File: barebones_chip.kicad_sch (KiCad schematic)
At the start: 2 parts, among them U1 RK3588

Commit message: fixed the power distribution by adding RK806 chips
Parts:
- added C112, C224, C280, C288, C289, C298, C305, C306, C316, C326, C327, C336, C338: 100nF, Capacitor_SMD:C_0201_0603Metric, symbol Device:C
- added C225, C232, C281, C296, C297, C304, C307, C308, C315, C323, C324, C325, C334, C337: 1uF, Capacitor_SMD:C_0201_0603Metric, symbol Device:C
- added C226, C290, C291, C309, C322: 4.7uF, Capacitor_SMD:C_0201_0603Metric, symbol Device:C
- added C227, C228, C229, C230, C282, C283, C284, C285, C286, C292, C293, C294, C299, C300, C301, C302, C310, C311, C312, C313, C318, C319, C320, C321, C329, C330, C332, C333: 10uF, Capacitor_SMD:C_0201_0603Metric, symbol Device:C
- added C231, C295, C303, C314, C317, C339: 22uF, Capacitor_SMD:C_0201_0603Metric, symbol Device:C
- added FL1: BLM18PG121SZ1D, BLM18PG121SZ1D:BEADC1608X95N, symbol BLM18PG121SZ1D:BLM18PG121SZ1D
- added R150, R151: 100k, Resistor_SMD:R_0603_1608Metric, symbol Device:R
- added R152, R153: 120k, Resistor_SMD:R_0603_1608Metric, symbol Device:R
- added R154, R155, R156: 22R, Resistor_SMD:R_0603_1608Metric, symbol Device:R
- added R96: 10k, Resistor_SMD:R_0603_1608Metric, symbol Device:R
Connections:
- net SPI_CS_PMIC: now reaches U1.K30 (SPI2_CS0_M2/I2C1_SDA_M1/PWM5_M0/UART0_TX_M1/GPIO0_B1_Z)
- net at U1.L29 (SPI2_MISO_M2/I2C0_SCL_M0/GPIO0_B3_Z): now also U1.N30 (SPI2_MOSI_M2/I2C0_SDA_M0/GPIO0_A6_Z), R155.1
- net INT_PMIC: now reaches U1.M30 (PMIC_INT_L/GPIO0_A7_U)
- net INT_PMIC: now also R96.1
- net at U1.N31 (SPI2_CLK_M2/SDMMC_PWREN/PMU_DEBUG/GPIO0_A5_D): now also R156.1
- net at U1.R32 (PMIC_SLEEP1/GPIO0_A2_D): now also R154.1
- net GND: now reaches U1.T24 (VSS_180)
- net GND: now also U1.A1 (VSS_1), U1.A11 (VSS_2), U1.A14 (VSS_3), U1.A34 (VSS_4), U1.AA10 (AVSS_16), U1.AA11 (VSS_250), U1.AA13 (VDD_GPU_0), U1.AA14 (VDD_GPU_7), U1.AA15 (VDD_GPU_11), U1.AA16 (VSS_251), U1.AA17 (VSS_252), U1.AA18 (VSS_253), U1.AA19 (VSS_254), U1.AA20 (VSS_255), U1.AA21 (VSS_256), U1.AA22 (VSS_257), U1.AA23 (VSS_258), U1.AA24 (VSS_259), U1.AA3 (VSS_248), U1.AA31 (VSS_260), U1.AA6 (VSS_249), U1.AA8 (AVSS_15), U1.AB10 (AVSS_20), U1.AB11 (VSS_263), U1.AB13 (VDD_GPU_1), U1.AB14 (VDD_GPU_6), U1.AB15 (VDD_GPU_10), U1.AB16 (VSS_264), U1.AB17 (VSS_265), U1.AB18 (VSS_266), U1.AB19 (VSS_267), U1.AB20 (VSS_268), U1.AB24 (VSS_269), U1.AB27 (VSS_270), U1.AB29 (VSS_271), U1.AB3 (VSS_261), U1.AB32 (VSS_272), U1.AB5 (VSS_262), U1.AB6 (AVSS_17), U1.AB7 (AVSS_18), U1.AB8 (AVSS_19), U1.AC10 (AVSS_23), U1.AC11 (VSS_275), U1.AC12 (VSS_276), U1.AC13 (VDD_GPU_2), U1.AC14 (VDD_GPU_5), U1.AC15 (VDD_GPU_9), U1.AC16 (VSS_277), U1.AC17 (VDD_LOGIC_5), U1.AC18 (VDD_LOGIC_4), U1.AC19 (VDD_LOGIC_3), U1.AC20 (VSS_278), U1.AC21 (VSS_279), U1.AC24 (VSS_280), U1.AC27 (VSS_281), U1.AC3 (VSS_273), U1.AC4 (VSS_274), U1.AC5 (AVSS_21), U1.AC8 (AVSS_22), U1.AD10 (AVSS_26), U1.AD11 (VSS_282), U1.AD12 (VSS_283), U1.AD13 (VDD_GPU_3), U1.AD14 (VDD_GPU_4), U1.AD15 (VDD_GPU_8), U1.AD16 (VSS_284), U1.AD17 (VDD_LOGIC_0), U1.AD18 (VDD_LOGIC_1), U1.AD19 (VDD_LOGIC_2), U1.AD20 (VSS_285), U1.AD21 (VSS_286), U1.AD24 (VSS_287), U1.AD25 (VSS_288), U1.AD26 (VSS_289), U1.AD5 (AVSS_24), U1.AD8 (AVSS_25), U1.AE11 (VSS_291), U1.AE12 (VSS_292), U1.AE13 (VSS_293), U1.AE14 (VSS_294), U1.AE15 (VSS_295), U1.AE16 (VSS_296), U1.AE18 (VSS_297), U1.AE19 (VSS_298), U1.AE20 (VSS_299), U1.AE21 (VSS_300), U1.AE24 (VSS_301), U1.AE26 (VSS_302), U1.AE3 (VSS_290), U1.AE6 (AVSS_27), U1.AE7 (AVSS_28), U1.AE9 (AVSS_29), U1.AF11 (AVSS_33), U1.AF12 (AVSS_34), U1.AF13 (AVSS_35), U1.AF14 (AVSS_36), U1.AF15 (AVSS_37), U1.AF16 (AVSS_38), U1.AF21 (AVSS_39), U1.AF22 (VSS_303), U1.AF24 (VSS_304), U1.AF25 (VSS_305), U1.AF27 (VSS_306), U1.AF28 (VSS_307), U1.AF29 (VSS_308), U1.AF30 (VSS_309), U1.AF31 (VSS_310), U1.AF32 (VSS_311), U1.AF4 (AVSS_30), U1.AF7 (AVSS_31), U1.AF8 (AVSS_32), U1.AG10 (AVSS_43), U1.AG12 (AVSS_44), U1.AG15 (AVSS_45), U1.AG18 (AVSS_46), U1.AG21 (AVSS_47), U1.AG22 (AVSS_48), U1.AG3 (AVSS_40), U1.AG30 (VSS_312), U1.AG6 (AVSS_41), U1.AG7 (AVSS_42), U1.AH11 (AVSS_51), U1.AH12 (AVSS_52), U1.AH15 (AVSS_53), U1.AH21 (AVSS_54), U1.AH22 (AVSS_55), U1.AH23 (AVSS_56), U1.AH4 (AVSS_49), U1.AH8 (AVSS_50), U1.AJ11 (AVSS_61), U1.AJ12 (AVSS_62), U1.AJ15 (AVSS_63), U1.AJ16 (AVSS_64), U1.AJ18 (AVSS_65), U1.AJ21 (AVSS_66), U1.AJ22 (AVSS_67), U1.AJ23 (AVSS_68), U1.AJ3 (AVSS_57), U1.AJ30 (VSS_313), U1.AJ7 (AVSS_58), U1.AJ8 (AVSS_59), U1.AJ9 (AVSS_60), U1.AK10 (AVSS_72), U1.AK11 (AVSS_73), U1.AK12 (AVSS_74), U1.AK13 (AVSS_75), U1.AK14 (AVSS_76), U1.AK23 (AVSS_77), U1.AK28 (VSS_314), U1.AK29 (VSS_315), U1.AK4 (AVSS_69), U1.AK5 (AVSS_70), U1.AK7 (AVSS_71), U1.AL11 (AVSS_81), U1.AL13 (AVSS_82), U1.AL23 (AVSS_83), U1.AL25 (VSS_316), U1.AL3 (AVSS_78), U1.AL4 (AVSS_79), U1.AL5 (AVSS_80), U1.AM18 (AVSS_87), U1.AM20 (AVSS_88), U1.AM22 (AVSS_89), U1.AM23 (AVSS_90), U1.AM24 (AVSS_91), U1.AM26 (AVSS_92), U1.AM28 (AVSS_93), U1.AM30 (VSS_317), U1.AM4 (AVSS_84), U1.AM8 (AVSS_85), U1.AM9 (AVSS_86), U1.AN12 (AVSS_95), U1.AN23 (AVSS_96), U1.AN31 (AVSS_97), U1.AN7 (AVSS_94), U1.AP1 (AVSS_98), U1.AP17 (AVSS_99), U1.AP23 (AVSS_100), U1.AP34 (AVSS_101), U1.B19 (VSS_6), U1.B24 (VSS_7), U1.B27 (VSS_8), U1.B33 (VSS_9), U1.B6 (VSS_5), U1.C10 (VSS_17), U1.C11 (VSS_18), U1.C12 (VSS_19), U1.C13 (VSS_20), U1.C14 (VSS_21), U1.C15 (VSS_22), U1.C16 (VSS_23), U1.C17 (VSS_24), U1.C18 (VSS_25), U1.C20 (VSS_26), U1.C21 (VSS_27), U1.C22 (VSS_28), U1.C23 (VSS_29), U1.C26 (VSS_30), U1.C28 (VSS_31), U1.C3 (VSS_10), U1.C30 (VSS_32), U1.C32 (VSS_33), U1.C4 (VSS_11), U1.C5 (VSS_12), U1.C6 (VSS_13), U1.C7 (VSS_14), U1.C8 (VSS_15), U1.C9 (VSS_16), U1.D23 (VSS_35), U1.D24 (VSS_36), U1.D3 (VSS_34), U1.D31 (VSS_37), U1.E12 (VSS_41), U1.E18 (VSS_42), U1.E20 (VSS_43), U1.E22 (VSS_44), U1.E23 (VSS_45), U1.E3 (VSS_38), U1.E32 (VSS_46), U1.E6 (VSS_39), U1.E8 (VSS_40), U1.F10 (VSS_50), U1.F11 (VSS_51), U1.F13 (VSS_52), U1.F14 (VSS_53), U1.F15 (VSS_54), U1.F16 (VSS_55), U1.F19 (VSS_56), U1.F20 (VSS_57), U1.F21 (VSS_58), U1.F22 (VSS_59), U1.F23 (VSS_60), U1.F3 (VSS_47), U1.F31 (VSS_61), U1.F7 (VSS_48), U1.F9 (VSS_49), U1.G10 (VSS_64), U1.G15 (VSS_65), U1.G19 (VSS_66), U1.G21 (VSS_67), U1.G22 (VSS_68), U1.G25 (VSS_69), U1.G3 (VSS_62), U1.G32 (VSS_70), U1.G6 (VSS_63), U1.H10 (VSS_73), U1.H12 (VSS_74), U1.H14 (VSS_75), U1.H19 (VSS_76), U1.H22 (VSS_77), U1.H25 (VSS_78), U1.H26 (VSS_79), U1.H28 (AVSS_1), U1.H3 (VSS_71), U1.H31 (AVSS_2), U1.H6 (VSS_72), U1.J10 (VSS_84), U1.J11 (VSS_85), U1.J12 (VSS_86), U1.J13 (VSS_87), U1.J14 (VSS_88), U1.J15 (VSS_89), U1.J16 (VSS_90), U1.J18 (VSS_91), U1.J19 (VSS_92), U1.J20 (VSS_93), U1.J21 (VSS_94), U1.J22 (VSS_95), U1.J23 (VSS_96), U1.J24 (VSS_97), U1.J25 (VSS_98), U1.J27 (AVSS_3), U1.J28 (AVSS_4), U1.J29 (AVSS_5), U1.J3 (VSS_80), U1.J32 (AVSS_6), U1.J4 (VSS_81), U1.J5 (VSS_82), U1.J6 (VSS_83), U1.K18 (VSS_103), U1.K19 (VDD_LOGIC_8), U1.K20 (VDD_LOGIC_9), U1.K21 (VSS_104), U1.K22 (VSS_105), U1.K26 (AVSS_7), U1.K3 (VSS_99), U1.K31 (AVSS_8), U1.K32 (AVSS_9), U1.K6 (VSS_100), U1.K8 (VSS_101), U1.K9 (VSS_102), U1.L1 (VSS_106), U1.L19 (VSS_110), U1.L20 (VSS_111), U1.L21 (VSS_112), U1.L22 (VSS_113), U1.L25 (VSS_114), U1.L26 (AVSS_10), U1.L3 (VSS_107), U1.L31 (AVSS_11), U1.L6 (VSS_108), U1.L9 (VSS_109), U1.M14 (VSS_118), U1.M15 (VSS_119), U1.M18 (VSS_120), U1.M20 (VSS_121), U1.M22 (VSS_122), U1.M25 (VSS_123), U1.M26 (AVSS_12), U1.M3 (VSS_115), U1.M32 (AVSS_13), U1.M6 (VSS_116), U1.M9 (VSS_117), U1.N11 (VSS_127), U1.N14 (VSS_128), U1.N15 (VSS_129), U1.N18 (VSS_130), U1.N20 (VSS_131), U1.N22 (VSS_132), U1.N25 (VSS_133), U1.N26 (VSS_134), U1.N29 (VSS_135), U1.N3 (VSS_124), U1.N32 (AVSS_14), U1.N6 (VSS_125), U1.N9 (VSS_126), U1.P1 (VSS_136), U1.P11 (VSS_141), U1.P14 (VSS_142), U1.P15 (VSS_143), U1.P18 (VSS_144), U1.P19 (VSS_145), U1.P20 (VSS_146), U1.P21 (VSS_147), U1.P22 (VSS_148), U1.P25 (VSS_149), U1.P26 (VSS_150), U1.P3 (VSS_137), U1.P34 (VSS_151), U1.P6 (VSS_138), U1.P8 (VSS_139), U1.P9 (VSS_140), U1.R11 (VSS_156), U1.R13 (VSS_157), U1.R15 (VSS_158), U1.R18 (VSS_159), U1.R19 (VSS_160), U1.R20 (VSS_161), U1.R21 (VSS_162), U1.R22 (VSS_163), U1.R23 (VSS_164), U1.R24 (VSS_165), U1.R25 (VSS_166), U1.R26 (VSS_167), U1.R28 (VSS_168), U1.R3 (VSS_152), U1.R33 (VSS_169), U1.R5 (VSS_153), U1.R8 (VSS_154), U1.R9 (VSS_155), U1.T11 (VSS_173), U1.T13 (VSS_174), U1.T15 (VSS_175), U1.T18 (VSS_176), U1.T19 (VSS_177), U1.T20 (VSS_178), U1.T23 (VSS_179), U1.T25 (VSS_181), U1.T26 (VSS_182), U1.T27 (VSS_183), U1.T3 (VSS_170), U1.T33 (VSS_184), U1.T6 (VSS_171), U1.T9 (VSS_172), U1.U12 (VSS_186), U1.U13 (VSS_187), U1.U15 (VSS_188), U1.U16 (VSS_189), U1.U17 (VSS_190), U1.U20 (VSS_191), U1.U23 (VSS_192), U1.U24 (VSS_193), U1.U3 (VSS_185), U1.U30 (VSS_194), U1.U31 (VSS_195), U1.U34 (VSS_196), U1.V10 (VSS_202), U1.V11 (VSS_203), U1.V15 (VSS_204), U1.V16 (VDD_LOGIC_6), U1.V17 (VDD_LOGIC_7), U1.V18 (VSS_205), U1.V19 (VSS_206), U1.V23 (VSS_207), U1.V24 (VSS_208), U1.V25 (VSS_209), U1.V27 (VSS_210), U1.V3 (VSS_197), U1.V30 (VSS_211), U1.V4 (VSS_198)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
- net at U1.T30 (PMIC_SLEEP5/GPIO0_C3_D): now also R151.2
- net at U1.T32 (PMIC_SLEEP4/GPIO0_C2_D): now also R150.2
- net VDD_GPU_S0: now reaches U1.AA12 (VDD_GPU_MEM_0)
- net VDD_GPU_S0: now also U1.AB12 (VDD_GPU_MEM_1), C112.2, C224.2, C225.2, C226.2, C227.2, C228.2, C229.2, C230.2, C231.2, C232.1
- net VDD_NPU_S0: now reaches U1.AB21 (VDD_NPU_6)
- net VDD_NPU_S0: now also U1.AB22 (VDD_NPU_5), U1.AB23 (VDD_NPU_2), U1.AC22 (VDD_NPU_4), U1.AC23 (VDD_NPU_1), U1.AD22 (VDD_NPU_3), U1.AD23 (VDD_NPU_0), U1.AE22 (VDD_NPU_MEM_0), U1.AE23 (VDD_NPU_MEM_1), C280.2, C281.2, C282.2, C283.2, C284.2, C285.2, C286.2
- net VDD_CPU_BIG1_S0: now reaches U1.K23 (VDD_CPU_BIG1_9)
- net VDD_CPU_BIG1_S0: now also U1.K24 (VDD_CPU_BIG1_0), U1.L23 (VDD_CPU_BIG1_8), U1.L24 (VDD_CPU_BIG1_1), U1.M23 (VDD_CPU_BIG1_7), U1.M24 (VDD_CPU_BIG1_2), U1.N23 (VDD_CPU_BIG1_6), U1.N24 (VDD_CPU_BIG1_3), U1.P23 (VDD_CPU_BIG1_5), U1.P24 (VDD_CPU_BIG1_4), C317.2, C318.2, C319.2, C320.2, C321.2, C322.2, C323.2, C325.2, C327.2, FL1.1
- net VDD_CPU_BIG0_S0: now reaches U1.M16 (VDD_CPU_BIG0_0)
- net VDD_CPU_BIG0_S0: now also U1.M17 (VDD_CPU_BIG0_9), U1.M19 (VDD_CPU_BIG0_MEM_0), U1.N16 (VDD_CPU_BIG0_1), U1.N17 (VDD_CPU_BIG0_8), U1.N19 (VDD_CPU_BIG0_MEM_1), U1.P16 (VDD_CPU_BIG0_2), U1.P17 (VDD_CPU_BIG0_7), U1.R16 (VDD_CPU_BIG0_3), U1.R17 (VDD_CPU_BIG0_6), U1.T16 (VDD_CPU_BIG0_4), U1.T17 (VDD_CPU_BIG0_5), C306.2, C307.2, C308.2, C309.2, C310.2, C311.2, C312.2, C313.2, C314.2, C315.1, C316.1
- net VDD_CPU_BIG1_MEM_S0: now reaches U1.M21 (VDD_CPU_BIG1_MEM_0)
- net VDD_CPU_BIG1_MEM_S0: now also U1.N21 (VDD_CPU_BIG1_MEM_1), C324.2, C326.2, C339.2, FL1.2
- net VDD_VDENC_S0: now reaches U1.R14 (VDD_VDENC_0)
- net VDD_VDENC_S0: now also U1.T14 (VDD_VDENC_1), U1.U14 (VDD_VDENC_2), U1.V12 (VDD_VDENC_MEM_0), U1.V13 (VDD_VDENC_MEM_1), U1.V14 (VDD_VDENC_3), U1.W13 (VDD_VDENC_5), U1.W14 (VDD_VDENC_4), C329.2, C330.2, C332.2, C333.2, C334.2, C336.2, C337.2, C338.2
- net VDD_LOG_S0: now reaches U1.T21 (VDD_CPU_LIT_MEM_1)
- net VDD_LOG_S0: now also U1.T22 (VDD_CPU_LIT_MEM_0), U1.U21 (VDD_CPU_LIT_7), U1.U22 (VDD_CPU_LIT_0), U1.V21 (VDD_CPU_LIT_6), U1.V22 (VDD_CPU_LIT_1), U1.W21 (VDD_CPU_LIT_5), U1.W22 (VDD_CPU_LIT_2), U1.Y21 (VDD_CPU_LIT_4), U1.Y22 (VDD_CPU_LIT_3), C288.2, C289.2, C290.1, C291.2, C292.2, C293.2, C294.2, C295.2, C296.2, C297.2, C298.1, C299.1, C300.1, C301.1, C302.1, C303.1, C304.1, C305.1
- net SPI_MISO_RK: now reaches U1.B25 (HDMI_TX1_SCL_M2/SPI2_MISO_M0/GPIO1_A4_D)
- net SPI_MOSI_RK: now reaches U1.B26 (HDMI_TX0_HPD_M0/SPI2_MOSI_M0/GPIO1_A5_D)
- net SPI_CLK_RK: now reaches U1.C24 (HDMI_TX1_HPD_M0/SPI2_CLK_M0/GPIO1_A6_D)
- net SPI_CS_RK: now reaches U1.C25 (PDM1_SDI0_M1/PCIE30X1_1_PERSTN_M2/PWM3_IR_M3/SPI2_CS0_M0/GPIO1_A7_U)
- net I2C4_SCL_M3: no longer names the net of U1.A27 (HDMI_TX1_SDA_M2/I2C4_SCL_M3/UART6_CTSN_M1/PWM1_M2/SPI4_CS0_M2/GPIO1_A3_D)
- new net PWRCTRL1_PMIC: R154.2
- new net PWRCTRL2_PMIC: R151.1, R152.2
- new net PWRCTRL3_PMIC: R150.1, R153.2
- new net SPI_CLK_PMIC: R156.2
- new net SPI_MOSI_PMIC: R155.2
- new net VCC_1V8_S0: R96.2
Other:
- moved on the sheet: U1A, U1B, U1C, U1D, U1V, U1W, U1X, U1Y

Commit message: routed the two 64Gb LPDDR4x RAM chips
Parts:
- added C143, C340, C344, C345, C346, C349, C357, C363, C364, C366, C368, C369: 100nF, Capacitor_SMD:C_0201_0603Metric, symbol Device:C
- added C343, C348, C350, C353, C354, C355, C356, C360, C362, C365, C367, C370, C371, C372: 1uF, Capacitor_SMD:C_0201_0603Metric, symbol Device:C
- added C347, C351, C358, C359: 10uF, Capacitor_SMD:C_0201_0603Metric, symbol Device:C
- added C352, C361: 4.7uF, Capacitor_SMD:C_0201_0603Metric, symbol Device:C
- added R157, R158, R159, R89: 200R, Resistor_SMD:R_0402_1005Metric, symbol Device:R
Connections:
- net GND: now also U1.L16 (DDR_CH1_PLL_AVSS), U1.M11 (DDR_CH0_PLL_AVSS), C143.1, C340.1, C343.1, C344.1, C345.1, C346.1, C347.1, C348.1, C349.1, C350.1, C351.1, C352.1, C353.1, C354.1, C355.1, C356.1, C357.1, C358.1, C359.1, C360.1, C361.1, C362.1, C363.1, C364.1, C365.1, C366.1, C367.1, C368.1, C369.1, C370.1, C371.1, C372.1, R157.2, R158.2, R159.2, R89.2
- net DDR_CH1_A4_C: now reaches U1.A10 (DDR_CH1_A4_C)
- net DDR_CH1_CKB_C: now reaches U1.A12 (DDR_CH1_CKB_C)
- net DDR_CH1_CKB_D: now reaches U1.A13 (DDR_CH1_CKB_D)
- net DDR_CH1_A4_D: now reaches U1.A15 (DDR_CH1_A4_D)
- net DDR_CH1_DQ2_D: now reaches U1.A16 (DDR_CH1_DQ2_D)
- net DDR_CH1_DQ0_D: now reaches U1.A17 (DDR_CH1_DQ0_D)
- net DDR_CH1_DQ6_D: now reaches U1.A18 (DDR_CH1_DQ6_D)
- net DDR_CH1_DQ4_D: now reaches U1.A19 (DDR_CH1_DQ4_D)
- net DDR_CH1_DQ10_C: now reaches U1.A2 (DDR_CH1_DQ10_C)
- net DDR_CH1_DQ12_D: now reaches U1.A20 (DDR_CH1_DQ12_D)
- net DDR_CH1_DQ14_D: now reaches U1.A21 (DDR_CH1_DQ14_D)
- net DDR_CH1_DQ8_D: now reaches U1.A22 (DDR_CH1_DQ8_D)
- net DDR_CH1_DQ10_D: now reaches U1.A23 (DDR_CH1_DQ10_D)
- net DDR_CH1_DQ8_C: now reaches U1.A3 (DDR_CH1_DQ8_C)
- net DDR_CH1_DQ14_C: now reaches U1.A4 (DDR_CH1_DQ14_C)
- net DDR_CH1_DQ12_C: now reaches U1.A5 (DDR_CH1_DQ12_C)
- net DDR_CH1_DQ4_C: now reaches U1.A6 (DDR_CH1_DQ4_C)
- net DDR_CH1_DQ6_C: now reaches U1.A7 (DDR_CH1_DQ6_C)
- net DDR_CH1_DQ0_C: now reaches U1.A8 (DDR_CH1_DQ0_C)
- net DDR_CH1_DQ2_C: now reaches U1.A9 (DDR_CH1_DQ2_C)
- net DDR_CH1_DQ3_C: now reaches U1.B10 (DDR_CH1_DQ3_C)
- net DDR_CH1_A5_C: now reaches U1.B11 (DDR_CH1_A5_C)
- net DDR_CH1_CK_C: now reaches U1.B12 (DDR_CH1_CK_C)
- net DDR_CH1_CK_D: now reaches U1.B13 (DDR_CH1_CK_D)
- net DDR_CH1_A5_D: now reaches U1.B14 (DDR_CH1_A5_D)
- net DDR_CH1_DQ3_D: now reaches U1.B15 (DDR_CH1_DQ3_D)
- net DDR_CH1_DQ1_D: now reaches U1.B16 (DDR_CH1_DQ1_D)
- net DDR_CH1_DQ7_D: now reaches U1.B17 (DDR_CH1_DQ7_D)
- net DDR_CH1_DQ5_D: now reaches U1.B18 (DDR_CH1_DQ5_D)
- net DDR_CH1_DQ11_C: now reaches U1.B2 (DDR_CH1_DQ11_C)
- net DDR_CH1_DQ13_D: now reaches U1.B20 (DDR_CH1_DQ13_D)
- net DDR_CH1_DQ15_D: now reaches U1.B21 (DDR_CH1_DQ15_D)
- net DDR_CH1_DQ9_D: now reaches U1.B22 (DDR_CH1_DQ9_D)
- net DDR_CH1_DQ11_D: now reaches U1.B23 (DDR_CH1_DQ11_D)
- net DDR_CH1_DQ9_C: now reaches U1.B3 (DDR_CH1_DQ9_C)
- net DDR_CH1_DQ15_C: now reaches U1.B4 (DDR_CH1_DQ15_C)
- net DDR_CH1_DQ13_C: now reaches U1.B5 (DDR_CH1_DQ13_C)
- net DDR_CH1_DQ5_C: now reaches U1.B7 (DDR_CH1_DQ5_C)
- net DDR_CH1_DQ7_C: now reaches U1.B8 (DDR_CH1_DQ7_C)
- net DDR_CH1_DQ1_C: now reaches U1.B9 (DDR_CH1_DQ1_C)
- net DDR_CH1_RESET_D: now reaches U1.C19 (DDR_CH1_RESET_D)
- net DDR_CH1_RESET_D: now also U1.F18 (DDR_CH1_ZQ_D), R158.1
- net DDR_CH1_LP4/4X_CKE0/LP5_CS0_C: now reaches U1.D11 (DDR_CH1_LP4/4X_CKE0/LP5_CS0_C)
- net DDR_CH1_A3_C: now reaches U1.D13 (DDR_CH1_A3_C)
- net DDR_CH1_LP4/4X_CKE0/LP5_CS0_D: now reaches U1.D16 (DDR_CH1_LP4/4X_CKE0/LP5_CS0_D)
- net DDR_CH1_LP4/4X_CS1_D: now reaches U1.D19 (DDR_CH1_LP4/4X_CS1_D)
- net DDR_CH1_DM0_D: now reaches U1.D20 (DDR_CH1_DM0_D)
- net DDR_CH1_DQS1P_D: now reaches U1.D21 (DDR_CH1_DQS1P_D)
- net DDR_CH1_DM1_D: now reaches U1.D22 (DDR_CH1_DM1_D)
- net DDR_CH1_DM1_C: now reaches U1.D4 (DDR_CH1_DM1_C)
- net DDR_CH1_DQS1N_C: now reaches U1.D5 (DDR_CH1_DQS1N_C)
- net DDR_CH1_DQS0N_C: now reaches U1.D9 (DDR_CH1_DQS0N_C)
- net DDR_CH1_RESET_C: now reaches U1.E10 (DDR_CH1_RESET_C)
- net DDR_CH1_RESET_C: now also U1.G8 (DDR_CH1_ZQ_C), R159.1
- net DDR_CH1_LP4/4X_CKE1/LP5_CS1_C: now reaches U1.E11 (DDR_CH1_LP4/4X_CKE1/LP5_CS1_C)
- net DDR_CH1_A2_C: now reaches U1.E13 (DDR_CH1_A2_C)
- net DDR_CH1_A3_D: now reaches U1.E14 (DDR_CH1_A3_D)
- net DDR_CH1_LP4/4X_CKE1/LP5_CS1_D: now reaches U1.E16 (DDR_CH1_LP4/4X_CKE1/LP5_CS1_D)
- net DDR_CH1_LP4/4X_CS0_D: now reaches U1.E19 (DDR_CH1_LP4/4X_CS0_D)
- net DDR_CH1_DQS1N_D: now reaches U1.E21 (DDR_CH1_DQS1N_D)
- net DDR_CH1_DQS1P_C: now reaches U1.E5 (DDR_CH1_DQS1P_C)
- net DDR_CH1_DQS0P_C: now reaches U1.E9 (DDR_CH1_DQS0P_C)
- net DDR_CH1_A1_C: now reaches U1.F12 (DDR_CH1_A1_C)
- net DDR_CH1_DM0_C: now reaches U1.F8 (DDR_CH1_DM0_C)
- net DDR_CH1_LP4/4X_CS0_C: now reaches U1.G11 (DDR_CH1_LP4/4X_CS0_C)
- net DDR_CH1_A0_C: now reaches U1.G12 (DDR_CH1_A0_C)
- net DDR_CH1_A2_D: now reaches U1.G13 (DDR_CH1_A2_D)
- net DDR_CH1_A1_D: now reaches U1.G14 (DDR_CH1_A1_D)
- net DDR_CH1_DQS0N_D: now reaches U1.G16 (DDR_CH1_DQS0N_D)
- net DDR_CH1_LP4/4X_CS1_C: now reaches U1.H11 (DDR_CH1_LP4/4X_CS1_C)
- net VDDQ_DDR_CKE_S3: now reaches U1.H13 (DDR_CH1_VDDQ_CKE)
- net VDDQ_DDR_CKE_S3: now also U1.N8 (DDR_CH0_VDDQ_CKE), C355.2, C372.2
- net DDR_CH1_A0_D: now reaches U1.H15 (DDR_CH1_A0_D)
- net DDR_CH1_DQS0P_D: now reaches U1.H16 (DDR_CH1_DQS0P_D)
- net VDDQ_DDR_S0: now reaches U1.K11 (DDR_CH1_VDDQ_0)
- net VDDQ_DDR_S0: now also U1.K12 (DDR_CH1_VDDQ_1), U1.K13 (DDR_CH1_VDDQ_2), U1.K14 (DDR_CH1_VDDQ_3), U1.K15 (DDR_CH1_VDDQ_4), U1.M10 (DDR_CH0_VDDQ_0), U1.N10 (DDR_CH0_VDDQ_1), U1.P10 (DDR_CH0_VDDQ_2), U1.R10 (DDR_CH0_VDDQ_3), U1.T10 (DDR_CH0_VDDQ_4), C343.2, C344.2, C345.2, C346.2, C347.2, C348.2, C358.2, C360.2, C362.2, C364.2, C366.2, C368.2
- net VCCA_1V8_S0: now reaches U1.K16 (DDR_CH1_PLL_AVDD1V8)
- net VCCA_1V8_S0: now also U1.M12 (DDR_CH0_PLL_AVDD1V8), C350.2, C370.2
- net VDD_DDR_S0: now reaches U1.L11 (DDR_CH1_VDD_0)
- net VDD_DDR_S0: now also U1.L12 (DDR_CH1_VDD_1), U1.L13 (DDR_CH1_VDD_2), U1.L14 (DDR_CH1_VDD_3), U1.L17 (DDR_CH1_VDD_MIF_0), U1.L18 (DDR_CH1_VDD_MIF_1), U1.N13 (DDR_CH0_VDD_MIF_0), U1.P12 (DDR_CH0_VDD_3), U1.P13 (DDR_CH0_VDD_MIF_1), U1.R12 (DDR_CH0_VDD_2), U1.T12 (DDR_CH0_VDD_1), U1.U11 (DDR_CH0_VDD_0), C349.2, C351.2, C352.2, C356.2, C357.2, C359.2, C361.2, C363.2, C365.2, C369.2
- net VDDQ_DDR_PLL_S0: now reaches U1.L15 (DDR_CH1_PLL_DVDD)
- net VDDQ_DDR_PLL_S0: now also U1.N12 (DDR_CH0_PLL_DVDD), C353.2, C371.2
- net VDDQ_DDR_CK_S0: now reaches U1.M13 (DDR_CH1_VDDQ_CK)
- net VDDQ_DDR_CK_S0: now also U1.L10 (DDR_CH0_VDDQ_CK), C354.2, C367.2
- net VCC_3V3_S3: now reaches U1.P28 (PMUIO2)
- net VCC_3V3_S3: now also C143.2
- net VCC_1V8_S3: now reaches U1.R27 (PMUIO2_1V8)
- net VCC_1V8_S3: now also C340.2
- net DDR_CH0_DQ14_A: now reaches U1.AA1 (DDR_CH0_DQ14_A)
- net DDR_CH0_DQ15_A: now reaches U1.AA2 (DDR_CH0_DQ15_A)
- net DDR_CH0_DQS1N_A: now reaches U1.AA4 (DDR_CH0_DQS1N_A)
- net DDR_CH0_DQS1P_A: now reaches U1.AA5 (DDR_CH0_DQS1P_A)
- net DDR_CH0_DQ9_A: now reaches U1.AB1 (DDR_CH0_DQ9_A)
- net DDR_CH0_DQ8_A: now reaches U1.AB2 (DDR_CH0_DQ8_A)
- net DDR_CH0_DM1_A: now reaches U1.AB4 (DDR_CH0_DM1_A)
- net DDR_CH0_DQ10_A: now reaches U1.AC1 (DDR_CH0_DQ10_A)
- net DDR_CH0_DQ11_A: now reaches U1.AC2 (DDR_CH0_DQ11_A)
- net DDR_CH0_DQ11_B: now reaches U1.B1 (DDR_CH0_DQ11_B)
- net DDR_CH0_DQ9_B: now reaches U1.C1 (DDR_CH0_DQ9_B)
- net DDR_CH0_DQ10_B: now reaches U1.C2 (DDR_CH0_DQ10_B)
- net DDR_CH0_DQ15_B: now reaches U1.D1 (DDR_CH0_DQ15_B)
- net DDR_CH0_DQ8_B: now reaches U1.D2 (DDR_CH0_DQ8_B)
- net DDR_CH0_DQ13_B: now reaches U1.E1 (DDR_CH0_DQ13_B)
- net DDR_CH0_DQ14_B: now reaches U1.E2 (DDR_CH0_DQ14_B)
- net DDR_CH0_DM1_B: now reaches U1.E4 (DDR_CH0_DM1_B)
- net DDR_CH0_DQ4_B: now reaches U1.F1 (DDR_CH0_DQ4_B)
- net DDR_CH0_DQ12_B: now reaches U1.F2 (DDR_CH0_DQ12_B)
- net DDR_CH0_DQS1N_B: now reaches U1.F4 (DDR_CH0_DQS1N_B)
- net DDR_CH0_DQS1P_B: now reaches U1.F5 (DDR_CH0_DQS1P_B)
- net DDR_CH0_DQ6_B: now reaches U1.G1 (DDR_CH0_DQ6_B)
- net DDR_CH0_DQ5_B: now reaches U1.G2 (DDR_CH0_DQ5_B)
- net DDR_CH0_DM0_B: now reaches U1.G4 (DDR_CH0_DM0_B)
- net DDR_CH0_DQ0_B: now reaches U1.H1 (DDR_CH0_DQ0_B)
- net DDR_CH0_DQ7_B: now reaches U1.H2 (DDR_CH0_DQ7_B)
- net DDR_CH0_RESET_B: now reaches U1.H7 (DDR_CH0_ZQ_B)
- net DDR_CH0_RESET_B: now also U1.K7 (DDR_CH0_RESET_B), R89.1
- net DDR_CH0_DQ2_B: now reaches U1.J1 (DDR_CH0_DQ2_B)
- net DDR_CH0_DQ1_B: now reaches U1.J2 (DDR_CH0_DQ1_B)
- net DDR_CH0_DQS0N_B: now reaches U1.J7 (DDR_CH0_DQS0N_B)
- net DDR_CH0_DQS0P_B: now reaches U1.J8 (DDR_CH0_DQS0P_B)
- net DDR_CH0_A4_B: now reaches U1.K1 (DDR_CH0_A4_B)
- net DDR_CH0_DQ3_B: now reaches U1.K2 (DDR_CH0_DQ3_B)
- net DDR_CH0_A5_B: now reaches U1.L2 (DDR_CH0_A5_B)
- net DDR_CH0_LP4/4X_CKE1/LP5_CS1_B: now reaches U1.L4 (DDR_CH0_LP4/4X_CKE1/LP5_CS1_B)
- net DDR_CH0_LP4/4X_CKE0/LP5_CS0_B: now reaches U1.L5 (DDR_CH0_LP4/4X_CKE0/LP5_CS0_B)
- net DDR_CH0_LP4/4X_CS0_B: now reaches U1.L7 (DDR_CH0_LP4/4X_CS0_B)
- net DDR_CH0_LP4/4X_CS1_B: now reaches U1.L8 (DDR_CH0_LP4/4X_CS1_B)
- net DDR_CH0_CKB_B: now reaches U1.M1 (DDR_CH0_CKB_B)
- net DDR_CH0_CK_B: now reaches U1.M2 (DDR_CH0_CK_B)
- net DDR_CH0_A1_B: now reaches U1.M5 (DDR_CH0_A1_B)
- net DDR_CH0_A0_B: now reaches U1.M8 (DDR_CH0_A0_B)
- net DDR_CH0_CKB_A: now reaches U1.N1 (DDR_CH0_CKB_A)
- net DDR_CH0_CK_A: now reaches U1.N2 (DDR_CH0_CK_A)
- net DDR_CH0_A3_B: now reaches U1.N4 (DDR_CH0_A3_B)
- net DDR_CH0_A2_B: now reaches U1.N5 (DDR_CH0_A2_B)
- net DDR_CH0_LP4/4X_CKE1/LP5_CS1_A: now reaches U1.N7 (DDR_CH0_LP4/4X_CKE1/LP5_CS1_A)
- net DDR_CH0_A5_A: now reaches U1.P2 (DDR_CH0_A5_A)
- net DDR_CH0_A2_A: now reaches U1.P4 (DDR_CH0_A2_A)
- net DDR_CH0_A3_A: now reaches U1.P5 (DDR_CH0_A3_A)
- net DDR_CH0_LP4/4X_CKE0/LP5_CS0_A: now reaches U1.P7 (DDR_CH0_LP4/4X_CKE0/LP5_CS0_A)
- net DDR_CH0_A4_A: now reaches U1.R1 (DDR_CH0_A4_A)
- net DDR_CH0_DQ3_A: now reaches U1.R2 (DDR_CH0_DQ3_A)
- net DDR_CH0_LP4/4X_CS0_A: now reaches U1.R6 (DDR_CH0_LP4/4X_CS0_A)
- net DDR_CH0_LP4/4X_CS1_A: now reaches U1.R7 (DDR_CH0_LP4/4X_CS1_A)
- net DDR_CH0_DQ2_A: now reaches U1.T1 (DDR_CH0_DQ2_A)
- net DDR_CH0_DQ1_A: now reaches U1.T2 (DDR_CH0_DQ1_A)
- net DDR_RESET: now reaches U1.T4 (DDR_CH0_RESET_A)
- net DDR_CH0_A0_A: now reaches U1.T7 (DDR_CH0_A0_A)
- net DDR_CH0_A1_A: now reaches U1.T8 (DDR_CH0_A1_A)
- net DDR_CH0_DQ0_A: now reaches U1.U1 (DDR_CH0_DQ0_A)
- net DDR_CH0_DQ7_A: now reaches U1.U2 (DDR_CH0_DQ7_A)
- net DDR_CH0_DQS0N_A: now reaches U1.U4 (DDR_CH0_DQS0N_A)
- net DDR_CH0_DQS0P_A: now reaches U1.U5 (DDR_CH0_DQS0P_A)
- net DDR_CH0_DQ6_A: now reaches U1.V1 (DDR_CH0_DQ6_A)
- net DDR_CH0_DQ5_A: now reaches U1.V2 (DDR_CH0_DQ5_A)
- net DDR_CH0_DQ4_A: now reaches U1.W1 (DDR_CH0_DQ4_A)
- net at U1.W8 (DDR_CH0_ZQ_A): now also R157.1
- net DDR_CH0_DQ12_A: now reaches U1.Y1 (DDR_CH0_DQ12_A)
- net DDR_CH0_DQ13_A: now reaches U1.Y2 (DDR_CH0_DQ13_A)
- net DDR_CH0_DM0_A: now reaches U1.Y4 (DDR_CH0_DM0_A)
- net SPI_CLK_RK: no longer names the net of U1.C24 (HDMI_TX1_HPD_M0/SPI2_CLK_M0/GPIO1_A6_D)
- net SPI_CS_RK: no longer names the net of U1.C25 (PDM1_SDI0_M1/PCIE30X1_1_PERSTN_M2/PWM3_IR_M3/SPI2_CS0_M0/GPIO1_A7_U)
- net SPI_MISO_RK: no longer names the net of U1.B25 (HDMI_TX1_SCL_M2/SPI2_MISO_M0/GPIO1_A4_D)
- net SPI_MOSI_RK: no longer names the net of U1.B26 (HDMI_TX0_HPD_M0/SPI2_MOSI_M0/GPIO1_A5_D)
- no-connect marks 0 -> 20
Other:
- moved on the sheet: C1, C112, C224, C225, C226, C227, C228, C229, C230, C231, C232, C280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

Commit message: added a USB 3.1 hub for the Type-A ports and a CLK generator for the PCIE 3.0/2.0
Parts:
- removed C1: 100nF, Capacitor_SMD:C_0201_0603Metric, symbol Device:C
- added C107, C108, C413, C414, C425, C427, C432, C434: 100nF, Capacitor_SMD:C_0201_0603Metric, symbol Device:C
- added C419, C420, C421: 18pF, Capacitor_SMD:C_0603_1608Metric, symbol Device:C
- added C422, C424, C443: 1uF, Capacitor_SMD:C_0603_1608Metric, symbol Device:C
- added C423, C442, C444, C445, C446: 100nF, Capacitor_SMD:C_0603_1608Metric, symbol Device:C
- added C426, C431, C433, C435: 4.7F, Capacitor_SMD:C_0201_0603Metric, symbol Device:C
- added C466, C467: 0.1uF, Capacitor_SMD:C_0201_0603Metric, symbol Device:C
- added R164: 22R, Resistor_SMD:R_0603_1608Metric, symbol Device:R
- added R165: 510k, Resistor_SMD:R_0603_1608Metric, symbol Device:R
- added R173, R174: 200R, Resistor_SMD:R_0402_1005Metric, symbol Device:R
- added Y1: C3E-24.000-12-3030-X-R, barebones:XTAL_C3E-24.000-12-3030-X-R, symbol C3E-24.000-12-3030-X-R:C3E-24.000-12-3030-X-R
Connections:
- net GND: now also U1.M29 (TVSS), U1.U19 (PLL_AVSS), C413.1, C414.1, C419.1, C420.2, C421.2, C422.2, C423.2, C424.2, C425.1, C426.1, C427.1, C431.1, C432.1, C433.1, C434.1, C435.1, C442.2, C443.2, C444.2, C445.2, C446.2, R173.2, R174.2, Y1.2 (GND), Y1.4 (GND)
- net VCCA_1V8_S0: now also U1.G23 (PCIE30_PORT0_AVDD1V8), U1.H23 (PCIE30_PORT1_AVDD1V8), U1.N27 (OSC_1V8), U1.U18 (PLL_AVDD1V8), C422.1, C423.1, C425.2, C426.2, C434.2, C435.2, C444.1
- net VCC_1V8_S0: now also U1.AA7 (VCCIO2_1V8), C414.2
- net VCC1V8_PMU_DDR_S3: now reaches U1.N28 (PMUIO1_1V8)
- net VCC1V8_PMU_DDR_S3: now also C445.1
- net VDD_0V75_S3: now reaches U1.P27 (PMU_0V75)
- net VDD_0V75_S3: now also C443.1, C446.1
- net SDMMC_DET: now reaches U1.P31 (SDMMC_DET/GPIO0_A4_U)
- net at U1.R34 (XIN_24M): now also C419.2, C421.1, R165.1, Y1.3
- net at U1.T34 (XOUT_24M): now also R164.2, R165.2
- net VDD_0V75_S0: now reaches U1.V20 (PLL_DVDD0V75)
- net VDD_0V75_S0: now also U1.G24 (PCIE30_PORT0_AVDD0V75), U1.H24 (PCIE30_PORT1_AVDD0V75), C424.1, C427.2, C431.2, C432.2, C433.2, C442.1
- net SDMMC_DAT1: now reaches U1.AD1 (SDMMC_D1/PDM1_SDI2_M0/JTAG_TMS_M1/I2C3_SDA_M4/UART2_RX_M1/PWM9_M1/GPIO4_D1_U)
- net SDMMC_DAT0: now reaches U1.AD2 (SDMMC_D0/PDM1_SDI3_M0/JTAG_TCK_M1/I2C3_SCL_M4/UART2_TX_M1/PWM8_M1/GPIO4_D0_U)
- net SDMMC_CLK: now reaches U1.AE1 (SDMMC_CLK/PDM1_CLK0_M0/TEST_CLKOUT_M0/MCU_JTAG_TMS_M0/CAN0_RX_M1/UART5_TX_M0/GPIO4_D5_D)
- net SDMMC_CMD: now reaches U1.AE2 (SDMMC_CMD/PDM1_CLK1_M0/MCU_JTAG_TCK_M0/CAN0_TX_M1/UART5_RX_M0/PWM7_IR_M1/GPIO4_D4_U)
- net SDMMC_DAT3: now reaches U1.AF1 (SDMMC_D3/PDM1_SDI0_M0/JTAG_TMS_M0/I2C8_SDA_M0/UART5_RTSN_M0/PWM10_M1/GPIO4_D3_U)
- net SDMMC_DAT2: now reaches U1.AF2 (SDMMC_D2/PDM1_SDI1_M0/JTAG_TCK_M0/I2C8_SCL_M0/UART5_CTSN_M0/GPIO4_D2_U)
- net VCCIO_SD_S0: now reaches U1.Y7 (VCCIO2)
- net VCCIO_SD_S0: now also C413.2
- net PCIE30_PORT1_REF_CLKP: now reaches U1.A28 (PCIE30_PORT1_REF_CLKP)
- net PCIE30_PORT1_TX0N: now reaches U1.A30 (PCIE30_PORT1_TX0N)
- net PCIE30_PORT1_RX0N: now reaches U1.A32 (PCIE30_PORT1_RX0N)
- net at U1.A33 (PCIE30_PORT1_RESREF): now also R173.1
- net PCIE30_PORT1_REF_CLKN: now reaches U1.B28 (PCIE30_PORT1_REF_CLKN)
- net PCIE30_PORT1_TX1N: now reaches U1.B29 (PCIE30_PORT1_TX1N)
- net PCIE30_PORT1_TX0P: now reaches U1.B30 (PCIE30_PORT1_TX0P)
- net PCIE30_PORT1_RX1N: now reaches U1.B31 (PCIE30_PORT1_RX1N)
- net PCIE30_PORT1_RX0P: now reaches U1.B32 (PCIE30_PORT1_RX0P)
- net at U1.B34 (PCIE30_PORT0_RESREF): now also R174.1
- net PCIE30_PORT1_TX1P: now reaches U1.C29 (PCIE30_PORT1_TX1P)
- net PCIE30_PORT1_RX1P: now reaches U1.C31 (PCIE30_PORT1_RX1P)
- net PCIE30_PORT0_TX1P: now reaches U1.C33 (PCIE30_PORT0_TX1P)
- net PCIE30_PORT0_TX1N: now reaches U1.C34 (PCIE30_PORT0_TX1N)
- net PCIE30_PORT0_RX0P: now reaches U1.D32 (PCIE30_PORT0_TX0P)
- net PCIE30_PORT0_RX0N: now reaches U1.D33 (PCIE30_PORT0_TX0N)
- net PCIE30_PORT0_REF_CLKP: now reaches U1.E33 (PCIE30_PORT0_REF_CLKP)
- net PCIE30_PORT0_REF_CLKN: now reaches U1.E34 (PCIE30_PORT0_REF_CLKN)
- net PCIE30_PORT0_RX1P: now reaches U1.F32 (PCIE30_PORT0_RX1P)
- net PCIE30_PORT0_RX1N: now reaches U1.F33 (PCIE30_PORT0_RX1N)
- net PCIE30_PORT0_TX0P: now reaches U1.G33 (PCIE30_PORT0_RX0P)
- net PCIE30_PORT0_TX0N: now reaches U1.G34 (PCIE30_PORT0_RX0N)
- net at U1.H29 (PCIE20_2_TXN/SATA30_2_TXN/USB30_2_SSTXN): now also C467.2
- net at U1.H30 (PCIE20_2_TXP/SATA30_2_TXP/USB30_2_SSTXP): now also C466.2
- net USB30_2_SSRXN: now reaches U1.J30 (PCIE20_2_RXN/SATA30_2_RXN/USB30_2_SSRXN)
- net USB30_2_SSRXP: now reaches U1.J31 (PCIE20_2_RXP/SATA30_2_RXP/USB30_2_SSRXP)
- net PCIE20_0_REFCLKP: now reaches U1.L32 (PCIE20_0_REFCLKP)
- net PCIE20_0_REFCLKN: now reaches U1.L33 (PCIE20_0_REFCLKN)
- net at U1.M33 (PCIE20_0_TXN/SATA30_0_TXN): now also C108.2
- net at U1.M34 (PCIE20_0_TXP/SATA30_0_TXP): now also C107.2
- net PCIE20_0_RXP: now reaches U1.N33 (PCIE20_0_RXP/SATA30_0_RXP)
- net PCIE20_0_RXN: now reaches U1.N34 (PCIE20_0_RXN/SATA30_0_RXN)
- net PCIE30x4_PWREN_H: now reaches U1.B25 (HDMI_TX1_SCL_M2/SPI2_MISO_M0/GPIO1_A4_D)
- net USB20_HOST0_DP: now reaches U1.AK6 (USB20_HOST0_DP)
- net USB20_HOST0_DM: now reaches U1.AL6 (USB20_HOST0_DM)
- net USB20_HOST1_DP: now reaches U1.AL7 (USB20_HOST1_DP)
- net USB20_HOST1_DM: now reaches U1.AM7 (USB20_HOST1_DM)
- new net: C420.1, R164.1, Y1.1
- new net PCIE20_0_TXN: C108.1
- new net PCIE20_0_TXP: C107.1
- new net USB30_2_SSTXN: C467.1
- new net USB30_2_SSTXP: C466.1
- no-connect marks 20 -> 22
Other:
- moved on the sheet: R154, R155, R156, R96, U1C, U1E, U1F, U1G
