File: barebones_chip.kicad_sch (KiCad schematic)
At the start: 142 parts, among them U1 RK3588, Y1 C3E-24.000-12-3030-X-R

Commit message: fixed the connection for the two HDMI ports and connected them to the RK3588 section Z
Parts:
- added C437, C438, C454, C455, C506, C508, C510, C533, C536, C540, C546, C547, C548: 100nF, Capacitor_SMD:C_0201_0603Metric, symbol Device:C
- added C465, C505, C507, C509, C537, C539, C542, C544, C545: 1uF, Capacitor_SMD:C_0201_0603Metric, symbol Device:C
- added C497, C498, C499, C500, C501, C502, C503, C504: 0.1uF, Capacitor_SMD:C_0201_0603Metric, symbol Device:C
- added C534, C535, C538, C541, C543: 4.7uF, Capacitor_SMD:C_0201_0603Metric, symbol Device:C
- added R211, R212, R213, R214: 10k, Resistor_SMD:R_0402_1005Metric, symbol Device:R
- added R220, R223, R224, R225: 200R, Resistor_SMD:R_0402_1005Metric, symbol Device:R
- added R221, R222: 4.7k, Resistor_SMD:R_0402_1005Metric, symbol Device:R
- added R226, R227, R246, R247: 8.2k, Resistor_SMD:R_0402_1005Metric, symbol Device:R
Connections:
- net GND: now also C437.1, C438.1, C454.1, C455.1, C465.1, C505.1, C506.1, C507.1, C508.1, C509.1, C510.1, C533.1, C534.1, C535.1, C536.1, C537.1, C538.1, C539.1, C540.1, C541.1, C542.1, C543.1, C544.1, C545.1, C546.1, C547.1, C548.1, R220.1, R223.1, R224.1, R225.1, R226.1, R227.1, R246.2, R247.2
- net PCIE20_0_RXN: now also C108.1; no longer U1.N34 (PCIE20_0_RXN/SATA30_0_RXN)
- net PCIE20_0_RXP: now also C107.1; no longer U1.N33 (PCIE20_0_RXP/SATA30_0_RXP)
- net PCIE20_0_TXN: now also U1.N34 (PCIE20_0_RXN/SATA30_0_RXN); no longer C108.1
- net PCIE20_0_TXP: now also U1.N33 (PCIE20_0_RXP/SATA30_0_RXP); no longer C107.1
- net USB30_2_SSRXN: now also C467.1; no longer U1.J30 (PCIE20_2_RXN/SATA30_2_RXN/USB30_2_SSRXN)
- net USB30_2_SSRXP: now also C466.1; no longer U1.J31 (PCIE20_2_RXP/SATA30_2_RXP/USB30_2_SSRXP)
- net USB30_2_SSTXN: now also U1.J30 (PCIE20_2_RXN/SATA30_2_RXN/USB30_2_SSRXN); no longer C467.1
- net USB30_2_SSTXP: now also U1.J31 (PCIE20_2_RXP/SATA30_2_RXP/USB30_2_SSRXP); no longer C466.1
- net VCCA_1V8_S0: now also U1.AG11 (USB20_AVDD_1V8), U1.AG13 (TYPEC1_DP1_VDDH_1V8), U1.AG14 (TYPEC0_DP0_VDDH_1V8), C437.2, C505.2, C506.2, C509.2, C510.2
- net VCC_1V8_S0: now also U1.AC6 (HDMI/EDP_TX0_VDD_CMN_1V8), U1.AC7 (HDMI/EDP_TX0_VDD_IO_1V8), U1.AD6 (HDMI/EDP_TX1_VDD_CMN_1V8), U1.AD7 (HDMI/EDP_TX1_VDD_IO_1V8), C538.2, C539.2, C540.2, C543.2, C545.2, C548.2
- net at U1.AG16 (TYPEC1_DP1_REXT): now also R227.2
- net VDDA_0V85_S0: now reaches U1.AH13 (TYPEC1_DP1_VDD_0V85)
- net VDDA_0V85_S0: now also U1.AH14 (TYPEC0_DP0_VDDA_0V85), U1.AJ13 (TYPEC1_DP1_VDDA_0V85), U1.AJ14 (TYPEC0_DP0_VDD_0V85), C455.2, C465.2, C507.2, C508.2
- net at U1.AH16 (TYPEC0_DP0_REXT): now also R226.2
- net USB_2_SBU1: now reaches U1.AL10 (TYPEC1_SBU1/DP1_AUXP)
- net USB_1_SBU1: now reaches U1.AL15 (TYPEC0_SBU1/DP0_AUXP)
- net USB_2_SBU2: now reaches U1.AM10 (TYPEC1_SBU2/DP1_AUXN)
- net USB_1_SBU2: now reaches U1.AM15 (TYPEC0_SBU2/DP0_AUXN)
- net USB_2_TX1P: now reaches U1.AN10 (TYPEC1_SSRX2P/DP1_TX2P)
- net at U1.AN11 (TYPEC1_SSTX2N/DP1_TX3N): now also C504.2
- net USB_1_TX1P: now reaches U1.AN13 (TYPEC0_SSRX1P/DP0_TX0P)
- net at U1.AN14 (TYPEC0_SSTX1N/DP0_TX1N): now also C498.2
- net USB_1_TX2P: now reaches U1.AN15 (TYPEC0_SSRX2P/DP0_TX2P)
- net at U1.AN16 (TYPEC0_SSTX2N/DP0_TX3N): now also C500.2
- net USB_2_TX2P: now reaches U1.AN8 (TYPEC1_SSRX1P/DP1_TX0P)
- net at U1.AN9 (TYPEC1_SSTX1N/DP1_TX1N): now also C502.2
- net USB_2_TX1N: now reaches U1.AP10 (TYPEC1_SSRX2N/DP1_TX2N)
- net at U1.AP11 (TYPEC1_SSTX2P/DP1_TX3P): now also C503.2
- net USB_1_TX1N: now reaches U1.AP13 (TYPEC0_SSRX1N/DP0_TX0N)
- net at U1.AP14 (TYPEC0_SSTX1P/DP0_TX1P): now also C497.2
- net USB_1_TX2N: now reaches U1.AP15 (TYPEC0_SSRX2N/DP0_TX2N)
- net at U1.AP16 (TYPEC0_SSTX2P/DP0_TX3P): now also C499.2
- net USB_2_TX2N: now reaches U1.AP8 (TYPEC1_SSRX1N/DP1_TX0N)
- net at U1.AP9 (TYPEC1_SSTX1P/DP1_TX1P): now also C501.2
- net VDDA_0V75_S0: now reaches U1.AA9 (HDMI/EDP_TX0_VDD_0V75)
- net VDDA_0V75_S0: now also U1.AB9 (HDMI/EDP_TX0_AVDD_0V75), U1.AC9 (HDMI/EDP_TX1_AVDD_0V75), U1.AD9 (HDMI/EDP_TX1_VDD_0V75), U1.AH10 (USB20_DVDD_0V75), C454.2, C533.2, C534.2, C535.2, C536.2, C537.2, C541.2, C542.2, C544.2, C546.2, C547.2
- net HDMI0_TX_SBDN/eDP0_TX_AUXN: now reaches U1.AG1 (HDMI_TX0_SBDN/EDP_TX0_AUXN)
- net HDMI0_TX_SBDP/eDP0_TX_AUXP: now reaches U1.AG2 (HDMI_TX0_SBDP/EDP_TX0_AUXP)
- net HDMI0_TX3N_PORT/eDP0_TX_D3N: now reaches U1.AH2 (HDMI_TX0_D3N/EDP_TX0_D3N)
- net HDMI0_TX3P_PORT/eDP0_TX_D3P: now reaches U1.AH3 (HDMI_TX0_D3P/EDP_TX0_D3P)
- net HDMI0_TX0N_PORT/eDP0_TX_D0N: now reaches U1.AJ1 (HDMI_TX0_D0N/EDP_TX0_D0N)
- net HDMI0_TX0P_PORT/eDP0_TX_D0P: now reaches U1.AJ2 (HDMI_TX0_D0P/EDP_TX0_D0P)
- net HDMI0_TX1N_PORT/eDP0_TX_D1N: now reaches U1.AK2 (HDMI_TX0_D1N/EDP_TX0_D1N)
- net HDMI0_TX1P_PORT/eDP0_TX_D1P: now reaches U1.AK3 (HDMI_TX0_D1P/EDP_TX0_D1P)
- net HDMI0_TX2N_PORT/eDP0_TX_D2N: now reaches U1.AL1 (HDMI_TX0_D2N/EDP_TX0_D2N)
- net HDMI0_TX2P_PORT/eDP0_TX_D2P: now reaches U1.AL2 (HDMI_TX0_D2P/EDP_TX0_D2P)
- net at U1.AM2 (HDMI/EDP_TX0_REXT): now also R246.1
- net HDMI1_TX3P_PORT/eDP1_TX_D3P: now reaches U1.AM3 (HDMI_TX1_D3P/EDP_TX1_D3P)
- net HDMI1_TX1P_PORT/eDP1_TX_D1P: now reaches U1.AM5 (HDMI_TX1_D1P/EDP_TX1_D1P)
- net at U1.AN1 (HDMI/EDP_TX1_REXT): now also R247.1
- net HDMI1_TX_SBDP/eDP1_TX_AUXP: now reaches U1.AN2 (HDMI_TX1_SBDP/EDP_TX1_AUXP)
- net HDMI1_TX3N_PORT/eDP1_TX_D3N: now reaches U1.AN3 (HDMI_TX1_D3N/EDP_TX1_D3N)
- net HDMI1_TX0P_PORT/eDP1_TX_D0P: now reaches U1.AN4 (HDMI_TX1_D0P/EDP_TX1_D0P)
- net HDMI1_TX1N_PORT/eDP1_TX_D1N: now reaches U1.AN5 (HDMI_TX1_D1N/EDP_TX1_D1N)
- net HDMI1_TX2P_PORT/eDP1_TX_D2P: now reaches U1.AN6 (HDMI_TX1_D2P/EDP_TX1_D2P)
- net HDMI1_TX_SBDN/eDP1_TX_AUXN: now reaches U1.AP2 (HDMI_TX1_SBDN/EDP_TX1_AUXN)
- net HDMI1_TX0N_PORT/eDP1_TX_D0N: now reaches U1.AP4 (HDMI_TX1_D0N/EDP_TX1_D0N)
- net HDMI1_TX2N_PORT/eDP1_TX_D2N: now reaches U1.AP6 (HDMI_TX1_D2N/EDP_TX1_D2N)
- net HDMITX0_CEC_M0: now reaches U1.AK24 (BT1120_D15/SPDIF1_TX_M2/PCIE20X1_2_PERSTN_M1/HDMI_TX0_CEC_M0/I2C8_SDA_M3/PWM6_M1/SPI3_CS1_M1/GPIO4_C1_D)
- net HDMITX0_HPDIN_M1: now reaches U1.B26 (HDMI_TX0_HPD_M0/SPI2_MOSI_M0/GPIO1_A5_D)
- net HDMITX1_HPDIN_M1: now reaches U1.C24 (HDMI_TX1_HPD_M0/SPI2_CLK_M0/GPIO1_A6_D)
- net I2C4_SCL_M1: now reaches U1.AB30 (GMAC0_PPSTRIG/FSPI_CS1N_M1/HDMI_TX1_SCL_M0/I2C4_SCL_M1/UART7_TX_M0/GPIO2_B5_U)
- net I2C4_SCL_M1: now also R212.2
- net I2C4_SDA_M1: now reaches U1.AB31 (GMAC0_PTP_REFCLK/FSPI_CS0N_M1/HDMI_TX1_SDA_M0/I2C4_SDA_M1/UART7_RX_M0/GPIO2_B4_U)
- net I2C4_SDA_M1: now also R211.2
- net HDMITX1_CEC_M2: now reaches U1.AC30 (GMAC0_PPSCLK/TEST_CLKOUT_M1/HDMI_TX1_CEC_M0/UART9_RX_M0/SPI1_CS1_M0/GPIO2_C4_D)
- net I2C5_SCL_M4: now reaches U1.AD33 (GMAC0_TXD0/I2S2_MCLK_M0/I2C5_SCL_M4/UART1_RX_M0/GPIO2_B6_D)
- net I2C5_SCL_M4: now also R213.2
- net I2C5_SDA_M4: now reaches U1.AD34 (GMAC0_TXD1/I2S2_SCLK_M0/I2C5_SDA_M4/UART1_TX_M0/GPIO2_B7_D)
- net I2C5_SDA_M4: now also R214.2
- net at U1.AG9 (USB20_HOST0_REXT): now also R224.2
- net at U1.AH9 (USB20_HOST1_REXT): now also R225.2
- net VCCA_3V3_S0: now reaches U1.AJ10 (USB20_AVDD_3V3)
- net VCCA_3V3_S0: now also C438.2, R221.1, R222.1
- net USB_2_OTG_DP: now reaches U1.AK9 (TYPEC1_USB20_OTG_DP)
- net USB_1_OTG_DP: now reaches U1.AL12 (TYPEC0_USB20_OTG_DP)
- net at U1.AL8 (TYPEC1_USB20_VBUSDET): now also R222.2
- net USB_2_OTG_DM: now reaches U1.AL9 (TYPEC1_USB20_OTG_DM)
- net USB_1_OTG_DM: now reaches U1.AM12 (TYPEC0_USB20_OTG_DM)
- net at U1.AM14 (TYPEC0_USB20_VBUSDET): now also R221.2
- net at U1.AP12 (TYPEC0_USB20_OTG0_REXT): now also R223.2
- net at U1.AP7 (TYPEC1_USB20_OTG1_REXT): now also R220.2
- new net USB_1_RX1N: C498.1
- new net USB_1_RX1P: C497.1
- new net USB_1_RX2N: C500.1
- new net USB_1_RX2P: C499.1
- new net USB_2_RX1N: C502.1
- new net USB_2_RX1P: C501.1
- new net USB_2_RX2N: C504.1
- new net USB_2_RX2P: C503.1
- new net VCC_1V8_SYS: R211.1, R212.1, R213.1, R214.1
- no-connect marks 22 -> 24
Other:
- moved on the sheet: U1A, U1B, U1C, U1F, U1J, U1K, U1L, U1M, U1O, U1P

Commit message: added the STM32L433RCT6 to act as the embedded controller
Parts:
- added C515, C516, C519, C520: 100nF, Capacitor_SMD:C_0201_0603Metric, symbol Device:C
- added C517, C518: 1uF, Capacitor_SMD:C_0201_0603Metric, symbol Device:C
- added R180: 200R, Resistor_SMD:R_0603_1608Metric, symbol Device:R
Connections:
- net GND: now also C515.1, C516.1, C517.1, C518.1, C519.1, C520.1, R180.1
- net VCCA_3V3_S0: now also U1.AE4 (HDMI_RX_VPH3V3), U1.AE5 (HDMI_RX_DVDD3V3), C517.2, C519.2
- net VCC_1V8_S0: now also U1.W25 (VCCIO5_1V8), C516.2
- net FSPI-D0: now reaches U1.AA29 (GMAC1_TXD2/SDIO_D0_M1/I2S3_MCLK/FSPI_D0_M2/I2C6_SDA_M4/PWM10_M0/SPI4_MISO_M1/GPIO3_A0_U)
- net FSPI-D1: now reaches U1.AA30 (GMAC1_TXD3/SDIO_D1_M1/I2S3_SCLK/AUDDSM_LN/FSPI_D1_M2/I2C6_SCL_M4/PWM11_IR_M0/SPI4_MOSI_M1/GPIO3_A1_U)
- net FSPI-D2: now reaches U1.AD27 (GMAC1_RXD2/SDIO_D2_M1/I2S3_LRCK/AUDDSM_LP/FSPI_D2_M2/UART8_TX_M1/SPI4_CLK_M1/GPIO3_A2_U)
- net FSPI-D3: now reaches U1.AE27 (GMAC1_RXD3/SDIO_D3_M1/I2S3_SDO/AUDDSM_RN/FSPI_D3_M2/UART8_RX_M1/SPI4_CS0_M1/GPIO3_A3_U)
- net HDMITX1_SCL_M1: now reaches U1.AG26 (CIF_D10/PCIE30X4_PERSTN_M2/HDMI_TX1_SCL_M1/SPI3_MISO_M3/GPIO3_C6_U)
- net HDMITX1_SDA_M1: now reaches U1.AH25 (CIF_D9/FSPI_CS1N_M2/PCIE30X4_WAKEN_M2/HDMI_TX1_SDA_M1/CAN2_TX_M0/UART5_RX_M1/SPI3_CS1_M3/GPIO3_C5_U)
- net FSPI-CS0: now reaches U1.AH26 (CIF_D8/FSPI_CS0N_M2/PCIE30X4_CLKREQN_M2/HDMI_TX1_CEC_M2/CAN2_RX_M0/UART5_TX_M1/SPI3_CS0_M3/GPIO3_C4_U)
- net FSPI-CLK: now reaches U1.AH30 (GMAC1_RXCLK/SDIO_CLK_M1/MIPI_CAMERA0_CLK_M1/FSPI_CLK_M2/I2C4_SDA_M0/UART8_CTSN_M1/GPIO3_A5_D)
- net VCC_3V3_S0: now reaches U1.W26 (VCCIO5)
- net VCC_3V3_S0: now also C515.2
- net I2C1_SCL_M0: now reaches U1.P29 (I2S1_MCLK_M1/JTAG_TCK_M2/I2C1_SCL_M0/UART2_TX_M0/PCIE30X1_1_CLKREQN_M0/GPIO0_B5_D)
- net I2C1_SDA_M0: now reaches U1.R29 (I2S1_SCLK_M1/JTAG_TMS_M2/I2C1_SDA_M0/UART2_RX_M0/PCIE30X1_1_WAKEN_M0/GPIO0_B6_D)
- net I2C0_SDA_M2: now reaches U1.W29 (I2S1_SDO1_M1/I2C0_SDA_M2/UART1_RX_M2/HDMI_RX_SCL_M0/SPI3_MOSI_M2/PCIE30X2_WAKEN_M0/HDMI_TX1_CEC_M1/GPIO0_D2_U)
- net I2C0_SCL_M2: now reaches U1.W30 (I2S1_SDO0_M1/CPU_BIG0_AVS/I2C0_SCL_M2/UART0_CTSN/UART1_TX_M2/HDMI_RX_SDA_M0/SPI0_CS0_M0/PCIE30X2_CLKREQN_M0/HDMI_TX0_CEC_M1/GPIO0_D1_U)
- net VCCA_0V75_S0: now reaches U1.AE8 (HDMI_RX_AVDD0V75)
- net VCCA_0V75_S0: now also C518.2, C520.2
- net at U1.AF3 (HDMI_RX_REXT): now also R180.2
- net HDMITX0_SDA_M0: now reaches U1.AJ25 (BT1120_D14/PCIE20X1_2_WAKEN_M1/HDMI_TX0_SDA_M0/I2C8_SCL_M3/SPI3_CS0_M1/GPIO4_C0_U)
- net PCIE30X4_WAKEn_M1_L: now reaches U1.AJ26 (BT1120_D11/PCIE30X4_WAKEN_M1/HDMI_RX_CEC_M0/SATA1_ACT_LED_M0/UART9_RX_M1/PWM12_M1/SPI3_MISO_M1/GPIO4_B5_D)
- net PCIE30X4_PERSTn_M1_L: now reaches U1.AJ27 (BT1120_D12/PCIE30X4_PERSTN_M1/HDMI_RX_HPDOUT_M0/SATA0_ACT_LED_M0/I2C5_SCL_M1/PWM13_M1/SPI3_MOSI_M1/GPIO4_B6_D)
- net HDMITX0_SCL_M0: now reaches U1.AJ28 (BT1120_D13/PCIE20X1_2_CLKREQN_M1/HDMI_TX0_SCL_M0/I2C5_SDA_M1/SPI3_CLK_M1/GPIO4_B7_U)
- net PCIE30X2_PERSTn_M1: now reaches U1.AK26 (CIF_CLKIN/BT1120_CLKOUT/I2S1_SDI3_M0/PCIE30X2_PERSTN_M1/I2C6_SDA_M3/UART8_TX_M0/SPI2_CS1_M1/GPIO4_B0_D)
- net PCIE30X1_0_PERSTn_M1_L: now reaches U1.AK27 (CIF_D5/BT1120_D5/I2S1_SDI0_M0/PCIE30X1_0_PERSTN_M1/I2C3_SDA_M2/UART3_TX_M2/SPI2_MOSI_M1/GPIO4_A5_D)
- net HDMI0_TX_ON_H: now reaches U1.AL24 (MIPI_CAMERA0_CLK_M0/SPDIF1_TX_M1/I2S1_SDO0_M0/PCIE30X1_0_BUTTON_RSTN/SATA2_ACT_LED_M0/I2C6_SCL_M3/UART8_RX_M0/SPI0_CS1_M1/GPIO4_B1_U)
- net PCIE30X4_CLKREQn_M1_L: now reaches U1.AL26 (CIF_CLKOUT/BT1120_D10/I2S1_SDO3_M0/PCIE30X4_CLKREQN_M1/DP0_HPDIN_M0/SPDIF0_TX_M1/UART9_TX_M1/PWM11_IR_M1/GPIO4_B4_U)
- net PCIE30X2_CLKREQn_M1: now reaches U1.AL27 (CIF_D6/BT1120_D6/I2S1_SDI1_M0/PCIE30X2_CLKREQN_M1/I2C5_SCL_M2/UART3_RX_M2/SPI2_CLK_M1/GPIO4_A6_D)
- net PCIE30X1_0_WAKEn_M1_L: now reaches U1.AL28 (CIF_D4/BT1120_D4/PCIE30X1_0_WAKEN_M1/I2C3_SCL_M2/UART0_RX_M2/SPI2_MISO_M1/GPIO4_A4_D)
- net PCIE30X1_0_CLKREQn_M1_L: now reaches U1.AL29 (CIF_D3/BT1120_D3/PCIE30X1_0_CLKREQN_M1/UART0_TX_M2/GPIO4_A3_D)
- net HDMI1_TX_ON_H: now reaches U1.AL30 (CIF_D1/BT1120_D1/I2S1_SCLK_M0/PCIE30X1_1_WAKEN_M1/UART9_CTSN_M1/SPI0_MOSI_M1/GPIO4_A1_D)
- net PCIE30X2_WAKEn_M1: now reaches U1.AM27 (CIF_D7/BT1120_D7/I2S1_SDI2_M0/PCIE30X2_WAKEN_M1/I2C5_SDA_M2/SPI2_CS0_M1/GPIO4_A7_D)
- net PCIE30x4_PWREN_H renamed PCIE30X4_PWREN_H
- no-connect marks 24 -> 32
Other:
- moved on the sheet: U1H

Commit message: added the display connector and its 12V power supply
Parts:
- renumbered C347 to C1, C362 to C10, C232 to C100, C304 to C101, C305 to C102, C538 to C103, C539 to C104, C540 to C105, C543 to C106, C545 to C107, C548 to C108, C112 to C109, C364 to C11, C224 to C110, C225 to C111, C226 to C112, C227 to C113, C228 to C114, C229 to C115, C230 to C116, C231 to C117, C329 to C118, C330 to C119, C366 to C12, C332 to C120, C333 to C121, C334 to C122, C338 to C123, C336 to C124, C280 to C125, C281 to C126, C282 to C127, C283 to C128, C284 to C129, C368 to C13, C285 to C130, C286 to C131, C324 to C132, C326 to C133, C317 to C134, C318 to C135, C319 to C136, C320 to C137, C321 to C138, C322 to C139, C370 to C14, C323 to C140, C325 to C141, C327 to C142, C296 to C143, C288 to C144, C289 to C145, C297 to C146, C291 to C147, C292 to C148, C293 to C149, C445 to C15, C294 to C150, C295 to C151, C315 to C152, C316 to C153, C337 to C154, C314 to C155, C313 to C156, C312 to C157, C311 to C158, C310 to C159, C443 to C16, C309 to C160, C308 to C161, C307 to C162, C306 to C163, C339 to C164, C446 to C17, C351 to C18, C352 to C19, C348 to C2, C349 to C20, C356 to C21, C357 to C22, C353 to C23, C419 to C24, C413 to C25, C359 to C26, C361 to C27, C363 to C28, C365 to C29, C343 to C3, C369 to C30, C371 to C31, C414 to C32, C354 to C33, C355 to C34, C420 to C35, C421 to C36, C422 to C37, C423 to C38, C367 to C39, C344 to C4, C372 to C40, C444 to C41, C424 to C42, C442 to C43, C437 to C44, C438 to C45, C454 to C46, C516 to C47, C515 to C48, C143 to C49, C345 to C5, C340 to C50, C519 to C51, C517 to C52, C520 to C53, C518 to C54, C432 to C55, C433 to C56, C434 to C57, C435 to C58, C507 to C59, C346 to C6, C508 to C60, C509 to C61, C510 to C62, C465 to C63, C455 to C64, C505 to C65, C506 to C66, C427 to C67, C431 to C68, C425 to C69, C350 to C7, C426 to C70, C107 to C71, C108 to C72, C497 to C73, C501 to C74, C466 to C75, C498 to C76, C502 to C77, C467 to C78, C499 to C79, C358 to C8, C503 to C80, C500 to C81, C504 to C82, C534 to C83, C535 to C84, C533 to C85, C541 to C86, C542 to C87, C546 to C88, C303 to C89, C360 to C9, C302 to C90, C301 to C91, C300 to C92, C299 to C93, C290 to C94, C298 to C95, C537 to C96, C536 to C97, C544 to C98, C547 to C99, R212 to R1, R155 to R10, R157 to R11, R89 to R12, R159 to R13, R158 to R14, R224 to R15, R225 to R16, R221 to R17, R222 to R18, R220 to R19, R211 to R2, R223 to R20, R180 to R21, R150 to R22, R151 to R23, R152 to R24, R153 to R25, R174 to R26, R173 to R27, R226 to R28, R227 to R29, R213 to R3, R246 to R30, R247 to R31, R214 to R4, R96 to R5, R154 to R6, R165 to R7, R156 to R8, R164 to R9
Connections:
- net HDMI0_TX_ON_H: no longer names the net of U1.AL24 (MIPI_CAMERA0_CLK_M0/SPDIF1_TX_M1/I2S1_SDO0_M0/PCIE30X1_0_BUTTON_RSTN/SATA2_ACT_LED_M0/I2C6_SCL_M3/UART8_RX_M0/SPI0_CS1_M1/GPIO4_B1_U)
- net HDMI0_TX_SBDN/eDP0_TX_AUXN: no longer names the net of U1.AG1 (HDMI_TX0_SBDN/EDP_TX0_AUXN)
- net HDMI0_TX_SBDP/eDP0_TX_AUXP: no longer names the net of U1.AG2 (HDMI_TX0_SBDP/EDP_TX0_AUXP)
- net HDMITX0_CEC_M0: no longer names the net of U1.AK24 (BT1120_D15/SPDIF1_TX_M2/PCIE20X1_2_PERSTN_M1/HDMI_TX0_CEC_M0/I2C8_SDA_M3/PWM6_M1/SPI3_CS1_M1/GPIO4_C1_D)
- net HDMITX0_HPDIN_M1: no longer names the net of U1.B26 (HDMI_TX0_HPD_M0/SPI2_MOSI_M0/GPIO1_A5_D)
- net HDMITX0_SCL_M0: no longer names the net of U1.AJ28 (BT1120_D13/PCIE20X1_2_CLKREQN_M1/HDMI_TX0_SCL_M0/I2C5_SDA_M1/SPI3_CLK_M1/GPIO4_B7_U)
- net HDMITX0_SDA_M0: no longer names the net of U1.AJ25 (BT1120_D14/PCIE20X1_2_WAKEN_M1/HDMI_TX0_SDA_M0/I2C8_SCL_M3/SPI3_CS0_M1/GPIO4_C0_U)
- no-connect marks 32 -> 34
