File: barebones_chip.kicad_sch (KiCad schematic)
At the start: 198 parts, among them U1 RK3588, Y1 C3E-24.000-12-3030-X-R

Commit message: added the PCF85063ATL/1,118 CMOS Real-Time Clock
Parts:
- added C522: 100nF, Capacitor_SMD:C_0201_0603Metric, symbol Device:C
Connections:
- net GND: now also C522.2
- net RTC_CLK_EN: now reaches U1.L30 (SPI2_CS1_M2/I2C1_SCL_M1/UART0_RX_M1/GPIO0_B0_Z)
- net RESETB: now reaches U1.M31 (NPOR)
- net RESETB: now also U1.P32 (TSADC_SHUT_ORG/TSADC_SHUT/GPIO0_A1_Z), C522.1
- net CPU_BIG0_VSEL: now reaches U1.R31 (PMIC_SLEEP2/GPIO0_A3_D)
- net USB_2_SBU1_DC: now reaches U1.P30 (I2S1_SDI0_M1/GPU_AVS/UART0_TX_M0/I2C4_SCL_M2/DP1_HPDIN_M1/PWM4_M0/PCIE30X1_0_PERSTN_M0/GPIO0_C5_U)
- net USB_1_SBU1_DC: now reaches U1.R30 (PDM0_CLK1_M1/PWM2_M0/UART0_RX_M0/I2C4_SDA_M2/DP0_HPDIN_M1/PCIE30X1_0_WAKEN_M0/GPIO0_C4_D)
- net NPU_VSEL: now reaches U1.U32 (PMIC_SLEEP3/GPIO0_C1_D)
- net CPU_BIG1_VSEL: now reaches U1.W28 (PMIC_SLEEP6/PDM0_SDI3_M1/GPIO0_D6_D)
- net INT_PMIC renamed PMIC_INT_L
- net PWRCTRL1_PMIC renamed PMIC_SLEEP1
- net SPI_CLK_PMIC renamed SPI2_CLK_M2
- net SPI_CS_PMIC renamed SPI2_CS0_M2
- net SPI_MOSI_PMIC renamed SPI2_MOSI_M2
- no-connect marks 34 -> 42
Other:
- moved on the sheet: C25, C32, R10, R22, R23, R24, R25, R5, R6, R8, U1C, U1D

Commit message: updated the Fuel Guage/BMS module for the 4S battery usage
Parts:
- added C253, C394: 100nF, Capacitor_SMD:C_0201_0603Metric, symbol Device:C
Connections:
- net GND: now also C253.1, C394.1
- net VCC_1V8_S0: now also U1.G20 (VCCIO1_1V8), U1.Y26 (VCCIO3_1V8), C253.2, C394.2
- net I2S0_SDI0: now reaches U1.D28 (I2S0_SDI0/GPIO1_D4_D)
- net I2S0_LRCK_TX: now reaches U1.D30 (I2S0_LRCK/I2C2_SCL_M3/UART4_RTSN/GPIO1_C5_D)
- net HP_INT: now reaches U1.E28 (I2S0_SDI1/PDM0_SDI3_M0/I2C1_SDA_M4/UART4_RX_M0/PWM1_M1/SPI1_CS0_M2/GPIO1_D3_D)
- net I2S0_SDO0: now reaches U1.E29 (I2S0_SDO0/I2C4_SCL_M4/UART4_CTSN/GPIO1_C7_D)
- net EDP_TX0_HDP: now reaches U1.E30 (PDM0_CLK1_M0/I2C2_SDA_M3/PWM11_IR_M2/SPI4_CS1_M0/GPIO1_C4_D)
- net I2S0_SCLK_TX: now reaches U1.E31 (I2S0_SCLK/I2C6_SCL_M1/UART3_CTSN/PWM7_IR_M2/SPI4_CS0_M0/GPIO1_C3_D)
- net I2C7_SCL_M0: now reaches U1.F26 (I2S0_SDO1/I2C7_SCL_M0/UART6_TX_M2/SPI1_MISO_M2/GPIO1_D0_D)
- net I2C7_SDA_M0: now reaches U1.F27 (I2S0_SDO2/I2S0_SDI3/PDM0_SDI1_M0/I2C7_SDA_M0/UART6_RX_M2/SPI1_MOSI_M2/GPIO1_D1_D)
- net I2S0_MLCK: now reaches U1.F30 (I2S0_MCLK/I2C6_SDA_M1/UART3_RTSN/PWM3_IR_M2/SPI4_CLK_M0/GPIO1_C2_D)
- net HP_DETECT: now reaches U1.G26 (PDM0_SDI0_M0/SPI1_CS1_M2/GPIO1_D5_D)
- no-connect marks 42 -> 59
Other:
- moved on the sheet: C1, C10, C11, C12, C13, C14, C15, C16, C17, C18, C19, C2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
