File: barebones_io.kicad_sch (KiCad schematic)
At the start: 229 parts, among them IC1 W25Q80DVSSIG, IC2 W25Q80DVSSIG, J1 12401610E4_2A, J10 10067847-001RLF, J11 G45AA1912100B1EU, J12 1-2199119-5, J13 SM02B-GHS-TB_LF__SN_, J14 SM02B-GHS-TB_LF__SN_, J2 12401610E4_2A, J3 1-2199119-5, J4 21992304, J5 G45AA1912100B1EU, J6 1040310811, J7 54-00007, J8 SJ2-35894B-SMT-TR, J9 54-00007, U16 TPS65987DDHRSHR, U17 TPS65987DDHRSHR, U19 TXS0104EYZTR, U21 TXS0104EYZTR, U25 TPD4E05U06DQAR, U26 TPD4E004DRYR, U42 TXS0104EYZTR, U43 TPS2553DBVR, U44 TPS2553DBVR, U45 PCA9306DCTR, U46 TPS2553DBVR, U47 PCA9306DCTR, U48 TPS2553DBVR, U52 PI6C557-05LEX, U53 PI6C557-05BLEX, U54 TPD4E004DRYR, U55 PI6C557-03ALEX, U56 TPD4E004DRYR, U57 TPD4E004DRYR, U58 GL3523-ONY30, U59 9FGV0641AKILFT, Y2 C2E-25.000-10-1530-X-R, Y3 C2E-25.000-10-1530-X-R, Y4 C2E-25.000-10-1530-X-R

Commit message: fixed the connection for the two HDMI ports and connected them to the RK3588 section Z
Parts:
- removed C216, C218, C220, C221: 100uF, Capacitor_SMD:C_0201_0603Metric, symbol Device:C
- removed C217, C222: 0.1uF, Capacitor_SMD:C_0201_0603Metric, symbol Device:C
- removed R118, R126, R134, R140, R73, R74: 10k, Resistor_SMD:R_0402_1005Metric, symbol Device:R
- removed R119, R141: 330k, Resistor_SMD:R_0402_1005Metric, symbol Device:R
- removed R120, R121, R122, R123, R124, R128, R129, R131, R132, R135, R136, R137, R138, R139: 2.2k, Resistor_SMD:R_0402_1005Metric, symbol Device:R
- removed R125, R133: 18k, Resistor_SMD:R_0402_1005Metric, symbol Device:R
- removed R127, R130: 27k, Resistor_SMD:R_0402_1005Metric, symbol Device:R
- removed U47: PCA9306DCTR, barebones:SOP65P400X130-8N, symbol PCA9306DCTR:PCA9306DCTR
- removed U48: TPS2553DBVR, barebones:SOT95P280X145-6N, symbol TPS2553DBVR:TPS2553DBVR
- removed Y2: C2E-25.000-10-1530-X-R, barebones:XTAL_C2E-25.000-10-1530-X-R, symbol C2E-25.000-10-1530-X-R:C2E-25.000-10-1530-X-R
- added C487, C488, C491, C492, C493, C494, C511, C512: 0.1uF, Capacitor_SMD:C_0201_0603Metric, symbol Device:C
- added C489, C490, C495, C496: 220pF, Capacitor_SMD:C_0201_0603Metric, symbol Device:C
- added C513, C514, C515, C516, C517, C518, C519, C520, C521, C522: 220nF, Capacitor_SMD:C_0201_0603Metric, symbol Device:C
- added C523, C526: 100pF, Capacitor_SMD:C_0201_0603Metric, symbol Device:C
- added C524, C528, C529, C530, C531, C532: 100uF, Capacitor_SMD:C_0201_0603Metric, symbol Device:C
- added C525, C527: 1uF, Capacitor_SMD:C_0201_0603Metric, symbol Device:C
- added D10, D16, D17, D9: SD103AWS-E3-08, SD103AWS-E3-08:SOD2713X115N, symbol SD103AWS-E3-08:SD103AWS-E3-08
- added IC3, IC4: FUSB302BMPX, barebones:QFN50P250X250X80-15N, symbol FUSB302BMPX:FUSB302BMPX
- added R205, R231, R234, R71: 10k, Resistor_SMD:R_0402_1005Metric, symbol Device:R
- added R206, R207, R208, R209, R210, R215, R216, R217, R218, R219: 2.2k, Resistor_SMD:R_0402_1005Metric, symbol Device:R
- added R228, R232, R233: 1k, Resistor_SMD:R_0402_1005Metric, symbol Device:R
- added R229, R230, R236, R237: 27k, Resistor_SMD:R_0402_1005Metric, symbol Device:R
- added R235: 1.8k, Resistor_SMD:R_0402_1005Metric, symbol Device:R
- added R238, R239, R240, R242, R243, R244: 47k, Resistor_SMD:R_0402_1005Metric, symbol Device:R
- added R241, R245: 1.2k, Resistor_SMD:R_0402_1005Metric, symbol Device:R
- added U51, U60: PCA9306DCTR, barebones:SOP65P400X130-8N, symbol PCA9306DCTR:PCA9306DCTR
- added U61: PI3DPX1207Q3ZHEX, barebones:QFN50P900X350X84-43N, symbol PI3DPX1207Q3ZHEX:PI3DPX1207Q3ZHEX
- added U62: OV9734-H16A, OV9734-H16A:BGA16N27X30P8X4_253X172X80N, symbol OV9734-H16A:OV9734-H16A
- added U63, U64, U65, U66, U67, U68, U69, U70, U71, U72, U73, U74, U75, U76, U77, U78, U79, U80: 2N7002KW, 2N7002KW:SOT323, symbol 2N7002KW:2N7002KW
- C428, C429: value 12pF -> 220nF
- C430, C439, C440: value 100nF -> 220nF
- C441: value 1uF -> 220nF
- R170: value 475R -> 499R
- R171, R172: value 10k -> 499R
- R175: value 2.2R -> 499R
- R176, R177, R178, R179, R180, R181, R182, R183: value 50R -> 499R
- R185, R186, R187, R188: value 33R -> 499R
- R189, R190: value 33R -> 10k
- R191: value 33R -> 1k
- R192: value 33R -> 1.8k
Connections:
- net GND: now also C487.2, C488.2, C489.2, C490.2, C491.2, C492.2, C493.2, C494.2, C495.2, C496.2, C524.1, C525.1, C527.1, C528.1, IC3.15 (EP_GND), IC3.8 (GND_1), IC3.9 (GND_2), IC4.15 (EP_GND), IC4.8 (GND_1), IC4.9 (GND_2), R240.1, R244.1, U51.1 (GND), U60.1 (GND), U61.43 (GND), U61.43.1 (GND), U61.43.10 (GND), U61.43.11 (GND), U61.43.12 (GND), U61.43.13 (GND), U61.43.14 (GND), U61.43.15 (GND), U61.43.16 (GND), U61.43.17 (GND), U61.43.18 (GND), U61.43.2 (GND), U61.43.3 (GND), U61.43.4 (GND), U61.43.5 (GND), U61.43.6 (GND), U61.43.7 (GND), U61.43.8 (GND), U61.43.9 (GND), U63.3, U64.3, U65.3, U66.3, U67.3, U68.3, U69.3, U70.3, U77.3, U78.3, U79.3, U80.3; no longer C428.1, C429.1, C430.1, C439.1, C440.1, C441.1, R170.2, R176.2, R177.2, R178.2, R179.2, R180.2, R181.2, R182.2, R183.2, U45.1 (GND), U46.2 (GND), U53.16 (GNDODA), U53.2 (S0), U53.3 (S1), U53.4 (S2), U53.9 (GNDXD)
- net HDMI_0_CEC: now also R229.1, U73.1
- net HDMI_0_SDA_1: now also R192.1, U72.1; no longer U45.5 (SDA2)
- net HDMI_1_CEC: now also R237.1, U76.1
- net HDMI_1_SDA_1: now also R235.1, U75.1
- net PCIE20_0_RXN: now also J4.43; no longer J4.37
- net PCIE20_0_RXP: now also J4.41; no longer J4.35
- net PCIE20_0_TXN: now also C512.1; no longer J4.43
- net PCIE20_0_TXP: now also C511.1; no longer J4.41
- net PCIE30_PORT0_REF_CLKN: no longer R182.1, R188.2
- net PCIE30_PORT0_REF_CLKP: no longer R183.1, R187.2
- net PCIE30_PORT1_REF_CLKN: no longer R180.1, R190.2
- net PCIE30_PORT1_REF_CLKP: no longer R181.1, R189.2
- net PCIE30_REFCLKN_SLOT_0: no longer R178.1, R192.2
- net PCIE30_REFCLKN_SLOT_1: no longer R176.1, R185.2
- net PCIE30_REFCLKP_SLOT_0: no longer R179.1, R191.2
- net PCIE30_REFCLKP_SLOT_1: no longer R177.1, R186.2
- net TMDS_CLOCK_0_DM: now also C522.1
- net TMDS_CLOCK_0_DP: now also C521.1
- net TMDS_CLOCK_1_DM: now also C514.1
- net TMDS_CLOCK_1_DP: now also C513.1
- net TMDS_DATA0_0_DM: now also C520.1
- net TMDS_DATA0_0_DP: now also C519.1
- net TMDS_DATA0_1_DM: now also C441.1
- net TMDS_DATA0_1_DP: now also C440.1
- net TMDS_DATA1_0_DM: now also C518.1
- net TMDS_DATA1_0_DP: now also C517.1
- net TMDS_DATA1_1_DM: now also C439.1
- net TMDS_DATA1_1_DP: now also C430.1
- net TMDS_DATA2_0_DM: now also C516.1
- net TMDS_DATA2_0_DP: now also C515.1
- net TMDS_DATA2_1_DM: now also C429.1
- net TMDS_DATA2_1_DP: now also C428.1
- net USB1_CC1: now also C490.1, IC3.10 (CC1_1), IC3.11 (CC1_2)
- net USB1_CC2: now also C489.1, IC3.1 (CC2_1), IC3.14 (CC2_2)
- net USB1_TX1N: now also D8.1 (IO1); no longer D7.4 (IO3)
- net USB1_TX1P: now also D8.2 (IO2); no longer D7.5 (IO4)
- net USB2_CC1: now also C496.1, IC4.10 (CC1_1), IC4.11 (CC1_2)
- net USB2_CC2: now also C495.1, IC4.1 (CC2_1), IC4.14 (CC2_2)
- net USB2_TX1N: now also D5.1 (IO1); no longer D6.4 (IO3)
- net USB2_TX1P: now also D5.2 (IO2); no longer D6.5 (IO4)
- net USB30_2_SSRXN: now also U58.46 (RXN1_P0); no longer C464.1
- net USB30_2_SSRXP: now also U58.47 (RXP1_P0); no longer C463.1
- net USB30_2_SSTXN: now also C464.1; no longer U58.46 (RXN1_P0)
- net USB30_2_SSTXP: now also C463.1; no longer U58.47 (RXP1_P0)
- net USB_1_RX1N: now also D7.4 (IO3); no longer D8.1 (IO1)
- net USB_1_RX1P: now also D7.5 (IO4); no longer D8.2 (IO2)
- net USB_2_RX1N: now also D6.4 (IO3); no longer D5.1 (IO1)
- net USB_2_RX1P: now also D6.5 (IO4); no longer D5.2 (IO2)
- net VBUS_A: now also IC3.2 (VBUS), IC4.2 (VBUS)
- net VCC_1V8_SYS: now also R205.1, R209.1, R210.1, R217.1, R219.1, R71.1, U51.2 (VREF1), U60.2 (VREF1); no longer U45.2 (VREF1)
- net VCC_3V3_SYS: now also C491.1, C493.1, IC3.3 (VDD_1), IC3.4 (VDD_2), IC4.3 (VDD_1), IC4.4 (VDD_2), R206.1, R207.1, R208.1, R215.1, R216.1, R218.1
- net VCC_5V0_PERIPH: no longer U45.7 (VREF2), U45.8 (EN), U46.1 (IN)
- net at U53.13 (~{CLK2}): no longer R192.1
- net at U53.11 (~{CLK3}): no longer R185.1
- net at R171.2: now also R170.2, U63.1; no longer U53.7 (~{PD})
- net at U53.12 (CLK3): no longer R186.1
- net at U53.5 (X1): no longer C428.2
- net PCIE20_1_CLKREQn_M1: now reaches J4.53
- net at U53.10 (IREF): no longer R170.1
- net at U53.14 (CLK2): no longer R191.1
- net at U53.17 (~{CLK1}): no longer R190.1
- net at U53.18 (CLK1): no longer R189.1
- net at U53.19 (~{CLK0}): no longer R188.1
- net at U53.20 (CLK0): no longer R187.1
- net at U53.6 (X2): no longer C429.2
- net at R172.2: now also R175.2, U64.1; no longer U53.8 (OE)
- net HDMI2_0_5V0: no longer names the net of U46.6 (OUT)
- net HDMI2_0_5V0: no longer J5.18 (+5V_POWER)
- net HDMI2_0_FAULT: no longer names the net of U46.4 (~{FAULT})
- net HDMI_0_SCL: no longer names the net of U45.3 (SCL1)
- net HDMI_0_SCL_1 renamed HDMI0_TX_SBDP
- net HDMI0_TX_SBDP: now also R190.1, C529.2, C531.2, U71.1
- net HDMI_0_SDA: no longer names the net of U45.4 (SDA1)
- net HDMI_1_SCL_1: no longer names the net of U45.6 (SCL2)
- net HDMI_1_SCL_1: no longer J11.15 (SCL)
- net HDMI_ENABLE: no longer names the net of U46.3 (EN)
- net HOT_PLUG_DETECT_0 renamed HDMI0_TX_SBDN
- net HDMI0_TX_SBDN: now also C530.2, C532.2, R241.1
- net HOT_PLUG_DETECT_1 renamed HDMI1_TX_SBDN
- net HDMI1_TX_SBDN: now also R245.1
- net PCIE30X1_0_PERSTN_M0 renamed PCIE20_1_RESETn_M1
- net PCIE20_1_RESETn_M1: no longer J4.22
- net PCIE30X1_0_WAKEN_M0 renamed PCIE20_1_WAKEn_M1
- removed net VCC3V3_PI6C_05: C430.2, C439.2, R171.1, R172.1, R175.2, U53.1 (VDDXD)
- new net: C526.1, R233.1, U75.2
- new net: R176.2, R177.2, U65.1
- new net: R178.2, R179.2, U66.1
- new net: R243.1, U79.2, U80.1
- new net: R180.2, R181.2, U67.1
- new net: R187.2, R188.2, U70.1
- new net: R244.2, R245.2, U80.2
- new net: C523.1, R228.1, U72.2
- new net: R185.2, R186.2, U69.1
- new net: R206.2, U51.7 (VREF2), U51.8 (EN)
- new net: R240.2, R241.2, U78.2
- new net: R215.2, U60.7 (VREF2), U60.8 (EN)
- new net: R182.2, R183.2, U68.1
- new net: R238.1, U77.2, U78.1
- new net: C511.2, J4.35
- new net: C512.2, J4.37
- new net: D10.1, R229.2
- new net: D17.1, R237.2
- new net FU_INT_L: IC3.5 (INT_N), R71.2
- new net FU_INT_L2: IC4.5 (INT_N), R205.2
- new net FU_SCL_1: IC3.6 (SCL), R218.2, U60.6 (SCL2)
- new net FU_SCL_2: IC4.6 (SCL), R207.2, U51.6 (SCL2)
- new net FU_SDA_1: IC3.7 (SDA), R216.2, U60.5 (SDA2)
- new net FU_SDA_2: IC4.7 (SDA), R208.2, U51.5 (SDA2)
- new net HDMI0_TX0N_PORT/eDP0_TX_D0N: C520.2, R186.1
- new net HDMI0_TX0P_PORT/eDP0_TX_D0P: C519.2, R185.1
- new net HDMI0_TX1N_PORT/eDP0_TX_D1N: C518.2, R183.1
- new net HDMI0_TX1P_PORT/eDP0_TX_D1P: C517.2, R182.1
- new net HDMI0_TX2N_PORT/eDP0_TX_D2N: C516.2, R181.1
- new net HDMI0_TX2P_PORT/eDP0_TX_D2P: C515.2, R180.1
- new net HDMI0_TX3N_PORT/eDP0_TX_D3N: C522.2, R188.1
- new net HDMI0_TX3P_PORT/eDP0_TX_D3P: C521.2, R187.1
- new net HDMI0_TX_ON_H: U67.2, U68.2, U69.2, U70.2
- new net HDMI0_TX_SBDN/eDP0_TX_AUXN: C530.1
- new net HDMI0_TX_SBDP/eDP0_TX_AUXP: C529.1
- new net HDMI1_TX0N_PORT/eDP1_TX_D0N: C441.2, R177.1
- new net HDMI1_TX0P_PORT/eDP1_TX_D0P: C440.2, R176.1
- new net HDMI1_TX1N_PORT/eDP1_TX_D1N: C439.2, R175.1
- new net HDMI1_TX1P_PORT/eDP1_TX_D1P: C430.2, R172.1
- new net HDMI1_TX2N_PORT/eDP1_TX_D2N: C429.2, R171.1
- new net HDMI1_TX2P_PORT/eDP1_TX_D2P: C428.2, R170.1
- new net HDMI1_TX3N_PORT/eDP1_TX_D3N: C514.2, R179.1
- new net HDMI1_TX3P_PORT/eDP1_TX_D3P: C513.2, R178.1
- new net HDMI1_TX_ON_H: U63.2, U64.2, U65.2, U66.2
- new net HDMI1_TX_SBDN/eDP1_TX_AUXN: C532.1
- new net HDMI1_TX_SBDP: J11.15 (SCL), R234.1, U74.1
- new net HDMI1_TX_SBDP/eDP1_TX_AUXP: C531.1
- new net HDMITX0_CEC_M0: R230.1, U73.3
- new net HDMITX0_HPDIN_M1: R239.1, U77.1
- new net HDMITX0_SCL_M0: R189.1, U71.3
- new net HDMITX0_SDA_M0: C523.2, R191.1, U72.3
- new net HDMITX1_CEC_M2: R236.1, U76.3
- new net HDMITX1_HPDIN_M1: R242.1, U79.1
- new net HDMITX1_SCL_M1: R231.1, U74.3
- new net HDMITX1_SDA_M1: C526.2, R232.1, U75.3
- new net I2C4_SCL_M1: R209.2, U51.3 (SCL1)
- new net I2C4_SDA_M1: R210.2, U51.4 (SDA1)
- new net I2C5_SCL_M4: R217.2, U60.3 (SCL1)
- new net I2C5_SDA_M4: R219.2, U60.4 (SDA1)
- new net VCC5V0_HDMI_TX0: D16.1, D9.1, R190.2, R192.2, R234.2, R235.2
- new net VCC5V0_SYS: D16.2, D9.2, U73.2, U76.2
- new net VCC5V_HDMI_TX0: C524.2, C525.2, C527.2, C528.2, J5.18 (+5V_POWER)
- new net VCC_1V8_S0: R238.2, R239.2, R242.2, R243.2
- new net VCC_3V3_S0: D10.2, D17.2, R189.2, R191.2, R228.2, R230.2, R231.2, R232.2, R233.2, R236.2, U71.2, U74.2
- new net VCC_5V0_SYS: C487.1, C488.1, C492.1, C494.1, IC3.12 (VCONN_1), IC3.13 (VCONN_2), IC4.12 (VCONN_1), IC4.13 (VCONN_2)
- new net VDD33: U61.12 (VDD33), U61.13 (VDD33), U61.26 (VDD33), U61.27 (VDD33), U61.31 (VDD33), U61.34 (VDD33), U61.35 (VDD33), U61.4 (VDD33), U61.5 (VDD33), U61.8 (VDD33)
- now unconnected: U53.15 (VDDODA)
- no-connect marks 150 -> 151
Other:
- note removed: "USE 1% TOLERANCE"
- moved on the sheet: C109, C110, C111, C184, C185, C208, C209, C210, C211, C391, C392, C393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

Commit message: added the STM32L433RCT6 to act as the embedded controller
Parts:
- removed C515, C516, C517, C518, C519, C520, C521, C522: 220nF, Capacitor_SMD:C_0201_0603Metric, symbol Device:C
- removed C523: 100pF, Capacitor_SMD:C_0201_0603Metric, symbol Device:C
- removed C524, C529, C530: 100uF, Capacitor_SMD:C_0201_0603Metric, symbol Device:C
- removed D10, D9: SD103AWS-E3-08, SD103AWS-E3-08:SOD2713X115N, symbol SD103AWS-E3-08:SD103AWS-E3-08
- removed D11, D12: TPD4E02B04DQAR, barebones:DIO_TPD4E02B04DQAR, symbol TPD4E02B04DQAR:TPD4E02B04DQAR
- removed J5: G45AA1912100B1EU, barebones:AMPHENOL_G45AA1912100B1EU, symbol G45AA1912100B1EU:G45AA1912100B1EU
- removed R180, R181, R182, R183, R185, R186, R187, R188: 499R, Resistor_SMD:R_0402_1005Metric, symbol Device:R
- removed R189, R190: 10k, Resistor_SMD:R_0402_1005Metric, symbol Device:R
- removed R191, R228: 1k, Resistor_SMD:R_0402_1005Metric, symbol Device:R
- removed R192: 1.8k, Resistor_SMD:R_0402_1005Metric, symbol Device:R
- removed R229, R230: 27k, Resistor_SMD:R_0402_1005Metric, symbol Device:R
- removed R238, R239, R240: 47k, Resistor_SMD:R_0402_1005Metric, symbol Device:R
- removed R241: 1.2k, Resistor_SMD:R_0402_1005Metric, symbol Device:R
- removed U67, U68, U69, U70, U71, U72, U73, U77, U78: 2N7002KW, 2N7002KW:SOT323, symbol 2N7002KW:2N7002KW
- added C549: 10uF, Capacitor_SMD:C_0201_0603Metric, symbol Device:C
- added C550, C552: 0.1uF, Capacitor_SMD:C_0201_0603Metric, symbol Device:C
- added C551: 4.7uF, Capacitor_SMD:C_0201_0603Metric, symbol Device:C
- added J15: 20455-040E-76, 20455-040E-76:IPEX_20455-040E-76, symbol 20455-040E-76:20455-040E-76
- added J5: SM05B-SRSS-TB_LF__SN_, SM05B-SRSS-TB_LF__SN_:JST_SM05B-SRSS-TB_LF__SN_, symbol SM05B-SRSS-TB_LF__SN_:SM05B-SRSS-TB_LF__SN_
- C525: value 1uF -> 100nF; footprint Capacitor_SMD:C_0201_0603Metric -> Capacitor_SMD:C_0603_1608Metric
- C531, C532: value 100uF -> 1uF
Connections:
- net GND: now also C525.2, C549.1, C550.1, C551.1, C552.1, J15.11, J15.14, J15.17, J15.2, J15.23, J15.24, J15.25, J15.26, J15.28, J15.29, J15.30, J15.31, J15.5, J15.8, J15.S1 (SHIELD), J15.S2 (SHIELD), J15.S3 (SHIELD), J15.S4 (SHIELD), J5.5, J5.S1 (SHIELD), J5.S2 (SHIELD); no longer C525.1
- net HDMI0_TX0N_PORT/eDP0_TX_D0N: now also J15.12
- net HDMI0_TX0P_PORT/eDP0_TX_D0P: now also J15.13
- net HDMI0_TX1N_PORT/eDP0_TX_D1N: now also J15.9
- net HDMI0_TX1P_PORT/eDP0_TX_D1P: now also J15.10
- net HDMI0_TX2N_PORT/eDP0_TX_D2N: now also J15.6
- net HDMI0_TX2P_PORT/eDP0_TX_D2P: now also J15.7
- net HDMI0_TX3N_PORT/eDP0_TX_D3N: now also J15.3
- net HDMI0_TX3P_PORT/eDP0_TX_D3P: now also J15.4
- net VCC_3V3_SYS: now also C551.2, C552.2, J15.18, J15.19, J15.20, J15.21
- net PCIE20_1_CLKREQn_M1 renamed PCIE30X1_0_CLKREQn_M1_L
- net PCIE20_1_RESETn_M1 renamed PCIE30X1_0_PERSTn_M1_L
- net PCIE20_1_WAKEn_M1 renamed PCIE30X1_0_WAKEn_M1_L
- net PCIE30X2_CLKREQn_M1_L renamed PCIE30X2_CLKREQn_M1
- net PCIE30X2_PERSTn_M1_L renamed PCIE30X2_PERSTn_M1
- net PCIE30X2_WAKEn_M1_L renamed PCIE30X2_WAKEn_M1
- net VCC5V_HDMI_TX0 renamed VCC5V_HDMI_TX1
- net VCC5V_HDMI_TX1: no longer C525.2
- new net EDP_TX0_AUX_N: J15.16
- new net EDP_TX0_AUX_P: J15.15
- new net EDP_TX0_BL_EN: J15.32
- new net EDP_TX0_BL_PWM: J15.33
- new net EDP_TX0_HDP: J15.27
- new net NRST_7: J5.4
- new net SWCLK_14: J5.3
- new net SWDIO_13: J5.2
- new net VCC_12V_EDP: C549.2, C550.2, J15.36, J15.37, J15.38, J15.39
- new net VCC_3V3_ALW: C525.1, J5.1
- no-connect marks 151 -> 153
Other:
- note added: "AUO B173ZAN03.3"
- note added: "EC PROGRAMMING PINS"
- moved on the sheet: C109, C110, C111, C219, C415, C428, C429, C430, C439, C440, C441, C511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

Commit message: added the display connector and its 12V power supply
Parts:
- removed C525: 100nF, Capacitor_SMD:C_0603_1608Metric, symbol Device:C
- removed C549: 10uF, Capacitor_SMD:C_0201_0603Metric, symbol Device:C
- removed C550, C552: 0.1uF, Capacitor_SMD:C_0201_0603Metric, symbol Device:C
- removed C551: 4.7uF, Capacitor_SMD:C_0201_0603Metric, symbol Device:C
- removed J5: SM05B-SRSS-TB_LF__SN_, SM05B-SRSS-TB_LF__SN_:JST_SM05B-SRSS-TB_LF__SN_, symbol SM05B-SRSS-TB_LF__SN_:SM05B-SRSS-TB_LF__SN_
- added C539: 100nF, Capacitor_SMD:C_0603_1608Metric, symbol Device:C
- added C541: 4.7uF, Capacitor_SMD:C_0201_0603Metric, symbol Device:C
- added C543, C544: 0.1uF, Capacitor_SMD:C_0201_0603Metric, symbol Device:C
- added C545: 10uF, Capacitor_SMD:C_0201_0603Metric, symbol Device:C
- added FPC1: FH12-6S-0.5SH, barebones:FPC-SMD_FH12-6S-0.5SH-55, symbol FH12-6S-0.5SH(55):FH12-6S-0.5SH
- added J14: SM05B-SRSS-TB_LF__SN_, SM05B-SRSS-TB_LF__SN_:JST_SM05B-SRSS-TB_LF__SN_, symbol SM05B-SRSS-TB_LF__SN_:SM05B-SRSS-TB_LF__SN_
- added J16: 524352671, barebones:CON_524352671_MOL, symbol 524352671:524352671
- added J17: 522070485, barebones:CON_522070485_MOL, symbol 522070485:522070485
- added J19: SM06B-SRSS-TB_LF__SN_, SM06B-SRSS-TB_LF__SN_:JST_SM06B-SRSS-TB_LF__SN_, symbol SM06B-SRSS-TB_LF__SN_:SM06B-SRSS-TB_LF__SN_
- added J20: 20682-040E-02, 20682-040E-02:IPEX_20682-040E-02, symbol 20682-040E-02:20682-040E-02
- added J7: 1-84953-4, 1-84953-4:TE_1-84953-4, symbol 1-84953-4:1-84953-4
- added R203: 1.5k, Resistor_SMD:R_0402_1005Metric, symbol Device:R
- renumbered C83 to C430, C85 to C431, C91 to C432, C92 to C433, C87 to C434, C89 to C435, C95 to C436, C109 to C437, C110 to C438, C111 to C439, C96 to C440, C511 to C441, C391 to C442, C512 to C443, C103 to C444, C392 to C445, C104 to C446, C393 to C447, C105 to C448, C417 to C449, C394 to C450, C106 to C451, C402 to C452, C403 to C453, C404 to C454, C399 to C455, C400 to C456, C401 to C457, C488 to C458, C487 to C459, C490 to C460, C489 to C461, C491 to C462, C452 to C463, C453 to C464, C464 to C465, C463 to C466, C447 to C467, C448 to C468, C478 to C469, C450 to C470, C451 to C471, C479 to C472, C472 to C473, C480 to C474, C471 to C475, C481 to C476, C470 to C477, C460 to C478, C482 to C479, C459 to C480, C469 to C481, C483 to C482, C468 to C483, C449 to C484, C461 to C485, C484 to C486, C462 to C487, C485 to C488, C84 to C489, C473 to C490, C486 to C491, C86 to C492, C474 to C493, C475 to C494, C93 to C495, C476 to C496, C94 to C497, C477 to C498, C88 to C499, C90 to C500, C97 to C501, C98 to C502, C219 to C503, C415 to C504, C184 to C505, C185 to C506, C458 to C507, C418 to C508, C457 to C509, C456 to C510, C416 to C511, C208 to C512, C209 to C513, C210 to C514, C211 to C515, C492 to C516, C494 to C517, C496 to C519, C495 to C520, C493 to C521, C531 to C526, C532 to C527, C527 to C528, C528 to C529, C526 to C530, C428 to C531, C429 to C532, C430 to C533, C439 to C534, C440 to C535, C441 to C536, C513 to C537, C514 to C538, D3 to D10, D4 to D11, D16 to D12, D17 to D13, D13 to D14, D14 to D15, D7 to D6, D8 to D7, D6 to D8, D5 to D9, IC3 to IC2, IC2 to IC3, J7 to J10, J9 to J11, J10 to J12, J14 to J13, J11 to J18, J12 to J2, J2 to J5, J8 to J6, J13 to J8, J6 to J9, R57 to R143, R58 to R144, R184 to R145, R69 to R146, R63 to R147, R65 to R148, R61 to R149, R67 to R150, R77 to R151, R78 to R152, R72 to R153, R79 to R154, R71 to R155, R216 to R156, R218 to R157, R215 to R158, R217 to R159, R219 to R160, R202 to R161, R201 to R162, R200 to R163, R193 to R164, R195 to R165, R197 to R166, R196 to R167, R198 to R168, R199 to R169, R203 to R170, R204 to R171, R194 to R172, R59 to R173, R60 to R174, R70 to R175, R64 to R176, R66 to R177, R62 to R178, R68 to R179, R101 to R180, R117 to R181, R205 to R182, R115 to R183, R112 to R184, R113 to R185, R116 to R186, R208 to R187, R207 to R188, R206 to R189, R209 to R190, R210 to R191, R231 to R192, R234 to R193, R242 to R194, R243 to R195, R232 to R196, R233 to R197, R245 to R198, R244 to R199, R236 to R200, R237 to R201, R235 to R202, R179 to R204, R178 to R205, R177 to R206, R176 to R207, R175 to R208, R172 to R209, R171 to R210, R170 to R211, U16 to U39, U19 to U40, U26 to U41, U60 to U42, U59 to U43, U25 to U44, U58 to U45, U42 to U46, U46 to U47, U61 to U48, U17 to U49, U21 to U50, U45 to U51, U62 to U52, U43 to U53, U53 to U55, U52 to U56, U55 to U57, U44 to U58, U57 to U59, U56 to U60, U51 to U61, U74 to U62, U79 to U63, U80 to U64, U76 to U65, U75 to U66, U66 to U67, U65 to U68, U64 to U69, U63 to U70, Y4 to Y3, Y3 to Y4
Connections:
- net EDP_TX0_AUX_N: now also J20.16; no longer J15.16
- net EDP_TX0_AUX_P: now also J20.15; no longer J15.15
- net EDP_TX0_BL_EN: now also FPC1.5; no longer J15.32
- net EDP_TX0_BL_PWM: now also FPC1.6; no longer J15.33
- net EDP_TX0_HDP: now also J20.27; no longer J15.27
- net GND: now also C539.2, C541.1, C543.1, C544.1, C545.1, FPC1.3, FPC1.4, FPC1.7, FPC1.8, J16.26, J16.P1, J16.P2, J17.P1, J17.P2, J19.6, J19.S1 (SHIELD), J19.S2 (SHIELD); no longer J15.11, J15.14, J15.17, J15.2, J15.23, J15.24, J15.25, J15.26, J15.28, J15.29, J15.30, J15.31, J15.5, J15.8, J15.S1 (SHIELD), J15.S2 (SHIELD), J15.S3 (SHIELD), J15.S4 (SHIELD)
- net HDMI0_TX0N_PORT/eDP0_TX_D0N: now also J20.12; no longer J15.12
- net HDMI0_TX0P_PORT/eDP0_TX_D0P: now also J20.13; no longer J15.13
- net HDMI0_TX1N_PORT/eDP0_TX_D1N: now also J20.9; no longer J15.9
- net HDMI0_TX1P_PORT/eDP0_TX_D1P: now also J20.10; no longer J15.10
- net HDMI0_TX2N_PORT/eDP0_TX_D2N: now also J20.6; no longer J15.6
- net HDMI0_TX2P_PORT/eDP0_TX_D2P: now also J20.7; no longer J15.7
- net HDMI0_TX3N_PORT/eDP0_TX_D3N: now also J20.3; no longer J15.3
- net HDMI0_TX3P_PORT/eDP0_TX_D3P: now also J20.4; no longer J15.4
- net NRST_7: now also J19.5
- net VCC_12V_EDP: now also C544.2, C545.2, FPC1.1, FPC1.2; no longer J15.36, J15.37, J15.38, J15.39
- net VCC_3V3_ALW: now also C539.1, J19.1
- net VCC_3V3_SYS: now also C541.2, C543.2, J20.18, J20.19, J20.20, J20.21; no longer J15.18, J15.19, J15.20, J15.21
- new net: J16.25, R203.1
- new net: J14.S1 (SHIELD), J14.S2 (SHIELD)
- new net: J15.S1 (SHIELD), J15.S2 (SHIELD), J15.S3 (SHIELD), J15.S4 (SHIELD)
- new net: J20.11, J20.14, J20.17, J20.2, J20.23, J20.24, J20.25, J20.26, J20.5, J20.8, J20.S1 (SHIELD), J20.S10 (SHIELD), J20.S11 (SHIELD), J20.S12 (SHIELD), J20.S13 (SHIELD), J20.S14 (SHIELD), J20.S15 (SHIELD), J20.S16 (SHIELD), J20.S17 (SHIELD), J20.S18 (SHIELD), J20.S19 (SHIELD), J20.S2 (SHIELD), J20.S20 (SHIELD), J20.S21 (SHIELD), J20.S22 (SHIELD), J20.S3 (SHIELD), J20.S4 (SHIELD), J20.S5 (SHIELD), J20.S6 (SHIELD), J20.S7 (SHIELD), J20.S8 (SHIELD), J20.S9 (SHIELD)
- new net: J7.S1 (SHIELD), J7.S2 (SHIELD)
- new net BACKLIGHT_DN: J17.3, J17.4
- new net BACKLIGHT_DP: J17.1, J17.2
- new net CAPS_P: R203.2
- new net KSI0: J16.1
- new net KSI1: J16.2
- new net KSI2: J16.3
- new net KSI3: J16.4
- new net KSI4: J16.5
- new net KSI5: J16.6
- new net KSI6: J16.7
- new net KSI7: J16.8
- new net KSO0: J16.9
- new net KSO1: J16.10
- new net KSO10: J16.19
- new net KSO11: J16.20
- new net KSO12: J16.21
- new net KSO13: J16.22
- new net KSO14: J16.23
- new net KSO15: J16.24
- new net KSO2: J16.11
- new net KSO3: J16.12
- new net KSO4: J16.13
- new net KSO5: J16.14
- new net KSO6: J16.15
- new net KSO7: J16.16
- new net KSO8: J16.17
- new net KSO9: J16.18
- new net SWCLK_49: J19.3
- new net SWDIO_46: J19.2
- new net SWO_14: J19.4
- no-connect marks 153 -> 163
Other:
- note added: "40-PIN eDP CONNECTOR"
- note added: "6-PIN BACKLIGHT CONNECTOR"
- note added: "AUO B160ZAN01.U DISPLAY"
- note added: "BACKLIGHT"
- note added: "MATRIX"
- note removed: "AUO B173ZAN03.3"
- note removed: "ROUTE TO EC IF IT NEEDS TO RESET THE USB CONTROLLER"
