File: barebones_io.kicad_sch (KiCad schematic)
At the start: 252 parts, among them IC1 W25Q80DVSSIG, IC2 FUSB302BMPX, IC3 W25Q80DVSSIG, IC4 FUSB302BMPX, J1 12401610E4_2A, J10 54-00007, J11 54-00007, J12 10067847-001RLF, J13 SM02B-GHS-TB_LF__SN_, J14 SM05B-SRSS-TB_LF__SN_, J15 20455-040E-76, J16 524352671, J17 522070485, J18 G45AA1912100B1EU, J19 SM06B-SRSS-TB_LF__SN_, J2 1-2199119-5, J20 20682-040E-02, J3 1-2199119-5, J4 21992304, J5 12401610E4_2A, J6 SJ2-35894B-SMT-TR, J7 1-84953-4, J8 SM02B-GHS-TB_LF__SN_, J9 1040310811, U39 TPS65987DDHRSHR, U40 TXS0104EYZTR, U41 TPD4E004DRYR, U42 PCA9306DCTR, U43 9FGV0641AKILFT, U44 TPD4E05U06DQAR, U45 GL3523-ONY30, U46 TXS0104EYZTR, U47 TPS2553DBVR, U48 PI3DPX1207Q3ZHEX, U49 TPS65987DDHRSHR, U50 TXS0104EYZTR, U51 PCA9306DCTR, U52 OV9734-H16A, U53 TPS2553DBVR, U54 TPD4E004DRYR, U55 PI6C557-05BLEX, U56 PI6C557-05LEX, U57 PI6C557-03ALEX, U58 TPS2553DBVR, U59 TPD4E004DRYR, U60 TPD4E004DRYR, U61 PCA9306DCTR, U62 2N7002KW, U63 2N7002KW, U64 2N7002KW, U65 2N7002KW, U66 2N7002KW, U67 2N7002KW, U68 2N7002KW, U69 2N7002KW, U70 2N7002KW, Y3 C2E-25.000-10-1530-X-R, Y4 C2E-25.000-10-1530-X-R

Commit message: added the PCF85063ATL/1,118 CMOS Real-Time Clock
Parts:
- added J21: SM02B-GHS-TB_LF__SN_, barebones:JST_SM02B-GHS-TB_LF__SN_, symbol SM02B-GHS-TB_LF__SN_:SM02B-GHS-TB_LF__SN_
- added R214, R215: 100k, Resistor_SMD:R_0402_1005Metric, symbol Device:R
Connections:
- net GND: now also J21.2
- net NRST_7: now also J19.4; no longer J19.5
- net SWO_14: now also J19.5; no longer J19.4
- net USB_1_SBU1: now also R214.1
- net USB_2_SBU1: now also R215.1
- new net USB_1_SBU1_DC: R214.2
- new net USB_2_SBU1_DC: R215.2
- new net V_BAT_CMOS: J21.1
Other:
- note added: "CMOS BATTERY"
- moved on the sheet: D6, D7, D8, D9

Commit message: updated the Fuel Guage/BMS module for the 4S battery usage
Parts:
- removed J21: SM02B-GHS-TB_LF__SN_, barebones:JST_SM02B-GHS-TB_LF__SN_, symbol SM02B-GHS-TB_LF__SN_:SM02B-GHS-TB_LF__SN_
Connections:
- net JACK_RING_1 renamed HP_JACK_RING_1
- net JACK_RING_2 renamed HP_JACK_RING_2
- net JACK_SLEEVE renamed HP_JACK_SLEEVE
- net JACK_SWITCH renamed HP_JACK_SWITCH
- net JACK_TIP renamed HP_JACK_TIP
Other:
- note removed: "CMOS BATTERY"
- moved on the sheet: J6
