File: barebones_mems.kicad_sch (KiCad schematic)
At the start: 4 parts, among them U12 MT53E1G32D2FW-046_AUT_B, U13 MT53E1G32D2FW-046_AUT_B, U14 MT53E1G32D2FW-046_AUT_B, U15 MT53E1G32D2FW-046_AUT_B

Commit message: routed the two 64Gb LPDDR4x RAM chips
Parts:
- removed U12, U13, U14, U15: MT53E1G32D2FW-046_AUT_B, barebones:BGA200C65X80P22X12_1500X1000X114N, symbol MT53E1G32D2FW-046_AUT_B:MT53E1G32D2FW-046_AUT_B
- added C341, C382: 4.7uF, Capacitor_SMD:C_0201_0603Metric, symbol Device:C
- added C342, C373, C374, C379, C380, C385, C387, C388, C389, C390: 100nF, Capacitor_SMD:C_0201_0603Metric, symbol Device:C
- added C375, C381: 22uF, Capacitor_SMD:C_0201_0603Metric, symbol Device:C
- added C376, C377, C383, C384: 10uF, Capacitor_SMD:C_0201_0603Metric, symbol Device:C
- added C378, C386: 1uF, Capacitor_SMD:C_0201_0603Metric, symbol Device:C
- added R160, R161, R81, R82: 200R, Resistor_SMD:R_0402_1005Metric, symbol Device:R
- added U12, U13: K4UCE3Q4AA-MGCL, barebones:BGA-200_L15.0-W10.0_K4F8E304HB-MGCJ, symbol K4UCE3Q4AA-MGCL:K4UCE3Q4AA-MGCL
Connections:
- new net: R82.1, U12.A8 (ZQ1)
- new net: R81.1, U12.A5 (ZQ0)
- new net: R161.1, U13.A8 (ZQ1)
- new net: R160.1, U13.A5 (ZQ0)
- new net DDR_CH0_A0_A: U12.H2 (CA0_a)
- new net DDR_CH0_A0_B: U12.R2 (CA0_b)
- new net DDR_CH0_A1_A: U12.J2 (CA1_a)
- new net DDR_CH0_A1_B: U12.P2 (CA1_b)
- new net DDR_CH0_A2_A: U12.H9 (CA2_a)
- new net DDR_CH0_A2_B: U12.R9 (CA2_b)
- new net DDR_CH0_A3_A: U12.H10 (CA3_a)
- new net DDR_CH0_A3_B: U12.R10 (CA3_b)
- new net DDR_CH0_A4_A: U12.H11 (CA4_a)
- new net DDR_CH0_A4_B: U12.R11 (CA4_b)
- new net DDR_CH0_A5_A: U12.J11 (CA5_a)
- new net DDR_CH0_A5_B: U12.P11 (CA5_b)
- new net DDR_CH0_CKB_A: U12.J9 (CK_c_a)
- new net DDR_CH0_CKB_B: U12.P9 (CK_c_b)
- new net DDR_CH0_CK_A: U12.J8 (CK_t_a)
- new net DDR_CH0_CK_B: U12.P8 (CK_t_b)
- new net DDR_CH0_DM0_A: U12.C3 (DMI0_a)
- new net DDR_CH0_DM0_B: U12.Y3 (DMI0_b)
- new net DDR_CH0_DM1_A: U12.C10 (DMI1_a)
- new net DDR_CH0_DM1_B: U12.Y10 (DMI1_b)
- new net DDR_CH0_DQ0_A: U12.B2 (DQ0_a)
- new net DDR_CH0_DQ0_B: U12.AA2 (DQ0_b)
- new net DDR_CH0_DQ10_A: U12.E11 (DQ10_a)
- new net DDR_CH0_DQ10_B: U12.V11 (DQ10_b)
- new net DDR_CH0_DQ11_A: U12.F11 (DQ11_a)
- new net DDR_CH0_DQ11_B: U12.U11 (DQ11_b)
- new net DDR_CH0_DQ12_A: U12.F9 (DQ12_a)
- new net DDR_CH0_DQ12_B: U12.U9 (DQ12_b)
- new net DDR_CH0_DQ13_A: U12.E9 (DQ13_a)
- new net DDR_CH0_DQ13_B: U12.V9 (DQ13_b)
- new net DDR_CH0_DQ14_A: U12.C9 (DQ14_a)
- new net DDR_CH0_DQ14_B: U12.Y9 (DQ14_b)
- new net DDR_CH0_DQ15_A: U12.B9 (DQ15_a)
- new net DDR_CH0_DQ15_B: U12.AA9 (DQ15_b)
- new net DDR_CH0_DQ1_A: U12.C2 (DQ1_a)
- new net DDR_CH0_DQ1_B: U12.Y2 (DQ1_b)
- new net DDR_CH0_DQ2_A: U12.E2 (DQ2_a)
- new net DDR_CH0_DQ2_B: U12.V2 (DQ2_b)
- new net DDR_CH0_DQ3_A: U12.F2 (DQ3_a)
- new net DDR_CH0_DQ3_B: U12.U2 (DQ3_b)
- new net DDR_CH0_DQ4_A: U12.F4 (DQ4_a)
- new net DDR_CH0_DQ4_B: U12.U4 (DQ4_b)
- new net DDR_CH0_DQ5_A: U12.E4 (DQ5_a)
- new net DDR_CH0_DQ5_B: U12.V4 (DQ5_b)
- new net DDR_CH0_DQ6_A: U12.C4 (DQ6_a)
- new net DDR_CH0_DQ6_B: U12.Y4 (DQ6_b)
- new net DDR_CH0_DQ7_A: U12.B4 (DQ7_a)
- new net DDR_CH0_DQ7_B: U12.AA4 (DQ7_b)
- new net DDR_CH0_DQ8_A: U12.B11 (DQ8_a)
- new net DDR_CH0_DQ8_B: U12.AA11 (DQ8_b)
- new net DDR_CH0_DQ9_A: U12.C11 (DQ9_a)
- new net DDR_CH0_DQ9_B: U12.Y11 (DQ9_b)
- new net DDR_CH0_DQS0N_A: U12.E3 (DQS0_c_a)
- new net DDR_CH0_DQS0N_B: U12.V3 (DQS0_c_b)
- new net DDR_CH0_DQS0P_A: U12.D3 (DQS0_t_a)
- new net DDR_CH0_DQS0P_B: U12.W3 (DQS0_t_b)
- new net DDR_CH0_DQS1N_A: U12.E10 (DQS1_c_a)
- new net DDR_CH0_DQS1N_B: U12.V10 (DQS1_c_b)
- new net DDR_CH0_DQS1P_A: U12.D10 (DQS1_t_a)
- new net DDR_CH0_DQS1P_B: U12.W10 (DQS1_t_b)
- new net DDR_CH0_LP4/4X_CKE0/LP5_CS0_A: U12.J4 (CKE0_a)
- new net DDR_CH0_LP4/4X_CKE0/LP5_CS0_B: U12.P4 (CKE0_b)
- new net DDR_CH0_LP4/4X_CKE1/LP5_CS1_A: U12.J5 (CKE1_a)
- new net DDR_CH0_LP4/4X_CKE1/LP5_CS1_B: U12.P5 (CKE1_b)
- new net DDR_CH0_LP4/4X_CS0_A: U12.H4 (CS0_a)
- new net DDR_CH0_LP4/4X_CS0_B: U12.R4 (CS0_b)
- new net DDR_CH0_LP4/4X_CS1_A: U12.H3 (CS1_a)
- new net DDR_CH0_LP4/4X_CS1_B: U12.R3 (CS1_b)
- new net DDR_CH1_A0_C: U13.H2 (CA0_a)
- new net DDR_CH1_A0_D: U13.R2 (CA0_b)
- new net DDR_CH1_A1_C: U13.J2 (CA1_a)
- new net DDR_CH1_A1_D: U13.P2 (CA1_b)
- new net DDR_CH1_A2_C: U13.H9 (CA2_a)
- new net DDR_CH1_A2_D: U13.R9 (CA2_b)
- new net DDR_CH1_A3_C: U13.H10 (CA3_a)
- new net DDR_CH1_A3_D: U13.R10 (CA3_b)
- new net DDR_CH1_A4_C: U13.H11 (CA4_a)
- new net DDR_CH1_A4_D: U13.R11 (CA4_b)
- new net DDR_CH1_A5_C: U13.J11 (CA5_a)
- new net DDR_CH1_A5_D: U13.P11 (CA5_b)
- new net DDR_CH1_CKB_C: U13.J9 (CK_c_a)
- new net DDR_CH1_CKB_D: U13.P9 (CK_c_b)
- new net DDR_CH1_CK_C: U13.J8 (CK_t_a)
- new net DDR_CH1_CK_D: U13.P8 (CK_t_b)
- new net DDR_CH1_DM0_C: U13.C3 (DMI0_a)
- new net DDR_CH1_DM0_D: U13.Y3 (DMI0_b)
- new net DDR_CH1_DM1_C: U13.C10 (DMI1_a)
- new net DDR_CH1_DM1_D: U13.Y10 (DMI1_b)
- new net DDR_CH1_DQ0_C: U13.B2 (DQ0_a)
- new net DDR_CH1_DQ0_D: U13.AA2 (DQ0_b)
- new net DDR_CH1_DQ10_C: U13.E11 (DQ10_a)
- new net DDR_CH1_DQ10_D: U13.V11 (DQ10_b)
- new net DDR_CH1_DQ11_C: U13.F11 (DQ11_a)
- new net DDR_CH1_DQ11_D: U13.U11 (DQ11_b)
- new net DDR_CH1_DQ12_C: U13.F9 (DQ12_a)
- new net DDR_CH1_DQ12_D: U13.U9 (DQ12_b)
- new net DDR_CH1_DQ13_C: U13.E9 (DQ13_a)
- new net DDR_CH1_DQ13_D: U13.V9 (DQ13_b)
- new net DDR_CH1_DQ14_C: U13.C9 (DQ14_a)
- new net DDR_CH1_DQ14_D: U13.Y9 (DQ14_b)
- new net DDR_CH1_DQ15_C: U13.B9 (DQ15_a)
- new net DDR_CH1_DQ15_D: U13.AA9 (DQ15_b)
- new net DDR_CH1_DQ1_C: U13.C2 (DQ1_a)
- new net DDR_CH1_DQ1_D: U13.Y2 (DQ1_b)
- new net DDR_CH1_DQ2_C: U13.E2 (DQ2_a)
- new net DDR_CH1_DQ2_D: U13.V2 (DQ2_b)
- new net DDR_CH1_DQ3_C: U13.F2 (DQ3_a)
- new net DDR_CH1_DQ3_D: U13.U2 (DQ3_b)
- new net DDR_CH1_DQ4_C: U13.F4 (DQ4_a)
- new net DDR_CH1_DQ4_D: U13.U4 (DQ4_b)
- new net DDR_CH1_DQ5_C: U13.E4 (DQ5_a)
- new net DDR_CH1_DQ5_D: U13.V4 (DQ5_b)
- new net DDR_CH1_DQ6_C: U13.C4 (DQ6_a)
- new net DDR_CH1_DQ6_D: U13.Y4 (DQ6_b)
- new net DDR_CH1_DQ7_C: U13.B4 (DQ7_a)
- new net DDR_CH1_DQ7_D: U13.AA4 (DQ7_b)
- new net DDR_CH1_DQ8_C: U13.B11 (DQ8_a)
- new net DDR_CH1_DQ8_D: U13.AA11 (DQ8_b)
- new net DDR_CH1_DQ9_C: U13.C11 (DQ9_a)
- new net DDR_CH1_DQ9_D: U13.Y11 (DQ9_b)
- new net DDR_CH1_DQS0N_C: U13.E3 (DQS0_c_a)
- new net DDR_CH1_DQS0N_D: U13.V3 (DQS0_c_b)
- new net DDR_CH1_DQS0P_C: U13.D3 (DQS0_t_a)
- new net DDR_CH1_DQS0P_D: U13.W3 (DQS0_t_b)
- new net DDR_CH1_DQS1N_C: U13.E10 (DQS1_c_a)
- new net DDR_CH1_DQS1N_D: U13.V10 (DQS1_c_b)
- new net DDR_CH1_DQS1P_C: U13.D10 (DQS1_t_a)
- new net DDR_CH1_DQS1P_D: U13.W10 (DQS1_t_b)
- new net DDR_CH1_LP4/4X_CKE0/LP5_CS0_C: U13.J4 (CKE0_a)
- new net DDR_CH1_LP4/4X_CKE0/LP5_CS0_D: U13.P4 (CKE0_b)
- new net DDR_CH1_LP4/4X_CKE1/LP5_CS1_C: U13.J5 (CKE1_a)
- new net DDR_CH1_LP4/4X_CKE1/LP5_CS1_D: U13.P5 (CKE1_b)
- new net DDR_CH1_LP4/4X_CS0_C: U13.H4 (CS0_a)
- new net DDR_CH1_LP4/4X_CS0_D: U13.R4 (CS0_b)
- new net DDR_CH1_LP4/4X_CS1_C: U13.H3 (CS1_a)
- new net DDR_CH1_LP4/4X_CS1_D: U13.R3 (CS1_b)
- new net DDR_RESET: U12.T11 (RESET_n), U13.T11 (RESET_n)
- new net GND: C341.2, C342.2, C373.2, C374.2, C375.2, C376.2, C377.2, C378.2, C379.2, C380.2, C381.2, C382.2, C383.2, C384.2, C385.2, C386.2, C387.2, C388.2, C389.2, C390.2, U12.A10 (VSS), U12.A3 (VSS), U12.AB10 (VSS), U12.AB3 (VSS), U12.AB5 (VSS), U12.AB8 (VSS), U12.C1 (VSS), U12.C12 (VSS), U12.C5 (VSS), U12.C8 (VSS), U12.D11 (VSS), U12.D2 (VSS), U12.D4 (VSS), U12.D9 (VSS), U12.E1 (VSS), U12.E12 (VSS), U12.E5 (VSS), U12.E8 (VSS), U12.G1 (VSS), U12.G10 (VSS), U12.G12 (VSS), U12.G2 (ODT_CA_a1)/2)), U12.G3 (VSS), U12.G5 (VSS), U12.G8 (VSS), U12.J1 (VSS), U12.J10 (VSS), U12.J12 (VSS), U12.J3 (VSS), U12.K11 (VSS), U12.K2 (VSS), U12.K4 (VSS), U12.K9 (VSS), U12.N11 (VSS), U12.N2 (VSS), U12.N4 (VSS), U12.N9 (VSS), U12.P1 (VSS), U12.P10 (VSS), U12.P12 (VSS), U12.P3 (VSS), U12.T1 (VSS), U12.T10 (VSS), U12.T12 (VSS), U12.T2 (ODT_CA_b1)/2)), U12.T3 (VSS), U12.T5 (VSS), U12.T8 (VSS), U12.V1 (VSS), U12.V12 (VSS), U12.V5 (VSS), U12.V8 (VSS), U12.W11 (VSS), U12.W2 (VSS), U12.W4 (VSS), U12.W9 (VSS), U12.Y1 (VSS), U12.Y12 (VSS), U12.Y5 (VSS), U12.Y8 (VSS), U13.A10 (VSS), U13.A3 (VSS), U13.AB10 (VSS), U13.AB3 (VSS), U13.AB5 (VSS), U13.AB8 (VSS), U13.C1 (VSS), U13.C12 (VSS), U13.C5 (VSS), U13.C8 (VSS), U13.D11 (VSS), U13.D2 (VSS), U13.D4 (VSS), U13.D9 (VSS), U13.E1 (VSS), U13.E12 (VSS), U13.E5 (VSS), U13.E8 (VSS), U13.G1 (VSS), U13.G10 (VSS), U13.G12 (VSS), U13.G2 (ODT_CA_a1)/2)), U13.G3 (VSS), U13.G5 (VSS), U13.G8 (VSS), U13.J1 (VSS), U13.J10 (VSS), U13.J12 (VSS), U13.J3 (VSS), U13.K11 (VSS), U13.K2 (VSS), U13.K4 (VSS), U13.K9 (VSS), U13.N11 (VSS), U13.N2 (VSS), U13.N4 (VSS), U13.N9 (VSS), U13.P1 (VSS), U13.P10 (VSS), U13.P12 (VSS), U13.P3 (VSS), U13.T1 (VSS), U13.T10 (VSS), U13.T12 (VSS), U13.T2 (ODT_CA_b1)/2)), U13.T3 (VSS), U13.T5 (VSS), U13.T8 (VSS), U13.V1 (VSS), U13.V12 (VSS), U13.V5 (VSS), U13.V8 (VSS), U13.W11 (VSS), U13.W2 (VSS), U13.W4 (VSS), U13.W9 (VSS), U13.Y1 (VSS), U13.Y12 (VSS), U13.Y5 (VSS), U13.Y8 (VSS)
- new net VCC_1V8_S3: C341.1, C342.1, C373.1, C374.1, C382.1, C385.1, C387.1, C390.1, U12.F1 (VDD1), U12.F12 (VDD1), U12.G4 (VDD1), U12.G9 (VDD1), U12.T4 (VDD1), U12.T9 (VDD1), U12.U1 (VDD1), U12.U12 (VDD1), U13.F1 (VDD1), U13.F12 (VDD1), U13.G4 (VDD1), U13.G9 (VDD1), U13.T4 (VDD1), U13.T9 (VDD1), U13.U1 (VDD1), U13.U12 (VDD1)
- new net VDDQ_DDR_S0: C375.1, C376.1, C377.1, C378.1, C379.1, C380.1, C381.1, C383.1, C384.1, C386.1, C388.1, C389.1, U12.AA10 (VDDQ), U12.AA3 (VDDQ), U12.AA5 (VDDQ), U12.AA8 (VDDQ), U12.B10 (VDDQ), U12.B3 (VDDQ), U12.B5 (VDDQ), U12.B8 (VDDQ), U12.D1 (VDDQ), U12.D12 (VDDQ), U12.D5 (VDDQ), U12.D8 (VDDQ), U12.F10 (VDDQ), U12.F3 (VDDQ), U12.U10 (VDDQ), U12.U3 (VDDQ), U12.W1 (VDDQ), U12.W12 (VDDQ), U12.W5 (VDDQ), U12.W8 (VDDQ), U13.AA10 (VDDQ), U13.AA3 (VDDQ), U13.AA5 (VDDQ), U13.AA8 (VDDQ), U13.B10 (VDDQ), U13.B3 (VDDQ), U13.B5 (VDDQ), U13.B8 (VDDQ), U13.D1 (VDDQ), U13.D12 (VDDQ), U13.D5 (VDDQ), U13.D8 (VDDQ), U13.F10 (VDDQ), U13.F3 (VDDQ), U13.U10 (VDDQ), U13.U3 (VDDQ), U13.W1 (VDDQ), U13.W12 (VDDQ), U13.W5 (VDDQ), U13.W8 (VDDQ)
- new net VDD_DDR_S0: R160.2, R161.2, R81.2, R82.2, U12.A4 (VDD2), U12.A9 (VDD2), U12.AB4 (VDD2), U12.AB9 (VDD2), U12.F5 (VDD2), U12.F8 (VDD2), U12.H1 (VDD2), U12.H12 (VDD2), U12.H5 (VDD2), U12.H8 (VDD2), U12.K1 (VDD2), U12.K10 (VDD2), U12.K12 (VDD2), U12.K3 (VDD2), U12.N1 (VDD2), U12.N10 (VDD2), U12.N12 (VDD2), U12.N3 (VDD2), U12.R1 (VDD2), U12.R12 (VDD2), U12.R5 (VDD2), U12.R8 (VDD2), U12.U5 (VDD2), U12.U8 (VDD2), U13.A4 (VDD2), U13.A9 (VDD2), U13.AB4 (VDD2), U13.AB9 (VDD2), U13.F5 (VDD2), U13.F8 (VDD2), U13.H1 (VDD2), U13.H12 (VDD2), U13.H5 (VDD2), U13.H8 (VDD2), U13.K1 (VDD2), U13.K10 (VDD2), U13.K12 (VDD2), U13.K3 (VDD2), U13.N1 (VDD2), U13.N10 (VDD2), U13.N12 (VDD2), U13.N3 (VDD2), U13.R1 (VDD2), U13.R12 (VDD2), U13.R5 (VDD2), U13.R8 (VDD2), U13.U5 (VDD2), U13.U8 (VDD2)
- no-connect marks 0 -> 34

Commit message: added the display connector and its 12V power supply
Parts:
- renumbered C341 to C374, C342 to C375, C373 to C376, C374 to C377, C382 to C378, C385 to C379, C387 to C380, C390 to C381, C375 to C382, C376 to C383, C377 to C384, C378 to C385, C379 to C386, C380 to C387, C381 to C388, C383 to C389, C384 to C390, C386 to C391, C388 to C392, C389 to C393, R81 to R122, R82 to R123, R160 to R124, R161 to R125, U12 to U32, U13 to U33
