File: barebones.kicad_pcb (KiCad board)
At the start: 2 copper layers, 350 x 250 mm, 440 parts, among them IC1 W25Q80DVSSIG, IC2 W25Q80DVSSIG, J1 12401610E4_2A, J10 G45AA1912100B1EU, J13 SM02B-GHS-TB_LF__SN_, J14 SM02B-GHS-TB_LF__SN_, J2 12401610E4_2A, J3 1-2199119-5, J4 21992304, J5 G45AA1912100B1EU, J6 1040310811, J7 54-00007, J8 SJ2-35894B-SMT-TR, J9 54-00007, Q1 STL40DN3LLH5, Q2 STL40DN3LLH5, Q3 STL40DN3LLH5, U1 RK3588, U10 ES8316, U11 BQ25731RSNR, U12 MT53E1G32D2FW-046_AUT_B, U13 MT53E1G32D2FW-046_AUT_B, U14 MT53E1G32D2FW-046_AUT_B, U15 MT53E1G32D2FW-046_AUT_B, U16 TPS65987DDHRSHR, U17 TPS65987DDHRSHR, U19 TXS0104EYZTR, U2 TPS54628DDAR, U21 TXS0104EYZTR, U25 TPD4E05U06DQAR, U26 TPD4E004DRYR, U3 TPS54628DDAR, U31 STM32H743VIH6, U35 2N7002KW, U36 2N7002KW, U37 LP5912-1.8DRVT, U38 TPA2012D2RTJT, U39 TPS54628DDAR, U4 TPS54628DDAR, U40 TPS54628DDAR, U42 TXS0104EYZTR, U43 TPS2553DBVR, U44 TPS2553DBVR, U45 PCA9306DCTR, U46 TPS2553DBVR, U47 TPS2553DBVR, U48 PCA9306DCTR, U5 TPS259474ARPWR, U6 TPS259474ARPWR, U7 TPS2121RUXR, U8 RK806-1_C5156483, U9 BQ28Z610DRZR

Commit message: routed the two 64Gb LPDDR4x RAM chips
Parts:
- removed C128, C143: 1uF, Capacitor_SMD:C_0603_1608Metric
- removed C132: 2.2uF, Capacitor_SMD:C_0603_1608Metric
- removed U13, U14, U15: MT53E1G32D2FW-046_AUT_B, barebones:BGA200C65X80P22X12_1500X1000X114N
- added C222: 0.1uF, Capacitor_SMD:C_0201_0603Metric, F.Cu at (424.7, 180.4)
- added C223: 0.1uF, Capacitor_SMD:C_0603_1608Metric, F.Cu at (460.6, 135.3)
- added C224: 100nF, Capacitor_SMD:C_0201_0603Metric, F.Cu at (446.8, 164.5)
- added C225: 1uF, Capacitor_SMD:C_0201_0603Metric, F.Cu at (446.8, 166.2)
- added C226: 4.7uF, Capacitor_SMD:C_0201_0603Metric, F.Cu at (446.8, 168.0)
- added C227: 10uF, Capacitor_SMD:C_0201_0603Metric, F.Cu at (446.8, 169.7)
- added C228: 10uF, Capacitor_SMD:C_0201_0603Metric, F.Cu at (446.8, 171.5)
- added C229: 10uF, Capacitor_SMD:C_0201_0603Metric, F.Cu at (446.8, 173.2)
- added C230: 10uF, Capacitor_SMD:C_0201_0603Metric, F.Cu at (446.8, 175.0)
- added C231: 22uF, Capacitor_SMD:C_0201_0603Metric, F.Cu at (446.8, 176.7)
- added C232: 1uF, Capacitor_SMD:C_0201_0603Metric, F.Cu at (446.8, 178.5)
- added C233: 1uF, Capacitor_SMD:C_0603_1608Metric, F.Cu at (425.5, 135.3)
- added C234: 47uF, Capacitor_SMD:C_0603_1608Metric, F.Cu at (425.5, 137.8)
- added C235: 1uF, Capacitor_SMD:C_0603_1608Metric, F.Cu at (425.5, 140.3)
- added C236: 22uF, Capacitor_SMD:C_0603_1608Metric, F.Cu at (425.5, 142.8)
- added C237: 22uF, Capacitor_SMD:C_0603_1608Metric, F.Cu at (425.5, 145.3)
- added C238: 1uF, Capacitor_SMD:C_0603_1608Metric, F.Cu at (425.5, 147.8)
- added C239: 1uF, Capacitor_SMD:C_0603_1608Metric, F.Cu at (425.5, 150.3)
- added C240: 22uF, Capacitor_SMD:C_0603_1608Metric, F.Cu at (425.5, 152.8)
- added C241: 22uF, Capacitor_SMD:C_0603_1608Metric, F.Cu at (425.5, 155.3)
- added C242: 1uF, Capacitor_SMD:C_0603_1608Metric, F.Cu at (425.5, 157.8)
- added C243: 10uF, Capacitor_SMD:C_0603_1608Metric, F.Cu at (425.5, 160.4)
- added C244: 100pF, Capacitor_SMD:C_0603_1608Metric, F.Cu at (429.5, 135.3)
- added C245: 47uF, Capacitor_SMD:C_0603_1608Metric, F.Cu at (429.5, 137.8)
- added C246: 47uF, Capacitor_SMD:C_0603_1608Metric, F.Cu at (429.5, 140.3)
- added C247: 10nF, Capacitor_SMD:C_0603_1608Metric, F.Cu at (429.5, 142.8)
- added C248: 0.1uF, Capacitor_SMD:C_0603_1608Metric, F.Cu at (429.5, 145.3)
- added C249: 1uF, Capacitor_SMD:C_0603_1608Metric, F.Cu at (429.5, 147.8)
- added C250: 0.1uF, Capacitor_SMD:C_0603_1608Metric, F.Cu at (429.5, 150.3)
- added C251: 47uF, Capacitor_SMD:C_0603_1608Metric, F.Cu at (429.5, 152.8)
- added C252: 47uF, Capacitor_SMD:C_0603_1608Metric, F.Cu at (429.5, 155.3)
- added C253: 0.1uF, Capacitor_SMD:C_0603_1608Metric, F.Cu at (429.5, 157.8)
- added C254: 10uF, Capacitor_SMD:C_0603_1608Metric, F.Cu at (429.5, 160.4)
- added C255: 100pF, Capacitor_SMD:C_0603_1608Metric, F.Cu at (433.5, 135.3)
- added C256: 1uF, Capacitor_SMD:C_0603_1608Metric, F.Cu at (433.5, 137.8)
- added C257: 22uF, Capacitor_SMD:C_0603_1608Metric, F.Cu at (433.5, 140.3)
- added C258: 22uF, Capacitor_SMD:C_0603_1608Metric, F.Cu at (433.5, 142.8)
- added C259: 22uF, Capacitor_SMD:C_0603_1608Metric, F.Cu at (433.5, 145.3)
- added C260: 22uF, Capacitor_SMD:C_0603_1608Metric, F.Cu at (433.5, 147.8)
- added C261: 22uF, Capacitor_SMD:C_0603_1608Metric, F.Cu at (433.5, 150.3)
- added C262: 22uF, Capacitor_SMD:C_0603_1608Metric, F.Cu at (433.5, 152.8)
- added C263: 22uF, Capacitor_SMD:C_0603_1608Metric, F.Cu at (433.5, 155.3)
- added C264: 22uF, Capacitor_SMD:C_0603_1608Metric, F.Cu at (433.5, 157.8)
- added C265: 1uF, Capacitor_SMD:C_0603_1608Metric, F.Cu at (433.5, 160.4)
- added C266: 22uF, Capacitor_SMD:C_0603_1608Metric, F.Cu at (437.5, 135.3)
- added C267: 22uF, Capacitor_SMD:C_0603_1608Metric, F.Cu at (437.5, 137.8)
- added C268: 22uF, Capacitor_SMD:C_0603_1608Metric, F.Cu at (437.5, 140.3)
- added C269: 22uF, Capacitor_SMD:C_0603_1608Metric, F.Cu at (437.5, 142.8)
- added C270: 22uF, Capacitor_SMD:C_0603_1608Metric, F.Cu at (437.5, 145.3)
- added C271: 22uF, Capacitor_SMD:C_0603_1608Metric, F.Cu at (437.5, 147.8)
- added C272: 22uF, Capacitor_SMD:C_0603_1608Metric, F.Cu at (437.5, 150.3)
- added C273: 1uF, Capacitor_SMD:C_0603_1608Metric, F.Cu at (437.5, 152.8)
- added C274: 22uF, Capacitor_SMD:C_0603_1608Metric, F.Cu at (437.5, 155.3)
- added C275: 22uF, Capacitor_SMD:C_0603_1608Metric, F.Cu at (437.5, 157.8)
- added C276: 22uF, Capacitor_SMD:C_0603_1608Metric, F.Cu at (437.5, 160.4)
- added C277: 22uF, Capacitor_SMD:C_0603_1608Metric, F.Cu at (441.5, 135.3)
- added C278: 22uF, Capacitor_SMD:C_0603_1608Metric, F.Cu at (441.5, 137.8)
- added C279: 22uF, Capacitor_SMD:C_0603_1608Metric, F.Cu at (441.5, 140.3)
- added C280: 100nF, Capacitor_SMD:C_0201_0603Metric, F.Cu at (446.8, 180.2)
- added C281: 1uF, Capacitor_SMD:C_0201_0603Metric, F.Cu at (446.8, 182.0)
- added C282: 10uF, Capacitor_SMD:C_0201_0603Metric, F.Cu at (449.2, 164.5)
- added C283: 10uF, Capacitor_SMD:C_0201_0603Metric, F.Cu at (449.2, 166.2)
- added C284: 10uF, Capacitor_SMD:C_0201_0603Metric, F.Cu at (449.2, 168.0)
- added C285: 10uF, Capacitor_SMD:C_0201_0603Metric, F.Cu at (449.2, 169.7)
- added C286: 10uF, Capacitor_SMD:C_0201_0603Metric, F.Cu at (449.2, 171.5)
- added C287: 10nF, Capacitor_SMD:C_0603_1608Metric, F.Cu at (441.5, 142.8)
- added C288: 100nF, Capacitor_SMD:C_0201_0603Metric, F.Cu at (449.2, 173.2)
- added C289: 100nF, Capacitor_SMD:C_0201_0603Metric, F.Cu at (449.2, 175.0)
- added C290: 4.7uF, Capacitor_SMD:C_0201_0603Metric, F.Cu at (449.2, 176.7)
- added C291: 4.7uF, Capacitor_SMD:C_0201_0603Metric, F.Cu at (449.2, 178.5)
- added C292: 10uF, Capacitor_SMD:C_0201_0603Metric, F.Cu at (449.2, 180.2)
- added C293: 10uF, Capacitor_SMD:C_0201_0603Metric, F.Cu at (449.2, 182.0)
- added C294: 10uF, Capacitor_SMD:C_0201_0603Metric, F.Cu at (451.7, 164.5)
- added C295: 22uF, Capacitor_SMD:C_0201_0603Metric, F.Cu at (451.7, 166.2)
- added C296: 1uF, Capacitor_SMD:C_0201_0603Metric, F.Cu at (451.7, 168.0)
- added C297: 1uF, Capacitor_SMD:C_0201_0603Metric, F.Cu at (451.7, 169.7)
- added C298: 100nF, Capacitor_SMD:C_0201_0603Metric, F.Cu at (451.7, 171.5)
- added C299: 10uF, Capacitor_SMD:C_0201_0603Metric, F.Cu at (451.7, 173.2)
- added C300: 10uF, Capacitor_SMD:C_0201_0603Metric, F.Cu at (451.7, 175.0)
- added C301: 10uF, Capacitor_SMD:C_0201_0603Metric, F.Cu at (451.7, 176.7)
- added C302: 10uF, Capacitor_SMD:C_0201_0603Metric, F.Cu at (451.7, 178.5)
- added C303: 22uF, Capacitor_SMD:C_0201_0603Metric, F.Cu at (451.7, 180.2)
- added C304: 1uF, Capacitor_SMD:C_0201_0603Metric, F.Cu at (451.7, 182.0)
- added C305: 100nF, Capacitor_SMD:C_0201_0603Metric, F.Cu at (454.1, 164.5)
- added C306: 100nF, Capacitor_SMD:C_0201_0603Metric, F.Cu at (454.1, 166.2)
- added C307: 1uF, Capacitor_SMD:C_0201_0603Metric, F.Cu at (454.1, 168.0)
- added C308: 1uF, Capacitor_SMD:C_0201_0603Metric, F.Cu at (454.1, 169.7)
- added C309: 4.7uF, Capacitor_SMD:C_0201_0603Metric, F.Cu at (454.1, 171.5)
- added C310: 10uF, Capacitor_SMD:C_0201_0603Metric, F.Cu at (454.1, 173.2)
- added C311: 10uF, Capacitor_SMD:C_0201_0603Metric, F.Cu at (454.1, 175.0)
- added C312: 10uF, Capacitor_SMD:C_0201_0603Metric, F.Cu at (454.1, 176.7)
- added C313: 10uF, Capacitor_SMD:C_0201_0603Metric, F.Cu at (454.1, 178.5)
- added C314: 22uF, Capacitor_SMD:C_0201_0603Metric, F.Cu at (454.1, 180.2)
- added C315: 1uF, Capacitor_SMD:C_0201_0603Metric, F.Cu at (454.1, 182.0)
- added C316: 100nF, Capacitor_SMD:C_0201_0603Metric, F.Cu at (456.6, 164.5)
- added C317: 22uF, Capacitor_SMD:C_0201_0603Metric, F.Cu at (456.6, 166.2)
- added C318: 10uF, Capacitor_SMD:C_0201_0603Metric, F.Cu at (456.6, 168.0)
- added C319: 10uF, Capacitor_SMD:C_0201_0603Metric, F.Cu at (456.6, 169.7)
- added C320: 10uF, Capacitor_SMD:C_0201_0603Metric, F.Cu at (456.6, 171.5)
- added C321: 10uF, Capacitor_SMD:C_0201_0603Metric, F.Cu at (456.6, 173.2)
- added C322: 4.7uF, Capacitor_SMD:C_0201_0603Metric, F.Cu at (456.6, 175.0)
- added C323: 1uF, Capacitor_SMD:C_0201_0603Metric, F.Cu at (456.6, 176.7)
- added C324: 1uF, Capacitor_SMD:C_0201_0603Metric, F.Cu at (456.6, 178.5)
- added C325: 1uF, Capacitor_SMD:C_0201_0603Metric, F.Cu at (456.6, 180.2)
- added C326: 100nF, Capacitor_SMD:C_0201_0603Metric, F.Cu at (456.6, 182.0)
- added C327: 100nF, Capacitor_SMD:C_0201_0603Metric, F.Cu at (459.0, 164.5)
- added C328: 4.7uF, Capacitor_SMD:C_0603_1608Metric, F.Cu at (441.5, 145.3)
- added C329: 10uF, Capacitor_SMD:C_0201_0603Metric, F.Cu at (459.0, 166.2)
- added C330: 10uF, Capacitor_SMD:C_0201_0603Metric, F.Cu at (459.0, 168.0)
- added C331: 4.7uF, Capacitor_SMD:C_0603_1608Metric, F.Cu at (441.5, 147.8)
- added C332: 10uF, Capacitor_SMD:C_0201_0603Metric, F.Cu at (459.0, 169.7)
- added C333: 10uF, Capacitor_SMD:C_0201_0603Metric, F.Cu at (459.0, 171.5)
- added C334: 1uF, Capacitor_SMD:C_0201_0603Metric, F.Cu at (459.0, 173.2)
- added C335: 1uF, Capacitor_SMD:C_0603_1608Metric, F.Cu at (441.5, 150.3)
- added C336: 100nF, Capacitor_SMD:C_0201_0603Metric, F.Cu at (459.0, 175.0)
- added C337: 1uF, Capacitor_SMD:C_0201_0603Metric, F.Cu at (459.0, 176.7)
- added C338: 100nF, Capacitor_SMD:C_0201_0603Metric, F.Cu at (459.0, 178.5)
- added C339: 22uF, Capacitor_SMD:C_0201_0603Metric, F.Cu at (459.0, 180.2)
- added J11: G45AA1912100B1EU, barebones:AMPHENOL_G45AA1912100B1EU, F.Cu at (432.3, 172.7)
- added L12: 0.22uH, Inductor_SMD:L_0805_2012Metric, F.Cu at (449.8, 141.8)
- added L13: 0.22uH, Inductor_SMD:L_0805_2012Metric, F.Cu at (449.8, 144.6)
- added L14: 0.22uH, Inductor_SMD:L_0805_2012Metric, F.Cu at (449.8, 147.3)
- added R114: 100, Resistor_SMD:R_0603_1608Metric, F.Cu at (441.5, 152.8)
- added R142: 2.2k, Resistor_SMD:R_0603_1608Metric, F.Cu at (441.5, 155.3)
- added R143: 2.2k, Resistor_SMD:R_0603_1608Metric, F.Cu at (441.5, 157.8)
- added R144: 2.2k, Resistor_SMD:R_0603_1608Metric, F.Cu at (441.5, 160.4)
- added R145: 100R, Resistor_SMD:R_0603_1608Metric, F.Cu at (445.6, 135.3)
- added R146: 100R, Resistor_SMD:R_0603_1608Metric, F.Cu at (445.6, 137.8)
- added R147: 2.2k, Resistor_SMD:R_0603_1608Metric, F.Cu at (445.6, 140.3)
- added R148: 2.2k, Resistor_SMD:R_0603_1608Metric, F.Cu at (445.6, 142.8)
- added R149: 100R, Resistor_SMD:R_0603_1608Metric, F.Cu at (445.6, 145.3)
- added R150: 100k, Resistor_SMD:R_0603_1608Metric, F.Cu at (462.3, 164.9)
- added R151: 100k, Resistor_SMD:R_0603_1608Metric, F.Cu at (462.3, 167.4)
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Connections:
- net /Power and Ground/CHIP_ENABLE renamed /Power and Ground/PMIC_EXT_EN
- net /Power and Ground/CHRG_PROT_EC renamed /Power and Ground/CHRG_PROT
- net /Power and Ground/MISO_RK renamed /Power and Ground/PWRCTRL3_PMIC
- net /Power and Ground/NLDO1 renamed NLDO1_RK
- net /Power and Ground/NLDO2 renamed NLDO2_RK
- net /Power and Ground/NLDO3 renamed NLDO3_RK
- net /Power and Ground/NLDO4 renamed NLDO4_RK
- net /Power and Ground/NLDO5 renamed NLDO5_RK
- net /Power and Ground/PLDO1 renamed PLDO1_RK
- net /Power and Ground/PLDO2 renamed PLDO2_RK
- net /Power and Ground/PLDO3 renamed PLDO3_RK
- net /Power and Ground/PLDO4 renamed PLDO4_RK
- net /Power and Ground/PLDO5 renamed PLDO5_RK
- net /Power and Ground/PWRCTRL1 renamed /Power and Ground/PWRCTRL1_PMIC
- net /Power and Ground/PWRCTRL2 renamed /Power and Ground/PWRCTRL2_PMIC
- C112 pad 1: Net-(J6-VDD) -> AGND
- C112 pad 2: VCC_3V3_SYS -> VDD_GPU_S0
- C114 pad 2: VCC_5V0_SYS -> VCC_4V0_SYS
- C115 pad 2: VCC_5V0_SYS -> VCC_4V0_SYS
- C116 pad 2: VCC_5V0_SYS -> VCC_4V0_SYS
- C117 pad 2: VCC_5V0_SYS -> VCC_4V0_SYS
- C118 pad 2: VCC_5V0_SYS -> VCC_4V0_SYS
- C119 pad 2: VCC_5V0_SYS -> VCC_4V0_SYS
- C120 pad 2: VCC_5V0_SYS -> VCC_4V0_SYS
- C121 pad 2: VCC_5V0_SYS -> VCC_4V0_SYS
- C125 pad 2: VCC_5V0_SYS -> VCC_4V0_SYS
- C126 pad 2: VCC_5V0_SYS -> VCC_4V0_SYS
- C127 pad 2: VCC_5V0_SYS -> VCC_4V0_SYS
- C129 pad 2: VCC_5V0_SYS -> VCC_4V0_SYS
- C130 pad 2: VCC_5V0_SYS -> VCC_4V0_SYS
- C131 pad 2: VCC_5V0_SYS -> VCC_4V0_SYS
- C140 pad 1: VCC_5V0_SYS -> VDD_DDR_S0
- C141 pad 1: VCC_5V0_SYS -> VDD_DDR_S0
- C142 pad 1: VCC_5V0_SYS -> VCC2_DDR_S3
- C144 pad 1: VCC_5V0_SYS -> VCC_2V0_PLDO_S3
- C145 pad 1: VCC_5V0_SYS -> VCC_2V0_PLDO_S3
- C146 pad 1: VCC_5V0_SYS -> VCC2_DDR_S3
- C148 pad 1: VCC_5V0_SYS -> VDD_VDENC_S0
- C149 pad 1: VCC_5V0_SYS -> VDD_VDENC_S0
- C150 pad 1: VCC_5V0_SYS -> VDD_VDENC_S0
- C151 pad 1: VCC_5V0_SYS -> VDD_LOG_S0
- C152 pad 1: VCC_5V0_SYS -> VDD_LOG_S0
- C153 pad 1: VCC_5V0_SYS -> VDD_LOG_S0
- C154 pad 1: VCC_5V0_SYS -> VDD_CPU_LIT_S0
- C155 pad 1: VCC_5V0_SYS -> VDD_CPU_LIT_S0
- C156 pad 1: VCC_5V0_SYS -> VDD_CPU_LIT_S0
- C157 pad 1: VCC_5V0_SYS -> VDD_GPU_S0
- C158 pad 1: VCC_5V0_SYS -> VDD_GPU_S0
- C159 pad 1: VCC_5V0_SYS -> VDD_GPU_S0
- C160 pad 1: VCC_5V0_SYS -> VCC_1V8_S3
- C161 pad 1: VCC_5V0_SYS -> VCC_1V8_S3
- C162 pad 1: VCC_5V0_SYS -> VDDQ_DDR_S0
- C163 pad 1: VCC_5V0_SYS -> VDDQ_DDR_S0
- C164 pad 1: VCC_5V0_SYS -> VCC_3V3_S3
- C165 pad 1: VCC_5V0_SYS -> VCC_3V3_S3
- C216 pad 2: /Peripheral IO Connectors/HDMI2_1_5V0 -> /Peripheral IO Connectors/HDMI2_0_5V0
- C217 pad 2: /Peripheral IO Connectors/HDMI2_1_5V0 -> /Peripheral IO Connectors/HDMI2_0_5V0
- C218 pad 2: /Peripheral IO Connectors/HDMI_1_CEC -> /Peripheral IO Connectors/HDMI_0_CEC
- C219 pad 1: AGND -> Net-(J10-VDD)
- C219 pad 2: /Peripheral IO Connectors/HDMI_0_CEC -> VCC_3V3_SYS
- C220 pad 2: /Peripheral IO Connectors/HDMI2_0_5V0 -> /Peripheral IO Connectors/HDMI_1_CEC
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
Commit message: added the display connector and its 12V power supply
Parts:
- removed D12, D13, D5: TPD4E02B04DQAR, barebones:DIO_TPD4E02B04DQAR
- removed D3, D4: TPD6E05U06RVZR, barebones:SON50P135X350X55-14N
- removed J14: SM02B-GHS-TB_LF__SN_, barebones:JST_SM02B-GHS-TB_LF__SN_
- removed J7: 54-00007, barebones:TENSILITY_54-00007
- removed L12, L13, L14, L8: 0.22uH, Inductor_SMD:L_0805_2012Metric
- removed U11: BQ25731RSNR, barebones:QFN40P400X400X80-33N
- removed U2, U22, U3: TPS54628DDAR, barebones:VREG_LM5017MR_NOPB
- removed U26: TPD4E004DRYR, barebones:PSON50P145X100X60-6N
- removed U35: 2N7002KW, barebones:SOT323
- removed U38: TPA2012D2RTJT, barebones:QFN50P400X400X80-21N270X270
- removed U5, U6: TPS259474ARPWR, barebones:IC_TPS259474ARPWR
- removed U9: BQ28Z610DRZR, barebones:IC_BQ27441DRZR-G1A
- added C128: 10uF, Capacitor_SMD:C_0201_0603Metric, F.Cu at (268.5, 177.4)
- added C132: 1uF, Capacitor_SMD:C_0201_0603Metric, F.Cu at (268.5, 184.4)
- added C143: 1uF, Capacitor_SMD:C_0201_0603Metric, F.Cu at (271.0, 179.2)
- added C340: 33nF, Capacitor_SMD:C_0603_1608Metric, F.Cu at (273.8, 135.4)
- added C341: 47uF, Capacitor_SMD:C_0603_1608Metric, F.Cu at (273.8, 137.9)
- added C342: 47uF, Capacitor_SMD:C_0603_1608Metric, F.Cu at (273.8, 140.4)
- added C343: 0.1uF, Capacitor_SMD:C_0603_1608Metric, F.Cu at (273.8, 142.9)
- added C344: 0.1uF, Capacitor_SMD:C_0603_1608Metric, F.Cu at (273.8, 145.4)
- added C345: 10nF, Capacitor_SMD:C_0603_1608Metric, F.Cu at (277.8, 102.8)
- added C346: 47uF, Capacitor_SMD:C_0603_1608Metric, F.Cu at (277.8, 105.3)
- added C347: 47uF, Capacitor_SMD:C_0603_1608Metric, F.Cu at (277.8, 107.8)
- added C348: 0.1uF, Capacitor_SMD:C_0603_1608Metric, F.Cu at (277.8, 110.3)
- added C349: 1uF, Capacitor_SMD:C_0603_1608Metric, F.Cu at (277.8, 112.8)
- added C350: 47uF, Capacitor_SMD:C_0603_1608Metric, F.Cu at (277.8, 115.3)
- added C351: 47uF, Capacitor_SMD:C_0603_1608Metric, F.Cu at (277.8, 117.8)
- added C352: 0.1uF, Capacitor_SMD:C_0603_1608Metric, F.Cu at (277.8, 120.3)
- added C353: 4.7uF, Capacitor_SMD:C_0603_1608Metric, F.Cu at (277.8, 122.8)
- added C354: 0.1uF, Capacitor_SMD:C_0603_1608Metric, F.Cu at (277.8, 125.3)
- added C355: 680pF, Capacitor_SMD:C_0603_1608Metric, F.Cu at (277.8, 127.9)
- added C356: 4.7uF, Capacitor_SMD:C_0603_1608Metric, F.Cu at (277.8, 130.4)
- added C357: 0.1uF, Capacitor_SMD:C_0603_1608Metric, F.Cu at (277.8, 132.9)
- added C358: 33uF, Capacitor_SMD:C_0603_1608Metric, F.Cu at (277.8, 135.4)
- added C359: 0.47uF, Capacitor_SMD:C_0603_1608Metric, F.Cu at (277.8, 137.9)
- added C360: 1uF, Capacitor_SMD:C_0201_0603Metric, F.Cu at (274.5, 154.6)
- added C361: 1uF, Capacitor_SMD:C_0201_0603Metric, F.Cu at (274.5, 156.3)
- added C362: 220nF, Capacitor_SMD:C_0201_0603Metric, F.Cu at (274.5, 158.1)
- added C363: 0.1uF, Capacitor_SMD:C_0603_1608Metric, F.Cu at (277.8, 140.4)
- added C364: 10nF, Capacitor_SMD:C_0603_1608Metric, F.Cu at (277.8, 142.9)
- added C365: 47uF, Capacitor_SMD:C_0603_1608Metric, F.Cu at (277.8, 145.4)
- added C366: 47uF, Capacitor_SMD:C_0603_1608Metric, F.Cu at (281.8, 102.8)
- added C367: 0.1uF, Capacitor_SMD:C_0603_1608Metric, F.Cu at (281.8, 105.3)
- added C368: 1uF, Capacitor_SMD:C_0603_1608Metric, F.Cu at (281.8, 107.8)
- added C369: 47uF, Capacitor_SMD:C_0603_1608Metric, F.Cu at (281.8, 110.3)
- added C370: 47uF, Capacitor_SMD:C_0603_1608Metric, F.Cu at (281.8, 112.8)
- added C371: 0.1uF, Capacitor_SMD:C_0603_1608Metric, F.Cu at (281.8, 115.3)
- added C372: 2.2uF, Capacitor_SMD:C_0603_1608Metric, F.Cu at (206.2, 205.7)
- added C373: 0.1uF, Capacitor_SMD:C_0603_1608Metric, F.Cu at (206.2, 208.2)
- added C374: 4.7uF, Capacitor_SMD:C_0201_0603Metric, F.Cu at (205.4, 194.6)
- added C375: 100nF, Capacitor_SMD:C_0201_0603Metric, F.Cu at (205.4, 196.3)
- added C376: 100nF, Capacitor_SMD:C_0201_0603Metric, F.Cu at (205.4, 198.1)
- added C377: 100nF, Capacitor_SMD:C_0201_0603Metric, F.Cu at (205.4, 199.8)
- added C378: 4.7uF, Capacitor_SMD:C_0201_0603Metric, F.Cu at (205.4, 201.6)
- added C379: 100nF, Capacitor_SMD:C_0201_0603Metric, F.Cu at (207.8, 194.6)
- added C380: 100nF, Capacitor_SMD:C_0201_0603Metric, F.Cu at (207.8, 196.3)
- added C381: 100nF, Capacitor_SMD:C_0201_0603Metric, F.Cu at (207.8, 198.1)
- added C382: 22uF, Capacitor_SMD:C_0201_0603Metric, F.Cu at (207.8, 199.8)
- added C383: 10uF, Capacitor_SMD:C_0201_0603Metric, F.Cu at (207.8, 201.6)
- added C384: 10uF, Capacitor_SMD:C_0201_0603Metric, F.Cu at (210.3, 194.6)
- added C385: 1uF, Capacitor_SMD:C_0201_0603Metric, F.Cu at (210.3, 196.3)
- added C386: 100nF, Capacitor_SMD:C_0201_0603Metric, F.Cu at (210.3, 198.1)
- added C387: 100nF, Capacitor_SMD:C_0201_0603Metric, F.Cu at (210.3, 199.8)
- added C388: 22uF, Capacitor_SMD:C_0201_0603Metric, F.Cu at (210.3, 201.6)
- added C389: 10uF, Capacitor_SMD:C_0201_0603Metric, F.Cu at (212.7, 194.6)
- added C390: 10uF, Capacitor_SMD:C_0201_0603Metric, F.Cu at (212.7, 196.3)
- added C391: 1uF, Capacitor_SMD:C_0201_0603Metric, F.Cu at (212.7, 198.1)
- added C392: 100nF, Capacitor_SMD:C_0201_0603Metric, F.Cu at (212.7, 199.8)
- added C393: 100nF, Capacitor_SMD:C_0201_0603Metric, F.Cu at (212.7, 201.6)
- added C394: 1uF, Capacitor_SMD:C_0603_1608Metric, F.Cu at (174.0, 178.4)
- added C395: 1uF, Capacitor_SMD:C_0603_1608Metric, F.Cu at (174.0, 180.9)
- added C396: 1uF, Capacitor_SMD:C_0603_1608Metric, F.Cu at (174.0, 183.4)
- added C397: 1uF, Capacitor_SMD:C_0603_1608Metric, F.Cu at (174.0, 185.9)
- added C398: 1uF, Capacitor_SMD:C_0603_1608Metric, F.Cu at (174.0, 188.5)
- added C399: 1uF, Capacitor_SMD:C_0603_1608Metric, F.Cu at (174.0, 191.0)
- added C400: 0.1uF, Capacitor_SMD:C_0603_1608Metric, F.Cu at (174.0, 193.5)
- added C401: 0.1uF, Capacitor_SMD:C_0603_1608Metric, F.Cu at (174.0, 196.0)
- added C402: 1uF, Capacitor_SMD:C_0603_1608Metric, F.Cu at (174.0, 198.5)
- added C403: 1uF, Capacitor_SMD:C_0603_1608Metric, F.Cu at (174.0, 201.0)
- added C404: 1uF, Capacitor_SMD:C_0603_1608Metric, F.Cu at (174.0, 203.5)
- added C405: 1uF, Capacitor_SMD:C_0603_1608Metric, F.Cu at (178.0, 178.4)
- added C406: 1uF, Capacitor_SMD:C_0603_1608Metric, F.Cu at (178.0, 180.9)
- added C407: 1uF, Capacitor_SMD:C_0603_1608Metric, F.Cu at (178.0, 183.4)
- added C408: 0.1uF, Capacitor_SMD:C_0603_1608Metric, F.Cu at (178.0, 185.9)
- added C409: 20pF, Capacitor_SMD:C_0603_1608Metric, F.Cu at (178.0, 188.5)
- added C410: 20pF, Capacitor_SMD:C_0603_1608Metric, F.Cu at (178.0, 191.0)
- added C411: 0.1uF, Capacitor_SMD:C_0603_1608Metric, F.Cu at (178.0, 193.5)
- added C412: 0.1uF, Capacitor_SMD:C_0603_1608Metric, F.Cu at (178.0, 196.0)
- added C413: 1uF, Capacitor_SMD:C_0603_1608Metric, F.Cu at (178.0, 198.5)
- added C414: 1uF, Capacitor_SMD:C_0603_1608Metric, F.Cu at (178.0, 201.0)
- added C415: 1uF, Capacitor_SMD:C_0603_1608Metric, F.Cu at (178.0, 203.5)
- added C416: 100nF, Capacitor_SMD:C_0603_1608Metric, F.Cu at (182.0, 178.4)
- added C417: 100nF, Capacitor_SMD:C_0603_1608Metric, F.Cu at (182.0, 180.9)
- added C418: 1uF, Capacitor_SMD:C_0603_1608Metric, F.Cu at (182.0, 183.4)
- added C419: 1uF, Capacitor_SMD:C_0603_1608Metric, F.Cu at (182.0, 185.9)
- added C420: 1uF, Capacitor_SMD:C_0603_1608Metric, F.Cu at (182.0, 188.5)
- added C421: 1uF, Capacitor_SMD:C_0603_1608Metric, F.Cu at (182.0, 191.0)
- added C422: 100nF, Capacitor_SMD:C_0603_1608Metric, F.Cu at (182.0, 193.5)
- added C423: 1uF, Capacitor_SMD:C_0603_1608Metric, F.Cu at (182.0, 196.0)
- added C424: 1uF, Capacitor_SMD:C_0603_1608Metric, F.Cu at (182.0, 198.5)
- added C425: 100nF, Capacitor_SMD:C_0603_1608Metric, F.Cu at (182.0, 201.0)
- added C426: 1uF, Capacitor_SMD:C_0603_1608Metric, F.Cu at (182.0, 203.5)
- added C427: 100nF, Capacitor_SMD:C_0603_1608Metric, F.Cu at (186.0, 178.4)
- added C428: 100nF, Capacitor_SMD:C_0603_1608Metric, F.Cu at (186.0, 180.9)
- added C429: 100nF, Capacitor_SMD:C_0603_1608Metric, F.Cu at (186.0, 183.4)
- added C430: 4.7uF, Capacitor_SMD:C_0201_0603Metric, F.Cu at (173.2, 142.7)
- added C431: 0.1uF, Capacitor_SMD:C_0201_0603Metric, F.Cu at (173.2, 144.5)
- added C432: 100nF, Capacitor_SMD:C_0201_0603Metric, F.Cu at (173.2, 146.2)
- added C433: 100nF, Capacitor_SMD:C_0201_0603Metric, F.Cu at (173.2, 148.0)
- added C434: 0.1uF, Capacitor_SMD:C_0201_0603Metric, F.Cu at (173.2, 149.7)
- added C435: 0.1uF, Capacitor_SMD:C_0201_0603Metric, F.Cu at (173.2, 151.5)
- added C436: 100nF, Capacitor_SMD:C_0201_0603Metric, F.Cu at (173.2, 153.2)
- added C437: 100nF, Capacitor_SMD:C_0201_0603Metric, F.Cu at (173.2, 155.0)
- added C438: 10uF, Capacitor_SMD:C_0201_0603Metric, F.Cu at (173.2, 156.7)
- added C439: 22uF, Capacitor_SMD:C_0201_0603Metric, F.Cu at (173.2, 158.5)
- added C440: 100nF, Capacitor_SMD:C_0201_0603Metric, F.Cu at (173.2, 160.2)
- added C441: 0.1uF, Capacitor_SMD:C_0201_0603Metric, F.Cu at (173.2, 162.0)
- added C442: 220nF, Capacitor_SMD:C_0201_0603Metric, F.Cu at (175.7, 142.7)
- added C443: 0.1uF, Capacitor_SMD:C_0201_0603Metric, F.Cu at (175.7, 144.5)
- added C444: 220nF, Capacitor_SMD:C_0201_0603Metric, F.Cu at (175.7, 146.2)
- added C445: 220nF, Capacitor_SMD:C_0201_0603Metric, F.Cu at (175.7, 148.0)
- added C446: 220nF, Capacitor_SMD:C_0201_0603Metric, F.Cu at (175.7, 149.7)
- added C447: 220nF, Capacitor_SMD:C_0201_0603Metric, F.Cu at (175.7, 151.5)
- added C448: 220nF, Capacitor_SMD:C_0201_0603Metric, F.Cu at (175.7, 153.2)
- added C449: 0.1uF, Capacitor_SMD:C_0201_0603Metric, F.Cu at (175.7, 155.0)
- added C450: 220nF, Capacitor_SMD:C_0201_0603Metric, F.Cu at (175.7, 156.7)
- added C451: 220nF, Capacitor_SMD:C_0201_0603Metric, F.Cu at (175.7, 158.5)
- added C452: 100nF, Capacitor_SMD:C_0201_0603Metric, F.Cu at (175.7, 160.2)
- added C453: 100nF, Capacitor_SMD:C_0201_0603Metric, F.Cu at (175.7, 162.0)
- added C454: 100nF, Capacitor_SMD:C_0201_0603Metric, F.Cu at (178.1, 142.7)
- added C455: 100nF, Capacitor_SMD:C_0201_0603Metric, F.Cu at (178.1, 144.5)
- added C456: 100nF, Capacitor_SMD:C_0201_0603Metric, F.Cu at (178.1, 146.2)
- added C457: 100nF, Capacitor_SMD:C_0201_0603Metric, F.Cu at (178.1, 148.0)
- added C458: 0.1uF, Capacitor_SMD:C_0201_0603Metric, F.Cu at (178.1, 149.7)
- added C459: 0.1uF, Capacitor_SMD:C_0201_0603Metric, F.Cu at (178.1, 151.5)
- added C460: 220pF, Capacitor_SMD:C_0201_0603Metric, F.Cu at (178.1, 153.2)
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Connections:
- net /Peripheral IO Connectors/USB20_HOST0_DN renamed /Peripheral IO Connectors/USB20_HOST0_DM
- C1 pad 1: unconnected-(C1-Pad1) -> AGND
- C1 pad 2: Net-(U1R-PCIE30_PORT0_TX0P) -> VDDQ_DDR_S0
- C10 pad 1: Net-(U2-SS) -> AGND
- C10 pad 2: AGND -> VDDQ_DDR_S0
- C100 pad 1: /Peripheral IO Connectors/PCIE30_PORT1_TX1P -> VDD_GPU_S0
- C100 pad 2: Net-(J3-P13) -> AGND
- C101 pad 1: /Peripheral IO Connectors/PCIE30_PORT1_TX0N -> VDD_LOG_S0
- C101 pad 2: Net-(J3-P23) -> AGND
- C102 pad 1: /Peripheral IO Connectors/PCIE30_PORT1_TX0P -> VDD_LOG_S0
- C102 pad 2: Net-(J3-P25) -> AGND
- C103 pad 1: /Peripheral IO Connectors/PCIE30_PORT0_TX1N -> AGND
- C103 pad 2: Net-(J3-P35) -> VCC_1V8_S0
- C104 pad 1: /Peripheral IO Connectors/PCIE30_PORT0_TX1P -> AGND
- C104 pad 2: Net-(J3-P37) -> VCC_1V8_S0
- C105 pad 1: /Peripheral IO Connectors/PCIE30_PORT0_TX0N -> AGND
- C105 pad 2: Net-(J3-P41) -> VCC_1V8_S0
- C106 pad 1: /Peripheral IO Connectors/PCIE30_PORT0_TX0P -> AGND
- C106 pad 2: Net-(J3-P43) -> VCC_1V8_S0
- C107 pad 1: /Peripheral IO Connectors/PCIE20_0_TXP -> AGND
- C107 pad 2: Net-(C107-Pad2) -> VCC_1V8_S0
- C108 pad 1: /Peripheral IO Connectors/PCIE20_0_TXN -> AGND
- C108 pad 2: Net-(C108-Pad2) -> VCC_1V8_S0
- C109 pad 2: VCC_3V3_SYS -> VDD_GPU_S0
- C11 pad 1: Net-(U3-SS) -> AGND
- C11 pad 2: AGND -> VDDQ_DDR_S0
- C110 pad 2: VCC_3V3_SYS -> VDD_GPU_S0
- C111 pad 2: VCC_3V3_SYS -> VDD_GPU_S0
- C113 pad 2: /Power and Ground/VIN_CHRG_4 -> VDD_GPU_S0
- C114 pad 2: VCC_4V0_SYS -> VDD_GPU_S0
- C115 pad 2: VCC_4V0_SYS -> VDD_GPU_S0
- C116 pad 2: VCC_4V0_SYS -> VDD_GPU_S0
- C117 pad 2: VCC_4V0_SYS -> VDD_GPU_S0
- C118 pad 2: VCC_4V0_SYS -> VDD_VDENC_S0
- C119 pad 2: VCC_4V0_SYS -> VDD_VDENC_S0
- C12 pad 1: Net-(U4-SS) -> AGND
- C12 pad 2: AGND -> VDDQ_DDR_S0
- C120 pad 2: VCC_4V0_SYS -> VDD_VDENC_S0
- C121 pad 2: VCC_4V0_SYS -> VDD_VDENC_S0
- C122 pad 2: NLDO5_RK -> VDD_VDENC_S0
- C123 pad 2: NLDO4_RK -> VDD_VDENC_S0
- C124 pad 2: NLDO3_RK -> VDD_VDENC_S0
- C125 pad 2: VCC_4V0_SYS -> VDD_NPU_S0
- C126 pad 2: VCC_4V0_SYS -> VDD_NPU_S0
- C127 pad 2: VCC_4V0_SYS -> VDD_NPU_S0
- C129 pad 2: VCC_4V0_SYS -> VDD_NPU_S0
- C13 pad 2: /Power and Ground/VIN_CHRG_4 -> VDDQ_DDR_S0
- C130 pad 2: VCC_4V0_SYS -> VDD_NPU_S0
- C131 pad 2: VCC_4V0_SYS -> VDD_NPU_S0
- C133 pad 2: PLDO1_RK -> VDD_CPU_BIG1_MEM_S0
- C134 pad 2: PLDO2_RK -> VDD_CPU_BIG1_S0
- C135 pad 2: PLDO3_RK -> VDD_CPU_BIG1_S0
- C136 pad 2: PLDO4_RK -> VDD_CPU_BIG1_S0
- C137 pad 2: PLDO5_RK -> VDD_CPU_BIG1_S0
- C138 pad 2: NLDO2_RK -> VDD_CPU_BIG1_S0
- C139 pad 2: NLDO1_RK -> VDD_CPU_BIG1_S0
- C14 pad 2: /Power and Ground/VIN_CHRG_4 -> VCCA_1V8_S0
- C140 pad 1: VDD_DDR_S0 -> AGND
- C140 pad 2: AGND -> VDD_CPU_BIG1_S0
- C141 pad 1: VDD_DDR_S0 -> AGND
- C141 pad 2: AGND -> VDD_CPU_BIG1_S0
- C142 pad 1: VCC2_DDR_S3 -> AGND
- C142 pad 2: AGND -> VDD_CPU_BIG1_S0
- C144 pad 1: VCC_2V0_PLDO_S3 -> AGND
- C144 pad 2: AGND -> VDD_LOG_S0
- C145 pad 1: VCC_2V0_PLDO_S3 -> AGND
- C145 pad 2: AGND -> VDD_LOG_S0
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Other:
- board size 350 x 250 mm -> 1 x 0.7 mm

Commit message: updated the Fuel Guage/BMS module for the 4S battery usage
Parts:
- removed C242: 4.7nF, Capacitor_SMD:C_0201_0603Metric
- removed C251: 33pF, Capacitor_SMD:C_0201_0603Metric
- removed C264: 680pF, Capacitor_SMD:C_0201_0603Metric
- removed C280, C281, C283, C290: 0.1uF, Capacitor_SMD:C_0201_0603Metric
- removed C282: 2.2uF, Capacitor_SMD:C_0201_0603Metric
- removed C291: 1uF, Capacitor_SMD:C_0201_0603Metric
- removed C395: 1uF, Capacitor_SMD:C_0603_1608Metric
- removed D1: MMSZ5V6T1G, barebones:MMSZ5V6T1G
- removed R126, R127: 33, Resistor_SMD:R_0603_1608Metric
- removed R128: 10k, Resistor_SMD:R_0603_1608Metric
- removed R64: 15k, Resistor_SMD:R_0603_1608Metric
- removed R77, R78: 10M, Resistor_SMD:R_0603_1608Metric
- removed R79, R81: 5.1k, Resistor_SMD:R_0603_1608Metric
- removed R80: FUSE, Resistor_SMD:R_0603_1608Metric
- removed R82: 10, Resistor_SMD:R_0603_1608Metric
- removed R83, R84, R85, R86, R87, R90, R95: 100, Resistor_SMD:R_0603_1608Metric
- removed R91: THERM, Resistor_SMD:R_0603_1608Metric
- removed TP1: RESETB, TestPoint:TestPoint_Pad_D1.5mm
- removed TP2, TP4: GND, TestPoint:TestPoint_Pad_D1.5mm
- removed TP3: POWER ON, TestPoint:TestPoint_Pad_D1.5mm
- added C539: 100nF, Capacitor_SMD:C_0603_1608Metric, F.Cu at (262.8, 173.2)
- added C540: 0.1uF, Capacitor_SMD:C_0402_1005Metric, F.Cu at (305.3, 111.8)
- added C541: 4.7uF, Capacitor_SMD:C_0201_0603Metric, F.Cu at (219.3, 158.2)
- added C542: 1uF, Capacitor_SMD:C_0603_1608Metric, F.Cu at (212.5, 185.5)
- added C543: 0.1uF, Capacitor_SMD:C_0201_0603Metric, F.Cu at (219.3, 160.0)
- added C544: 0.1uF, Capacitor_SMD:C_0201_0603Metric, F.Cu at (219.3, 161.7)
- added C545: 10uF, Capacitor_SMD:C_0201_0603Metric, F.Cu at (219.3, 163.5)
- added C556: 4.7nF, Capacitor_SMD:C_0402_1005Metric, F.Cu at (330.3, 141.9)
- added C557: 680pF, Capacitor_SMD:C_0402_1005Metric, F.Cu at (330.3, 143.7)
- added C558: 15pF, Capacitor_SMD:C_0402_1005Metric, F.Cu at (330.3, 145.4)
- added C559: 33pF, Capacitor_SMD:C_0402_1005Metric, F.Cu at (332.8, 129.7)
- added C561: 0.1uF, Capacitor_SMD:C_0402_1005Metric, F.Cu at (336.6, 272.4)
- added C562: 0.1uF, Capacitor_SMD:C_0402_1005Metric, F.Cu at (476.4, 272.9)
- added C563: 0.1uF, Capacitor_SMD:C_0402_1005Metric, F.Cu at (397.6, 271.4)
- added C564: 0.1uF, Capacitor_SMD:C_0402_1005Metric, F.Cu at (501.6, 275.3)
- added C565: 0.1uF, Capacitor_SMD:C_0402_1005Metric, F.Cu at (515.2, 268.8)
- added C566: 2.2uF, Capacitor_SMD:C_0402_1005Metric, F.Cu at (476.4, 270.9)
- added C567: 0.1uF, Capacitor_SMD:C_0402_1005Metric, F.Cu at (369.5, 270.2)
- added C568: 0.1uF, Capacitor_SMD:C_0402_1005Metric, F.Cu at (369.5, 269.1)
- added D16: BAT54CW, Package_TO_SOT_SMD:SOT-323_SC-70, F.Cu at (238.3, 223.3)
- added D21: 1N4148W, Diode_SMD:D_SOD-123, F.Cu at (354.7, 268.6)
- added FPC1: FH12-6S-0.5SH, barebones:FPC-SMD_FH12-6S-0.5SH-55, F.Cu at (264.8, 153.8)
- added J21: SM02B-GHS-TB_LF__SN_, barebones:JST_SM02B-GHS-TB_LF__SN_, F.Cu at (332.1, 115.1)
- added J22: SJ2-35894B-SMT-TR, barebones:CUI_SJ2-35894B-SMT-TR, F.Cu at (227.3, 184.5)
- added J23: 874381343, barebones:MOLEX_874381343, F.Cu at (416.6, 268.9)
- added NT3: NetTie_2, NetTie:NetTie-2_SMD_Pad0.5mm, F.Cu at (229.9, 194.0)
- added NT4: NetTie_2, NetTie:NetTie-2_SMD_Pad0.5mm, F.Cu at (229.9, 195.5)
- added PAD0: NEUTRAL, barebones:7x10-PAD, F.Cu at (519.0, 279.4)
- added PAD1: BATT_1P, barebones:7x10-PAD, F.Cu at (458.1, 279.4)
- added PAD2: BATT_2P, barebones:7x10-PAD, F.Cu at (397.1, 279.4)
- added PAD3: BATT_3P, barebones:7x10-PAD, F.Cu at (373.1, 279.4)
- added PAD4: BATT_4P, barebones:7x10-PAD, F.Cu at (312.1, 279.4)
- added PAD5: BATT_4N, barebones:7x10-PAD, F.Cu at (336.1, 279.4)
- added PAD6: BATT_3N, barebones:7x10-PAD, F.Cu at (434.1, 279.4)
- added PAD7: BATT_2N, barebones:7x10-PAD, F.Cu at (495.1, 279.4)
- added Q5: CSD18504Q5A, barebones:MOSFET_CSD19531Q5A, F.Cu at (320.1, 267.9)
- added Q6: CSD18504Q5A, barebones:MOSFET_CSD19531Q5A, F.Cu at (327.2, 267.9)
- added R212: 1k, Resistor_SMD:R_0603_1608Metric, F.Cu at (242.4, 217.8)
- added R213: 2.2k, Resistor_SMD:R_0402_1005Metric, F.Cu at (241.8, 222.6)
- added R214: 100k, Resistor_SMD:R_0402_1005Metric, F.Cu at (238.0, 140.1)
- added R215: 100k, Resistor_SMD:R_0402_1005Metric, F.Cu at (238.0, 142.0)
- added R216: 4.7k, Resistor_SMD:R_0603_1608Metric, F.Cu at (216.5, 190.5)
- added R217: 4.7k, Resistor_SMD:R_0603_1608Metric, F.Cu at (216.5, 193.0)
- added R218: 4.7k, Resistor_SMD:R_0603_1608Metric, F.Cu at (216.5, 195.5)
- added R219: 10k, Resistor_SMD:R_0603_1608Metric, F.Cu at (216.5, 198.1)
- added R225: 5.1k, Resistor_SMD:R_0402_1005Metric, F.Cu at (482.5, 266.1)
- added R226: 100R, Resistor_SMD:R_0402_1005Metric, F.Cu at (324.8, 271.6)
- added R236: 100, Resistor_SMD:R_0402_1005Metric, F.Cu at (315.1, 270.2)
- added R237: 100, Resistor_SMD:R_0402_1005Metric, F.Cu at (336.6, 273.4)
- added R238: 100, Resistor_SMD:R_0402_1005Metric, F.Cu at (397.6, 272.5)
- added R239: 100, Resistor_SMD:R_0402_1005Metric, F.Cu at (500.4, 275.3)
- added R240: 300, Resistor_SMD:R_0402_1005Metric, F.Cu at (369.5, 268.1)
- added R241: 100, Resistor_SMD:R_0402_1005Metric, F.Cu at (515.1, 266.0)
- added R242: 10M, Resistor_SMD:R_0402_1005Metric, F.Cu at (315.1, 269.1)
- added R243: 100, Resistor_SMD:R_0402_1005Metric, F.Cu at (515.2, 270.8)
- added R244: 10M, Resistor_SMD:R_0402_1005Metric, F.Cu at (482.5, 265.1)
- added R245: 100, Resistor_SMD:R_0402_1005Metric, F.Cu at (504.6, 270.7)
- added R246: 100, Resistor_SMD:R_0402_1005Metric, F.Cu at (504.6, 269.5)
- added R247: 100, Resistor_SMD:R_0402_1005Metric, F.Cu at (493.8, 272.6)
- added R248: 10M, Resistor_SMD:R_0402_1005Metric, F.Cu at (375.9, 269.1)
- added TP11: SMBD, TestPoint:TestPoint_Pad_D1.0mm, F.Cu at (509.9, 266.1)
- added TP12: SMBC, TestPoint:TestPoint_Pad_D1.0mm, F.Cu at (507.8, 266.1)
- added TP13: GND, TestPoint:TestPoint_Pad_D1.0mm, F.Cu at (512.0, 266.1)
- added U72: PCA9306DCTR, barebones:SOP65P400X130-8N, F.Cu at (248.3, 216.0)
- added U73: BQ40Z50RSMR-R2, barebones:QFN40P400X400X100-33N, F.Cu at (492.4, 268.6)
- added U77: NXFT15XH103FA2B025, barebones:NXFT15XH103FA2B025, F.Cu at (322.5, 283.2)
- added U78: NXFT15XH103FA2B025, barebones:NXFT15XH103FA2B025, F.Cu at (506.9, 283.2)
- added U79: NXFT15XH103FA2B025, barebones:NXFT15XH103FA2B025, F.Cu at (445.3, 283.2)
- added U80: NXFT15XH103FA2B025, barebones:NXFT15XH103FA2B025, F.Cu at (384.9, 283.2)
- C165, C166, C180, C181, C184, C185, C189, C190, C195, C196, C198, C220, C221, C222, C223, C224, C225, C226, C227, C228, C231, C232, C235, C237, C238, C240, C241, C243, C254, C255, C256, C257, C258, C259, C260, C261, C262, C268, C269, C272, C273, C274, C275, C276, C360, C361, C362: footprint Capacitor_SMD:C_0201_0603Metric -> Capacitor_SMD:C_0402_1005Metric
- C167, C168, C169, C170, C171, C172, C173, C174, C175, C176, C177, C178, C179, C182, C183, C186, C187, C188, C191, C192, C193, C194, C197, C199, C200, C201, C202, C203, C204, C205, C206, C207, C208, C209, C210, C211, C212, C213, C214, C215, C216, C217, C218, C219, C229, C230, C233, C234, C236, C239, C244, C245, C246, C247, C248, C249, C250, C252, C263, C265, C266, C267, C270, C271, C277, C278, C279, C284, C285, C286, C287, C288, C289, C292, C293, C294, C295, C296, C297, C298, C299, C300, C301, C302, C303, C304, C305, C306, C307, C308, C309, C310, C311, C312, C313, C314, C315, C316, C317, C318, C319, C320, C321, C322, C323, C324, C325, C326, C327, C328, C329, C330, C331, C332, C333, C334, C335, C336, C337, C338, C339, C340, C341, C342, C343, C344, C345, C346, C347, C348, C349, C350, C351, C352, C353, C354, C355, C356, C357, C358, C359, C363, C364, C365, C366, C367, C368, C369, C370, C371: footprint Capacitor_SMD:C_0603_1608Metric -> Capacitor_SMD:C_0402_1005Metric
- C253: value 15pF -> 100nF
- C394: value 1uF -> 100nF; footprint Capacitor_SMD:C_0603_1608Metric -> Capacitor_SMD:C_0201_0603Metric
- C396, C398, C402, C404: value 1uF -> 10uF
- C397, C399, C405, C406, C407: value 1uF -> 100nF
- C400, C401: value 0.1uF -> 10uF
- C403: value 1uF -> 4.7uF
- C518: value 100nF -> 0.1uF
- C522: value 4.7uF -> 100nF
- C523, C525: value 0.1uF -> 10uF; footprint Capacitor_SMD:C_0201_0603Metric -> Capacitor_SMD:C_0603_1608Metric
- C524: value 10uF -> 0.1uF; footprint Capacitor_SMD:C_0201_0603Metric -> Capacitor_SMD:C_0603_1608Metric
- Q3: value STL40DN3LLH5 -> AO3401A; footprint barebones:TRANS_STL40DN3LLH5 -> Package_TO_SOT_SMD:SOT-23
- R100, R101, R102, R103, R104, R105, R106, R107, R108, R109, R110, R111, R112, R113, R114, R115, R116, R117, R32, R33, R34, R35, R36, R37, R38, R39, R40, R41, R42, R43, R44, R45, R46, R47, R48, R49, R50, R52, R53, R54, R55, R56, R57, R58, R60, R61, R62, R63, R65, R66, R67, R69, R70, R71, R72, R73, R74, R88, R89, R92, R96, R97, R98, R99: footprint Resistor_SMD:R_0603_1608Metric -> Resistor_SMD:R_0402_1005Metric
- R129: value 2.2k -> 330k
- R130: value 2.2k -> 10k
- R132: value 2.2k -> 4.7k
- R59: value 40.2k -> WSL25122L000FEA; footprint Resistor_SMD:R_0603_1608Metric -> barebones:RES_WSL25122L000FEA
- R75: value 100k -> 40.2k; footprint Resistor_SMD:R_0603_1608Metric -> Resistor_SMD:R_0402_1005Metric
- R76: value 100k -> 15k; footprint Resistor_SMD:R_0603_1608Metric -> Resistor_SMD:R_0402_1005Metric
- R93: value WSL25122L000FEA -> 5.1k; footprint barebones:RES_WSL25122L000FEA -> Resistor_SMD:R_0402_1005Metric
- R94: value 100 -> 5.1k; footprint Resistor_SMD:R_0603_1608Metric -> Resistor_SMD:R_0402_1005Metric
- U15: value 2N7002KW -> BQ78350DBTR-R1; footprint barebones:SOT323 -> barebones:SOP50P640X120-30N
- U16: value 2N7002KW -> BQ7692000PW; footprint barebones:SOT323 -> barebones:SOP65P640X120-20N
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Connections:
- net /Embedded Controller and Internal Audio/AMP_MUTE renamed /Embedded Controller and Internal Audio/SPK_MUTE
- net /Embedded Controller and Internal Audio/ES_ASDOUT renamed /Embedded Controller and Internal Audio/I2S0_SDI0
- net /Embedded Controller and Internal Audio/ES_DSIN renamed /Embedded Controller and Internal Audio/I2S0_SDO0
- net /Embedded Controller and Internal Audio/ES_LRCK renamed /Embedded Controller and Internal Audio/I2S0_LRCK_TX
- net /Embedded Controller and Internal Audio/ES_MCLK renamed /Embedded Controller and Internal Audio/I2S0_MLCK
- net /Embedded Controller and Internal Audio/ES_SCLK renamed /Embedded Controller and Internal Audio/I2S0_SCLK_TX
- net /Embedded Controller and Internal Audio/I2C4_SCL_M1 renamed /Embedded Controller and Internal Audio/I2C1_SCL_M2
- net /Embedded Controller and Internal Audio/I2C4_SDA_M1 renamed /Embedded Controller and Internal Audio/I2C1_SDA_M2
- net /Embedded Controller and Internal Audio/LED_INDICATOR renamed /Memory and Control/LED_INDICATOR
- net /Embedded Controller and Internal Audio/SWCLK_14 renamed /Embedded Controller and Internal Audio/SWCLK_49
- net /Embedded Controller and Internal Audio/SWDIO_13 renamed /Embedded Controller and Internal Audio/SWDIO_46
- net /High Speed IO/INT_PMIC renamed /High Speed IO/PMIC_INT_L
- net /High Speed IO/PWRCTRL1_PMIC renamed /High Speed IO/PMIC_SLEEP1
- net /High Speed IO/SPI_CLK_PMIC renamed /High Speed IO/SPI2_CLK_M2
- net /High Speed IO/SPI_CS_PMIC renamed /High Speed IO/SPI2_CS0_M2
- net /High Speed IO/SPI_MOSI_PMIC renamed /High Speed IO/SPI2_MOSI_M2
- net /Peripheral IO Connectors/JACK_RING_1 renamed /Peripheral IO Connectors/HP_JACK_RING_1
- net /Peripheral IO Connectors/JACK_RING_2 renamed /Peripheral IO Connectors/HP_JACK_RING_2
- net /Peripheral IO Connectors/JACK_SLEEVE renamed /Peripheral IO Connectors/HP_JACK_SLEEVE
- net /Peripheral IO Connectors/JACK_SWITCH renamed /Peripheral IO Connectors/HP_JACK_SWITCH
- net /Peripheral IO Connectors/JACK_TIP renamed /Peripheral IO Connectors/HP_JACK_TIP
- net /Power and Ground/CHARGE_CNTRL renamed /Power and Ground/CHRG_CTRL
- net /Power and Ground/PWRCTRL1_PMIC renamed /Power and Ground/PMIC_SLEEP1
- net /Power and Ground/SPI_CLK_PMIC renamed /Power and Ground/SPI2_CLK_M2
- net Net-(U14-ACN) renamed /Power and Ground/ACN
- net Net-(U14-ACP) renamed /Power and Ground/ACP
- net Net-(U14-IBAT) renamed /Power and Ground/IBAT
- net VCCA_1V2_S0 renamed VDDA_1V2_S0
- C245 pad 2: VCCA_1V8_S0 -> VCC_1V8_S0
- C253 pad 2: /Power and Ground/COMP2 -> VCC_1V8_S0
- C394 pad 1: /Embedded Controller and Internal Audio/LIN1 -> AGND
- C394 pad 2: /Embedded Controller and Internal Audio/CODEC_MIC -> VCC_1V8_S0
- C397 pad 1: AGND -> VCC_1V8_S0
- C397 pad 2: VCC_3V3_SYS -> AGND
- C398 pad 1: /Embedded Controller and Internal Audio/JACK_SLEEVE -> VCC_1V8_S0
- C398 pad 2: /Embedded Controller and Internal Audio/JACK_MIC_1 -> AGND
- C399 pad 1: AGND -> /Embedded Controller and Internal Audio/CPVSSP
- C399 pad 2: VCC_3V3_SYS -> AGND
- C400 pad 1: AGND -> /Embedded Controller and Internal Audio/CPVSSP
- C400 pad 2: VCC_5V0_PERIPH -> AGND
- C401 pad 2: VCC_5V0_PERIPH -> /Embedded Controller and Internal Audio/DACVREF
- C402 pad 2: /Embedded Controller and Internal Audio/VMID -> /Embedded Controller and Internal Audio/ADCVREF
- C403 pad 2: VCC_5V0_PERIPH -> /Embedded Controller and Internal Audio/VMID
- C404 pad 1: /Embedded Controller and Internal Audio/MICBIAS -> AGND
- C404 pad 2: AGND -> /Embedded Controller and Internal Audio/MICBIAS
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Routing:
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Other:
- board size 1 x 0.7 mm -> 217 x 22.5 mm
