File: barebones_power.kicad_sch (KiCad schematic)
At the start: 267 parts, among them Q1 STL40DN3LLH5, Q2 STL40DN3LLH5, Q3 STL40DN3LLH5, U11 BQ25731RSNR, U2 TPS54628DDAR, U27 IHLP1616ABERR47M01, U28 IHLP1616ABERR47M01, U29 IHLP1616ABERR47M01, U3 TPS54628DDAR, U32 IHLP1616ABERR47M01, U33 IHLP1616ABERR47M01, U34 IHLP1616ABERR47M01, U35 2N7002KW, U36 2N7002KW, U37 LP5912-1.8DRVT, U39 TPS54628DDAR, U4 TPS54628DDAR, U40 TPS54628DDAR, U41 LM3940IMPX-3.3_NOPB, U5 TPS259474ARPWR, U6 TPS259474ARPWR, U7 TPS2121RUXR, U8 RK806-1_C5156483, U9 BQ28Z610DRZR

Commit message: Fixed version control merge issues
Parts:
- L1, L10, L2, L3, L9: footprint barebones:IND_XAL7030-472MEB -> XAL7030-472MEB:IND_XAL7030-472MEB
Changed lines of the file:
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@@
 			)
 		)
-		(property "Footprint" "barebones:IND_XAL7030-472MEB"
+		(property "Footprint" "XAL7030-472MEB:IND_XAL7030-472MEB"
 			(at 125.73 266.7 0)
 			(hide yes)
@@
 			)
 		)
-		(property "Footprint" "barebones:IND_XAL7030-472MEB"
+		(property "Footprint" "XAL7030-472MEB:IND_XAL7030-472MEB"
 			(at 124.46 228.6 0)
 			(hide yes)
@@
 			)
 		)
-		(property "Footprint" "barebones:IND_XAL7030-472MEB"
+		(property "Footprint" "XAL7030-472MEB:IND_XAL7030-472MEB"
 			(at 283.21 273.05 0)
 			(hide yes)
@@
 			)
 		)
-		(property "Footprint" "barebones:IND_XAL7030-472MEB"
+		(property "Footprint" "XAL7030-472MEB:IND_XAL7030-472MEB"
 			(at 124.46 186.69 0)
 			(hide yes)
@@
 			)
 		)
-		(property "Footprint" "barebones:IND_XAL7030-472MEB"
+		(property "Footprint" "XAL7030-472MEB:IND_XAL7030-472MEB"
 			(at 124.46 138.43 0)
 			(hide yes)

Commit message: fixed the power distribution by adding RK806 chips
Parts:
- removed C128, C143: 1uF, Capacitor_SMD:C_0603_1608Metric, symbol Device:C
- removed C132: 2.2uF, Capacitor_SMD:C_0603_1608Metric, symbol Device:C
- removed R81, R82: 5.1k, Resistor_SMD:R_0603_1608Metric, symbol Device:R
- removed R89: 10, Resistor_SMD:R_0603_1608Metric, symbol Device:R
- removed R96: 100k, Resistor_SMD:R_0603_1608Metric, symbol Device:R
- added C233, C235, C238, C239, C242, C249, C256, C265, C273, C335: 1uF, Capacitor_SMD:C_0603_1608Metric, symbol Device:C
- added C234, C245, C246, C251, C252: 47uF, Capacitor_SMD:C_0603_1608Metric, symbol Device:C
- added C236, C237, C240, C241, C257, C258, C259, C260, C261, C262, C263, C264, C266, C267, C268, C269, C270, C271, C272, C274, C275, C276, C277, C278, C279: 22uF, Capacitor_SMD:C_0603_1608Metric, symbol Device:C
- added C243, C254: 10uF, Capacitor_SMD:C_0603_1608Metric, symbol Device:C
- added C244, C255: 100pF, Capacitor_SMD:C_0603_1608Metric, symbol Device:C
- added C247, C287: 10nF, Capacitor_SMD:C_0603_1608Metric, symbol Device:C
- added C248, C250, C253: 0.1uF, Capacitor_SMD:C_0603_1608Metric, symbol Device:C
- added C328, C331: 4.7uF, Capacitor_SMD:C_0603_1608Metric, symbol Device:C
- added L11: XAL7030-472MEB, XAL7030-472MEB:IND_XAL7030-472MEB, symbol XAL7030-472MEB:XAL7030-472MEB
- added L12, L13, L14: 0.22uH, Inductor_SMD:L_0805_2012Metric, symbol Device:L
- added R114: 100, Resistor_SMD:R_0603_1608Metric, symbol Device:R
- added R142, R143, R144, R147, R148: 2.2k, Resistor_SMD:R_0603_1608Metric, symbol Device:R
- added R145, R146, R149: 100R, Resistor_SMD:R_0603_1608Metric, symbol Device:R
- added R55: 56k, Resistor_SMD:R_0603_1608Metric, symbol Device:R
- added R56: 10k, Resistor_SMD:R_0603_1608Metric, symbol Device:R
- added U18, U23: RK860-2, barebones:WLCSP-20_L2.0-W1.6-R5-C4-P0.40-TL, symbol RK860-2:RK860-2
- added U20: RK860-3, easyeda2kicad:WLCSP-20_L2.0-W1.6-R5-C4-P0.40-TL, symbol RK860-3:RK860-3
- added U22: TPS54628DDAR, barebones:VREG_LM5017MR_NOPB, symbol TPS54628DDAR:TPS54628DDAR
- added U24: 1N5819WT, easyeda2kicad:SOD-523_L1.2-W0.8-LS1.6-RD, symbol 1N5819WT:1N5819WT_C5451630
- C157: value 22uF -> 47uF
- R87, R88: value 100k -> 200k
- R90, R91, R94, R95: value 100k -> 100
- R92: value 100k -> 110k
- R97: value 100k -> 2.2k
Connections:
- net FB5: no longer R87.2, R88.1
- net FB6: now also C244.2
- net GND: now also R85.2, R86.2, C234.2, C236.2, C237.2, C240.2, C241.2, C243.2, C245.1, C246.1, C247.2, C248.1, C249.1, C251.1, C252.1, C253.1, C254.2, C257.2, C258.2, C259.2, C260.2, C261.2, C262.2, C263.2, C264.2, C266.2, C267.2, C268.2, C269.2, C270.2, C271.2, C272.2, C274.2, C275.2, C276.2, C277.2, C278.2, C279.2, C287.1, C331.1, C335.1, R56.1, U18.A1 (VSEL), U18.B2 (GND), U18.B3 (GND), U18.B4 (AGND), U18.C1 (GND), U18.C2 (GND), U18.C3 (GND), U18.C4 (GND), U20.A1 (VSEL), U20.B2 (GND), U20.B3 (GND), U20.B4 (AGND), U20.C1 (GND), U20.C2 (GND), U20.C3 (GND), U20.C4 (GND), U22.5 (GND), U23.A1 (VSEL), U23.B2 (GND), U23.B3 (GND), U23.B4 (AGND), U23.C1 (GND), U23.C2 (GND), U23.C3 (GND), U23.C4 (GND), U24.2 (A); no longer R91.2, R95.2, R97.2
- net RESETB: now also R84.2, C287.2; no longer R86.2
- net VDC: now also R87.1, R88.1, C331.2
- net VSYS_MAIN: now also C245.2, C246.2, C248.2, U22.8 (VIN)
- net CHIP_ENABLE renamed PMIC_EXT_EN
- net PMIC_EXT_EN: now also U18.A2 (EN), U20.A2 (EN), U22.1 (EN), U23.A2 (EN)
- net CHRG_PROT_EC renamed CHRG_PROT
- removed net FB1: R94.2, R95.1, U8.48 (FB1)
- removed net FB2: R90.2, R91.1, U8.38 (FB2)
- net FB9 renamed I2C1_SCL_M0
- net I2C1_SCL_M0: now also U18.A3 (SCL); no longer U8.66 (FB9)
- net INT_RK renamed INT_PMIC
- net INT_PMIC: now also R83.2; no longer R85.2
- net MISO_RK renamed PWRCTRL3_PMIC
- net MOSI_RK renamed SPI_MOSI_PMIC
- net SPI_MOSI_PMIC: now also R85.1; no longer R83.2
- net PWRCTRL1 renamed PWRCTRL1_PMIC
- net PWRCTRL2 renamed PWRCTRL2_PMIC
- net SCL_CLK_RK renamed SPI_CLK_PMIC
- net SPI_CLK_PMIC: no longer R84.2
- net VCCA renamed SPI_CS_PMIC
- net SPI_CS_PMIC: now also R86.1; no longer U8.21 (VCCA)
- removed net VCCIO_RK: R83.1, R84.1, R85.1, R86.1, U8.20 (VCCIO)
- removed net VCC_5V0_SYS: C114.2, C115.2, C116.2, C117.2, C118.2, C119.2, C120.2, C121.2, C125.2, C126.2, C127.2, C129.2, C130.2, C131.2, C140.1, C141.1, C142.1, C144.1, C145.1, C146.1, C148.1, C149.1, C150.1, C151.1, C152.1, C153.1, C154.1, C155.1, C156.1, C157.1, C158.1, C159.1, C160.1, C161.1, C162.1, C163.1, C164.1, C165.1, C29.2, C32.2, C35.2, L1.2, L5.2, L6.2, L7.2, L8.2, R1.1, R87.1, R90.1, R92.1, R94.1, U27.2, U28.2, U29.2, U32.2, U33.2, U34.2, U8.1 (VCC9), U8.13 (VCC13), U8.22 (VCC4), U8.24 (VOUT4), U8.25 (VOUT10), U8.27 (VCC10), U8.28 (VCC6), U8.30 (VOUT6), U8.33 (VCC2), U8.34 (VCC2), U8.37 (VOUT2), U8.41 (VOUT7), U8.43 (VCC7), U8.44 (VCC5), U8.46 (VOUT5), U8.49 (VOUT1), U8.5 (VOUT8), U8.52 (VCC1), U8.53 (VCC1), U8.54 (VCC3), U8.56 (VOUT3), U8.59 (VCC11), U8.64 (VCC12), U8.67 (VOUT9), U8.7 (VCC8), U8.9 (VCC14)
- new net: R55.2, R56.2, U22.2 (VFB)
- new net: C249.2, U22.3 (VREG5)
- new net: C247.1, U22.4 (SS)
- new net: C250.2, L11.1, U22.6 (SW)
- new net: C250.1, U22.7 (VBST)
- new net: C328.1, R87.2, U24.1 (K)
- new net I2C0_SCL_M2: R143.1, R147.1, U20.A3 (SCL), U23.A3 (SCL)
- new net I2C0_SDA_M2: R144.1, R148.1, U20.B1 (SDA), U23.B1 (SDA)
- new net I2C1_SDA_M0: R142.1, U18.B1 (SDA)
- new net SW0_LX: L14.1, U23.D3 (LX), U23.D4 (LX), U23.E3 (LX), U23.E4 (LX)
- new net SW1_LX: L12.1, U18.D3 (LX), U18.D4 (LX), U18.E3 (LX), U18.E4 (LX)
- new net SW2_LX: L13.1, U20.D3 (LX), U20.D4 (LX), U20.E3 (LX), U20.E4 (LX)
- new net VCC2_DDR_S3: C142.1, C146.1, C243.1, C244.1, R92.1, U29.2, U8.30 (VOUT6)
- new net VCCIO: U8.20 (VCCIO)
- new net VCC_1V8_S0: R142.2, R143.2, R144.2, R147.2, R148.2, R97.2
- new net VCC_1V8_S3: C160.1, C161.1, R83.1, R84.1, U32.2, U8.25 (VOUT10)
- new net VCC_2V0_PLDO_S3: C144.1, C145.1, U28.2, U8.41 (VOUT7)
- new net VCC_3V3_S3: C164.1, C165.1, U34.2, U8.5 (VOUT8)
- new net VCC_4V0_SYS: C114.2, C115.2, C116.2, C117.2, C118.2, C119.2, C120.2, C121.2, C125.2, C126.2, C127.2, C129.2, C130.2, C131.2, C262.1, C263.1, C264.1, C266.1, C272.1, C274.1, C29.2, C32.2, C328.2, C335.2, C35.2, L1.2, R1.1, U18.D1 (VIN), U18.D2 (VIN), U18.E1 (VIN), U18.E2 (VIN), U20.D1 (VIN), U20.D2 (VIN), U20.E1 (VIN), U20.E2 (VIN), U23.D1 (VIN), U23.D2 (VIN), U23.E1 (VIN), U23.E2 (VIN), U8.1 (VCC9), U8.13 (VCC13), U8.21 (VCCA), U8.22 (VCC4), U8.27 (VCC10), U8.28 (VCC6), U8.33 (VCC2), U8.34 (VCC2), U8.43 (VCC7), U8.44 (VCC5), U8.52 (VCC1), U8.53 (VCC1), U8.54 (VCC3), U8.59 (VCC11), U8.64 (VCC12), U8.7 (VCC8), U8.9 (VCC14)
- new net VDDQ_DDR_S0: C162.1, C163.1, C254.1, C255.1, C255.2, U33.2, U8.66 (FB9), U8.67 (VOUT9)
- new net VDD_CPU_BIG0_S0: C256.1, C256.2, C257.1, C258.1, C259.1, C260.1, C261.1, L12.2, R145.1, R145.2, U18.A4 (VOUT)
- new net VDD_CPU_BIG1_S0: C265.1, C265.2, C267.1, C268.1, C269.1, C270.1, C271.1, L13.2, R146.1, R146.2, U20.A4 (VOUT)
- new net VDD_CPU_LIT_S0: C154.1, C155.1, C156.1, C233.1, C236.1, L7.2, R90.1
- new net VDD_DDR_S0: C140.1, C141.1, C241.1, C242.1, R114.1, U27.2
- new net VDD_GPU_S0: C157.1, C158.1, C159.1, C234.1, C235.1, C251.2, C252.2, C253.2, L11.2, L8.2, R55.1, R94.1
- new net VDD_LOG_S0: C151.1, C152.1, C153.1, C237.1, C238.1, L6.2, R91.1
- new net VDD_NPU_S0: C273.1, C273.2, C275.1, C276.1, C277.1, C278.1, C279.1, L14.2, R149.1, R149.2, U23.A4 (VOUT)
- new net VDD_VDENC_S0: C148.1, C149.1, C150.1, C239.1, C240.1, L5.2, R95.1
- new net VOUT1: C235.2, R94.2, U8.49 (VOUT1)
- new net VOUT2: C233.2, R90.2, U8.37 (VOUT2)
- new net VOUT3: C238.2, R91.2, U8.56 (VOUT3)
- new net VOUT4: C239.2, R95.2, U8.24 (VOUT4)
- new net VOUT5: C242.2, R114.2, U8.46 (VOUT5)
- no-connect marks 6 -> 8
Other:
- note added: "4V BUCK CONVERTER"
- note added: "5V BUCK CONVERTER FOR GPU"
- note removed: "MAYBE NEEDS 7.4V"
- moved on the sheet: C10, C11, C113, C114, C115, C116, C117, C118, C119, C12, C120, C121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

Commit message: added a USB 3.1 hub for the Type-A ports and a CLK generator for the PCIE 3.0/2.0
Parts:
- added C100, C397, C398, C407, C412, C99: 100nF, Capacitor_SMD:C_0603_1608Metric, symbol Device:C
- added C101, C102, C395, C396, C406, C409, C410, C411: 10uF, Capacitor_SMD:C_0603_1608Metric, symbol Device:C
- added C405, C408: 33nF, Capacitor_SMD:C_0603_1608Metric, symbol Device:C
- added C436: 1uF, Capacitor_SMD:C_0603_1608Metric, symbol Device:C
- added L15, L16: XAL7030-472MEB, XAL7030-472MEB:IND_XAL7030-472MEB, symbol XAL7030-472MEB:XAL7030-472MEB
- added R162, R76: 10k, Resistor_SMD:R_0603_1608Metric, symbol Device:R
- added R163, R75: 31.3k, Resistor_SMD:R_0603_1608Metric, symbol Device:R
- added U14, U15: TPS62933DRLR, barebones:SOTFL50P160X60-8N, symbol TPS62933DRLR:TPS62933DRLR
Connections:
- net PLDO2_RK is gone; now on net VCCA_1V8_S0: C134.2, U8.58 (PLDO2)
- net GND: now also C101.1, C102.1, C395.1, C396.1, C397.1, C398.1, C405.1, C406.1, C407.1, C408.1, C409.1, C410.1, C411.1, C412.1, C436.1, R162.1, R76.1, U14.4 (GND), U15.4 (GND)
- net VCC_2V0_PLDO_S3: now also C126.2, U8.59 (VCC11)
- net VCC_4V0_SYS: no longer C114.2, C119.2, C126.2, U8.13 (VCC13), U8.59 (VCC11), U8.9 (VCC14)
- net VCC_5V0_PERIPH: now also C395.2, C397.2, C406.2, C407.2, U14.3 (VIN), U15.3 (VIN)
- net NLDO1_RK renamed VDD_0V75_S3
- net NLDO2_RK renamed VCCA_DDR_PLL_S0
- net NLDO3_RK renamed VCCA_0V75_S0
- net NLDO4_RK renamed VCCA_0V85_S0
- net NLDO5_RK renamed VDD_0V75_S0
- net PLDO1_RK renamed VCCA_1V8_S0
- net PLDO3_RK renamed VCCA_1V2_S0
- net PLDO4_RK renamed VCCA_3V3_S0
- net PLDO5_RK renamed VCCIO_SD_S0
- net VCCIO renamed VCC_1V8_S3_PLDO6
- net VCC_1V8_S3_PLDO6: now also C436.2
- net VCC_1V8_S3 renamed VCC1V8_PMU_DDR_S3
- new net: R75.2, R76.2, U14.8 (FB)
- new net: C99.2, L15.1, U14.5 (SW)
- new net: C99.1, U14.6 (BST)
- new net: C405.2, U14.7 (SS)
- new net: C100.2, L16.1, U15.5 (SW)
- new net: R162.2, R163.2, U15.8 (FB)
- new net: C408.2, U15.7 (SS)
- new net: C100.1, U15.6 (BST)
- new net PCIE30x4_PWREN_H: U14.2 (EN), U15.2 (EN)
- new net VCC3V3_PCIE30: C101.2, C102.2, C396.2, C398.2, L15.2, R75.1
- new net VCC3V3_PCIE30_1: C409.2, C410.2, C411.2, C412.2, L16.2, R163.1
- new net VCC_1V1_NLDO_S3: C114.2, C119.2, U8.13 (VCC13), U8.9 (VCC14)
- no-connect marks 8 -> 10
Other:
- note added: "VCC1V8_PMU_DDR_S3"

Commit message: added the STM32L433RCT6 to act as the embedded controller
Parts:
- removed C113, C147, C205, C206, C245, C246, C251, C252: 47uF, Capacitor_SMD:C_0603_1608Metric, symbol Device:C
- removed C168, C247: 10nF, Capacitor_SMD:C_0603_1608Metric, symbol Device:C
- removed C192, C207, C248, C250, C253: 0.1uF, Capacitor_SMD:C_0603_1608Metric, symbol Device:C
- removed C249: 1uF, Capacitor_SMD:C_0603_1608Metric, symbol Device:C
- removed L10, L11: XAL7030-472MEB, XAL7030-472MEB:IND_XAL7030-472MEB, symbol XAL7030-472MEB:XAL7030-472MEB
- removed R100, R111, R56: 10k, Resistor_SMD:R_0603_1608Metric, symbol Device:R
- removed R110: 13.3k, Resistor_SMD:R_0603_1608Metric, symbol Device:R
- removed R37: 18k, Resistor_SMD:R_0603_1608Metric, symbol Device:R
- removed R38: 15k, Resistor_SMD:R_0603_1608Metric, symbol Device:R
- removed U22, U40: TPS54628DDAR, barebones:VREG_LM5017MR_NOPB, symbol TPS54628DDAR:TPS54628DDAR
- added C212, C213: 4.7uF, Capacitor_SMD:C_0603_1608Metric, symbol Device:C
- added C214, C216: 0.1uF, Capacitor_SMD:C_0603_1608Metric, symbol Device:C
- added C215: 680pF, Capacitor_SMD:C_0603_1608Metric, symbol Device:C
- added D18: B0530W-7-F, B0530W-7-F:SOD3715X145N, symbol B0530W-7-F:B0530W-7-F
- added L18: LQH5BPN100MT0L, LQH5BPN100MT0L:IND_LQH5BPN100MT0L, symbol LQH5BPN100MT0L:LQH5BPN100MT0L
- added R118, R119: 10k, Resistor_SMD:R_0603_1608Metric, symbol Device:R
- added R73: 87.6k, Resistor_SMD:R_0603_1608Metric, symbol Device:R
- added U47: TPS61170DRVR, TPS61170DRVR:SON65P200X200X80-7N, symbol TPS61170DRVR:TPS61170DRVR
- C190: value 0.1uF -> 0.47uF
- C191: value 1uF -> 33uF
- R18: value 33.2k -> 56k
- R55: value 56k -> 10k
Connections:
- net CMPIN_EC is gone; now on net GND: U11.14 (CMPIN)
- net GND: now also R55.1, C212.1, C213.1, C214.1, C215.1, C216.1, R118.1, U47.3 (GND), U47.7 (THERMALPAD)
- net VCC_3V3_ALW: now also C191.2, U41.3 (OUT); no longer C181.2, C182.2, C183.2, L9.2, R18.1
- net VDD_GPU_S0: no longer R55.1
- net VSYS_MAIN: now also C212.2, C214.2, U47.5 (CTRL), U47.6 (VIN); no longer C190.2
- net at R55.2: now also R18.2, U39.2 (VFB)
- net VCC_5V0_ALW: now reaches U41.1 (IN)
- net VCC_5V0_ALW: now also C181.2, C182.2, C183.2, C190.2, L9.2, R18.1
- net BUCK_5V_PWRON renamed BUCK_PWRON
- net CMPOUT_EC: no longer names the net of U11.15 (CMPOUT)
- net PCIE30x4_PWREN_H renamed PCIE30X4_PWREN_H
- new net: L18.1, R118.2, R73.2, U47.1 (FB)
- new net: C215.2, R119.1
- new net: R119.2, U47.2 (COMP)
- new net EDP_SW: D18.A, L18.2, U47.4 (SW)
- new net VCC_12V_EDP: C213.2, C216.2, D18.C, R73.1
- no-connect marks 10 -> 11
Other:
- note added: "3V3 LDO FOR EC"
- note added: "5V BUCK CONVERTER FOR EC"
- note added: "REMOVE ALL USES OF VCC_1V8_SYS"
- note removed: "1V8 BUCK CONVERTER"
- note removed: "3V3 BUCK CONVERTER FOR EC"
- note removed: "5V BUCK CONVERTER FOR GPU"
- note removed: "VCC1V8_PMU_DDR_S3"
- moved on the sheet: C100, C101, C102, C12, C15, C175, C176, C177, C178, C179, C18, C180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

Commit message: added the display connector and its 12V power supply
Parts:
- added C360, C361: 1uF, Capacitor_SMD:C_0201_0603Metric, symbol Device:C
- added C362: 220nF, Capacitor_SMD:C_0201_0603Metric, symbol Device:C
- added D4: B0530W-7-F, B0530W-7-F:SOD3715X145N, symbol B0530W-7-F:B0530W-7-F
- added L15: LQH32PH220MNCL, LQH32PH220MNCL:IND_LQH32PH220MNCL, symbol LQH32PH220MNCL:LQH32PH220MNCL
- added R115: 10R, Resistor_SMD:R_0603_1608Metric, symbol Device:R
- added U28: TPS61160ADRVT, TPS61160ADRVT:SON65P200X200X80-7N, symbol TPS61160ADRVT:TPS61160ADRVT
- renumbered C8 to C165, C25 to C166, C240 to C167, C148 to C168, C149 to C169, C150 to C170, C241 to C171, C140 to C172, C141 to C173, C239 to C174, C242 to C175, C244 to C176, C146 to C177, C142 to C178, C243 to C179, C26 to C180, C22 to C181, C115 to C182, C335 to C183, C38 to C184, C39 to C185, C328 to C186, C144 to C187, C145 to C188, C9 to C189, C24 to C190, C116 to C191, C160 to C192, C161 to C193, C331 to C194, C28 to C195, C27 to C196, C117 to C197, C23 to C198, C237 to C199, C151 to C200, C152 to C201, C153 to C202, C238 to C203, C255 to C204, C139 to C205, C118 to C206, C162 to C207, C163 to C208, C254 to C209, C138 to C210, C114 to C211, C233 to C212, C236 to C213, C154 to C214, C155 to C215, C156 to C216, C124 to C217, C164 to C218, C165 to C219, C57 to C220, C58 to C221, C59 to C222, C60 to C223, C63 to C224, C64 to C225, C65 to C226, C61 to C227, C62 to C228, C119 to C229, C123 to C230, C52 to C231, C53 to C232, C130 to C233, C133 to C234, C51 to C235, C120 to C236, C67 to C237, C74 to C238, C122 to C239, C55 to C240, C56 to C241, C46 to C242, C54 to C243, C131 to C244, C134 to C245, C159 to C246, C158 to C247, C157 to C248, C234 to C249, C235 to C250, C49 to C251, C121 to C252, C50 to C253, C66 to C254, C69 to C255, C70 to C256, C72 to C257, C73 to C258, C75 to C259, C77 to C260, C79 to C261, C81 to C262, C436 to C263, C47 to C264, C135 to C265, C287 to C266, C129 to C267, C80 to C268, C82 to C269, C136 to C270, C125 to C271, C48 to C272, C71 to C273, C68 to C274, C76 to C275, C78 to C276, C137 to C277, C126 to C278, C127 to C279, C42 to C280, C44 to C281, C41 to C282, C40 to C283, C273 to C284, C275 to C285, C276 to C286, C277 to C287, C278 to C288, C279 to C289, C43 to C290, C45 to C291, C272 to C292, C274 to C293, C256 to C294, C257 to C295, C258 to C296, C259 to C297, C260 to C298, C261 to C299, C262 to C300, C263 to C301, C19 to C302, C99 to C303, C10 to C304, C29 to C305, C32 to C306, C35 to C307, C395 to C308, C397 to C309, C101 to C310, C102 to C311, C396 to C312, C398 to C313, C16 to C314, C265 to C315, C267 to C316, C268 to C317, C269 to C318, C270 to C319, C271 to C320, C405 to C321, C2 to C322, C5 to C323, C13 to C324, C264 to C325, C266 to C326, C100 to C327, C20 to C328, C406 to C329, C407 to C330, C11 to C331, C30 to C332, C33 to C333, C36 to C334, C409 to C335, C410 to C336, C411 to C337, C412 to C338, C17 to C339, C408 to C340, C3 to C341, C6 to C342, C14 to C343, C180 to C344, C177 to C345, C181 to C346, C182 to C347, C183 to C348, C179 to C349, C175 to C350, C176 to C351, C178 to C352, C213 to C353, C216 to C354, C215 to C355, C212 to C356, C214 to C357, C191 to C358, C190 to C359, C21 to C363, C12 to C364, C31 to C365, C34 to C366, C37 to C367, C18 to C368, C4 to C369, C7 to C370, C15 to C371, D18 to D3, L5 to L1, L13 to L10, L16 to L11, L2 to L12, L9 to L13, L18 to L14, L3 to L16, L6 to L2, L7 to L3, L8 to L5, L14 to L6, L12 to L7, L1 to L8, L15 to L9, Q2 to Q1, Q3 to Q2, Q1 to Q3, R4 to R100, R75 to R101, R143 to R102, R144 to R103, R76 to R104, R146 to R105, R2 to R106, R5 to R107, R163 to R108, R162 to R109, R18 to R110, R55 to R111, R73 to R112, R118 to R113, R119 to R114, R3 to R116, R6 to R117, R95 to R32, R114 to R33, R92 to R34, R7 to R35, R8 to R36, R93 to R37, R9 to R38, R15 to R39, R10 to R40, R87 to R41, R11 to R42, R12 to R43, R88 to R44, R17 to R45, R13 to R46, R16 to R47, R14 to R48, R91 to R49, R90 to R50, R35 to R52, R36 to R53, R43 to R54, R48 to R55, R44 to R56, R50 to R57, R86 to R58, R39 to R59, R94 to R60, R83 to R61, R84 to R62, R85 to R63, R40 to R64, R34 to R65, R47 to R66, R41 to R67, R53 to R68, R45 to R69, R46 to R70, R49 to R71, R42 to R72, R52 to R73, R54 to R74, R99 to R75, R98 to R76, R26 to R77, R29 to R78, R24 to R79, R30 to R80, R19 to R81, R22 to R82, R21 to R83, R27 to R84, R25 to R85, R28 to R86, R23 to R87, R147 to R88, R148 to R89, R20 to R90, R31 to R91, R149 to R92, R80 to R93, R32 to R94, R33 to R95, R97 to R96, R142 to R97, R145 to R98, R1 to R99, U6 to U10, U33 to U11, U8 to U12, U34 to U13, U11 to U14, U36 to U15, U35 to U16, U9 to U17, U23 to U18, U18 to U19, U27 to U2, U2 to U20, U14 to U21, U20 to U22, U15 to U23, U3 to U24, U39 to U25, U47 to U26, U41 to U27, U4 to U29, U29 to U3, U5 to U4, U28 to U5, U32 to U6, U37 to U7, U7 to U8, U24 to U9
Connections:
- net GND: now also C360.1, C361.1, C362.1, R115.2, U28.3 (GND), U28.7 (THERMALPAD)
- new net: C362.2, U28.2 (COMP)
- new net BACKLIGHT_DN: R115.1, U28.1 (FB)
- new net BACKLIGHT_DP: C361.2, D4.C
- new net BACKLIGHT_PWM: U28.5 (CTRL)
- new net PWM_SW: D4.A, L15.2, U28.4 (SW)
- new net PWM_VIN: C360.2, L15.1, U28.6 (VIN)
Other:
- moved on the sheet: C355, R114

Commit message: added the PCF85063ATL/1,118 CMOS Real-Time Clock
Parts:
- removed R75, R76: 100k, Resistor_SMD:R_0603_1608Metric, symbol Device:R
- removed TP1: RESETB, TestPoint:TestPoint_Pad_D1.5mm, symbol Connector:TestPoint
- removed TP2, TP4: GND, TestPoint:TestPoint_Pad_D1.5mm, symbol Connector:TestPoint
- removed TP3: POWER ON, TestPoint:TestPoint_Pad_D1.5mm, symbol Connector:TestPoint
- removed U15, U16: 2N7002KW, barebones:SOT323, symbol 2N7002KW:2N7002KW
Connections:
- net GND: no longer U18.A1 (VSEL), U19.A1 (VSEL)
- net INT_PMIC: no longer U12.19 (INT)
- net SPI_CS_PMIC: no longer U12.18 (CS)
- net SPI_MOSI_PMIC: no longer U12.15 (MOSI/SDA)
- net PWRCTRL1_PMIC renamed PMIC_SLEEP1
- net PWRON_RK renamed PWRON
- net SPI_CLK_PMIC renamed SPI2_CLK_M2
- new net CPU_BIG0_VSEL: U19.A1 (VSEL)
- new net NPU_VSEL: U18.A1 (VSEL)
- new net PMIC_INT_L: U12.19 (INT)
- new net SPI2_CS0_M2: U12.18 (CS)
- new net SPI2_MOSI_M2: U12.15 (MOSI/SDA)
Other:
- note added: "CPU_BIG0_VSEL"

Commit message: updated the Fuel Guage/BMS module for the 4S battery usage
Parts:
- removed C242: 4.7nF, Capacitor_SMD:C_0201_0603Metric, symbol Device:C
- removed C251: 33pF, Capacitor_SMD:C_0201_0603Metric, symbol Device:C
- removed C253: 15pF, Capacitor_SMD:C_0201_0603Metric, symbol Device:C
- removed C264: 680pF, Capacitor_SMD:C_0201_0603Metric, symbol Device:C
- removed C280, C281, C283, C290: 0.1uF, Capacitor_SMD:C_0201_0603Metric, symbol Device:C
- removed C282: 2.2uF, Capacitor_SMD:C_0201_0603Metric, symbol Device:C
- removed C291: 1uF, Capacitor_SMD:C_0201_0603Metric, symbol Device:C
- removed D1: MMSZ5V6T1G, barebones:MMSZ5V6T1G, symbol MMSZ5V6T1G:MMSZ5V6T1G
- removed Q3: STL40DN3LLH5, barebones:TRANS_STL40DN3LLH5, symbol STL40DN3LLH5:STL40DN3LLH5
- removed R59: 40.2k, Resistor_SMD:R_0603_1608Metric, symbol Device:R
- removed R64: 15k, Resistor_SMD:R_0603_1608Metric, symbol Device:R
- removed R77, R78: 10M, Resistor_SMD:R_0603_1608Metric, symbol Device:R
- removed R79, R81: 5.1k, Resistor_SMD:R_0603_1608Metric, symbol Device:R
- removed R80: FUSE, Resistor_SMD:R_0603_1608Metric, symbol Device:R
- removed R82: 10, Resistor_SMD:R_0603_1608Metric, symbol Device:R
- removed R83, R84, R85, R86, R87, R90, R95: 100, Resistor_SMD:R_0603_1608Metric, symbol Device:R
- removed R91: THERM, Resistor_SMD:R_0603_1608Metric, symbol Device:R
- removed R93: WSL25122L000FEA, barebones:RES_WSL25122L000FEA, symbol WSL25122L000FEA:WSL25122L000FEA
- added C540, C561, C562, C563, C564, C565, C567, C568: 0.1uF, Capacitor_SMD:C_0402_1005Metric, symbol Device:C
- added C556: 4.7nF, Capacitor_SMD:C_0402_1005Metric, symbol Device:C
- added C557: 680pF, Capacitor_SMD:C_0402_1005Metric, symbol Device:C
- added C558: 15pF, Capacitor_SMD:C_0402_1005Metric, symbol Device:C
- added C559: 33pF, Capacitor_SMD:C_0402_1005Metric, symbol Device:C
- added C566: 2.2uF, Capacitor_SMD:C_0402_1005Metric, symbol Device:C
- added D21: 1N4148W, Diode_SMD:D_SOD-123, symbol Diode:1N4148W
- added J21: SM02B-GHS-TB_LF__SN_, barebones:JST_SM02B-GHS-TB_LF__SN_, symbol SM02B-GHS-TB_LF__SN_:SM02B-GHS-TB_LF__SN_
- added J23: 874381343, barebones:MOLEX_874381343, symbol 874381343:874381343
- added PAD0: NEUTRAL, barebones:7x10-PAD, symbol Connector:TestPoint
- added PAD1: BATT_1P, barebones:7x10-PAD, symbol Connector:TestPoint
- added PAD2: BATT_2P, barebones:7x10-PAD, symbol Connector:TestPoint
- added PAD3: BATT_3P, barebones:7x10-PAD, symbol Connector:TestPoint
- added PAD4: BATT_4P, barebones:7x10-PAD, symbol Connector:TestPoint
- added PAD5: BATT_4N, barebones:7x10-PAD, symbol Connector:TestPoint
- added PAD6: BATT_3N, barebones:7x10-PAD, symbol Connector:TestPoint
- added PAD7: BATT_2N, barebones:7x10-PAD, symbol Connector:TestPoint
- added Q3: AO3401A, Package_TO_SOT_SMD:SOT-23, symbol Transistor_FET:AO3401A
- added Q5, Q6: CSD18504Q5A, barebones:MOSFET_CSD19531Q5A, symbol CSD18504Q5A:CSD18504Q5A
- added R225, R93: 5.1k, Resistor_SMD:R_0402_1005Metric, symbol Device:R
- added R226: 100R, Resistor_SMD:R_0402_1005Metric, symbol Device:R
- added R236, R237, R238, R239, R241, R243, R245, R246, R247: 100, Resistor_SMD:R_0402_1005Metric, symbol Device:R
- added R240: 300, Resistor_SMD:R_0402_1005Metric, symbol Device:R
- added R242, R244, R248: 10M, Resistor_SMD:R_0402_1005Metric, symbol Device:R
- added R59: WSL25122L000FEA, barebones:RES_WSL25122L000FEA, symbol WSL25122L000FEA:WSL25122L000FEA
- added R75: 40.2k, Resistor_SMD:R_0402_1005Metric, symbol Device:R
- added R76: 15k, Resistor_SMD:R_0402_1005Metric, symbol Device:R
- added TP11: SMBD, TestPoint:TestPoint_Pad_D1.0mm, symbol Connector:TestPoint
- added TP12: SMBC, TestPoint:TestPoint_Pad_D1.0mm, symbol Connector:TestPoint
- added TP13: GND, TestPoint:TestPoint_Pad_D1.0mm, symbol Connector:TestPoint
- added U15: BQ78350DBTR-R1, barebones:SOP50P640X120-30N, symbol BQ78350DBTR-R1:BQ78350DBTR-R1
- added U16: BQ7692000PW, barebones:SOP65P640X120-20N, symbol BQ7692000PW:BQ7692000PW
- added U73: BQ40Z50RSMR-R2, barebones:QFN40P400X400X100-33N, symbol BQ40Z50RSMR-R2:BQ40Z50RSMR-R2
- added U74: TPD4E004DRYR, barebones:PSON50P145X100X60-6N, symbol TPD4E004DRYR:TPD4E004DRYR
- added U77, U78, U79, U80: NXFT15XH103FA2B025, barebones:NXFT15XH103FA2B025, symbol NXFT15XH103FA2B025:NXFT15XH103FA2B025
- C165, C166, C180, C181, C184, C185, C189, C190, C195, C196, C198, C220, C221, C222, C223, C224, C225, C226, C227, C228, C231, C232, C235, C237, C238, C240, C241, C243, C254, C255, C256, C257, C258, C259, C260, C261, C262, C268, C269, C272, C273, C274, C275, C276, C360, C361, C362: footprint Capacitor_SMD:C_0201_0603Metric -> Capacitor_SMD:C_0402_1005Metric; KiLib_Generator (none) -> SMD_2terminal_chip_molded
- C167, C168, C169, C170, C171, C172, C173, C174, C175, C176, C177, C178, C179, C182, C183, C186, C187, C188, C191, C192, C193, C194, C197, C199, C200, C201, C202, C203, C204, C205, C206, C207, C208, C209, C210, C211, C212, C213, C214, C215, C216, C217, C218, C219, C229, C230, C233, C234, C236, C239, C244, C245, C246, C247, C248, C249, C250, C252, C263, C265, C266, C267, C270, C271, C277, C278, C279, C284, C285, C286, C287, C288, C289, C292, C293, C294, C295, C296, C297, C298, C299, C300, C301, C302, C303, C304, C305, C306, C307, C308, C309, C310, C311, C312, C313, C314, C315, C316, C317, C318, C319, C320, C321, C322, C323, C324, C325, C326, C327, C328, C329, C330, C331, C332, C333, C334, C335, C336, C337, C338, C339, C340, C341, C342, C343, C344, C345, C346, C347, C348, C349, C350, C351, C352, C353, C354, C355, C356, C357, C358, C359, C363, C364, C365, C366, C367, C368, C369, C370, C371: footprint Capacitor_SMD:C_0603_1608Metric -> Capacitor_SMD:C_0402_1005Metric; KiLib_Generator (none) -> SMD_2terminal_chip_molded
- R100, R101, R102, R103, R104, R105, R106, R107, R108, R109, R110, R111, R112, R113, R114, R115, R116, R117, R32, R33, R34, R35, R36, R37, R38, R39, R40, R41, R42, R43, R44, R45, R46, R47, R48, R49, R50, R52, R53, R54, R55, R56, R57, R58, R60, R61, R62, R63, R65, R66, R67, R69, R70, R71, R72, R73, R74, R88, R89, R92, R96, R97, R98, R99: footprint Resistor_SMD:R_0603_1608Metric -> Resistor_SMD:R_0402_1005Metric; KiLib_Generator (none) -> SMD_2terminal_chip_molded
- R94: value 100 -> 5.1k; footprint Resistor_SMD:R_0603_1608Metric -> Resistor_SMD:R_0402_1005Metric; KiLib_Generator (none) -> SMD_2terminal_chip_molded
Connections:
- net COMP1: now also C559.1, R75.2
- net COMP2: now also C558.1, R76.1
- net GND: now also C540.1, C556.2, C557.2, C558.2, C559.2, C564.1, C566.1, J21.2, PAD0.1, R243.2, R59.1, TP13.1, U73.14 (NC), U73.17 (~{DISP}), U73.23 (PTC), U73.24 (PTCEN), U73.29 (NC), U73.33 (EXP), U73.33_1 (EXP), U73.7 (NC), U73.9 (VSS), U74.3 (GND), U77.P$1, U78.P$1, U79.P$1, U80.P$1; no longer D2.A
- net TS1: now also U73.10 (TS1), U78.P$2; no longer U17.4 (T81)
- net VC1: now also C562.1, C564.2, R239.1, U73.5 (VC1); no longer R94.2, U17.12 (VC1)
- net VC2: now also C562.2, C563.1, R238.1, U73.4 (VC2); no longer U17.11 (VC2)
- net VCCA_1V8_S0: no longer C245.2, U12.58 (PLDO2)
- net VCC_1V8_S0: now also C245.2, U12.58 (PLDO2)
- net IBAT: now reaches C240.1, U14.9 (IBAT)
- net ACN: now reaches C235.2, R56.1, U14.2 (ACN)
- net ACP: now reaches C231.2, C232.2, C235.1, R54.1, U14.3 (ACP)
- net BATT-: no longer names the net of U17.1 (VSS)
- net BATT-: no longer U17.13 (PWPD)
- net BATT_NEUTRAL renamed PCHG
- net PCHG: now also U73.30 (PCHG)
- net CHARGE_CNTRL renamed CHRG_CTRL
- net VCCA_1V2_S0 renamed VDDA_1V2_S0
- new net: C566.2, U73.1 (PBI)
- new net: R247.1, U73.16 (~{PRES}/~{SHUTDN})
- new net: R245.2, U73.18 (SMBD)
- new net: R246.2, U73.19 (SMBC)
- new net: Q5.4, R242.1, R93.2
- new net: Q3.2 (S), Q5.5, Q5.6, Q5.7, Q5.8, Q6.5, Q6.6, Q6.7, Q6.8, R226.2
- new net: C557.1, R76.2
- new net: C556.1, R75.1
- new net: Q3.1 (G), R248.1, R94.2
- new net: Q6.4, R225.2, R244.1
- new net: J23.5_1 (5), J23.5_2 (5)
- new net: J23.9_1 (9), J23.9_2 (9)
- new net: C567.2, C568.1
- new net: Q3.3 (D), R240.1
- new net BAT: D21.1 (K), U73.32 (BAT)
- new net BATT_1P: PAD1.1, PAD7.1, R239.2
- new net BATT_2P: PAD2.1, PAD6.1, R238.2
- new net BATT_3P: PAD3.1, PAD5.1, R237.2
- new net BATT_4P: C568.2, D21.2 (A), PAD4.1, Q5.1, Q5.2, Q5.3, R236.2, R240.2, R242.2
- new net BATT_PRES: J23.6_1 (6), J23.6_2 (6), R247.2, U74.1
- new net CHG: R93.1, U73.31 (CHG)
- new net DSG: R225.1, U73.28 (DSG)
- new net PACK_N: J23.10_1 (10), J23.10_2 (10), J23.11_1 (11), J23.11_2 (11), J23.12_1 (12), J23.12_2 (12), J23.13_1 (13), J23.13_2 (13), R241.2, R59.2
- new net PACK_P: C567.1, J23.1_1 (1), J23.1_2 (1), J23.2_1 (2), J23.2_2 (2), J23.3_1 (3), J23.3_2 (3), J23.4_1 (4), J23.4_2 (4), Q6.1, Q6.2, Q6.3, R244.2, U73.27 (PACK)
- new net SMBC_BATT: J23.8_1 (8), J23.8_2 (8), R246.1, TP12.1, U74.5
- new net SMBD_BATT: J23.7_1 (7), J23.7_2 (7), R245.1, TP11.1, U74.4
- new net SRN_BATT: C565.1, R241.1, U73.6 (SRN)
- new net SRP_BATT: C565.2, R243.1, U73.8 (SRP)
- new net TS2: U73.11 (TS2), U79.P$2
- new net TS3: U73.12 (TS3), U80.P$2
- new net TS4: U73.13 (TS4), U77.P$2
- new net VC3: C561.1, C563.2, R237.1, U73.3 (VC3)
- new net VC4: C561.2, R236.1, U73.2 (VC4)
- new net VCC: R226.1, R248.2, U73.26 (VCC)
- new net V_BAT_CMOS: C540.2, J21.1
- no-connect marks 11 -> 19
Other:
- note added: "CMOS BATTERY"
- note removed: "REPLACE WITH FUSE"
- note removed: "REPLACE WITH THERMISTOR"
- note removed: "TO EMBEDDED CONTROLLER"
- moved on the sheet: C165, C166, C180, C181, C220, C221, C222, C223, C224, C225, C226, C227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
