File: hardware/motherboard/barebones.kicad_pcb (KiCad board)
At the start: 2 copper layers, 217 x 22.5 mm, 884 parts, among them IC1 W25Q80DVSSIG, IC2 FUSB302BMPX, IC3 W25Q80DVSSIG, IC4 FUSB302BMPX, J1 12401610E4_2A, J10 54-00007, J11 54-00007, J13 SM02B-GHS-TB_LF__SN_, J16 524352671, J17 522070485, J18 G45AA1912100B1EU, J2 1-2199119-5, J21 SM02B-GHS-TB_LF__SN_, J22 SJ2-35894B-SMT-TR, J23 874381343, J3 1-2199119-5, J4 21992304, J5 12401610E4_2A, J6 SJ2-35894B-SMT-TR, J8 SM02B-GHS-TB_LF__SN_, J9 1040310811, Q1 STL40DN3LLH5, Q2 STL40DN3LLH5, Q3 AO3401A, Q5 CSD18504Q5A, Q6 CSD18504Q5A, U1 RK3588, U10 TPS259474ARPWR, U12 RK806-1_C5156483, U14 BQ25731RSNR, U15 BQ78350DBTR-R1, U16 BQ7692000PW, U17 BQ28Z610DRZR, U18 RK860-2, U19 RK860-2, U20 TPS54628DDAR, U21 TPS62933DRLR, U23 TPS62933DRLR, U24 TPS54628DDAR, U25 TPS54628DDAR, U29 TPS54628DDAR, U30 W25Q256JWEIQ, U31 PCF85063ATL/1,118, U32 K4UCE3Q4AA-MGCL, U33 K4UCE3Q4AA-MGCL, U34 ES8316, U36 PCA9306DCTR, U37 TPA2012D2RTJT, U39 TPS65987DDHRSHR, U4 TPS259474ARPWR, U40 TXS0104EYZTR, U41 TPD4E004DRYR, U42 PCA9306DCTR, U43 9FGV0641AKILFT, U44 TPD4E05U06DQAR, U45 GL3523-ONY30, U46 TXS0104EYZTR, U47 TPS2553DBVR, U48 PI3DPX1207Q3ZHEX, U49 TPS65987DDHRSHR, U50 TXS0104EYZTR, U51 PCA9306DCTR, U53 TPS2553DBVR, U54 TPD4E004DRYR, U55 PI6C557-05BLEX, U58 TPS2553DBVR, U59 TPD4E004DRYR, U60 TPD4E004DRYR, U61 PCA9306DCTR, U7 LP5912-1.8DRVT, U72 PCA9306DCTR, U73 BQ40Z50RSMR-R2, U77 NXFT15XH103FA2B025, U78 NXFT15XH103FA2B025, U79 NXFT15XH103FA2B025, U8 TPS2121RUXR, U80 NXFT15XH103FA2B025, Y1 C3E-24.000-12-3030-X-R, Y3 C2E-25.000-10-1530-X-R, Y4 C2E-25.000-10-1530-X-R

Commit message: updated last changes
Parts:
- removed C100, C104, C107, C111, C14, C385, C391, C484, C59, C61, C63, C96, C98: 1uF, Capacitor_SMD:C_0201_0603Metric
- removed C103, C106, C112, C94: 4.7uF, Capacitor_SMD:C_0201_0603Metric
- removed C105, C108, C13, C381, C386, C387, C392, C393, C394, C48, C55, C57, C67, C69, C71, C88, C97, C99: 100nF, Capacitor_SMD:C_0201_0603Metric
- removed C113, C116, C118, C119, C120, C121, C149, C150, C156, C157, C383, C384, C389, C390, C93: 10uF, Capacitor_SMD:C_0201_0603Metric
- removed C117, C382, C388: 22uF, Capacitor_SMD:C_0201_0603Metric
- removed C311, C312: 10uF, Capacitor_SMD:C_0402_1005Metric
- removed C313: 100nF, Capacitor_SMD:C_0402_1005Metric
- removed C324, C363: 0.1uF, Capacitor_SMD:C_0402_1005Metric
- removed C333: 47uF, Capacitor_SMD:C_0402_1005Metric
- removed C340: 33nF, Capacitor_SMD:C_0402_1005Metric
- removed C364: 10nF, Capacitor_SMD:C_0402_1005Metric
- removed C397, C406: 100nF, Capacitor_SMD:C_0603_1608Metric
- removed C398: 10uF, Capacitor_SMD:C_0603_1608Metric
- removed C480, C481, C483, C485, C487, C490, C493, C494, C496, C498, C506, C515, C516, C517, C75: 0.1uF, Capacitor_SMD:C_0201_0603Metric
- removed C505, C514: 100uF, Capacitor_SMD:C_0201_0603Metric
- removed C519, C520: 220pF, Capacitor_SMD:C_0201_0603Metric
- removed C56, C58, C68, C70: 4.7F, Capacitor_SMD:C_0201_0603Metric
- removed D2: MMSZ5V6T1G, barebones:MMSZ5V6T1G
- removed D21: 1N4148W, Diode_SMD:D_SOD-123
- removed FPC1: FH12-6S-0.5SH, barebones:FPC-SMD_FH12-6S-0.5SH-55
- removed IC1, IC3: W25Q80DVSSIG, barebones:SOIC8-FLASH
- removed IC2, IC4: FUSB302BMPX, barebones:QFN50P250X250X80-15N
- removed J13, J21: SM02B-GHS-TB_LF__SN_, barebones:JST_SM02B-GHS-TB_LF__SN_
- removed J22: SJ2-35894B-SMT-TR, barebones:CUI_SJ2-35894B-SMT-TR
- removed J23: 874381343, barebones:MOLEX_874381343
- removed L5: 0.22uH, Inductor_SMD:L_0805_2012Metric
- removed NT1, NT2, NT3, NT4: NetTie_2, NetTie:NetTie-2_SMD_Pad0.5mm
- removed PAD0: NEUTRAL, barebones:7x10-PAD
- removed PAD1: BATT_1P, barebones:7x10-PAD
- removed PAD2: BATT_2P, barebones:7x10-PAD
- removed PAD3: BATT_3P, barebones:7x10-PAD
- removed PAD4: BATT_4P, barebones:7x10-PAD
- removed PAD5: BATT_4N, barebones:7x10-PAD
- removed PAD6: BATT_3N, barebones:7x10-PAD
- removed PAD7: BATT_2N, barebones:7x10-PAD
- removed Q5, Q6: CSD18504Q5A, barebones:MOSFET_CSD19531Q5A
- removed R1, R100, R104, R107, R109, R111, R117, R151, R164, R2, R3, R36, R39, R4, R40, R43, R47, R48, R63, R69, R70, R71: 10k, Resistor_SMD:R_0402_1005Metric
- removed R101, R108: 31.3k, Resistor_SMD:R_0402_1005Metric
- removed R102, R103, R213, R88, R89, R96, R97: 2.2k, Resistor_SMD:R_0402_1005Metric
- removed R105, R98: 100R, Resistor_SMD:R_0402_1005Metric
- removed R106, R110, R99: 56k, Resistor_SMD:R_0402_1005Metric
- removed R116: 33.2k, Resistor_SMD:R_0402_1005Metric
- removed R122, R123, R124, R125, R26: 200R, Resistor_SMD:R_0402_1005Metric
- removed R129: 330k, Resistor_SMD:R_0603_1608Metric
- removed R130: 10k, Resistor_SMD:R_0603_1608Metric
- removed R150: 4.7k, Resistor_SMD:R_0402_1005Metric
- removed R196, R197: 1k, Resistor_SMD:R_0402_1005Metric
- removed R202: 1.8k, Resistor_SMD:R_0402_1005Metric
- removed R38, R46: 174k, Resistor_SMD:R_0402_1005Metric
- removed R42: 27.4k, Resistor_SMD:R_0402_1005Metric
- removed R59: WSL25122L000FEA, barebones:RES_WSL25122L000FEA
- removed TP10: MISO, TestPoint:TestPoint_Pad_D1.5mm
- removed TP11: SMBD, TestPoint:TestPoint_Pad_D1.0mm
- removed TP12: SMBC, TestPoint:TestPoint_Pad_D1.0mm
- removed TP13: GND, TestPoint:TestPoint_Pad_D1.0mm
- removed TP9: MOSI, TestPoint:TestPoint_Pad_D1.5mm
- removed U21, U23: TPS62933DRLR, barebones:SOTFL50P160X60-8N
- removed U24, U25, U29: TPS54628DDAR, barebones:VREG_LM5017MR_NOPB
- removed U39, U49: TPS65987DDHRSHR, barebones:IC_TPS65987DDHRSHR
- removed U40, U46, U50: TXS0104EYZTR, barebones:BGA12N50P4X3_186X136X62N
- removed U42, U51, U61, U72: PCA9306DCTR, barebones:SOP65P400X130-8N
- removed U44: TPD4E05U06DQAR, barebones:IC_TPD4E05U06DQAR
- removed U45: GL3523-ONY30, barebones:QFN-48_L6.0-W6.0-P0.40-BL-EP3.8
- removed U47, U58: TPS2553DBVR, barebones:SOT95P280X145-6N
- removed U48: PI3DPX1207Q3ZHEX, barebones:QFN50P900X350X84-43N
- removed U55: PI6C557-05BLEX, barebones:TSSOP-20_L6.5-W4.4-P0.65-LS6.4-BL
- removed U59, U60: TPD4E004DRYR, barebones:PSON50P145X100X60-6N
- removed U73: BQ40Z50RSMR-R2, barebones:QFN40P400X400X100-33N
- removed U78, U80: NXFT15XH103FA2B025, barebones:NXFT15XH103FA2B025
- removed Y4: C2E-25.000-10-1530-X-R, barebones:XTAL_C2E-25.000-10-1530-X-R
- added BT1: BK-912-G, barebones:BAT_BK-912-G, F.Cu at (420.4, 209.8)
- added C242: 1uF, Capacitor_SMD:C_0603_1608Metric, F.Cu at (187.7, 98.9)
- added C251: 0.1uF, Capacitor_SMD:C_0603_1608Metric, F.Cu at (188.8, 107.4)
- added C264: 1uF, Capacitor_SMD:C_0201_0603Metric, B.Cu at (301.9, 155.8)
- added C280: 1uF, Capacitor_SMD:C_0201_0603Metric, B.Cu at (310.2, 163.7)
- added C281: 1uF, Capacitor_SMD:C_0201_0603Metric, B.Cu at (312.7, 160.3)
- added C282: 0.1uF, Capacitor_SMD:C_0201_0603Metric, B.Cu at (310.4, 162.1)
- added C283: 0.1uF, Capacitor_SMD:C_0201_0603Metric, B.Cu at (306.3, 160.0)
- added C290: 1uF, Capacitor_SMD:C_0201_0603Metric, B.Cu at (303.9, 171.2)
- added C291: 0.1uF, Capacitor_SMD:C_0201_0603Metric, B.Cu at (303.9, 172.0)
- added C395: 12.5pF, Capacitor_SMD:C_0603_1608Metric, F.Cu at (302.0, 185.9)
- added C546: 1uF, Capacitor_SMD:C_0201_0603Metric, F.Cu at (377.3, 148.6)
- added C547: 10uF, Capacitor_SMD:C_0603_1608Metric, F.Cu at (176.0, 109.7)
- added C548: 10uF, Capacitor_SMD:C_0603_1608Metric, F.Cu at (259.4, 123.8)
- added C549: 1uF, Capacitor_SMD:C_0402_1005Metric, F.Cu at (399.2, 168.9)
- added C550: 0.1uF, Capacitor_SMD:C_0201_0603Metric, F.Cu at (398.9, 170.8)
- added C551: 0.1uF, Capacitor_SMD:C_0201_0603Metric, F.Cu at (398.9, 172.9)
- added C553: 0.1uF, Capacitor_SMD:C_0201_0603Metric, F.Cu at (371.5, 83.2)
- added C554: 10uF, Capacitor_SMD:C_0603_1608Metric, F.Cu at (176.4, 97.6)
- added C555: 20pF, Capacitor_SMD:C_0201_0603Metric, F.Cu at (405.3, 172.0)
- added C560: 0.1uF, Capacitor_SMD:C_0201_0603Metric, F.Cu at (398.9, 175.9)
- added C569: 0.1uF, Capacitor_SMD:C_0201_0603Metric, F.Cu at (226.1, 159.6)
- added C570: 0.1uF, Capacitor_SMD:C_0201_0603Metric, F.Cu at (360.6, 83.3)
- added C571: 0.1uF, Capacitor_SMD:C_0201_0603Metric, F.Cu at (231.6, 164.2)
- added C572: 0.1uF, Capacitor_SMD:C_0201_0603Metric, F.Cu at (226.1, 158.6)
- added C573: 10uF, Capacitor_SMD:C_0603_1608Metric, F.Cu at (425.3, 168.4)
- added C574: 1uF, Capacitor_SMD:C_0402_1005Metric, F.Cu at (447.7, 161.3)
- added C575: 0.1uF, Capacitor_SMD:C_0402_1005Metric, F.Cu at (197.2, 185.9)
- added C576: 22uF, Capacitor_SMD:C_0402_1005Metric, F.Cu at (193.8, 176.9)
- added C577: 10uF, Capacitor_SMD:C_0603_1608Metric, F.Cu at (146.7, 103.9)
- added C578: 10uF, Capacitor_SMD:C_0603_1608Metric, F.Cu at (131.8, 102.6)
- added C579: 22uF, Capacitor_SMD:C_0603_1608Metric, F.Cu at (140.8, 108.3)
- added C580: 22uF, Capacitor_SMD:C_0603_1608Metric, F.Cu at (140.8, 96.6)
- added C581: 0.1uF, Capacitor_SMD:C_0201_0603Metric, B.Cu at (282.6, 165.9)
- added C582: 22uF, Capacitor_SMD:C_0603_1608Metric, F.Cu at (131.8, 106.1)
- added C583: 1uF, Capacitor_SMD:C_0402_1005Metric, F.Cu at (168.7, 112.6)
- added C584: 0.1uF, Capacitor_SMD:C_0402_1005Metric, F.Cu at (162.5, 111.0)
- added C585: 10uF, Capacitor_SMD:C_0603_1608Metric, F.Cu at (174.7, 97.6)
- added C586: 0.1uF, Capacitor_SMD:C_0402_1005Metric, F.Cu at (173.2, 97.0)
- added C587: 1uF, Capacitor_SMD:C_0402_1005Metric, F.Cu at (166.8, 100.4)
- added C588: 0.1uF, Capacitor_SMD:C_0402_1005Metric, F.Cu at (162.6, 98.4)
- added C589: 22uF, Capacitor_SMD:C_0402_1005Metric, F.Cu at (196.4, 176.9)
- added C590: 1uF, Capacitor_SMD:C_0201_0603Metric, F.Cu at (447.3, 86.4)
- added C591: 33nF, Capacitor_SMD:C_0201_0603Metric, F.Cu at (194.3, 183.0)
- added C592: 100nF, Capacitor_SMD:C_0402_1005Metric, F.Cu at (187.2, 170.7)
- added C593: 10uF, Capacitor_SMD:C_0402_1005Metric, F.Cu at (187.2, 171.8)
- added C594: 100nF, Capacitor_SMD:C_0402_1005Metric, F.Cu at (187.2, 175.3)
- added C595: 12pF, Capacitor_SMD:C_0402_1005Metric, F.Cu at (224.1, 154.3)
- added C596: 12pF, Capacitor_SMD:C_0402_1005Metric, F.Cu at (223.4, 149.9)
- added C597: 100nF, Capacitor_SMD:C_0402_1005Metric, F.Cu at (187.2, 173.0)
- added C598: 10uF, Capacitor_SMD:C_0402_1005Metric, F.Cu at (187.2, 174.1)
- added C599: 100nF, Capacitor_SMD:C_0402_1005Metric, F.Cu at (187.2, 201.0)
- added C600: 100nF, Capacitor_SMD:C_0402_1005Metric, F.Cu at (187.2, 206.7)
- added C601: 22uF, Capacitor_SMD:C_0603_1608Metric, F.Cu at (131.8, 97.3)
- added C602: 12pF, Capacitor_SMD:C_0201_0603Metric, B.Cu at (381.7, 128.2)
- added C603: 0.1uF, Capacitor_SMD:C_0402_1005Metric, F.Cu at (193.7, 219.7)
- added C604: 10uF, Capacitor_SMD:C_0402_1005Metric, F.Cu at (195.9, 219.7)
- added C605: 0.1uF, Capacitor_SMD:C_0201_0603Metric, F.Cu at (145.3, 98.7)
- added C606: 100nF, Capacitor_SMD:C_0402_1005Metric, F.Cu at (187.2, 202.1)
- added C607: 0.1uF, Capacitor_SMD:C_0402_1005Metric, F.Cu at (130.7, 125.7)
- added C608: 10uF, Capacitor_SMD:C_0402_1005Metric, F.Cu at (130.7, 126.9)
- added C609: 120uF, Capacitor_SMD:C_0402_1005Metric, F.Cu at (138.5, 126.8)
- added C610: 10uF, Capacitor_SMD:C_0402_1005Metric, F.Cu at (427.3, 135.1)
- added C611: 0.1uF, Capacitor_SMD:C_0402_1005Metric, F.Cu at (427.3, 136.2)
- added C612: 120uF, Capacitor_SMD:C_0402_1005Metric, F.Cu at (433.9, 135.1)
- added C613: 0.1uF, Capacitor_SMD:C_0201_0603Metric, F.Cu at (361.5, 83.3)
- added C614: 4.7uF, Capacitor_SMD:C_0402_1005Metric, F.Cu at (362.5, 83.5)
- added C615: 1uF, Capacitor_SMD:C_0402_1005Metric, F.Cu at (447.1, 171.2)
- added C616: 100nF, Capacitor_SMD:C_0402_1005Metric, F.Cu at (187.2, 205.6)
- added C617: 10uF, Capacitor_SMD:C_0402_1005Metric, F.Cu at (187.2, 203.3)
- added C618: 10uF, Capacitor_SMD:C_0402_1005Metric, F.Cu at (187.2, 204.4)
- added C621: 0.1uF, Capacitor_SMD:C_0201_0603Metric, F.Cu at (446.1, 195.7)
- added C622: 20pF, Capacitor_SMD:C_0201_0603Metric, F.Cu at (405.3, 177.1)
- added C623: 12pF, Capacitor_SMD:C_0201_0603Metric, B.Cu at (381.7, 123.7)
- added C624: 0.1uF, Capacitor_SMD:C_0201_0603Metric, F.Cu at (148.1, 103.1)
- added C625: 0.1uF, Capacitor_SMD:C_0201_0603Metric, F.Cu at (238.9, 162.0)
- added C626: 0.1uF, Capacitor_SMD:C_0201_0603Metric, F.Cu at (230.3, 164.2)
- added C627: 0.1uF, Capacitor_SMD:C_0201_0603Metric, F.Cu at (235.1, 151.9)
- added C628: 0.1uF, Capacitor_SMD:C_0201_0603Metric, F.Cu at (230.9, 151.9)
- added C629: 0.1uF, Capacitor_SMD:C_0201_0603Metric, F.Cu at (238.9, 161.1)
- added C630: 0.1uF, Capacitor_SMD:C_0201_0603Metric, F.Cu at (233.4, 164.2)
- added C631: 0.1uF, Capacitor_SMD:C_0201_0603Metric, F.Cu at (226.1, 157.3)
- added C632: 0.1uF, Capacitor_SMD:C_0201_0603Metric, F.Cu at (231.9, 151.9)
- added C633: 0.1uF, Capacitor_SMD:C_0201_0603Metric, F.Cu at (235.5, 164.2)
- added C634: 0.1uF, Capacitor_SMD:C_0201_0603Metric, F.Cu at (226.1, 160.6)
- added C635: 0.1uF, Capacitor_SMD:C_0201_0603Metric, F.Cu at (229.5, 164.2)
- added C636: 0.1uF, Capacitor_SMD:C_0201_0603Metric, F.Cu at (236.2, 151.9)
- added C637: 0.1uF, Capacitor_SMD:C_0201_0603Metric, F.Cu at (144.4, 98.7)
- added C638: 0.1uF, Capacitor_SMD:C_0201_0603Metric, B.Cu at (283.8, 165.9)
- added C639: 0.1uF, Capacitor_SMD:C_0201_0603Metric, B.Cu at (283.8, 161.9)
- added C640: 0.1uF, Capacitor_SMD:C_0201_0603Metric, B.Cu at (282.6, 161.9)
- added C641: 0.1uF, Capacitor_SMD:C_0201_0603Metric, B.Cu at (277.4, 165.9)
- added C642: 0.1uF, Capacitor_SMD:C_0201_0603Metric, B.Cu at (278.6, 165.9)
- added C643: 0.1uF, Capacitor_SMD:C_0201_0603Metric, B.Cu at (278.6, 161.9)
- added C644: 0.1uF, Capacitor_SMD:C_0201_0603Metric, B.Cu at (277.4, 161.9)
- added C645: 22uF, Capacitor_SMD:C_0603_1608Metric, B.Cu at (286.7, 163.2)
- added C646: 10uF, Capacitor_SMD:C_0402_1005Metric, B.Cu at (276.6, 163.9)
- added C647: 10uF, Capacitor_SMD:C_0402_1005Metric, B.Cu at (284.6, 163.9)
- added C648: 0.1uF, Capacitor_SMD:C_0201_0603Metric, B.Cu at (277.2, 157.7)
- added C649: 0.1uF, Capacitor_SMD:C_0201_0603Metric, B.Cu at (277.2, 158.7)
- added C650: 0.1uF, Capacitor_SMD:C_0201_0603Metric, B.Cu at (284.0, 158.7)
- added C651: 0.1uF, Capacitor_SMD:C_0201_0603Metric, B.Cu at (284.0, 157.7)
- added C652: 0.1uF, Capacitor_SMD:C_0201_0603Metric, B.Cu at (277.1, 169.1)
- added C653: 0.1uF, Capacitor_SMD:C_0201_0603Metric, B.Cu at (277.1, 170.1)
- added C654: 0.1uF, Capacitor_SMD:C_0201_0603Metric, B.Cu at (284.0, 170.1)
- added C655: 0.1uF, Capacitor_SMD:C_0201_0603Metric, B.Cu at (284.0, 169.1)
- added C656: 4.7uF, Capacitor_SMD:C_0402_1005Metric, B.Cu at (280.1, 163.9)
- added C657: 0.1uF, Capacitor_SMD:C_0201_0603Metric, B.Cu at (280.3, 166.8)
- added C658: 0.1uF, Capacitor_SMD:C_0201_0603Metric, B.Cu at (280.3, 161.0)
- added C659: 4.7uF, Capacitor_SMD:C_0402_1005Metric, B.Cu at (300.9, 145.2)
- added C660: 22uF, Capacitor_SMD:C_0603_1608Metric, B.Cu at (301.9, 139.7)
- added C661: 22uF, Capacitor_SMD:C_0603_1608Metric, B.Cu at (301.9, 151.7)
- added C662: 0.1uF, Capacitor_SMD:C_0201_0603Metric, B.Cu at (298.0, 145.3)
- added C663: 10uF, Capacitor_SMD:C_0402_1005Metric, B.Cu at (307.3, 145.7)
- added C664: 10uF, Capacitor_SMD:C_0402_1005Metric, B.Cu at (300.9, 141.7)
- added C665: 0.1uF, Capacitor_SMD:C_0201_0603Metric, B.Cu at (303.9, 145.3)
- added C666: 10uF, Capacitor_SMD:C_0402_1005Metric, B.Cu at (294.9, 145.7)
- added C667: 10uF, Capacitor_SMD:C_0402_1005Metric, B.Cu at (300.9, 149.7)
- added C668: 0.1uF, Capacitor_SMD:C_0201_0603Metric, B.Cu at (298.9, 148.8)
- added C669: 0.1uF, Capacitor_SMD:C_0201_0603Metric, B.Cu at (294.8, 149.2)
- added C670: 0.1uF, Capacitor_SMD:C_0201_0603Metric, B.Cu at (298.9, 143.7)
- added C671: 0.1uF, Capacitor_SMD:C_0201_0603Metric, B.Cu at (295.6, 142.1)
- added C672: 0.1uF, Capacitor_SMD:C_0201_0603Metric, B.Cu at (302.9, 147.7)
- added C673: 0.1uF, Capacitor_SMD:C_0201_0603Metric, B.Cu at (294.8, 142.1)
- added C674: 0.1uF, Capacitor_SMD:C_0201_0603Metric, B.Cu at (302.9, 142.4)
- added C675: 0.1uF, Capacitor_SMD:C_0201_0603Metric, B.Cu at (306.1, 149.2)
- added C676: 0.1uF, Capacitor_SMD:C_0201_0603Metric, B.Cu at (298.9, 147.7)
- added C677: 0.1uF, Capacitor_SMD:C_0201_0603Metric, B.Cu at (307.1, 149.2)
- added C678: 0.1uF, Capacitor_SMD:C_0201_0603Metric, B.Cu at (298.9, 142.4)
- added C679: 0.1uF, Capacitor_SMD:C_0201_0603Metric, B.Cu at (295.6, 149.2)
- added C680: 0.1uF, Capacitor_SMD:C_0201_0603Metric, B.Cu at (302.9, 148.8)
- added C681: 0.1uF, Capacitor_SMD:C_0201_0603Metric, B.Cu at (307.1, 142.1)
- added C682: 0.1uF, Capacitor_SMD:C_0201_0603Metric, B.Cu at (302.9, 143.7)
- added C683: 0.1uF, Capacitor_SMD:C_0201_0603Metric, B.Cu at (306.2, 142.1)
- added C684: 10uF, Capacitor_SMD:C_0402_1005Metric, F.Cu at (197.0, 219.7)
- added C685: 0.1uF, Capacitor_SMD:C_0402_1005Metric, F.Cu at (197.0, 217.2)
- added C686: 33nF, Capacitor_SMD:C_0201_0603Metric, F.Cu at (194.2, 214.5)
- added C687: 22uF, Capacitor_SMD:C_0402_1005Metric, F.Cu at (193.5, 208.0)
- added C688: 22uF, Capacitor_SMD:C_0402_1005Metric, F.Cu at (196.1, 208.0)
- added C689: 1uF, Capacitor_SMD:C_0201_0603Metric, F.Cu at (448.5, 109.6)
- added C690: 0.1uF, Capacitor_SMD:C_0402_1005Metric, B.Cu at (122.5, 215.4)
- added C691: 10uF, Capacitor_SMD:C_0402_1005Metric, B.Cu at (121.4, 215.4)
- added C692: 10uF, Capacitor_SMD:C_0402_1005Metric, B.Cu at (120.3, 215.4)
- added C693: 0.1uF, Capacitor_SMD:C_0402_1005Metric, B.Cu at (120.3, 213.1)
- added C694: 33nF, Capacitor_SMD:C_0201_0603Metric, B.Cu at (123.3, 210.3)
- added C695: 22uF, Capacitor_SMD:C_0402_1005Metric, B.Cu at (123.8, 203.8)
- added C696: 22uF, Capacitor_SMD:C_0402_1005Metric, B.Cu at (121.1, 203.8)
- added C697: 0.1uF, Capacitor_SMD:C_0201_0603Metric, F.Cu at (453.5, 87.6)
- added C698: 0.1uF, Capacitor_SMD:C_0201_0603Metric, F.Cu at (398.9, 169.9)
- added C699: 10uF, Capacitor_SMD:C_0402_1005Metric, F.Cu at (219.6, 80.7)
- added C700: 10uF, Capacitor_SMD:C_0402_1005Metric, F.Cu at (219.6, 81.8)
- added C701: 0.1uF, Capacitor_SMD:C_0402_1005Metric, F.Cu at (222.1, 81.8)
- added C702: 33nF, Capacitor_SMD:C_0201_0603Metric, F.Cu at (224.9, 78.9)
- added C703: 47uF, Capacitor_SMD:C_0402_1005Metric, F.Cu at (231.1, 80.9)
- added C704: 47uF, Capacitor_SMD:C_0402_1005Metric, F.Cu at (231.1, 78.3)
- added C705: 0.1uF, Capacitor_SMD:C_0201_0603Metric, F.Cu at (430.5, 59.4)
- added C706: 0.1uF, Capacitor_SMD:C_0201_0603Metric, F.Cu at (430.5, 58.5)
- added C707: 1uF, Capacitor_SMD:C_0402_1005Metric, F.Cu at (447.1, 195.9)
- added C708: 1uF, Capacitor_SMD:C_0402_1005Metric, F.Cu at (384.4, 161.6)
- added C709: 0.1uF, Capacitor_SMD:C_0201_0603Metric, F.Cu at (385.5, 161.8)
- added C710: 1uF, Capacitor_SMD:C_0402_1005Metric, F.Cu at (399.2, 177.8)
- added C711: 0.1uF, Capacitor_SMD:C_0201_0603Metric, F.Cu at (398.9, 176.8)
- added C712: 1uF, Capacitor_SMD:C_0402_1005Metric, F.Cu at (379.7, 177.8)
- added C713: 0.1uF, Capacitor_SMD:C_0201_0603Metric, F.Cu at (379.9, 176.8)
- added C714: 1uF, Capacitor_SMD:C_0402_1005Metric, F.Cu at (393.8, 161.6)
- added C715: 0.1uF, Capacitor_SMD:C_0201_0603Metric, F.Cu at (394.9, 161.8)
- added C716: 0.1uF, Capacitor_SMD:C_0201_0603Metric, F.Cu at (435.4, 58.8)
- added C717: 0.1uF, Capacitor_SMD:C_0201_0603Metric, F.Cu at (430.8, 55.0)
- added C718: 0.1uF, Capacitor_SMD:C_0201_0603Metric, F.Cu at (430.8, 54.1)
- added C719: 0.1uF, Capacitor_SMD:C_0201_0603Metric, F.Cu at (435.4, 53.8)
- added C720: 0.1uF, Capacitor_SMD:C_0201_0603Metric, F.Cu at (408.5, 52.1)
- added C721: 0.1uF, Capacitor_SMD:C_0201_0603Metric, F.Cu at (408.5, 51.2)
- added C722: 0.1uF, Capacitor_SMD:C_0201_0603Metric, F.Cu at (413.1, 51.0)
- added C724: 0.1uF, Capacitor_SMD:C_0201_0603Metric, F.Cu at (398.6, 80.6)
- added D1: SMAJ15CA, Diode_SMD:D_SMA, F.Cu at (166.9, 94.1)
- added D13: SD103AWS-E3-08, barebones:SOD2713X115N, F.Cu at (435.2, 98.3)
- added D17: SMAJ15CA, Diode_SMD:D_SMA, F.Cu at (166.7, 106.2)
- added D19: TPD6E05U06RVZR, barebones:SON50P135X350X55-14N, F.Cu at (139.3, 157.0)
- added D20: SD103AWS-E3-08, barebones:SOD2713X115N, F.Cu at (454.8, 88.5)
- added D3: B0530W-7-F, barebones:SOD3715X145N, F.Cu at (348.1, 81.6)
- added D4: B0530W-7-F, barebones:SOD3715X145N, F.Cu at (364.1, 214.1)
- added D5: TPD1E05U06DPYR, barebones:DIO_TPD1E05U06DPYR, F.Cu at (336.7, 160.0)
- added FL1: BLM18PG121SZ1D, barebones:BEADC1608X95N, B.Cu at (299.4, 155.0)
- added FL2: BLM18PG121SZ1D, barebones:BEADC1608X95N, F.Cu at (435.9, 166.7)
- added FL3: BLM18PG121SZ1D, barebones:BEADC1608X95N, F.Cu at (399.7, 167.5)
- added H1: MountingHole_Pad, MountingHole:MountingHole_2.2mm_M2_Pad_Via, F.Cu at (449.6, 216.2)
- added H2: MountingHole_Pad, MountingHole:MountingHole_2.2mm_M2_Pad_Via, F.Cu at (452.0, 77.0)
- added H3: MountingHole_Pad, MountingHole:MountingHole_2.2mm_M2_Pad_Via, F.Cu at (106.2, 77.2)
- added H4: MountingHole_Pad, MountingHole:MountingHole_2.2mm_M2_Pad_Via, F.Cu at (108.4, 214.5)
- added H5: MountingHole_Pad, MountingHole:MountingHole_2.2mm_M2_Pad_Via, F.Cu at (302.1, 133.4)
- added J12: 10067847-001RLF, barebones:AMPHENOL_10067847-001RLF, F.Cu at (106.4, 157.2)
- added J14: S2B-PH-K-S_LF__SN_, barebones:JST_S2B-PH-K-S_LF__SN_, F.Cu at (107.3, 198.9)
- added J15: S2B-PH-K-S_LF__SN_, barebones:JST_S2B-PH-K-S_LF__SN_, F.Cu at (449.7, 204.2)
- added J19: SM06B-SRSS-TB_LF__SN_, barebones:JST_SM06B-SRSS-TB_LF__SN_, F.Cu at (448.7, 192.2)
- added J24: FH12-30S-0.5SH_55_, barebones:HIROSE_FH12-30S-0.5SH_55_, F.Cu at (370.5, 146.3)
- added J25: F33X-1AAJ1-E8951, barebones:AMPHENOL_F33X-1AAJ1-E8951, F.Cu at (386.8, 215.1)
- added J7: 5034801200, barebones:CON_5034801200_MOL, F.Cu at (395.6, 73.9)
- added L11: DFE201610E-R47M=P2, barebones:INDC2016X100N, F.Cu at (146.7, 194.1)
- added L12: DFE252010F-R22M=P2, barebones:IND-SMD_L2.5-W2.0_MHCD252012B-2R2M-A8L, F.Cu at (146.5, 202.8)
- added L13: DFE252010F-R22M=P2, barebones:IND-SMD_L2.5-W2.0_MHCD252012B-2R2M-A8L, F.Cu at (141.6, 187.7)
- added L14: LQH5BPN100MT0L, barebones:IND_LQH5BPN100MT0L, F.Cu at (343.6, 81.4)
- added L15: LQH32PH220MNCL, barebones:IND_LQH32PH220MNCL, F.Cu at (359.8, 215.2)
- added L16: DFE252010F-R22M=P2, barebones:IND-SMD_L2.5-W2.0_MHCD252012B-2R2M-A8L, F.Cu at (129.1, 204.8)
- added L17: XAL7030-472MEB, barebones:IND_XAL7030-472MEB, F.Cu at (569.5, 324.2)
- added L18: DFE252010F-R22M=P2, barebones:IND-SMD_L2.5-W2.0_MHCD252012B-2R2M-A8L, F.Cu at (138.0, 215.5)
- added L19: DFE252010F-R22M=P2, barebones:IND-SMD_L2.5-W2.0_MHCD252012B-2R2M-A8L, F.Cu at (129.6, 215.5)
- added L20: DFEG7030D-4R7M=P3, barebones:IND_DFEG7030D-4R7M=P3, F.Cu at (200.9, 106.7)
- added L21: DFE201610E-R47M=P2, barebones:INDC2016X100N, F.Cu at (146.1, 197.2)
- added L22: DFE201610E-R47M=P2, barebones:INDC2016X100N, F.Cu at (126.2, 195.0)
- added L23: DFE201610E-R47M=P2, barebones:INDC2016X100N, F.Cu at (130.3, 187.9)
- added L24: DFE201610E-R47M=P2, barebones:INDC2016X100N, F.Cu at (134.9, 204.5)
- added L25: DFE201610E-R47M=P2, barebones:INDC2016X100N, F.Cu at (138.7, 204.5)
- added L26: XAL6030-332MEC, barebones:IND_XAL6030-332MEC, F.Cu at (227.6, 95.0)
- added L4: FDSD0420-H-2R2M=P3, barebones:IND_FDSD0420-H-2R2M=P3, B.Cu at (122.5, 206.7)
- added L9: DFE252010F-R22M=P2, barebones:IND-SMD_L2.5-W2.0_MHCD252012B-2R2M-A8L, F.Cu at (138.2, 187.7)
- added LED1: SK6812SIDE-A, barebones:LED-SMD_4P-L4.0-W1.6-L, F.Cu at (159.7, 217.8)
- added Q11: CSD18543Q3A, barebones:TRANS_CSD18543Q3A, F.Cu at (193.5, 103.1)
- added Q12: CSD18543Q3A, barebones:TRANS_CSD18543Q3A, F.Cu at (193.5, 108.1)
- added Q13: CSD18543Q3A, barebones:TRANS_CSD18543Q3A, F.Cu at (207.1, 101.0)
- added Q14: CSD18543Q3A, barebones:TRANS_CSD18543Q3A, F.Cu at (207.1, 106.0)
- added Q4: MMBT3904, Package_TO_SOT_SMD:SOT-23, F.Cu at (333.8, 159.6)
- added Q7: CSD25402Q3A, barebones:TRANS_CSD25402Q3A, F.Cu at (169.9, 110.1)
- added Q8: CSD25402Q3A, barebones:TRANS_CSD25402Q3A, F.Cu at (170.1, 97.9)
- added Q9: CSD25402Q3A, barebones:TRANS_CSD25402Q3A, F.Cu at (165.5, 97.9)
- added R221: 10k, Resistor_SMD:R_0201_0603Metric, F.Cu at (398.9, 173.9)
- added R222: 22R, Resistor_SMD:R_0201_0603Metric, F.Cu at (379.9, 175.9)
- added R223: 22R, Resistor_SMD:R_0201_0603Metric, F.Cu at (384.6, 181.6)
- added R224: 10k, Resistor_SMD:R_0201_0603Metric, F.Cu at (393.1, 181.6)
- added R227: 30.1k, Resistor_SMD:R_0402_1005Metric, F.Cu at (236.8, 113.2)
- added R228: 10k, Resistor_SMD:R_0201_0603Metric, F.Cu at (233.4, 110.7)
- added R229: 4.7k, Resistor_SMD:R_0201_0603Metric, F.Cu at (408.5, 111.7)
- added R230: 4.7k, Resistor_SMD:R_0201_0603Metric, F.Cu at (416.5, 105.2)
- added R231: 4.7k, Resistor_SMD:R_0201_0603Metric, F.Cu at (412.3, 129.2)
- added R232: 4.7k, Resistor_SMD:R_0201_0603Metric, F.Cu at (409.7, 129.2)
- added R233: 4.7k, Resistor_SMD:R_0201_0603Metric, F.Cu at (416.5, 123.0)
- added R234: 4.7k, Resistor_SMD:R_0201_0603Metric, F.Cu at (416.5, 142.4)
- added R235: 4.7k, Resistor_SMD:R_0201_0603Metric, F.Cu at (408.8, 147.2)
- added R249: 10k, Resistor_SMD:R_0201_0603Metric, B.Cu at (387.5, 103.1)
- added R250: 10k, Resistor_SMD:R_0201_0603Metric, B.Cu at (376.4, 129.3)
- added R251: 10k, Resistor_SMD:R_0402_1005Metric, F.Cu at (222.1, 77.9)
- added R252: 31.3k, Resistor_SMD:R_0402_1005Metric, F.Cu at (224.7, 77.9)
- added R253: 10k, Resistor_SMD:R_0201_0603Metric, F.Cu at (445.6, 88.9)
- added R255: 10k, Resistor_SMD:R_0402_1005Metric, F.Cu at (130.7, 128.4)
- added R256: 20.2k, Resistor_SMD:R_0402_1005Metric, F.Cu at (138.6, 128.4)
- added R257: 10k, Resistor_SMD:R_0402_1005Metric, F.Cu at (431.9, 133.4)
- added R258: 20.2k, Resistor_SMD:R_0402_1005Metric, F.Cu at (432.9, 138.3)
- added R259: 10k, Resistor_SMD:R_0201_0603Metric, F.Cu at (398.6, 81.5)
- added R260: 10k, Resistor_SMD:R_0201_0603Metric, F.Cu at (390.3, 81.5)
- added R261: 10k, Resistor_SMD:R_0201_0603Metric, F.Cu at (445.6, 89.8)
- added R262: 1.8k, Resistor_SMD:R_0201_0603Metric, F.Cu at (453.0, 89.0)
- added R263: 1.8k, Resistor_SMD:R_0201_0603Metric, F.Cu at (453.0, 90.0)
- added R264: 200k, Resistor_SMD:R_0201_0603Metric, F.Cu at (452.6, 87.6)
- added R269: 200R, Resistor_SMD:R_0201_0603Metric, F.Cu at (398.6, 79.7)
- added R271: 10k, Resistor_SMD:R_0201_0603Metric, F.Cu at (398.6, 82.5)
- added R272: 10k, Resistor_SMD:R_0201_0603Metric, F.Cu at (390.3, 82.5)
- added R64: 100k, Resistor_SMD:R_0402_1005Metric, F.Cu at (126.4, 198.0)
- added R82: 4.7k, Resistor_SMD:R_0201_0603Metric, F.Cu at (200.2, 121.6)
- added S2: TL3342F160QG, barebones:SW_TL3342F160QG, F.Cu at (395.2, 106.7)
- added S3: TL3342F160QG, barebones:SW_TL3342F160QG, F.Cu at (395.2, 124.7)
- added S4: TL3342F160QG, barebones:SW_TL3342F160QG, F.Cu at (395.2, 142.7)
- added S5: TL3342F160QG, barebones:SW_TL3342F160QG, B.Cu at (383.9, 115.9)
- added S6: TL3342F160QG, barebones:SW_TL3342F160QG, B.Cu at (384.0, 106.7)
- added S7: 1571983-4, barebones:SW_1571983-4, B.Cu at (545.3, 307.7)
- added S8: 1-1571983-0, barebones:SW_1-1571983-0, B.Cu at (259.8, 79.6)
- added SW1: EC05E1220401, barebones:SW-SMD_EC05E1220401, F.Cu at (411.0, 107.8)
- added SW2: EC05E1220401, barebones:SW-SMD_EC05E1220401, F.Cu at (411.0, 125.8)
- added SW3: EC05E1220401, barebones:SW-SMD_EC05E1220401, F.Cu at (411.0, 143.8)
- added TP2: 3V3, TestPoint:TestPoint_Pad_D1.0mm, B.Cu at (372.6, 110.3)
- added TP3: BOOT0, TestPoint:TestPoint_Pad_D1.0mm, B.Cu at (376.3, 110.3)
- added TP4: NRST, TestPoint:TestPoint_Pad_D1.0mm, B.Cu at (368.5, 107.6)
- added U11: PCA9306DCTR, barebones:SOP65P400X130-8N, F.Cu at (449.3, 88.7)
- added U13: STM32U083MCT6, barebones:TQFP-80_L12.0-W12.0-P0.50-LS14.0-BL, F.Cu at (389.4, 172.1)
- added U2: W25Q16JVUXIQ_TR, barebones:IC_W25Q16JVUXIQ_TR, F.Cu at (147.2, 99.9)
- added U22: RK860-3, barebones:WLCSP-20_L2.0-W1.6-R5-C4-P0.40-TL, F.Cu at (144.7, 212.9)
- added U26: TPS61170DRVR, barebones:SON65P200X200X80-7N, F.Cu at (344.9, 77.2)
- added U28: TPS61160ADRVT, barebones:SON65P200X200X80-7N, F.Cu at (363.3, 216.7)
- added U3: TLV75533PDBVR, barebones:SOT95P280X145-5N, F.Cu at (560.6, 322.1)
- added U35: TS3A227EYFFR, barebones:BGA16N40P4X4_175X175X62N, F.Cu at (445.0, 158.1)
- added U38: TPS65988DHRSHR, barebones:IC_TPS65987DDHRSHR, F.Cu at (139.4, 102.3)
- added U5: TPS56837RPAR, barebones:CONV_TPS56837RPAR, F.Cu at (234.1, 113.6)
- added U6: TPS62933DRLR, barebones:SOTFL50P160X60-8N, F.Cu at (195.3, 185.5)
- added U65: 2N7002KW, barebones:SOT323, F.Cu at (437.5, 98.3)
- added U67: 2N7002KW, barebones:SOT323, F.Cu at (440.7, 109.4)
- added U68: 2N7002KW, barebones:SOT323, F.Cu at (438.0, 109.4)
- added U69: 2N7002KW, barebones:SOT323, F.Cu at (438.2, 86.6)
- added U70: 2N7002KW, barebones:SOT323, F.Cu at (440.9, 86.6)
- added U71: DRV5032DUDBZR, barebones:SOT-23-3_L2.9-W1.3-P1.90-LS2.4-BR, F.Cu at (440.2, 218.0)
- added U74: 2N7002KW, barebones:SOT323, F.Cu at (174.0, 105.7)
- added U85: TPS2557DRBR, barebones:SON65P300X300X100-9N, F.Cu at (431.0, 135.9)
- added U86: TPS2557DRBR, barebones:SON65P300X300X100-9N, F.Cu at (134.8, 127.1)
- added U9: 1N5819WT, barebones:SOD-523_L1.2-W0.8-LS1.6-RD, B.Cu at (143.9, 201.1)
- added VR1: TPS7A7002DDAR, barebones:VREG_TPS7A7002DDAR, F.Cu at (554.0, 333.5)
- added Y5: ABS07-32.768KHZ-T, barebones:XTAL_ABS07-32.768KHZ-T, F.Cu at (301.7, 189.0)
- added Y6: ABS07-32.768KHZ-T, barebones:XTAL_ABS07-32.768KHZ-T, F.Cu at (404.8, 174.5)
- added Y7: C2E-25.000-10-1530-X-R, barebones:XTAL_C2E-25.000-10-1530-X-R, F.Cu at (223.7, 152.1)
- added Y8: C2E-25.000-10-1530-X-R, barebones:XTAL_C2E-25.000-10-1530-X-R, B.Cu at (382.3, 126.0)
- C1, C114, C115, C129, C130, C131, C135, C136, C138, C164, C18, C19, C26, C27, C378, C437, C438, C439, C441, C443, C86, C89: footprint Capacitor_SMD:C_0201_0603Metric -> Capacitor_SMD:C_0402_1005Metric; moved to B.Cu
- C10, C101, C126, C132, C162, C29, C40: value 1uF -> 0.1uF; moved to B.Cu
- C102, C109, C11, C110, C12, C124, C125, C133, C20, C25, C30, C32, C4, C44, C45, C46, C47, C5, C51, C522, C53, C6, C60, C62, C64, C85, C95: value 100nF -> 0.1uF; moved to B.Cu
- C122, C143, C146, C152, C154, C7: value 1uF -> 10uF; footprint Capacitor_SMD:C_0201_0603Metric -> Capacitor_SMD:C_0402_1005Metric; moved to B.Cu
- C123, C142, C144, C145, C153, C375: value 100nF -> 10uF; footprint Capacitor_SMD:C_0201_0603Metric -> Capacitor_SMD:C_0402_1005Metric; moved to B.Cu
- C127, C128: value 10uF -> 0.1uF; moved to B.Cu
- C134: value 22uF -> 0.1uF; moved to B.Cu
- C137, C158, C159, C8: value 10uF -> 1uF; moved to B.Cu
- C139, C147, C374: value 4.7uF -> 10uF; footprint Capacitor_SMD:C_0201_0603Metric -> Capacitor_SMD:C_0402_1005Metric; moved to B.Cu
- C140, C161, C167, C168, C169, C170, C171, C172, C173, C177, C178, C179, C182, C183, C186, C187, C188, C191, C192, C193, C194, C197, C199, C2, C200, C201, C202, C205, C206, C207, C208, C209, C21, C210, C211, C213, C214, C215, C216, C217, C218, C219, C229, C23, C230, C233, C234, C236, C239, C244, C245, C246, C247, C248, C249, C252, C263, C265, C266, C267, C270, C271, C272, C274, C275, C276, C277, C278, C279, C286, C287, C288, C296, C297, C298, C299, C3, C31, C316, C319, C320, C33, C336, C337, C34, C39, C400, C401, C402, C434, C435, C507, C508, C509, C510, C52, C525, C54, C65, C73, C76, C77, C78, C79, C80, C81, C82, C9, D10, D11, J2, J3, R145, R152, R153, R154, R41, R44, R61, R62, Y1: moved to B.Cu
- C141, C87: value 1uF -> 4.7uF; footprint Capacitor_SMD:C_0201_0603Metric -> Capacitor_SMD:C_0402_1005Metric; moved to B.Cu
- C148: value 10uF -> 4.7uF; footprint Capacitor_SMD:C_0201_0603Metric -> Capacitor_SMD:C_0402_1005Metric; moved to B.Cu
- C15, C17, C38, C41, C422, C43, C539: value 100nF -> 0.1uF; footprint Capacitor_SMD:C_0603_1608Metric -> Capacitor_SMD:C_0201_0603Metric; moved to B.Cu
- C151: value 22uF -> 10uF; footprint Capacitor_SMD:C_0201_0603Metric -> Capacitor_SMD:C_0402_1005Metric; moved to B.Cu
- C155: value 22uF -> 4.7uF; footprint Capacitor_SMD:C_0201_0603Metric -> Capacitor_SMD:C_0402_1005Metric; moved to B.Cu
- C16, C424: value 1uF -> 0.1uF; footprint Capacitor_SMD:C_0603_1608Metric -> Capacitor_SMD:C_0201_0603Metric; moved to B.Cu
- C160, C430, C83, C84: value 4.7uF -> 0.1uF; moved to B.Cu
- C163, C22, C28, C50, C66: value 100nF -> 1uF; moved to B.Cu
- C165, C166, C185, C204, C222, C224, C226: footprint Capacitor_SMD:C_0402_1005Metric -> Capacitor_SMD:C_0201_0603Metric; moved to B.Cu
- C176, C240, C241, C354, C355, C357, C362, C556, C557, C558, C559: footprint Capacitor_SMD:C_0402_1005Metric -> Capacitor_SMD:C_0201_0603Metric
- C180, C196: value 4.7nF -> 0.1uF; footprint Capacitor_SMD:C_0402_1005Metric -> Capacitor_SMD:C_0201_0603Metric; moved to B.Cu
- C181, C198, C304: value 10nF -> 0.1uF; footprint Capacitor_SMD:C_0402_1005Metric -> Capacitor_SMD:C_0201_0603Metric; moved to B.Cu
- C184, C190, C220: value 1uF -> 0.1uF; footprint Capacitor_SMD:C_0402_1005Metric -> Capacitor_SMD:C_0201_0603Metric; moved to B.Cu
- C189, C315: value 1uF -> 22uF; moved to B.Cu
- C195: value 0.1uF -> 22uF; moved to B.Cu
- C221, C223, C225, C307: value 0.1uF -> 1uF; footprint Capacitor_SMD:C_0402_1005Metric -> Capacitor_SMD:C_0201_0603Metric; moved to B.Cu
- C227, C228, C237, C238: footprint Capacitor_SMD:C_0402_1005Metric -> Capacitor_SMD:C_0603_1608Metric
- C24, C35: value 18pF -> 1uF; footprint Capacitor_SMD:C_0603_1608Metric -> Capacitor_SMD:C_0201_0603Metric; moved to B.Cu
- C253, C338, C405: value 100nF -> 10uF; moved to B.Cu
- C254, C255, C256, C257, C258: value 10uF -> 0.1uF; footprint Capacitor_SMD:C_0402_1005Metric -> Capacitor_SMD:C_0603_1608Metric
- C259, C261, C310: value 10uF -> 1uF; footprint Capacitor_SMD:C_0402_1005Metric -> Capacitor_SMD:C_0201_0603Metric; moved to B.Cu
- C260, C262: value 10uF -> 0.1uF; footprint Capacitor_SMD:C_0402_1005Metric -> Capacitor_SMD:C_0201_0603Metric; moved to B.Cu
- C268, C269: value 33uF -> 0.1uF; footprint Capacitor_SMD:C_0402_1005Metric -> Capacitor_SMD:C_0201_0603Metric; moved to B.Cu
- C285, C289: value 22uF -> 47uF; moved to B.Cu
- C295: value 22uF -> 0.1uF; footprint Capacitor_SMD:C_0402_1005Metric -> Capacitor_SMD:C_0201_0603Metric; moved to B.Cu
- C302, C567, C568: value 0.1uF -> 1uF
- C303, C309, C417: value 100nF -> 22uF; moved to B.Cu
- C305, C306, C370: value 47uF -> 1uF; footprint Capacitor_SMD:C_0402_1005Metric -> Capacitor_SMD:C_0201_0603Metric; moved to B.Cu
- C308: value 10uF -> 22uF; moved to B.Cu
- C314: value 1uF -> 0.1uF
- C321: value 33nF -> 0.1uF
- C322: value 47uF -> 0.1uF; moved to B.Cu
- C323: value 47uF -> 0.1uF
- C325, C326: value 22uF -> 10uF; footprint Capacitor_SMD:C_0402_1005Metric -> Capacitor_SMD:C_0603_1608Metric; moved to B.Cu
- C327: value 100nF -> 1uF; footprint Capacitor_SMD:C_0402_1005Metric -> Capacitor_SMD:C_0201_0603Metric; moved to B.Cu
- C328: value 0.1uF -> 10uF; footprint Capacitor_SMD:C_0402_1005Metric -> Capacitor_SMD:C_0603_1608Metric; moved to B.Cu
- C329: footprint Capacitor_SMD:C_0402_1005Metric -> Capacitor_SMD:C_0603_1608Metric; moved to B.Cu
- C330: value 100nF -> 10uF; footprint Capacitor_SMD:C_0402_1005Metric -> Capacitor_SMD:C_0603_1608Metric; moved to B.Cu
- C331: value 10nF -> 10uF; footprint Capacitor_SMD:C_0402_1005Metric -> Capacitor_SMD:C_0603_1608Metric; moved to B.Cu
- C332: value 47uF -> 10uF; footprint Capacitor_SMD:C_0402_1005Metric -> Capacitor_SMD:C_0603_1608Metric; moved to B.Cu
- C334: value 0.1uF -> 33uF; footprint Capacitor_SMD:C_0402_1005Metric -> Capacitor_SMD:C_0603_1608Metric; moved to B.Cu
- C335: value 10uF -> 33uF; footprint Capacitor_SMD:C_0402_1005Metric -> Capacitor_SMD:C_0603_1608Metric; moved to B.Cu
- C339, C415: value 1uF -> 10uF; moved to B.Cu
- C341, C342, C350, C351: value 47uF -> 10uF
- C344: value 0.1uF -> 47nF; footprint Capacitor_SMD:C_0402_1005Metric -> Capacitor_SMD:C_0201_0603Metric
- C345: value 10nF -> 0.1uF
- C346: value 47uF -> 150pF
- C347, C366: value 47uF -> 22uF; footprint Capacitor_SMD:C_0402_1005Metric -> Capacitor_SMD:C_0603_1608Metric
- C348, C367: value 0.1uF -> 22uF; footprint Capacitor_SMD:C_0402_1005Metric -> Capacitor_SMD:C_0603_1608Metric
- C349, C368: value 1uF -> 22uF; footprint Capacitor_SMD:C_0402_1005Metric -> Capacitor_SMD:C_0603_1608Metric
- C358: value 33uF -> 0.1uF
- C359: value 0.47uF -> 47nF; footprint Capacitor_SMD:C_0402_1005Metric -> Capacitor_SMD:C_0201_0603Metric
- C36, C37, C42: footprint Capacitor_SMD:C_0603_1608Metric -> Capacitor_SMD:C_0201_0603Metric; moved to B.Cu
- C365: value 47uF -> 150pF; footprint Capacitor_SMD:C_0402_1005Metric -> Capacitor_SMD:C_0201_0603Metric
- C369: value 47uF -> 10uF; moved to B.Cu
- C371, C466, C540: value 0.1uF -> 10uF; moved to B.Cu
- C376, C377, C379, C380, C72: value 100nF -> 4.7uF; footprint Capacitor_SMD:C_0201_0603Metric -> Capacitor_SMD:C_0402_1005Metric; moved to B.Cu
- C396, C408: footprint Capacitor_SMD:C_0603_1608Metric -> Capacitor_SMD:C_0201_0603Metric
- C399, C407, C416, C425: value 100nF -> 0.1uF; footprint Capacitor_SMD:C_0603_1608Metric -> Capacitor_SMD:C_0201_0603Metric
- C403, C412, C418, C420, C423, C426, C542: footprint Capacitor_SMD:C_0603_1608Metric -> Capacitor_SMD:C_0402_1005Metric
- C409, C410: value 20pF -> 0.1uF; footprint Capacitor_SMD:C_0603_1608Metric -> Capacitor_SMD:C_0201_0603Metric
- C413: value 1uF -> 0.1uF; footprint Capacitor_SMD:C_0603_1608Metric -> Capacitor_SMD:C_0201_0603Metric
- C414: value 1uF -> 12.5pF
- C419: value 1uF -> 4.7uF; footprint Capacitor_SMD:C_0603_1608Metric -> Capacitor_SMD:C_0201_0603Metric; moved to B.Cu
- C421: value 1uF -> 10uF; footprint Capacitor_SMD:C_0603_1608Metric -> Capacitor_SMD:C_0402_1005Metric; moved to B.Cu
- C427: value 100nF -> 0.1uF; footprint Capacitor_SMD:C_0603_1608Metric -> Capacitor_SMD:C_0402_1005Metric
- C428, C429: value 100nF -> 1uF; footprint Capacitor_SMD:C_0603_1608Metric -> Capacitor_SMD:C_0402_1005Metric
- C431, C432, C433, C436, C440, C442, C444, C445, C446, C447, C448, C449, C450, C451, C452, C453, C455, C456, C458, C463, C464, C469, C470, C471, C472, C474, C476, C479, C482, C486, C488, C491, C495, C497, C501, C502, C503, C504, C511, C528, C541: footprint Capacitor_SMD:C_0201_0603Metric -> Capacitor_SMD:C_0402_1005Metric
- C454: value 100nF -> 10uF; footprint Capacitor_SMD:C_0201_0603Metric -> Capacitor_SMD:C_0402_1005Metric
- C457: value 100nF -> 100uF; footprint Capacitor_SMD:C_0201_0603Metric -> Capacitor_SMD:C_0402_1005Metric
- C459: value 0.1uF -> 100nF; footprint Capacitor_SMD:C_0201_0603Metric -> Capacitor_SMD:C_0402_1005Metric; moved to B.Cu
- C460: value 220pF -> 10uF; footprint Capacitor_SMD:C_0201_0603Metric -> Capacitor_SMD:C_0603_1608Metric
- C461: value 220pF -> 0.1uF; footprint Capacitor_SMD:C_0201_0603Metric -> Capacitor_SMD:C_0402_1005Metric
- C462: value 0.1uF -> 10uF; footprint Capacitor_SMD:C_0201_0603Metric -> Capacitor_SMD:C_0402_1005Metric; moved to B.Cu
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Connections:
- net /Embedded Controller and Internal Audio/I2S0_LRCK_TX renamed /I2S0_LRCK
- net /Embedded Controller and Internal Audio/I2S0_SCLK_TX renamed /I2S0_SCLK
- net /Embedded Controller and Internal Audio/SPK_MUTE renamed /SPK_MUTE
- net /High Speed IO/HP_DETECT renamed /HP_DETECT
- net /High Speed IO/HP_INT renamed /HP_INT
- net /High Speed IO/I2S0_LRCK_TX renamed /I2S0_LRCK_TX
- net /High Speed IO/I2S0_SCLK_TX renamed /I2S0_SCLK_TX
- net /Peripheral IO Connectors/HDMI1_TX_SBDN renamed /Peripheral IO Connectors/HDMI_1_TX_SBDN
- net /Peripheral IO Connectors/PCIE30_REFCLKN_SLOT_0 renamed /PCIE30_REFCLKN_SLOT_0
- net /Peripheral IO Connectors/PCIE30_REFCLKN_SLOT_1 renamed /PCIE30_REFCLKN_SLOT_1
- net /Peripheral IO Connectors/PCIE30_REFCLKP_SLOT_0 renamed /PCIE30_REFCLKP_SLOT_0
- net /Peripheral IO Connectors/PCIE30_REFCLKP_SLOT_1 renamed /PCIE30_REFCLKP_SLOT_1
- net /Power and Ground/CHRG_OK_EC renamed /CHRG_OK_EC
- C1 pad 1: AGND -> GND
- C1 pad 2: VDDQ_DDR_S0 -> VDDQ_DDR_CK_S0
- C10 pad 1: AGND -> GND
- C10 pad 2: VDDQ_DDR_S0 -> VDDQ_DDR_CK_S0
- C101 pad 1: VDD_LOG_S0 -> GND
- C101 pad 2: AGND -> VDD_CPU_BIG1_S0
- C102 pad 1: VDD_LOG_S0 -> GND
- C102 pad 2: AGND -> VDD_CPU_BIG1_S0
- C109 pad 1: AGND -> GND
- C109 pad 2: VDD_GPU_S0 -> VDD_CPU_BIG0_S0
- C11 pad 1: AGND -> GND
- C11 pad 2: VDDQ_DDR_S0 -> VDDQ_DDR_CK_S0
- C110 pad 1: AGND -> GND
- C110 pad 2: VDD_GPU_S0 -> VDD_CPU_BIG0_S0
- C114 pad 1: AGND -> GND
- C114 pad 2: VDD_GPU_S0 -> VDD_CPU_LIT_S0
- C115 pad 1: AGND -> GND
- C115 pad 2: VDD_GPU_S0 -> VDD_VDENC_S0
- C12 pad 1: AGND -> GND
- C12 pad 2: VDDQ_DDR_S0 -> VDDQ_DDR_CK_S0
- C122 pad 1: AGND -> GND
- C123 pad 1: AGND -> GND
- C123 pad 2: VDD_VDENC_S0 -> VDD_CPU_LIT_S0
- C124 pad 1: AGND -> GND
- C124 pad 2: VDD_VDENC_S0 -> VDD_GPU_S0
- C125 pad 1: AGND -> GND
- C125 pad 2: VDD_NPU_S0 -> VDD_LOG_S0
- C126 pad 1: AGND -> GND
- C126 pad 2: VDD_NPU_S0 -> VDD_GPU_S0
- C127 pad 1: AGND -> GND
- C127 pad 2: VDD_NPU_S0 -> VCC_1V8_S0
- C128 pad 1: AGND -> GND
- C129 pad 1: AGND -> GND
- C129 pad 2: VDD_NPU_S0 -> VDD_CPU_LIT_S0
- C130 pad 1: AGND -> GND
- C130 pad 2: VDD_NPU_S0 -> VDD_GPU_S0
- C131 pad 1: AGND -> GND
- C131 pad 2: VDD_NPU_S0 -> VDD_CPU_LIT_S0
- C132 pad 1: AGND -> GND
- C132 pad 2: VDD_CPU_BIG1_MEM_S0 -> VDD_GPU_S0
- C133 pad 1: AGND -> GND
- C133 pad 2: VDD_CPU_BIG1_MEM_S0 -> VDD_NPU_S0
- C134 pad 1: AGND -> GND
- C134 pad 2: VDD_CPU_BIG1_S0 -> VDD_LOG_S0
- C135 pad 1: AGND -> GND
- C135 pad 2: VDD_CPU_BIG1_S0 -> VDD_GPU_S0
- C136 pad 1: AGND -> GND
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Routing:
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Other:
- board size 217 x 22.5 mm -> 354 x 150 mm
- copper layers 2 -> 12
- board text added: "PRIMARY STORAGE"
- board text added: "SECONDARY STORAGE"
- board text added: "WIFI/BLUETOOTH MODULE"
