File: hardware/motherboard/barebones.kicad_pcb (KiCad board)
At the start: 12 copper layers, 354 x 150 mm, 984 parts, among them J1 12401610E4_2A, J10 54-00007, J11 54-00007, J12 10067847-001RLF, J14 S2B-PH-K-S_LF__SN_, J15 S2B-PH-K-S_LF__SN_, J16 SM04B-SRSS-TB_LF__SN_, J17 2200981671, J18 G45AA1912100B1EU, J19 SM06B-SRSS-TB_LF__SN_, J2 1-2199119-5, J24 FH12-30S-0.5SH_55_, J25 F33X-1AAJ1-E8951, J3 1-2199119-5, J4 SJ3-350114B, J5 12401610E4_2A, J6 2199119-4, J7 5034801200, J8 SJ3-350114B, J9 20455-040E-76, Q1 BSS138, Q11 CSD18543Q3A, Q12 CSD18543Q3A, Q13 CSD18543Q3A, Q14 CSD18543Q3A, Q2 CSD25402Q3A, Q3 BSS138, Q4 MMBT3904, Q7 CSD25402Q3A, Q8 CSD25402Q3A, Q9 CSD25402Q3A, SW1 EC05E1220401, SW2 EC05E1220401, SW3 EC05E1220401, U1 RK3588, U10 TPS62933DRLR, U11 PCA9306DCTR, U12 RK806-1, U13 STM32U083MCT6, U14 BQ25731RSNR, U15 TPS22919DCK, U16 TPS22919DCK, U17 TPS22919DCK, U18 RK860-2, U19 RK860-2, U2 W25Q16JVUXIQ_TR, U20 PCA9306DCTR, U22 RK860-3, U26 TPS61170DRVR, U28 TPS61160ADRVT, U3 TLV75533PDBVR, U30 W25Q256JWEIQ, U31 PCF85063ATL/1,118, U32 K4UCE3Q4AA-MGCL, U33 K4UCE3Q4AA-MGCL, U34 ES8316, U35 TS3A227EYFFR, U36 STM32F411CEU6, U37 TPA2012D2RTJT, U38 TPS65988DHRSHR, U4 TPS56837RPAR, U41 TPD4E004DRYR, U43 9FGV0641AKILFT, U5 TPS56837RPAR, U53 TPS54628DDAR, U54 TPD4E004DRYR, U6 TPS62933DRLR, U65 2N7002KW, U67 2N7002KW, U68 2N7002KW, U69 2N7002KW, U7 TPS62933DRLR, U70 2N7002KW, U71 DRV5032DUDBZR, U74 2N7002KW, U77 2N7002KW, U79 USB5744_2G, U8 TPS62933DRLR, U85 TPS2557DRBR, U86 TPS2557DRBR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

Commit message: started routing on LPDDR4x RAM
Parts:
- removed C167, C168, C169, C170, C171, C172, C173, C439, C489, C576, C589: 22uF, Capacitor_SMD:C_0402_1005Metric
- removed C354, C357, C507: 0.1uF, Capacitor_SMD:C_0201_0603Metric
- removed C355: 680pF, Capacitor_SMD:C_0201_0603Metric
- removed C356: 4.7uF, Capacitor_SMD:C_0402_1005Metric
- removed C358, C575: 0.1uF, Capacitor_SMD:C_0402_1005Metric
- removed C359: 47nF, Capacitor_SMD:C_0201_0603Metric
- removed C360, C361: 1uF, Capacitor_SMD:C_0402_1005Metric
- removed C362: 220nF, Capacitor_SMD:C_0201_0603Metric
- removed C365: 150pF, Capacitor_SMD:C_0201_0603Metric
- removed C367, C368: 22uF, Capacitor_SMD:C_0603_1608Metric
- removed C414: 12.5pF, Capacitor_SMD:C_0603_1608Metric
- removed C437, C459: 100nF, Capacitor_SMD:C_0402_1005Metric
- removed C438, C462, C527, C530: 10uF, Capacitor_SMD:C_0402_1005Metric
- removed C457: 100uF, Capacitor_SMD:C_0402_1005Metric
- removed C65, C66: 1uF, Capacitor_SMD:C_0201_0603Metric
- removed D4: B0530W-7-F, barebones:SOD3715X145N
- removed J14: S2B-PH-K-S_LF__SN_, barebones:JST_S2B-PH-K-S_LF__SN_
- removed R112: 87.6k, Resistor_SMD:R_0402_1005Metric
- removed R113, R239: 10k, Resistor_SMD:R_0402_1005Metric
- removed R114, R228: 10k, Resistor_SMD:R_0201_0603Metric
- removed R115: 10R, Resistor_SMD:R_0201_0603Metric
- removed R119: 10k, Resistor_SMD:R_0603_1608Metric
- removed R227: 30.1k, Resistor_SMD:R_0402_1005Metric
- removed R238: 4.7k, Resistor_SMD:R_0201_0603Metric
- removed R240: 49.9k, Resistor_SMD:R_0402_1005Metric
- removed R241: 73.2k, Resistor_SMD:R_0402_1005Metric
- removed R45: 0R, Capacitor_SMD:C_0201_0603Metric
- removed SW3: EC05E1220401, barebones:SW-SMD_EC05E1220401
- removed TP2: 3V3, TestPoint:TestPoint_Pad_D1.0mm
- removed TP3: BOOT0, TestPoint:TestPoint_Pad_D1.0mm
- removed TP4: NRST, TestPoint:TestPoint_Pad_D1.0mm
- removed TP7: SWDIO, TestPoint:TestPoint_Pad_D1.0mm
- removed TP8: SWCLK, TestPoint:TestPoint_Pad_D1.0mm
- removed U10, U6, U7, U8: TPS62933DRLR, barebones:SOTFL50P160X60-8N
- removed U5: TPS56837RPAR, barebones:CONV_TPS56837RPAR
- added C149: 10uF, Capacitor_SMD:C_0603_1608Metric, B.Cu at (364.6, 348.3)
- added C150: 10uF, Capacitor_SMD:C_0603_1608Metric, B.Cu at (364.6, 350.8)
- added C156: 10uF, Capacitor_SMD:C_0603_1608Metric, B.Cu at (378.5, 346.4)
- added C157: 10uF, Capacitor_SMD:C_0603_1608Metric, B.Cu at (378.5, 348.1)
- added C311: 22uF, Capacitor_SMD:C_0603_1608Metric, F.Cu at (237.8, 352.5)
- added C312: 22uF, Capacitor_SMD:C_0603_1608Metric, F.Cu at (268.0, 349.2)
- added C313: 22uF, Capacitor_SMD:C_0603_1608Metric, F.Cu at (269.7, 349.2)
- added C324: 10uF, Capacitor_SMD:C_0805_2012Metric, F.Cu at (178.5, 330.4)
- added C333: 22uF, Capacitor_SMD:C_0805_2012Metric, F.Cu at (195.9, 307.7)
- added C340: 22uF, Capacitor_SMD:C_0805_2012Metric, F.Cu at (152.8, 321.1)
- added C363: 56pF, Capacitor_SMD:C_0402_1005Metric, F.Cu at (155.2, 33.1)
- added C381: 47uF, Capacitor_SMD:C_1210_3225Metric, F.Cu at (161.0, 44.0)
- added C382: 0.1uF, Capacitor_SMD:C_0402_1005Metric, F.Cu at (158.7, 42.6)
- added C383: 0.1uF, Capacitor_SMD:C_0402_1005Metric, F.Cu at (158.7, 30.7)
- added C384: 47uF, Capacitor_SMD:C_1210_3225Metric, F.Cu at (164.4, 44.0)
- added C385: 47uF, Capacitor_SMD:C_1210_3225Metric, F.Cu at (164.4, 29.3)
- added C386: 0.047uF, Capacitor_SMD:C_0402_1005Metric, F.Cu at (155.2, 35.2)
- added C387: 4.7uF, Capacitor_SMD:C_0402_1005Metric, F.Cu at (154.1, 40.5)
- added C397: 12.5pF, Capacitor_SMD:C_0402_1005Metric, F.Cu at (311.2, 338.8)
- added C48: 1uF, Capacitor_SMD:C_0201_0603Metric, B.Cu at (272.5, 315.3)
- added C480: 10uF, Capacitor_SMD:C_0603_1608Metric, B.Cu at (238.7, 310.5)
- added C481: 22uF, Capacitor_SMD:C_0805_2012Metric, B.Cu at (237.8, 319.5)
- added C483: 10uF, Capacitor_SMD:C_0603_1608Metric, B.Cu at (238.7, 316.9)
- added C484: 10uF, Capacitor_SMD:C_0603_1608Metric, B.Cu at (238.7, 305.9)
- added C485: 22uF, Capacitor_SMD:C_0805_2012Metric, B.Cu at (250.8, 290.6)
- added C487: 10uF, Capacitor_SMD:C_0603_1608Metric, B.Cu at (254.7, 289.5)
- added C490: 10uF, Capacitor_SMD:C_0603_1608Metric, B.Cu at (264.9, 289.5)
- added C493: 22uF, Capacitor_SMD:C_0805_2012Metric, B.Cu at (259.8, 294.2)
- added C494: 10uF, Capacitor_SMD:C_0603_1608Metric, B.Cu at (261.7, 289.5)
- added C496: 10uF, Capacitor_SMD:C_0603_1608Metric, B.Cu at (258.5, 289.5)
- added C514: 0.1uF, Capacitor_SMD:C_0402_1005Metric, F.Cu at (119.5, 133.9)
- added C55: 4.7uF, Capacitor_SMD:C_0603_1608Metric, B.Cu at (287.1, 313.6)
- added C552: 10uF, Capacitor_SMD:C_0402_1005Metric, F.Cu at (230.1, 29.7)
- added C56: 0.1uF, Capacitor_SMD:C_0201_0603Metric, B.Cu at (297.2, 311.2)
- added C57: 0.1uF, Capacitor_SMD:C_0201_0603Metric, B.Cu at (297.2, 312.2)
- added C58: 0.1uF, Capacitor_SMD:C_0201_0603Metric, B.Cu at (295.5, 313.7)
- added C59: 0.1uF, Capacitor_SMD:C_0201_0603Metric, B.Cu at (296.4, 313.7)
- added C61: 0.1uF, Capacitor_SMD:C_0201_0603Metric, B.Cu at (286.4, 307.5)
- added C619: 1uF, Capacitor_SMD:C_0603_1608Metric, B.Cu at (95.7, 95.2)
- added C620: 1uF, Capacitor_SMD:C_0603_1608Metric, B.Cu at (94.5, 113.5)
- added C63: 0.1uF, Capacitor_SMD:C_0201_0603Metric, B.Cu at (291.4, 308.1)
- added C67: 0.1uF, Capacitor_SMD:C_0201_0603Metric, B.Cu at (290.6, 308.1)
- added C68: 0.1uF, Capacitor_SMD:C_0201_0603Metric, B.Cu at (293.4, 306.0)
- added C69: 4.7uF, Capacitor_SMD:C_0603_1608Metric, B.Cu at (291.2, 305.3)
- added C70: 10pF, Capacitor_SMD:C_0201_0603Metric, B.Cu at (297.2, 308.5)
- added C71: 0.1uF, Capacitor_SMD:C_0201_0603Metric, B.Cu at (292.5, 306.0)
- added C723: 0.1uF, Capacitor_SMD:C_0402_1005Metric, B.Cu at (96.8, 113.0)
- added C725: 10uF, Capacitor_SMD:C_0805_2012Metric, F.Cu at (104.7, 125.6)
- added C726: 0.1uF, Capacitor_SMD:C_0402_1005Metric, F.Cu at (155.2, 137.2)
- added C727: 0.1uF, Capacitor_SMD:C_0201_0603Metric, B.Cu at (234.7, 307.9)
- added C728: 0.1uF, Capacitor_SMD:C_0201_0603Metric, B.Cu at (242.7, 307.9)
- added C729: 0.1uF, Capacitor_SMD:C_0201_0603Metric, B.Cu at (256.6, 293.5)
- added C730: 0.1uF, Capacitor_SMD:C_0201_0603Metric, B.Cu at (256.6, 285.5)
- added C731: 22uF, Capacitor_SMD:C_0805_2012Metric, F.Cu at (140.8, 317.1)
- added C732: 22uF, Capacitor_SMD:C_0805_2012Metric, F.Cu at (138.5, 317.1)
- added C733: 22uF, Capacitor_SMD:C_0805_2012Metric, B.Cu at (104.6, 128.3)
- added C734: 22uF, Capacitor_SMD:C_0805_2012Metric, B.Cu at (108.8, 134.2)
- added C735: 22uF, Capacitor_SMD:C_0805_2012Metric, B.Cu at (108.8, 137.2)
- added C736: 22uF, Capacitor_SMD:C_0805_2012Metric, B.Cu at (108.8, 140.1)
- added C737: 22uF, Capacitor_SMD:C_0805_2012Metric, B.Cu at (104.6, 137.1)
- added C738: 22uF, Capacitor_SMD:C_0805_2012Metric, B.Cu at (104.6, 134.2)
- added C739: 22uF, Capacitor_SMD:C_0805_2012Metric, B.Cu at (104.6, 131.3)
- added C740: 22uF, Capacitor_SMD:C_0805_2012Metric, B.Cu at (108.7, 143.0)
- added C741: 0.1uF, Capacitor_SMD:C_0402_1005Metric, F.Cu at (156.3, 137.2)
- added C742: 10uF, Capacitor_SMD:C_0603_1608Metric, F.Cu at (153.5, 137.8)
- added C743: 22uF, Capacitor_SMD:C_0805_2012Metric, B.Cu at (104.6, 143.0)
- added C744: 22uF, Capacitor_SMD:C_0805_2012Metric, B.Cu at (104.6, 140.1)
- added C745: 0.1uF, Capacitor_SMD:C_0402_1005Metric, F.Cu at (156.3, 152.0)
- added C746: 0.1uF, Capacitor_SMD:C_0402_1005Metric, F.Cu at (155.2, 152.0)
- added C747: 10uF, Capacitor_SMD:C_0603_1608Metric, F.Cu at (153.9, 151.4)
- added C75: 2.2uF, Capacitor_SMD:C_0402_1005Metric, B.Cu at (290.2, 313.9)
- added C752: 150uF, Capacitor_Tantalum_SMD:CP_EIA-7343-20_Kemet-V, F.Cu at (508.2, 126.8)
- added C753: 0.1uF, Capacitor_SMD:C_0201_0603Metric, F.Cu at (135.1, 309.1)
- added D12: SMAJ22A, Diode_SMD:D_SMA, B.Cu at (95.2, 107.7)
- added D2: SMAJ22A, Diode_SMD:D_SMA, B.Cu at (95.7, 87.9)
- added J13: BM04B-SRSS-TB_LF__SN_, barebones:JST_BM04B-SRSS-TB_LF__SN_, B.Cu at (395.0, 94.8)
- added J20: 5055671571, barebones:CONN_505567_15_MOL, F.Cu at (321.3, 218.1)
- added J23: 10137062-00021LF, barebones:AMPHENOL_10137062-00021LF, F.Cu at (105.7, 108.2)
- added J26: 10137062-00021LF, barebones:AMPHENOL_10137062-00021LF, F.Cu at (105.7, 89.5)
- added L5: XFL4015-471MEC, barebones:IND-SMD_L4.0-W4.0_XFL4020-102MEB, F.Cu at (544.8, 297.6)
- added L8: XAL7030-152MEC, barebones:INDDFN750X750X310-2N, F.Cu at (170.8, 36.6)
- added Q5: BSS138, Package_TO_SOT_SMD:SOT-23, F.Cu at (278.2, 34.6)
- added R122: 10k, Resistor_SMD:R_0402_1005Metric, B.Cu at (290.3, 340.8)
- added R196: 10k, Resistor_SMD:R_0201_0603Metric, F.Cu at (155.4, 36.4)
- added R197: 49.9k, Resistor_SMD:R_0201_0603Metric, F.Cu at (155.9, 41.2)
- added R202: 10k, Resistor_SMD:R_0402_1005Metric, F.Cu at (232.9, 29.7)
- added R213: 57.6k, Resistor_SMD:R_0402_1005Metric, F.Cu at (156.3, 33.1)
- added R220: 10k, Resistor_SMD:R_0402_1005Metric, F.Cu at (157.4, 33.1)
- added R254: 10k, Resistor_SMD:R_0201_0603Metric, B.Cu at (367.1, 178.8)
- added R26: 10k, Resistor_SMD:R_0201_0603Metric, B.Cu at (286.4, 309.4)
- added R36: 10k, Resistor_SMD:R_0201_0603Metric, B.Cu at (286.4, 311.2)
- added R38: 10k, Resistor_SMD:R_0201_0603Metric, B.Cu at (286.4, 312.1)
- added R39: 10k, Resistor_SMD:R_0201_0603Metric, B.Cu at (286.4, 308.4)
- added R40: 10k, Resistor_SMD:R_0201_0603Metric, B.Cu at (291.5, 309.5)
- added R42: 10k, Resistor_SMD:R_0201_0603Metric, B.Cu at (286.4, 310.3)
- added R43: 10k, Resistor_SMD:R_0201_0603Metric, B.Cu at (291.5, 310.5)
- added R46: 10k, Resistor_SMD:R_0201_0603Metric, B.Cu at (291.5, 312.6)
- added R47: 10k, Resistor_SMD:R_0201_0603Metric, B.Cu at (297.2, 309.5)
- added R48: 10k, Resistor_SMD:R_0201_0603Metric, B.Cu at (294.6, 313.7)
- added R59: 22R, Resistor_SMD:R_0201_0603Metric, B.Cu at (292.3, 308.1)
- added R63: 47k, Resistor_SMD:R_0201_0603Metric, B.Cu at (293.2, 308.1)
- added U21: DF40C-30DP-0.4V51, barebones:HIROSE_DF40C-30DP-0.4V-58, F.Cu at (565.8, 308.6)
- added U23: KLMCG4JETD-B041, barebones:BGA-153_L13.0-W11.5-P0.50-TL_KLM8G1GEME-B041, F.Cu at (291.9, 308.8)
- added U24: TPS56C215RNNR, barebones:QFN50P350X350X100-18N, F.Cu at (159.1, 36.7)
- added U29: TPS62933DRLR, barebones:SOTFL50P160X60-8N, F.Cu at (266.3, 30.0)
- added U39: TPS62933DRLR, barebones:SOTFL50P160X60-8N, F.Cu at (134.5, 311.3)
- added U40: TPS62933DRLR, barebones:SOTFL50P160X60-8N, F.Cu at (167.4, 177.1)
- added U42: TPS62933DRLR, barebones:SOTFL50P160X60-8N, F.Cu at (167.4, 209.4)
- added U44: TPS62933DRLR, barebones:SOTFL50P160X60-8N, F.Cu at (266.3, 44.6)
- C1, C114, C115, C122, C123, C129, C130, C131, C135, C136, C138, C139, C142, C143, C144, C145, C146, C147, C151, C152, C153, C154, C18, C182, C19, C191, C197, C205, C206, C210, C211, C217, C229, C230, C233, C234, C236, C239, C244, C245, C252, C26, C263, C265, C267, C27, C270, C271, C277, C278, C279, C292, C293, C300, C301, C421, C454, C588, C593, C598, C607, C610, C618, C685, C7: footprint Capacitor_SMD:C_0402_1005Metric -> Capacitor_SMD:C_0603_1608Metric
- C141: footprint Capacitor_SMD:C_0402_1005Metric -> Capacitor_SMD:C_0201_0603Metric
- C164, C275, C276, C608, C89, C90, C91, C92: footprint Capacitor_SMD:C_0402_1005Metric -> Capacitor_SMD:C_0805_2012Metric
- C165, C166, C176, C2, C21, C22, C23, C24, C259, C28, C280, C281, C3, C31, C33, C34, C35, C37, C39, C42, C50, C52, C54, C591, C605, C624, C637, C686, C8, C9: footprint Capacitor_SMD:C_0201_0603Metric -> Capacitor_SMD:C_0402_1005Metric
- C177, C178, C179, C187, C188, C189, C192, C193, C195, C199, C200, C201, C207, C208, C213, C214, C215, C216, C218, C219, C246, C247, C249, C319, C320, C337, C691, C692, C695, C696: footprint Capacitor_SMD:C_0402_1005Metric -> Capacitor_SMD:C_0805_2012Metric; moved to F.Cu
- C202: value 22uF -> 10uF; footprint Capacitor_SMD:C_0402_1005Metric -> Capacitor_SMD:C_0805_2012Metric; moved to F.Cu
- C204, C509, C672: footprint Capacitor_SMD:C_0201_0603Metric -> Capacitor_SMD:C_0402_1005Metric; moved to F.Cu
- C209, C336, C338, C339: value 10uF -> 22uF; footprint Capacitor_SMD:C_0402_1005Metric -> Capacitor_SMD:C_0805_2012Metric; moved to F.Cu
- C242, C251, C254, C417, C468, C577, C578, C579, C580, C582, C601: footprint Capacitor_SMD:C_0603_1608Metric -> Capacitor_SMD:C_0805_2012Metric
- C248: value 47uF -> 22uF; footprint Capacitor_SMD:C_0402_1005Metric -> Capacitor_SMD:C_0805_2012Metric; moved to F.Cu
- C253: footprint Capacitor_SMD:C_0201_0603Metric -> Capacitor_SMD:C_0603_1608Metric
- C255, C256: value 0.1uF -> 1uF; footprint Capacitor_SMD:C_0603_1608Metric -> Capacitor_SMD:C_0402_1005Metric; moved to B.Cu
- C257, C258: value 0.1uF -> 10uF; moved to B.Cu
- C274, C322, C441, C443, C508, C510, C525, C694, D10, D11, L4, R145, R152, R153, R154, R157, R188, R218, R61, R73, S8: moved to F.Cu
- C285, C286, C287, C288, C289, C296, C297, C298, C299, C303, C308, C309, C315, C316, C690: footprint Capacitor_SMD:C_0402_1005Metric -> Capacitor_SMD:C_0603_1608Metric; moved to F.Cu
- C317, C318: value 22uF -> 10uF; footprint Capacitor_SMD:C_0402_1005Metric -> Capacitor_SMD:C_0603_1608Metric; moved to B.Cu
- C325, C326, C328, C329, C348, C349: footprint Capacitor_SMD:C_0603_1608Metric -> Capacitor_SMD:C_1210_3225Metric
- C330, C331, C332: value 10uF -> 22uF; footprint Capacitor_SMD:C_0603_1608Metric -> Capacitor_SMD:C_0805_2012Metric; moved to F.Cu
- C334: value 33uF -> 22uF; footprint Capacitor_SMD:C_0603_1608Metric -> Capacitor_SMD:C_0805_2012Metric; moved to F.Cu
- C335: value 33uF -> 47uF; footprint Capacitor_SMD:C_0603_1608Metric -> Capacitor_SMD:C_0805_2012Metric; moved to F.Cu
- C341, C342: footprint Capacitor_SMD:C_0402_1005Metric -> Capacitor_SMD:C_1210_3225Metric; moved to B.Cu
- C343, C503: footprint Capacitor_SMD:C_0402_1005Metric -> Capacitor_SMD:C_0805_2012Metric; moved to B.Cu
- C347: value 22uF -> 0.1uF; footprint Capacitor_SMD:C_0603_1608Metric -> Capacitor_SMD:C_0402_1005Metric; moved to B.Cu
- C350, C351: value 10uF -> 22uF; footprint Capacitor_SMD:C_0402_1005Metric -> Capacitor_SMD:C_0603_1608Metric
- C353: value 4.7uF -> 22uF; footprint Capacitor_SMD:C_0402_1005Metric -> Capacitor_SMD:C_0603_1608Metric
- C366: value 22uF -> 47uF; footprint Capacitor_SMD:C_0603_1608Metric -> Capacitor_SMD:C_1210_3225Metric
- C369, C371, C374, C375: value 10uF -> 47uF; footprint Capacitor_SMD:C_0402_1005Metric -> Capacitor_SMD:C_1210_3225Metric; moved to F.Cu
- C372, C373: footprint Capacitor_SMD:C_0603_1608Metric -> Capacitor_SMD:C_0402_1005Metric; moved to B.Cu
- C395, C524: footprint Capacitor_SMD:C_0603_1608Metric -> Capacitor_SMD:C_0402_1005Metric
- C396, C399, C403, C404, C412, C413, C418, C420, C423, C425, C426, C431, C449, C458, C465, C473, C475, C511, C513, C523, C542, C544, C545, C546, C549, C550, C551, C555, C560, C563, C564, C573, C621, C622, C698, C707, C708, C709, C710, C711, C712, C713, C714, C715, C717, C718, C719, C720, C721, C722, D5, FL2, FL3, J19, J24, J25, L15, Q4, R132, R141, R156, R185, R192, R193, R219, R221, R222, R223, R224, R226, R243, R244, R58, R64, TP5, TP6, U13, U16, U17, U28, U34, U37, Y6: moved to B.Cu
- C452, C453, C455, C456, C492, C495, C497, C501, C502, C592, C594, C597, C599, C600, C606, C616: value 100nF -> 0.1uF
- C504: value 100nF -> 0.1uF; footprint Capacitor_SMD:C_0402_1005Metric -> Capacitor_SMD:C_0603_1608Metric; moved to B.Cu
- C540: value 10uF -> 0.1uF; moved to F.Cu
- C567: value 1uF -> 0.1uF; moved to B.Cu
- C568: value 1uF -> 10uF
- C604, C617, C687: footprint Capacitor_SMD:C_0402_1005Metric -> Capacitor_SMD:C_1206_3216Metric
- C609, C612: value 120uF -> 0.1uF; footprint Capacitor_SMD:C_0402_1005Metric -> Capacitor_SMD:C_0805_2012Metric
- C645, C660, C661: value 22uF -> 0.1uF; footprint Capacitor_SMD:C_0603_1608Metric -> Capacitor_SMD:C_0201_0603Metric
- C646, C647, C663, C664, C666, C667: value 10uF -> 0.1uF; footprint Capacitor_SMD:C_0402_1005Metric -> Capacitor_SMD:C_0201_0603Metric
- C674: value 0.1uF -> 33nF; moved to F.Cu
- C676, C678: value 0.1uF -> 22uF; footprint Capacitor_SMD:C_0201_0603Metric -> Capacitor_SMD:C_1210_3225Metric; moved to F.Cu
- C679: value 0.1uF -> 10uF; footprint Capacitor_SMD:C_0201_0603Metric -> Capacitor_SMD:C_1206_3216Metric; moved to F.Cu
- C680, C681: value 0.1uF -> 22uF; footprint Capacitor_SMD:C_0201_0603Metric -> Capacitor_SMD:C_1206_3216Metric; moved to F.Cu
- C682, C683: value 0.1uF -> 10uF; footprint Capacitor_SMD:C_0201_0603Metric -> Capacitor_SMD:C_0603_1608Metric; moved to F.Cu
- C684: value 10uF -> 22uF; footprint Capacitor_SMD:C_0402_1005Metric -> Capacitor_SMD:C_1206_3216Metric
- C688: value 22uF -> 10uF; footprint Capacitor_SMD:C_0402_1005Metric -> Capacitor_SMD:C_1206_3216Metric
- C693: footprint Capacitor_SMD:C_0402_1005Metric -> Capacitor_SMD:C_0201_0603Metric; moved to F.Cu
- C703, C704: footprint Capacitor_SMD:C_0402_1005Metric -> Capacitor_SMD:C_1210_3225Metric
- J1: value 12401610E4_2A -> DF40C-34DP-0.4V_58_; footprint barebones:AMPHENOL_12401610E4_2A -> barebones:HIROSE_DF40C-34DP-0.4V_58_
- J5: value 12401610E4_2A -> SM04B-SRSS-TB_LF__SN_; footprint barebones:AMPHENOL_12401610E4_2A -> barebones:JST_SM04B-SRSS-TB_LF__SN_
- L7: value XAL6030-332MEC -> FDSD0420-H-2R2M=P3
- Q11, Q12, Q13, Q14: footprint barebones:TRANS_CSD18543Q3A -> Package_SON:VSON-8_3.3x3.3mm_P0.65mm_NexFET
- R118, R120, R121: footprint Resistor_SMD:R_0603_1608Metric -> Resistor_SMD:R_0402_1005Metric; moved to B.Cu
- R143, R144, R146, R147, R174, R179, R183: footprint Resistor_SMD:R_0201_0603Metric -> Resistor_SMD:R_0402_1005Metric
- R182: value 100k -> 10k; footprint Resistor_SMD:R_0201_0603Metric -> Resistor_SMD:R_0402_1005Metric
- R187: footprint Resistor_SMD:R_0402_1005Metric -> Resistor_SMD:R_0201_0603Metric; moved to F.Cu
- R212: footprint Resistor_SMD:R_0603_1608Metric -> Resistor_SMD:R_0402_1005Metric
- R225: value 10k -> 140k; footprint Resistor_SMD:R_0201_0603Metric -> Resistor_SMD:R_0402_1005Metric
- R234: value 4.7k -> 10k; footprint Resistor_SMD:R_0201_0603Metric -> Resistor_SMD:R_0402_1005Metric
- R235: value 4.7k -> 52.3k; footprint Resistor_SMD:R_0201_0603Metric -> Resistor_SMD:R_0402_1005Metric
- R256, R258: value 20.2k -> 20k
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Connections:
- net /DDR_CH1_CKB_C renamed /DDR_CH1_CK_C_N
- net /DDR_CH1_CKB_D renamed /DDR_CH1_CK_D_N
- net /DDR_CH1_CK_C renamed /DDR_CH1_CK_C_P
- net /DDR_CH1_CK_D renamed /DDR_CH1_CK_D_P
- net /DDR_CH1_DQS0N_C renamed /DDR_CH1_DQS0_C_N
- net /DDR_CH1_DQS0N_D renamed /DDR_CH1_DQS0_D_N
- net /DDR_CH1_DQS0P_C renamed /DDR_CH1_DQS0_C_P
- net /DDR_CH1_DQS0P_D renamed /DDR_CH1_DQS0_D_P
- net /DDR_CH1_DQS1N_C renamed /DDR_CH1_DQS1_C_N
- net /DDR_CH1_DQS1N_D renamed /DDR_CH1_DQS1_D_N
- net /DDR_CH1_DQS1P_C renamed /DDR_CH1_DQS1_C_P
- net /DDR_CH1_DQS1P_D renamed /DDR_CH1_DQS1_D_P
- net Net-(J10-SSTX+) renamed /Peripheral IO Connectors/USB3_0_SSTX_P
- C153 pad 2: VDD_CPU_BIG0_S0 -> VDD_NPU_S0
- C154 pad 2: VDD_CPU_BIG0_S0 -> VDD_NPU_S0
- C202 pad 1: VDD_LOG_S0 -> VDDQ_DDR_CK_S0
- C209 pad 1: VDDQ_DDR_CK_S0 -> VCC_3V3_S3
- C248 pad 1: VDD_GPU_S0 -> VCC1V8_PMU_DDR_S3
- C255 pad 1: /SYS_PWR -> GND
- C255 pad 2: GND -> VDDA_0V85_S0
- C256 pad 1: /SYS_PWR -> GND
- C256 pad 2: GND -> VCCA_1V8_S0
- C257 pad 1: /SYS_PWR -> GND
- C257 pad 2: GND -> VDD_LOG_S0
- C258 pad 1: /SYS_PWR -> GND
- C258 pad 2: GND -> VDD_LOG_S0
- C273 pad 2: /Power and Ground/VSYS_MAIN -> VIN
- C274 pad 1: /Power and Ground/VSYS_MAIN -> VIN
- C284 pad 1: Net-(C284-Pad1) -> VDD_NPU_S0
- C285 pad 1: Net-(C284-Pad1) -> VDD_NPU_S0
- C286 pad 1: Net-(C284-Pad1) -> VDD_NPU_S0
- C287 pad 1: Net-(C284-Pad1) -> VDD_NPU_S0
- C288 pad 1: Net-(C284-Pad1) -> VDD_NPU_S0
- C289 pad 1: Net-(C284-Pad1) -> VDD_NPU_S0
- C292 pad 1: VCC_5V0_SYS -> VCC_4V0_SYS
- C293 pad 1: VCC_5V0_SYS -> VCC_4V0_SYS
- C294 pad 1: Net-(C294-Pad1) -> VDD_CPU_BIG0_S0
- C296 pad 1: Net-(C294-Pad1) -> VDD_CPU_BIG0_S0
- C297 pad 1: Net-(C294-Pad1) -> VDD_CPU_BIG0_S0
- C298 pad 1: Net-(C294-Pad1) -> VDD_CPU_BIG0_S0
- C299 pad 1: Net-(C294-Pad1) -> VDD_CPU_BIG0_S0
- C300 pad 1: VCC_5V0_SYS -> VCC_4V0_SYS
- C301 pad 1: VCC_5V0_SYS -> VCC_4V0_SYS
- C302 pad 1: Net-(C302-Pad1) -> VDD_CPU_BIG1_S0
- C303 pad 1: Net-(C302-Pad1) -> VDD_CPU_BIG1_S0
- C308 pad 1: Net-(C302-Pad1) -> VDD_CPU_BIG1_S0
- C309 pad 1: Net-(C302-Pad1) -> VDD_CPU_BIG1_S0
- C315 pad 1: Net-(C302-Pad1) -> VCC_4V0_SYS
- C316 pad 1: Net-(C294-Pad1) -> VCC_4V0_SYS
- C317 pad 1: VCC_5V0_SYS -> GND
- C317 pad 2: GND -> VDD_LOG_S0
- C318 pad 1: VCC_5V0_SYS -> GND
- C318 pad 2: GND -> VDD_LOG_S0
- C319 pad 1: VCC_3V3_S3 -> VDD_VDENC_S0
- C320 pad 1: Net-(C302-Pad1) -> VDD_VDENC_S0
- C325 pad 2: /Power and Ground/VSYS_MAIN -> VIN
- C326 pad 2: /Power and Ground/VSYS_MAIN -> VIN
- C328 pad 2: /Power and Ground/VSYS_MAIN -> VIN
- C329 pad 2: /Power and Ground/VSYS_MAIN -> VIN
- C330 pad 1: GND -> VCC_2V0_PLDO_S3
- C330 pad 2: /Power and Ground/VSYS_MAIN -> GND
- C331 pad 1: GND -> VDD_DDR_S0
- C331 pad 2: /Power and Ground/VSYS_MAIN -> GND
- C332 pad 1: GND -> VDD_DDR_S0
- C332 pad 2: /Power and Ground/VSYS_MAIN -> GND
- C334 pad 1: GND -> VDD_DDR_S0
- C334 pad 2: /Power and Ground/VSYS_MAIN -> GND
- C335 pad 1: GND -> VDD_GPU_S0
- C335 pad 2: /Power and Ground/VSYS_MAIN -> GND
- C336 pad 1: GND -> VDD_LOG_S0
- C336 pad 2: VDD_NPU_S0 -> GND
- C337 pad 1: GND -> VDDQ_DDR_CK_S0
- C337 pad 2: VDD_NPU_S0 -> GND
- C338 pad 1: GND -> VCC_3V3_S3
- C338 pad 2: VDD_NPU_S0 -> GND
- C339 pad 1: GND -> VDD_VDENC_S0
- C339 pad 2: VDD_NPU_S0 -> GND
- C341 pad 2: /Power and Ground/VSYS_MAIN -> VIN
- C342 pad 2: /Power and Ground/VSYS_MAIN -> VIN
- C343 pad 2: /Power and Ground/VSYS_MAIN -> VIN
- C347 pad 1: GND -> Net-(U44-BST)
- C347 pad 2: VCC_5V0_SYS -> Net-(U44-SW)
- C350 pad 1: GND -> VDD_CPU_BIG0_S0
- C350 pad 2: VCC_5V0_SYS -> GND
- C351 pad 1: GND -> VDD_NPU_S0
- C351 pad 2: VCC_5V0_SYS -> GND
- C352 pad 1: GND -> Net-(U24-BOOT)
- C352 pad 2: VCC_5V0_SYS -> /Power and Ground/MAIN_SW
- C353 pad 1: GND -> VDD_CPU_BIG1_S0
- C353 pad 2: VCC_12V_EDP -> GND
- C369 pad 2: VDD_LOG_S0 -> VCC_4V0_SYS
- C371 pad 2: VDD_LOG_S0 -> VCC_4V0_SYS
- C374 pad 2: VDD_LOG_S0 -> VCC_4V0_SYS
- C375 pad 2: VDD_LOG_S0 -> VIN
- C503 pad 1: Net-(J12-VDD) -> GND
- C504 pad 1: Net-(J12-VDD) -> GND
- C540 pad 1: VDD2_DDR_S3 -> GND
- C540 pad 2: GND -> Net-(U44-EN)
- C567 pad 1: VBUS_A -> /Peripheral IO Connectors/USB1_VBUS
- C568 pad 1: VBUS_A -> GND
- C568 pad 2: GND -> VIN
- C584 pad 1: VBUS_A -> /Peripheral IO Connectors/USB2_VBUS
- C588 pad 1: VBUS_A -> /Peripheral IO Connectors/USB1_VBUS
- C604 pad 2: VCC_5V0_SYS -> VIN
- C617 pad 2: VCC3V3_PCIE30_1 -> VIN
- C645 pad 1: VDDQ_DDR_CK_S0 -> VDD2_DDR_S3
- C646 pad 1: VDDQ_DDR_CK_S0 -> VDD2_DDR_S3
- C647 pad 1: VDDQ_DDR_CK_S0 -> VDD2_DDR_S3
- C672 pad 1: VDD2_DDR_S3 -> GND
- C672 pad 2: GND -> VIN
- C674 pad 1: VDD2_DDR_S3 -> GND
- C674 pad 2: GND -> Net-(U44-SS)
- C676 pad 1: VDD2_DDR_S3 -> GND
- C676 pad 2: GND -> VCC_12V_EDP
- C678 pad 1: VDD2_DDR_S3 -> GND
- C678 pad 2: GND -> VCC_12V_EDP
- C679 pad 1: VDDQ_DDR_CK_S0 -> GND
- C679 pad 2: GND -> VIN
- C680 pad 1: VDD2_DDR_S3 -> GND
- C680 pad 2: GND -> VCC3V3_PCIE30_1
- C681 pad 1: VDDQ_DDR_CK_S0 -> GND
- C681 pad 2: GND -> VCC3V3_PCIE30_1
- C682 pad 1: VDD2_DDR_S3 -> GND
- C682 pad 2: GND -> VCC3V3_PCIE30_1
- C683 pad 1: VDDQ_DDR_CK_S0 -> GND
- C683 pad 2: GND -> VCC3V3_PCIE30_1
- C684 pad 2: VCC_5V0_SYS -> VCC3V3_PCIE30
- C685 pad 2: VCC_5V0_SYS -> VIN
- C687 pad 2: VCC3V3_PCIE30_1 -> VCC3V3_PCIE30
- C688 pad 2: VCC3V3_PCIE30_1 -> VIN
- C690 pad 2: Net-(U8-EN) -> VIN
- C691 pad 2: VCC_5V0_SYS -> VIN
- C692 pad 2: VCC_5V0_SYS -> VIN
- C693 pad 2: VCC_5V0_SYS -> VIN
- C699 pad 2: /Power and Ground/VSYS_MAIN -> VIN
- C700 pad 2: /Power and Ground/VSYS_MAIN -> VIN
- C701 pad 2: /Power and Ground/VSYS_MAIN -> VIN
- D10 pad 1: (no net) -> /Peripheral IO Connectors/USB3_0_RX_N
- D10 pad 11: /Peripheral IO Connectors/USB3_0_DP -> /Peripheral IO Connectors/USB3_0_DN
- D10 pad 12: /Peripheral IO Connectors/USB3_0_DN -> /Peripheral IO Connectors/USB3_0_DP
- D10 pad 2: (no net) -> /Peripheral IO Connectors/USB3_0_RX_P
- D10 pad 3: (no net) -> /Peripheral IO Connectors/USB3_0_DP
- D10 pad 4: (no net) -> /Peripheral IO Connectors/USB3_0_DN
- D10 pad 6: (no net) -> /Peripheral IO Connectors/USB3_0_TX_N
- D10 pad 7: (no net) -> /Peripheral IO Connectors/USB3_0_TX_P
- D10 pad 8: /Peripheral IO Connectors/USB3_0_TX_N -> /Peripheral IO Connectors/USB3_0_TX_P
- D10 pad 9: /Peripheral IO Connectors/USB3_0_TX_P -> /Peripheral IO Connectors/USB3_0_TX_N
- D11 pad 1: (no net) -> /Peripheral IO Connectors/USB3_1_RX_N
- D11 pad 2: (no net) -> /Peripheral IO Connectors/USB3_1_RX_P
- D11 pad 3: (no net) -> /Peripheral IO Connectors/USB3_1_DP
- D11 pad 4: (no net) -> /Peripheral IO Connectors/USB3_1_DN
- D11 pad 6: (no net) -> /Peripheral IO Connectors/USB3_1_TX_N
- D11 pad 7: (no net) -> /Peripheral IO Connectors/USB3_1_TX_P
- D11 pad 8: /Peripheral IO Connectors/USB3_1_TX_N -> /Peripheral IO Connectors/USB3_1_TX_P
- D11 pad 9: /Peripheral IO Connectors/USB3_1_TX_P -> /Peripheral IO Connectors/USB3_1_TX_N
- D14 pad 10: unconnected-(D14-NC-Pad10) -> /Peripheral IO Connectors/TMDS_DATA2_1_DP
- D14 pad 6: unconnected-(D14-NC-Pad6) -> /Peripheral IO Connectors/TMDS_DATA1_1_DM
- D14 pad 7: unconnected-(D14-NC-Pad7) -> /Peripheral IO Connectors/TMDS_DATA1_1_DP
- D14 pad 9: unconnected-(D14-NC-Pad9) -> /Peripheral IO Connectors/TMDS_DATA2_1_DM
- D15 pad 10: unconnected-(D15-NC-Pad10) -> /Peripheral IO Connectors/TMDS_DATA0_1_DP
- D15 pad 6: unconnected-(D15-NC-Pad6) -> /Peripheral IO Connectors/TMDS_CLOCK_1_DM
- D15 pad 7: unconnected-(D15-NC-Pad7) -> /Peripheral IO Connectors/TMDS_CLOCK_1_DP
- D15 pad 9: unconnected-(D15-NC-Pad9) -> /Peripheral IO Connectors/TMDS_DATA0_1_DM
- D19 pad 1: (no net) -> /SDMMC_DAT2
- D19 pad 2: (no net) -> /SDMMC_DAT3
- D19 pad 3: (no net) -> /SDMMC_CMD
- D19 pad 4: (no net) -> /SDMMC_CLK
- D19 pad 6: (no net) -> /SDMMC_DAT0
- D19 pad 7: (no net) -> /SDMMC_DAT1
- D3 pad A: /Power and Ground/EDP_SW -> unconnected-(D3-PadA)
- D3 pad C: VCC_12V_EDP -> unconnected-(D3-PadC)
- D6 pad 1: /USB_1_RX2N -> /Peripheral IO Connectors/USB1_TX2N
- D6 pad 10: unconnected-(D6-NC-Pad10) -> /Peripheral IO Connectors/USB1_TX2N
- D6 pad 2: /USB_1_RX2P -> /Peripheral IO Connectors/USB1_TX2P
- D6 pad 4: /USB_1_RX1N -> /USB_1_RX2P
- D6 pad 5: /USB_1_RX1P -> /USB_1_RX2N
- D6 pad 6: unconnected-(D6-NC-Pad6) -> /USB_1_RX2N
- D6 pad 7: unconnected-(D6-NC-Pad7) -> /USB_1_RX2P
- D6 pad 9: unconnected-(D6-NC-Pad9) -> /Peripheral IO Connectors/USB1_TX2P
- D7 pad 10: unconnected-(D7-NC-Pad10) -> /Peripheral IO Connectors/USB1_TX1N
- D7 pad 4: /Peripheral IO Connectors/USB1_TX2N -> /USB_1_RX1P
- D7 pad 5: /Peripheral IO Connectors/USB1_TX2P -> /USB_1_RX1N
- D7 pad 6: unconnected-(D7-NC-Pad6) -> /USB_1_RX1N
- D7 pad 7: unconnected-(D7-NC-Pad7) -> /USB_1_RX1P
- D7 pad 9: unconnected-(D7-NC-Pad9) -> /Peripheral IO Connectors/USB1_TX1P
- D8 pad 1: /USB_2_RX2N -> /Peripheral IO Connectors/USB2_TX1N
- D8 pad 10: unconnected-(D8-NC-Pad10) -> /Peripheral IO Connectors/USB2_TX1N
- D8 pad 2: /USB_2_RX2P -> /Peripheral IO Connectors/USB2_TX1P
- D8 pad 4: /USB_2_RX1N -> /USB_2_RX1P
- D8 pad 5: /USB_2_RX1P -> /USB_2_RX1N
- D8 pad 6: unconnected-(D8-NC-Pad6) -> /USB_2_RX1N
- D8 pad 7: unconnected-(D8-NC-Pad7) -> /USB_2_RX1P
- D8 pad 9: unconnected-(D8-NC-Pad9) -> /Peripheral IO Connectors/USB2_TX1P
- D9 pad 1: /Peripheral IO Connectors/USB2_TX1N -> /Peripheral IO Connectors/USB2_TX2N
- D9 pad 10: unconnected-(D9-NC-Pad10) -> /Peripheral IO Connectors/USB2_TX2N
- D9 pad 2: /Peripheral IO Connectors/USB2_TX1P -> /Peripheral IO Connectors/USB2_TX2P
- D9 pad 4: /Peripheral IO Connectors/USB2_TX2N -> /USB_2_RX2P
- D9 pad 5: /Peripheral IO Connectors/USB2_TX2P -> /USB_2_RX2N
- D9 pad 6: unconnected-(D9-NC-Pad6) -> /USB_2_RX2N
- D9 pad 7: unconnected-(D9-NC-Pad7) -> /USB_2_RX2P
- D9 pad 9: unconnected-(D9-NC-Pad9) -> /Peripheral IO Connectors/USB2_TX2P
- J10 pad 8: Net-(J10-SSTX-) -> /Peripheral IO Connectors/USB3_0_SSTX_N
- J12 pad 4: Net-(J12-VDD) -> VCC_3V3_S3
- J15 pad 1: /Embedded Controller and Internal Audio/SPK_OUT_R_1+ -> unconnected-(J15-Pad1)
- J15 pad 2: /Embedded Controller and Internal Audio/SPK_OUT_R_1- -> unconnected-(J15-Pad2)
- J17 pad 1: /Power and Ground/PACK_P -> unconnected-(J17-Pad1)
- J17 pad 12: GND -> unconnected-(J17-Pad12)
- J17 pad 13: GND -> unconnected-(J17-Pad13)
- J17 pad 14: GND -> unconnected-(J17-Pad14)
- J17 pad 15: GND -> unconnected-(J17-Pad15)
- J17 pad 16: GND -> unconnected-(J17-Pad16)
- J17 pad 2: /Power and Ground/PACK_P -> unconnected-(J17-Pad2)
- J17 pad 3: /Power and Ground/PACK_P -> unconnected-(J17-Pad3)
- J17 pad 4: /Power and Ground/PACK_P -> unconnected-(J17-Pad4)
- J17 pad 5: /Power and Ground/PACK_P -> unconnected-(J17-Pad5)
- J17 pad 7: /BATT_PRES -> unconnected-(J17-Pad7)
- J17 pad 8: /SMBD_BATT -> unconnected-(J17-Pad8)
- J17 pad 9: /SMBC_BATT -> unconnected-(J17-Pad9)
- J25 pad 30: /BACKLIGHT_DP -> VCC_5V0_SYS
- J25 pad 32: /BACKLIGHT_DP -> VCC_5V0_SYS
- L10 pad 2: Net-(C302-Pad1) -> VDD_CPU_BIG1_S0
- L14 pad 1: Net-(U26-FB) -> unconnected-(L14-Pad1)
- L14 pad 2: /Power and Ground/EDP_SW -> unconnected-(L14-Pad2)
- L15 pad 1: VCC_5V0_SYS -> unconnected-(L15-Pad1)
- L15 pad 2: /Power and Ground/PWM_SW -> unconnected-(L15-Pad2)
- L18 pad 2: Net-(C284-Pad1) -> VDD_NPU_S0
- L19 pad 2: Net-(C294-Pad1) -> VDD_CPU_BIG0_S0
- L7 pad 1: /Power and Ground/B_SW_1 -> Net-(U44-SW)
- L7 pad 2: VCC_4V0_SYS -> VCC_12V_EDP
- Q13 pad 5: /Power and Ground/VSYS_MAIN -> VIN
- Q2 pad 1: VBUS_A -> /Peripheral IO Connectors/USB2_VBUS
- Q2 pad 2: VBUS_A -> /Peripheral IO Connectors/USB2_VBUS
- Q2 pad 3: VBUS_A -> /Peripheral IO Connectors/USB2_VBUS
- Q9 pad 1: VBUS_A -> /Peripheral IO Connectors/USB1_VBUS
- Q9 pad 2: VBUS_A -> /Peripheral IO Connectors/USB1_VBUS
- Q9 pad 3: VBUS_A -> /Peripheral IO Connectors/USB1_VBUS
- R182 pad 1: GND -> /GPIO3_B5_U
- R182 pad 2: /12C1_EXTI_EC -> VCC_3V3_S0
- R183 pad 1: GND -> /PCIE30X4_PWREN_H
- R183 pad 2: /GPIO3_B5_U -> Net-(U44-EN)
- R187 pad 2: Net-(U8-EN) -> Net-(U39-EN)
- R225 pad 1: GND -> VCC_12V_EDP
- R225 pad 2: /BUCK_PWRON -> Net-(U44-FB)
- R234 pad 1: /Macro Pad/EN_BTN_2 -> Net-(U24-PGOOD)
- R234 pad 2: VCC_3V3_S3 -> Net-(U24-VREG5)
- R235 pad 1: /Macro Pad/EN_CHAN_A_2 -> Net-(U24-VREG5)
- R235 pad 2: VCC_3V3_S3 -> Net-(U24-MODE)
- R242 pad 1: /Power and Ground/VSYS_MAIN -> VIN
- R260 pad 1: /I2C3_SCL_M0 -> /Peripheral IO Connectors/I2C8_SCL_M2
- R272 pad 1: /I2C3_SDA_M0 -> /Peripheral IO Connectors/I2C8_SDA_M2
- R68 pad 1: /Power and Ground/VSYS_MAIN -> VIN
- R73 pad 1: /Power and Ground/VSYS_MAIN -> VIN
- R92 pad 2: Net-(C284-Pad1) -> VDD_NPU_S0
- R93 pad 2: Net-(C294-Pad1) -> VDD_CPU_BIG0_S0
- R94 pad 2: Net-(C302-Pad1) -> VDD_CPU_BIG1_S0
- U1 pad AA32: unconnected-(U1C-EMMC_D5/I2C1_SDA_M3/UART5_TX_M2/GPIO2_D5_U-PadAA32) -> /High Speed IO/EMMC_D5
- U1 pad AA33: unconnected-(U1C-EMMC_D3/FSPI_D3_M0/GPIO2_D3_U-PadAA33) -> /High Speed IO/EMMC_D3
- U1 pad AA34: unconnected-(U1C-EMMC_RSTN/I2C2_SCL_M2/UART5_RTSN_M1/GPIO2_A3_D-PadAA34) -> /High Speed IO/EMMC_RSTN
- U1 pad AL9: /USB_2_OTG_DM -> /USB_2_OTG_DN
- U1 pad AM12: /USB_1_OTG_DM -> /USB_1_OTG_DN
- U1 pad C25: unconnected-(U1F-PDM1_SDI0_M1/PCIE30X1_1_PERSTN_M2/PWM3_IR_M3/SPI2_CS0_M0/GPIO1_A7_U-PadC25) -> /MIC_DAT
- U1 pad C27: unconnected-(U1F-PDM1_SDI1_M1/PCIE30X4_CLKREQN_M3/SPI2_CS1_M0/GPIO1_B0_U-PadC27) -> /INT_ALS
- U1 pad E24: unconnected-(U1F-PDM1_CLK0_M1/PCIE30X1_0_PERSTN_M2/UART7_RX_M2/SPI0_CS0_M2/GPIO1_B4_U-PadE24) -> /MIC_CLK
- U1 pad E26: unconnected-(U1F-MIPI_CAMERA1_CLK_M0/SPDIF0_TX_M0/PCIE30X2_WAKEN_M3/HDMI_RX_HPDOUT_M2/I2C5_SCL_M3/UART1_TX_M1/GPIO1_B6_U-PadE26) -> /CAM_SW
- U1 pad E27: unconnected-(U1F-MIPI_CAMERA2_CLK_M0/SPDIF1_TX_M0/PCIE30X2_PERSTN_M3/HDMI_RX_CEC_M2/SATA2_ACT_LED_M1/I2C5_SDA_M3/UART1_RX_M1/PWM13_M2/GPIO1_B7_U-PadE27) -> /MIC_SW
- U1 pad F24: unconnected-(U1F-MIPI_CAMERA3_CLK_M0/HDMI_RX_SCL_M2/I2C8_SCL_M2/UART1_RTSN_M1/PWM14_M2/GPIO1_D6_U-PadF24) -> /I2C8_SCL_M2
- U1 pad F25: unconnected-(U1F-MIPI_CAMERA4_CLK_M0/PCIE30X2_CLKREQN_M3/HDMI_RX_SDA_M2/I2C8_SDA_M2/UART1_CTSN_M1/PWM15_IR_M3/GPIO1_D7_U-PadF25) -> /I2C8_SDA_M2
- U1 pad G27: /I2C3_SCL_M0 -> unconnected-(U1L-I2C3_SCL_M0/UART3_TX_M0/SPI4_MOSI_M0/GPIO1_C1_Z-PadG27)
- U1 pad G29: /I2C3_SDA_M0 -> unconnected-(U1L-I2C3_SDA_M0/UART3_RX_M0/SPI4_MISO_M0/GPIO1_C0_Z-PadG29)
- U1 pad T31: /MIC_CLK -> unconnected-(U1I-PDM0_CLK0_M1/PWM1_M0/I2C2_SDA_M0/CAN0_RX_M0/SPI0_MOSI_M0/PCIE30X1_0_CLKREQN_M0/GPIO0_C0_D-PadT31)
- U1 pad V26: unconnected-(U1C-EMMCIO_1V8-PadV26) -> VCC1V8_PMU_DDR_S3
- U1 pad V31: /MIC_DAT -> unconnected-(U1I-I2S1_SDI2_M1/PDM0_SDI0_M1/I2C6_SDA_M0/UART1_RTSN_M2/PWM6_M0/SPI0_MISO_M0/PCIE30X4_WAKEN_M0/GPIO0_C7_D-PadV31)
- U1 pad V32: unconnected-(U1C-EMMC_D2/FSPI_D2_M0/GPIO2_D2_U-PadV32) -> /High Speed IO/EMMC_D2
- U1 pad V33: unconnected-(U1C-EMMC_D7/FSPI_CS1N_M0/GPIO2_D7_U-PadV33) -> /High Speed IO/EMMC_D7
- U1 pad V34: unconnected-(U1C-EMMC_CLKOUT/GPIO2_A1_D-PadV34) -> /High Speed IO/EMMC_CLKOUT
- U1 pad W32: unconnected-(U1C-EMMC_D6/FSPI_CS0N_M0/GPIO2_D6_U-PadW32) -> /High Speed IO/EMMC_D6
- U1 pad W33: unconnected-(U1C-EMMC_D1/FSPI_D1_M0/GPIO2_D1_U-PadW33) -> /High Speed IO/EMMC_D1
- U1 pad W34: unconnected-(U1C-EMMC_CMD/FSPI_CLK_M0/GPIO2_A0_U-PadW34) -> /High Speed IO/EMMC_CMD
- U1 pad Y32: unconnected-(U1C-EMMC_D4/I2C1_SCL_M3/UART5_RX_M2/GPIO2_D4_U-PadY32) -> /High Speed IO/EMMC_D4
- U1 pad Y33: unconnected-(U1C-EMMC_D0/FSPI_D0_M0/GPIO2_D0_U-PadY33) -> /High Speed IO/EMMC_D0
- U1 pad Y34: unconnected-(U1C-EMMC_DATA_STROBE/I2C2_SDA_M2/UART5_CTSN_M1/GPIO2_A2_D-PadY34) -> /High Speed IO/EMMC_DATA_STROBE
- U13 pad 18: /INT_ALS -> unconnected-(U13-PA1-Pad18)
- U13 pad 45: unconnected-(U13-PD10-Pad45) -> /12C1_EXTI_EC
- U14 pad 22: /Power and Ground/VSYS_MAIN -> VIN
- U18 pad D1: VCC_5V0_SYS -> VCC_4V0_SYS
- U18 pad D2: VCC_5V0_SYS -> VCC_4V0_SYS
- U18 pad E1: VCC_5V0_SYS -> VCC_4V0_SYS
- U18 pad E2: VCC_5V0_SYS -> VCC_4V0_SYS
- U19 pad D1: VCC_5V0_SYS -> VCC_4V0_SYS
- U19 pad D2: VCC_5V0_SYS -> VCC_4V0_SYS
- U19 pad E1: VCC_5V0_SYS -> VCC_4V0_SYS
- U19 pad E2: VCC_5V0_SYS -> VCC_4V0_SYS
- U20 pad 3: /I2C3_SCL_M0 -> /Peripheral IO Connectors/I2C8_SCL_M2
- U20 pad 4: /I2C3_SDA_M0 -> /Peripheral IO Connectors/I2C8_SDA_M2
- U22 pad D1: VCC_5V0_SYS -> VCC_4V0_SYS
- U22 pad D2: VCC_5V0_SYS -> VCC_4V0_SYS
- U22 pad E1: VCC_5V0_SYS -> VCC_4V0_SYS
- U22 pad E2: VCC_5V0_SYS -> VCC_4V0_SYS
- U26 pad 1: Net-(U26-FB) -> unconnected-(U26-FB-Pad1)
- U26 pad 2: Net-(U26-COMP) -> unconnected-(U26-COMP-Pad2)
- U26 pad 3: GND -> unconnected-(U26-GND-Pad3)
- U26 pad 4: /Power and Ground/EDP_SW -> unconnected-(U26-SW-Pad4)
- U26 pad 5: /EDP_PWM11_M1 -> unconnected-(U26-CTRL-Pad5)
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Routing:
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- added copper zone on F.Cu, net /Peripheral IO Connectors/TPS1_LDO_3V3
- added copper zone on F.Cu, net /Peripheral IO Connectors/USB1_VBUS
- added copper zone on In3.Cu, net /Peripheral IO Connectors/USB1_VBUS
- added copper zone on In6.Cu, net /Peripheral IO Connectors/USB1_VBUS
- added copper zone on F.Cu, net /Peripheral IO Connectors/USB2_VBUS
- added copper zone on In3.Cu, net /Peripheral IO Connectors/USB2_VBUS
- added copper zone on In6.Cu, net /Peripheral IO Connectors/USB2_VBUS
- added copper zone on B.Cu, net /Peripheral IO Connectors/USB3_0_VBUS
- added copper zone on F.Cu, net /Peripheral IO Connectors/USB3_0_VBUS
- added copper zone on B.Cu, net /Peripheral IO Connectors/USB3_1_S1
- added copper zone on In6.Cu, net /Peripheral IO Connectors/USB3_1_S1
- added copper zone on F.Cu, net /Peripheral IO Connectors/USB3_1_VBUS
- added copper zone on F.Cu, net /Power and Ground/B_SW_0
- added copper zone on F.Cu, net /Power and Ground/MAIN_SW
- added copper zone on B.Cu, net /Power and Ground/PACK_P
- added copper zone on F.Cu, net /Power and Ground/PACK_P
- added copper zone on F.Cu, net /Power and Ground/SW0_LX
- added copper zone on F.Cu, net /Power and Ground/SW1
- added copper zone on F.Cu, net /Power and Ground/SW10
- added copper zone on F.Cu, net /Power and Ground/SW1_LX
- added copper zone on F.Cu, net /Power and Ground/SW2
- added copper zone on F.Cu, net /Power and Ground/SW3
- added copper zone on F.Cu, net /Power and Ground/SW4
- added copper zone on F.Cu, net /Power and Ground/SW5
- added copper zone on F.Cu, net /Power and Ground/SW6
- added copper zone on F.Cu, net /Power and Ground/SW7
- added copper zone on F.Cu, net /Power and Ground/SW8
- added copper zone on F.Cu, net /Power and Ground/SW9
- added copper zone on F.Cu, net /Power and Ground/VIN_CHRG_1
- added copper zone on F.Cu, net /Power and Ground/VIN_CHRG_2
- added copper zone on F.Cu, net /Power and Ground/VIN_CHRG_3
- added copper zone on F.Cu, net /SYS_PWR
- added copper zone on F.Cu, net Net-(C583-Pad1)
- added copper zone on F.Cu, net Net-(C586-Pad2)
- added copper zone on F.Cu, net Net-(C587-Pad1)
- added copper zone on F.Cu, net Net-(U29-SW)
- added copper zone on F.Cu, net Net-(U39-SW)
- added copper zone on F.Cu, net Net-(U40-SW)
- added copper zone on F.Cu, net Net-(U42-SW)
- added copper zone on F.Cu, net VCC1V8_PMU_DDR_S3
- added copper zone on F.Cu, net VCC3V3_PCIE30
- added copper zone on F.Cu, net VCC3V3_PCIE30_1
- added copper zone on F.Cu, net VCC_12V_EDP
- added copper zone on F.Cu, net VCC_1V1_NLDO_S3
- added copper zone on F.Cu, net VCC_2V0_PLDO_S3
- added copper zone on F.Cu, net VCC_3V3_ALW
- added copper zone on B.Cu, net VCC_3V3_S3
- added copper zone on F.Cu, net VCC_3V3_S3
- added copper zone on B.Cu, net VCC_3V3_SYS
- added copper zone on F.Cu, net VCC_3V3_SYS
- added copper zone on B.Cu, net VCC_4V0_SYS
- added copper zone on F.Cu, net VCC_4V0_SYS
- added copper zone on In3.Cu, net VCC_4V0_SYS
- added copper zone on In6.Cu, net VCC_4V0_SYS
- added copper zone on B.Cu, net VCC_5V0_SYS
- added copper zone on F.Cu, net VCC_5V0_SYS
- added copper zone on In3.Cu, net VCC_5V0_SYS
- added copper zone on In6.Cu, net VCC_5V0_SYS
- added copper zone on F.Cu, net VDD2_DDR_S3
- added copper zone on F.Cu, net VDDQ_DDR_CK_S0
- added copper zone on F.Cu, net VDD_CPU_BIG0_S0
- added copper zone on F.Cu, net VDD_CPU_BIG1_S0
- added copper zone on F.Cu, net VDD_CPU_LIT_S0
- added copper zone on F.Cu, net VDD_DDR_S0
- added copper zone on F.Cu, net VDD_GPU_S0
- added copper zone on F.Cu, net VDD_LOG_S0
- added copper zone on F.Cu, net VDD_NPU_S0
- added copper zone on F.Cu, net VDD_VDENC_S0
- added copper zone on B.Cu, net VIN
- added copper zone on F.Cu, net VIN
- added copper zone on In3.Cu, net VIN
- added copper zone on In6.Cu, net VIN
Other:
- board size 354 x 150 mm -> 424.5 x 336.3 mm
- copper layers 12 -> 8
- board text added: "AUDIO OUT"
- board text added: "BATTERY CONNECTOR"
- board text added: "BIG0 PMIC"
- board text added: "BIG1 PMIC"
- board text added: "BOOT0"
- board text added: "CLOCK GENERATOR"
- board text added: "DISPLAY CONNECTOR"
- board text added: "DP1.4 / USB3.2 GEN 1 PORT"
- board text added: "ECU DEBUG"
- board text added: "HDMI 2.1"
- board text added: "INDICATOR LED"
- board text added: "MIC IN"
- board text added: "NPU PMIC"
- board text added: "NRST"
- board text added: "PMIC"
- board text added: "PWR BUTTON"
- board text added: "RK3588"
- board text added: "SDMMC 3.0"
- board text added: "SPEAKER"
- board text added: "USB 3.2 GEN 1"
- board text added: "USB3.2 GEN 1"
- board text added: "WEBCAM CONNECTOR"
- board text added: "barebones"
