File: hardware/motherboard/barebones_chip.kicad_sch (KiCad schematic)
At the start: 201 parts, among them U1 RK3588, Y1 C3E-24.000-12-3030-X-R

Commit message: arranged the schematics in every sheet
Parts:
- removed R1, R2, R3, R4: 10k, Resistor_SMD:R_0402_1005Metric, symbol Device:R
Connections:
- net VDDQ_DDR_S0 is gone; now on net VDDQ_DDR_CK_S0: C1.2, C10.2, C11.2, C12.2, C13.2, C2.2, C3.2, C4.2, C5.2, C6.2, C8.2, C9.2, U1.K11 (DDR_CH1_VDDQ_0), U1.K12 (DDR_CH1_VDDQ_1), U1.K13 (DDR_CH1_VDDQ_2), U1.K14 (DDR_CH1_VDDQ_3), U1.K15 (DDR_CH1_VDDQ_4), U1.M10 (DDR_CH0_VDDQ_0), U1.N10 (DDR_CH0_VDDQ_1), U1.P10 (DDR_CH0_VDDQ_2), U1.R10 (DDR_CH0_VDDQ_3), U1.T10 (DDR_CH0_VDDQ_4)
- net GPIO3_B3_U: now reaches U1.AC28 (GMAC1_TXD0/I2S2_SDO_M1/UART2_RTSN/GPIO3_B3_U)
- net GPIO3_B4_U: now reaches U1.AC29 (GMAC1_TXD1/I2S2_MCLK_M1/UART2_CTSN/GPIO3_B4_U)
- net GPIO3_B5_U: now reaches U1.AD29 (GMAC1_TXEN/I2S2_SCLK_M1/CAN1_RX_M0/UART3_TX_M1/PWM12_M0/GPIO3_B5_U)
- net I2C4_SDA_M3: now reaches U1.A26 (VOP_POST_EMPTY/I2C4_SDA_M3/UART6_RTSN_M1/PWM0_M2/SPI4_CLK_M2/GPIO1_A2_D)
- net I2C4_SCL_M3: now reaches U1.A27 (HDMI_TX1_SDA_M2/I2C4_SCL_M3/UART6_CTSN_M1/PWM1_M2/SPI4_CS0_M2/GPIO1_A3_D)
Other:
- moved on the sheet: C10, C11, C12, C13, C14, C23, C26, C27, C28, C29, C30, C31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

Commit message: updated last changes
Parts:
- removed C100, C104, C107, C111, C14, C59, C61, C63, C96, C98: 1uF, Capacitor_SMD:C_0201_0603Metric, symbol Device:C
- removed C103, C106, C112, C94: 4.7uF, Capacitor_SMD:C_0201_0603Metric, symbol Device:C
- removed C105, C108, C13, C394, C48, C55, C57, C67, C69, C71, C88, C97, C99: 100nF, Capacitor_SMD:C_0201_0603Metric, symbol Device:C
- removed C113, C116, C118, C119, C120, C121, C149, C150, C156, C157, C93: 10uF, Capacitor_SMD:C_0201_0603Metric, symbol Device:C
- removed C117: 22uF, Capacitor_SMD:C_0201_0603Metric, symbol Device:C
- removed C56, C58, C68, C70: 4.7F, Capacitor_SMD:C_0201_0603Metric, symbol Device:C
- removed C75: 0.1uF, Capacitor_SMD:C_0201_0603Metric, symbol Device:C
- removed R26: 200R, Resistor_SMD:R_0402_1005Metric, symbol Device:R
- added C165, C166, C221, C223, C225, C259, C261, C264, C280, C281, C290, C305, C306, C307, C310, C327, C370: 1uF, Capacitor_SMD:C_0201_0603Metric, symbol Device:C
- added C180, C181, C184, C185, C190, C196, C198, C220, C222, C224, C226, C260, C262, C268, C269, C282, C283, C291, C295, C304: 0.1uF, Capacitor_SMD:C_0201_0603Metric, symbol Device:C
- added C336, C337, C338, C339, C369, C371, C374, C375: 10uF, Capacitor_SMD:C_0402_1005Metric, symbol Device:C
- added C376, C377, C378, C379, C380: 4.7uF, Capacitor_SMD:C_0402_1005Metric, symbol Device:C
- added R35: 8.2k, Resistor_SMD:R_0201_0603Metric, symbol Device:R
- C1, C114, C115, C129, C130, C131, C135, C136, C138, C164, C18, C19, C26, C27, C86, C89: footprint Capacitor_SMD:C_0201_0603Metric -> Capacitor_SMD:C_0402_1005Metric; KiLib_Generator (none) -> SMD_2terminal_chip_molded
- C10, C101, C126, C132, C162, C29, C40: value 1uF -> 0.1uF; KiLib_Generator (none) -> SMD_2terminal_chip_molded
- C102, C109, C11, C110, C12, C124, C125, C133, C20, C30, C32, C4, C44, C45, C46, C47, C5, C51, C522, C53, C6, C85, C95: value 100nF -> 0.1uF; KiLib_Generator (none) -> SMD_2terminal_chip_molded
- C122, C143, C146, C152, C154, C7: value 1uF -> 10uF; footprint Capacitor_SMD:C_0201_0603Metric -> Capacitor_SMD:C_0402_1005Metric; KiLib_Generator (none) -> SMD_2terminal_chip_molded
- C123, C142, C144, C145, C153: value 100nF -> 10uF; footprint Capacitor_SMD:C_0201_0603Metric -> Capacitor_SMD:C_0402_1005Metric; KiLib_Generator (none) -> SMD_2terminal_chip_molded
- C127, C128: value 10uF -> 0.1uF; KiLib_Generator (none) -> SMD_2terminal_chip_molded
- C134: value 22uF -> 0.1uF; KiLib_Generator (none) -> SMD_2terminal_chip_molded
- C137, C158, C159, C8: value 10uF -> 1uF; KiLib_Generator (none) -> SMD_2terminal_chip_molded
- C139, C147: value 4.7uF -> 10uF; footprint Capacitor_SMD:C_0201_0603Metric -> Capacitor_SMD:C_0402_1005Metric; KiLib_Generator (none) -> SMD_2terminal_chip_molded
- C140, C161, C2, C21, C23, C3, C31, C33, C34, C39, C52, C54, C65, C73, C76, C77, C78, C79, C80, C81, C82, C9: KiLib_Generator (none) -> SMD_2terminal_chip_molded
- C141, C87: value 1uF -> 4.7uF; footprint Capacitor_SMD:C_0201_0603Metric -> Capacitor_SMD:C_0402_1005Metric; KiLib_Generator (none) -> SMD_2terminal_chip_molded
- C148: value 10uF -> 4.7uF; footprint Capacitor_SMD:C_0201_0603Metric -> Capacitor_SMD:C_0402_1005Metric; KiLib_Generator (none) -> SMD_2terminal_chip_molded
- C15, C17, C38, C41, C43: value 100nF -> 0.1uF; footprint Capacitor_SMD:C_0603_1608Metric -> Capacitor_SMD:C_0201_0603Metric
- C151: value 22uF -> 10uF; footprint Capacitor_SMD:C_0201_0603Metric -> Capacitor_SMD:C_0402_1005Metric; KiLib_Generator (none) -> SMD_2terminal_chip_molded
- C155: value 22uF -> 4.7uF; footprint Capacitor_SMD:C_0201_0603Metric -> Capacitor_SMD:C_0402_1005Metric; KiLib_Generator (none) -> SMD_2terminal_chip_molded
- C16: value 1uF -> 0.1uF; footprint Capacitor_SMD:C_0603_1608Metric -> Capacitor_SMD:C_0201_0603Metric; KiLib_Generator (none) -> SMD_2terminal_chip_molded
- C160, C83, C84: value 4.7uF -> 0.1uF; KiLib_Generator (none) -> SMD_2terminal_chip_molded
- C163, C22, C28, C66: value 100nF -> 1uF; KiLib_Generator (none) -> SMD_2terminal_chip_molded
- C24, C35: value 18pF -> 1uF; footprint Capacitor_SMD:C_0603_1608Metric -> Capacitor_SMD:C_0201_0603Metric; KiLib_Generator (none) -> SMD_2terminal_chip_molded
- C25, C60, C62, C64: value 100nF -> 0.1uF
- C253: value 100nF -> 10uF; KiLib_Generator (none) -> SMD_2terminal_chip_molded
- C36, C37, C42: footprint Capacitor_SMD:C_0603_1608Metric -> Capacitor_SMD:C_0201_0603Metric
- C49: value 100nF -> 18pF
- C50: value 100nF -> 1uF
- C72: value 100nF -> 4.7uF; footprint Capacitor_SMD:C_0201_0603Metric -> Capacitor_SMD:C_0402_1005Metric; KiLib_Generator (none) -> SMD_2terminal_chip_molded
- C74: value 0.1uF -> 4.7uF; footprint Capacitor_SMD:C_0201_0603Metric -> Capacitor_SMD:C_0402_1005Metric; KiLib_Generator (none) -> SMD_2terminal_chip_molded
- C90, C91, C92: value 10uF -> 22uF; footprint Capacitor_SMD:C_0201_0603Metric -> Capacitor_SMD:C_0402_1005Metric; KiLib_Generator (none) -> SMD_2terminal_chip_molded
- FL1: footprint BLM18PG121SZ1D:BEADC1608X95N -> barebones:BEADC1608X95N
- R10, R21, R22, R23, R24, R25, R5, R6, R8, R9: footprint Resistor_SMD:R_0603_1608Metric -> Resistor_SMD:R_0201_0603Metric
- R11, R12, R13, R14, R15, R16, R17, R18, R19, R20, R27, R28, R29, R31: footprint Resistor_SMD:R_0402_1005Metric -> Resistor_SMD:R_0201_0603Metric
- R30: value 8.2k -> 200R; footprint Resistor_SMD:R_0402_1005Metric -> Resistor_SMD:R_0201_0603Metric
- R7: footprint Resistor_SMD:R_0603_1608Metric -> Resistor_SMD:R_0402_1005Metric
Connections:
- net GND: now also C101.1, C102.1, C152.1, C153.1, C16.1, C25.2, C35.1, C49.2, C50.2, C60.2, C62.2, C64.2, C72.1, C74.1, C89.1, C90.1, C91.1, C92.1, C95.1, R16.2, R19.2, C165.1, C166.1, C181.1, C184.1, C185.1, C190.1, C196.1, C198.1, C220.1, C221.1, C222.1, C223.1, C224.1, C225.1, C226.1, C259.1, C260.1, C261.1, C262.1, C264.1, C268.1, C269.1, C280.1, C281.1, C282.1, C283.1, C290.1, C291.1, C295.1, C304.1, C305.1, C306.1, C307.1, C310.1, C327.1, C336.1, C337.1, C338.1, C339.1, C369.1, C370.1, C371.1, C374.1, C375.1, C376.1, C377.1, C378.1, C379.1, C380.1, R35.2; no longer C101.2, C102.2, C152.2, C153.2, C16.2, C25.1, C35.2, C49.1, C50.1, C60.1, C62.1, C64.1, C83.1, C84.1, C85.1, C89.2, C90.2, C91.2, C92.2, C95.2, R16.1, R19.1, U1.AA13 (VDD_GPU_0), U1.AA14 (VDD_GPU_7), U1.AA15 (VDD_GPU_11), U1.AB13 (VDD_GPU_1), U1.AB14 (VDD_GPU_6), U1.AB15 (VDD_GPU_10), U1.AC13 (VDD_GPU_2), U1.AC14 (VDD_GPU_5), U1.AC15 (VDD_GPU_9), U1.AC17 (VDD_LOGIC_5), U1.AC18 (VDD_LOGIC_4), U1.AC19 (VDD_LOGIC_3), U1.AD13 (VDD_GPU_3), U1.AD14 (VDD_GPU_4), U1.AD15 (VDD_GPU_8), U1.AD17 (VDD_LOGIC_0), U1.AD18 (VDD_LOGIC_1), U1.AD19 (VDD_LOGIC_2), U1.K19 (VDD_LOGIC_8), U1.K20 (VDD_LOGIC_9), U1.V16 (VDD_LOGIC_6), U1.V17 (VDD_LOGIC_7)
- net PCIE20_0_RXN: now also C85.1; no longer C72.1
- net PCIE20_0_RXP: now also C84.1
- net PWRCTRL2_PMIC: now also R23.2; no longer R23.1
- net SPI2_CLK_M2: now also R10.2; no longer R8.2
- net SPI2_MOSI_M2: now also R8.2; no longer R10.2
- net USB30_2_SSRXP: now also C83.1
- net USB_2_RX1N: now also C82.1; no longer C77.1
- net USB_2_RX1P: now also C180.1; no longer C74.1
- net USB_2_RX2N: now also C77.1; no longer C82.1
- net VCCA_1V8_S0: now also C33.2, C34.2, C72.2, C74.2, U1.K27 (PCIE20_SATA30_USB30_2_AVDD_1V8), U1.L27 (PCIE20_SATA30_1_AVDD_1V8), U1.M27 (PCIE20_SATA30_0_AVDD_1V8), C165.2, C185.2, C196.2, C259.2, C269.2, C281.2, C283.2, C304.2; no longer C62.2, C66.2, C7.2
- net VCCA_3V3_S0: now also R18.2; no longer R18.1
- net VCCIO_SD_S0: now also C40.2; no longer C25.2
- net VCC_1V8_S0: now also C127.2, C158.2, C159.2, C160.2, C25.1, C60.1, C62.1, U1.H20 (VCCIO4_1V8), U1.H21 (VCCIO4), C377.2, C378.2; no longer C253.2
- net VCC_1V8_S3: now also C184.2; no longer C50.2
- net VCC_3V3_S0: now also C64.1
- net VCC_3V3_S3: now also C181.2; no longer C49.2
- net VDDA_0V75_S0: now also C161.2, C162.2, C163.2, C220.2, C221.2, C222.2, C225.2, C226.2, C379.2, C380.2; no longer C83.2, C84.2, C85.2, C86.2, C87.2
- net VDDA_0V85_S0: now also C253.2, C66.2, U1.K28 (PCIE20_SATA30_USB30_2_AVDD_0V85), U1.L28 (PCIE20_SATA30_1_AVDD_0V85), U1.M28 (PCIE20_SATA30_0_AVDD_0V85), C166.2, C190.2, C198.2, C262.2, C280.2; no longer C60.2, C64.2
- net VDDQ_DDR_CKE_S3: now also C24.2, C39.2; no longer C34.2, C40.2
- net VDDQ_DDR_CK_S0: now also C22.2, C31.2, C7.2; no longer C33.2, C39.2
- net VDDQ_DDR_PLL_S0: now also C35.2; no longer C31.2
- net VDD_0V75_S0: now also C86.2, C87.2, C282.2, C295.2
- net VDD_0V75_S3: now also C50.1; no longer C16.1
- net VDD_CPU_BIG0_S0: now also C109.2, C110.2, C151.2, C152.2, C153.2, C154.2, C91.2, C290.2, C291.2, C307.2, C310.2; no longer C152.1, C153.1, C158.2, C159.2, C160.2, C161.2, C162.2, C163.2
- net VDD_CPU_BIG1_MEM_S0: now also C264.2, C268.2; no longer C132.2, C133.2
- net VDD_CPU_BIG1_S0: now also C101.2, C102.2, C144.2, C145.2, C146.2, C147.2, C148.2, C90.2, C305.2, C306.2; no longer C134.2, C135.2, C136.2, C137.2, C138.2, C139.2, C140.2, C141.2, C142.2
- net VDD_DDR_S0: now also C16.2; no longer C22.2
- net VDD_GPU_S0: now also C124.2, C126.2, C130.2, C132.2, C135.2, C138.2, C139.2, C92.2, U1.AA13 (VDD_GPU_0), U1.AA14 (VDD_GPU_7), U1.AA15 (VDD_GPU_11), U1.AB13 (VDD_GPU_1), U1.AB14 (VDD_GPU_6), U1.AB15 (VDD_GPU_10), U1.AC13 (VDD_GPU_2), U1.AC14 (VDD_GPU_5), U1.AC15 (VDD_GPU_9), U1.AD13 (VDD_GPU_3), U1.AD14 (VDD_GPU_4), U1.AD15 (VDD_GPU_8); no longer C109.2, C110.2, C114.2, C115.2
- net VDD_LOG_S0: now also C125.2, C134.2, C137.2, C140.2, U1.AC17 (VDD_LOGIC_5), U1.AC18 (VDD_LOGIC_4), U1.AC19 (VDD_LOGIC_3), U1.AD17 (VDD_LOGIC_0), U1.AD18 (VDD_LOGIC_1), U1.AD19 (VDD_LOGIC_2), U1.K19 (VDD_LOGIC_8), U1.K20 (VDD_LOGIC_9), U1.V16 (VDD_LOGIC_6), U1.V17 (VDD_LOGIC_7), C369.2, C371.2, C374.2, C375.2, C376.2; no longer C101.1, C102.1, C143.2, C144.2, C145.2, C146.2, C147.2, C148.2, C151.2, C89.1, C90.1, C91.1, C92.1, C95.1, U1.T21 (VDD_CPU_LIT_MEM_1), U1.T22 (VDD_CPU_LIT_MEM_0), U1.U21 (VDD_CPU_LIT_7), U1.U22 (VDD_CPU_LIT_0), U1.V21 (VDD_CPU_LIT_6), U1.V22 (VDD_CPU_LIT_1), U1.W21 (VDD_CPU_LIT_5), U1.W22 (VDD_CPU_LIT_2), U1.Y21 (VDD_CPU_LIT_4), U1.Y22 (VDD_CPU_LIT_3)
- net VDD_NPU_S0: now also C133.2, C136.2, C327.2, C336.2, C337.2, C338.2, C339.2; no longer C125.2, C126.2, C127.2, C129.2, C130.2, C131.2
- net VDD_VDENC_S0: now also C115.2, C142.2, C143.2, C260.2, C261.2, C370.2; no longer C123.2, C124.2, C154.2
- net at U1.L29 (SPI2_MISO_M2/I2C0_SCL_M0/GPIO0_B3_Z), U1.N30 (SPI2_MOSI_M2/I2C0_SDA_M0/GPIO0_A6_Z): now also R8.1; no longer R10.1
- net at U1.N31 (SPI2_CLK_M2/SDMMC_PWREN/PMU_DEBUG/GPIO0_A5_D): now also R10.1; no longer R8.1
- net at C36.1, R7.1, U1.R34 (XIN_24M)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: no longer C24.2
- net at U1.M34 (PCIE20_0_TXP/SATA30_0_TXP): now also C84.2
- net at R9.1, Y1.1: now also C49.1; no longer C35.1
- net at U1.AP9 (TYPEC1_SSTX1P/DP1_TX1P): now also C180.2; no longer C74.2
- net at U1.T30 (PMIC_SLEEP5/GPIO0_C3_D): now also R23.1; no longer R23.2
- net MIC_CLK: now reaches U1.T31 (PDM0_CLK0_M1/PWM1_M0/I2C2_SDA_M0/CAN0_RX_M0/SPI0_MOSI_M0/PCIE30X1_0_CLKREQN_M0/GPIO0_C0_D)
- net MIC_DAT: now reaches U1.V31 (I2S1_SDI2_M1/PDM0_SDI0_M1/I2C6_SDA_M0/UART1_RTSN_M2/PWM6_M0/SPI0_MISO_M0/PCIE30X4_WAKEN_M0/GPIO0_C7_D)
- net at U1.AL8 (TYPEC1_USB20_VBUSDET): now also R18.1; no longer R18.2
- net at U1.AN11 (TYPEC1_SSTX2N/DP1_TX3N): now also C77.2; no longer C82.2
- net at U1.AN9 (TYPEC1_SSTX1N/DP1_TX1N): now also C82.2; no longer C77.2
- net at U1.AM2 (HDMI/EDP_TX0_REXT): now also R35.1; no longer R30.1
- net at U1.B34 (PCIE30_PORT0_RESREF): now also R30.1
- net at U1.AP7 (TYPEC1_USB20_OTG1_REXT): now also R19.1; no longer R19.2
- net at U1.H30 (PCIE20_2_TXP/SATA30_2_TXP/USB30_2_SSTXP): now also C83.2
- net at U1.M33 (PCIE20_0_TXN/SATA30_0_TXN): now also C85.2; no longer C72.2
- net I2C3_SCL_M0: now reaches U1.G27 (I2C3_SCL_M0/UART3_TX_M0/SPI4_MOSI_M0/GPIO1_C1_Z)
- net I2C3_SDA_M0: now reaches U1.G29 (I2C3_SDA_M0/UART3_RX_M0/SPI4_MISO_M0/GPIO1_C0_Z)
- net at U1.AH9 (USB20_HOST1_REXT): now also R16.1; no longer R16.2
- new net VDD_CPU_LIT_S0: C114.2, C123.2, C129.2, C131.2, C141.2, C223.2, C224.2, C89.2, C95.2, U1.T21 (VDD_CPU_LIT_MEM_1), U1.T22 (VDD_CPU_LIT_MEM_0), U1.U21 (VDD_CPU_LIT_7), U1.U22 (VDD_CPU_LIT_0), U1.V21 (VDD_CPU_LIT_6), U1.V22 (VDD_CPU_LIT_1), U1.W21 (VDD_CPU_LIT_5), U1.W22 (VDD_CPU_LIT_2), U1.Y21 (VDD_CPU_LIT_4), U1.Y22 (VDD_CPU_LIT_3)
- no-connect marks 59 -> 61
Other:
- moved on the sheet: C1, C15, C164, C2, C32, C37, C4, C522, C78, FL1, R31, U1A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
