File: hardware/motherboard/barebones_chip.kicad_sch (KiCad schematic)
At the start: 203 parts, among them U1 RK3588, Y1 C3E-24.000-12-3030-X-R

Commit message: started routing on LPDDR4x RAM
Parts:
- removed C336, C337, C338, C339, C369, C371, C374, C375: 10uF, Capacitor_SMD:C_0402_1005Metric, symbol Device:C
- removed C65, C66: 1uF, Capacitor_SMD:C_0201_0603Metric, symbol Device:C
- added C149, C150, C156, C157, C257, C258, C317, C318: 10uF, Capacitor_SMD:C_0603_1608Metric, symbol Device:C
- added C255, C256: 1uF, Capacitor_SMD:C_0402_1005Metric, symbol Device:C
- added C48: 1uF, Capacitor_SMD:C_0201_0603Metric, symbol Device:C
- added C55, C69: 4.7uF, Capacitor_SMD:C_0603_1608Metric, symbol Device:C
- added C56, C57, C58, C59, C61, C63, C67, C68, C71: 0.1uF, Capacitor_SMD:C_0201_0603Metric, symbol Device:C
- added C70: 10pF, Capacitor_SMD:C_0201_0603Metric, symbol Device:C
- added C75: 2.2uF, Capacitor_SMD:C_0402_1005Metric, symbol Device:C
- added J1: DF40C-34DP-0.4V_58_, barebones:HIROSE_DF40C-34DP-0.4V_58_, symbol DF40C-34DP-0.4V_58_:DF40C-34DP-0.4V_58_
- added R26, R36, R38, R39, R40, R42, R43, R46, R47, R48: 10k, Resistor_SMD:R_0201_0603Metric, symbol Device:R
- added R59: 22R, Resistor_SMD:R_0201_0603Metric, symbol Device:R
- added R63: 47k, Resistor_SMD:R_0201_0603Metric, symbol Device:R
- added U21: DF40C-30DP-0.4V51, barebones:HIROSE_DF40C-30DP-0.4V-58, symbol DF40C-30DP-0.4V-58:DF40C-30DP-0.4V51
- added U23: KLMCG4JETD-B041, barebones:BGA-153_L13.0-W11.5-P0.50-TL_KLM8G1GEME-B041, symbol KLMCG4JETD-B041:KLMCG4JETD-B041
- C1, C114, C115, C122, C123, C129, C130, C131, C135, C136, C138, C139, C142, C143, C144, C145, C146, C147, C151, C152, C153, C154, C18, C19, C26, C27, C7: footprint Capacitor_SMD:C_0402_1005Metric -> Capacitor_SMD:C_0603_1608Metric
- C141: footprint Capacitor_SMD:C_0402_1005Metric -> Capacitor_SMD:C_0201_0603Metric
- C164, C89, C90, C91, C92: footprint Capacitor_SMD:C_0402_1005Metric -> Capacitor_SMD:C_0805_2012Metric
- C165, C166, C2, C21, C22, C23, C24, C259, C28, C280, C281, C3, C31, C33, C34, C35, C37, C39, C42, C50, C52, C54, C8, C9: footprint Capacitor_SMD:C_0201_0603Metric -> Capacitor_SMD:C_0402_1005Metric
- C253: footprint Capacitor_SMD:C_0201_0603Metric -> Capacitor_SMD:C_0603_1608Metric
Connections:
- net GND: now also C149.1, C150.1, C156.1, C157.1, C255.1, C256.1, C257.1, C258.1, C317.1, C318.1, C48.1, C55.1, C56.1, C57.1, C58.1, C59.1, C61.1, C63.1, C67.1, C68.1, C69.1, C70.1, C71.1, C75.1, R63.2, U23.A6 (VSS), U23.C4 (VSS), U23.E7 (VSS), U23.G5 (VSS), U23.H10 (VSS), U23.J5 (VSS), U23.K8 (VSS), U23.N2 (VSS), U23.N5 (VSS), U23.P4 (VSS), U23.P6 (VSS)
- net MIC_CLK: now also U1.E24 (PDM1_CLK0_M1/PCIE30X1_0_PERSTN_M2/UART7_RX_M2/SPI0_CS0_M2/GPIO1_B4_U); no longer U1.T31 (PDM0_CLK0_M1/PWM1_M0/I2C2_SDA_M0/CAN0_RX_M0/SPI0_MOSI_M0/PCIE30X1_0_CLKREQN_M0/GPIO0_C0_D)
- net MIC_DAT: now also U1.C25 (PDM1_SDI0_M1/PCIE30X1_1_PERSTN_M2/PWM3_IR_M3/SPI2_CS0_M0/GPIO1_A7_U); no longer U1.V31 (I2S1_SDI2_M1/PDM0_SDI0_M1/I2C6_SDA_M0/UART1_RTSN_M2/PWM6_M0/SPI0_MISO_M0/PCIE30X4_WAKEN_M0/GPIO0_C7_D)
- net VCCA_1V8_S0: now also C256.2
- net VCC_1V8_S3: now also U1.V26 (EMMCIO_1V8), C48.2, C55.2, C56.2, C57.2, C58.2, C59.2, C61.2, R26.1, R36.1, R38.1, R39.1, R40.1, R42.1, R43.1, R46.1, R48.1, U23.C6 (VCCQ), U23.M4 (VCCQ), U23.N4 (VCCQ), U23.P3 (VCCQ), U23.P5 (VCCQ)
- net VCC_3V3_S3: now also C63.2, C67.2, C68.2, C69.2, C71.2, R47.1, U23.E6 (VCC), U23.F5 (VCC), U23.J10 (VCC), U23.K9 (VCC)
- net VDDA_0V85_S0: now also C255.2
- net VDD_CPU_BIG0_S0: now also C149.2, C150.2; no longer C153.2, C154.2
- net VDD_LOG_S0: now also C257.2, C258.2, C317.2, C318.2
- net VDD_NPU_S0: now also C153.2, C154.2, C156.2, C157.2
- net EMMC_D5: now reaches U1.AA32 (EMMC_D5/I2C1_SDA_M3/UART5_TX_M2/GPIO2_D5_U)
- net EMMC_D5: now also R42.2, U23.B4 (DAT5), U23.C3 (NC), U23.D1 (NC), U23.D2 (NC)
- net EMMC_D3: now reaches U1.AA33 (EMMC_D3/FSPI_D3_M0/GPIO2_D3_U)
- net EMMC_D3: now also R46.2, U23.A1 (NC), U23.B2 (DAT3)
- net EMMC_RSTN: now reaches U1.AA34 (EMMC_RSTN/I2C2_SCL_M2/UART5_RTSN_M1/GPIO2_A3_D)
- net EMMC_RSTN: now also R48.2, U23.K1 (NC), U23.K2 (NC), U23.K3 (NC), U23.K5 (RSTN)
- net EMMC_D2: now reaches U1.V32 (EMMC_D2/FSPI_D2_M0/GPIO2_D2_U)
- net EMMC_D2: now also R26.2, U23.A5 (DAT2)
- net EMMC_D7: now reaches U1.V33 (EMMC_D7/FSPI_CS1N_M0/GPIO2_D7_U)
- net EMMC_D7: now also R39.2, U23.A7 (RFU), U23.A8 (NC), U23.B6 (DAT7), U23.B7 (NC)
- net EMMC_CLKOUT: now reaches U1.V34 (EMMC_CLKOUT/GPIO2_A1_D)
- net EMMC_CLKOUT: now also C70.2, U23.M6 (CLK), U23.P8 (NC)
- net EMMC_D6: now reaches U1.W32 (EMMC_D6/FSPI_CS0N_M0/GPIO2_D6_U)
- net EMMC_D6: now also R40.2, U23.A9 (NC), U23.B5 (DAT6), U23.B8 (NC), U23.C5 (NC), U23.C7 (NC), U23.D4 (NC), U23.E1 (NC), U23.E2 (NC), U23.E3 (NC)
- net EMMC_D1: now reaches U1.W33 (EMMC_D1/FSPI_D1_M0/GPIO2_D1_U)
- net EMMC_D1: now also R36.2, U23.A4 (DAT1)
- net EMMC_CMD: now reaches U1.W34 (EMMC_CMD/FSPI_CLK_M0/GPIO2_A0_U)
- net EMMC_CMD: now also R47.2, U23.M5 (CMD), U23.P7 (RFU)
- net EMMC_D4: now reaches U1.Y32 (EMMC_D4/I2C1_SCL_M3/UART5_RX_M2/GPIO2_D4_U)
- net EMMC_D4: now also R43.2, U23.A2 (NC), U23.B3 (DAT4)
- net EMMC_D0: now reaches U1.Y33 (EMMC_D0/FSPI_D0_M0/GPIO2_D0_U)
- net EMMC_D0: now also R38.2, U23.A3 (DAT0)
- net EMMC_DATA_STROBE: now reaches U1.Y34 (EMMC_DATA_STROBE/I2C2_SDA_M2/UART5_CTSN_M1/GPIO2_A2_D)
- net EMMC_DATA_STROBE: now also R59.1, R63.1
- net INT_ALS: now reaches U1.C27 (PDM1_SDI1_M1/PCIE30X4_CLKREQN_M3/SPI2_CS1_M0/GPIO1_B0_U)
- net CAM_SW: now reaches U1.E26 (MIPI_CAMERA1_CLK_M0/SPDIF0_TX_M0/PCIE30X2_WAKEN_M3/HDMI_RX_HPDOUT_M2/I2C5_SCL_M3/UART1_TX_M1/GPIO1_B6_U)
- net MIC_SW: now reaches U1.E27 (MIPI_CAMERA2_CLK_M0/SPDIF1_TX_M0/PCIE30X2_PERSTN_M3/HDMI_RX_CEC_M2/SATA2_ACT_LED_M1/I2C5_SDA_M3/UART1_RX_M1/PWM13_M2/GPIO1_B7_U)
- net I2C8_SCL_M2: now reaches U1.F24 (MIPI_CAMERA3_CLK_M0/HDMI_RX_SCL_M2/I2C8_SCL_M2/UART1_RTSN_M1/PWM14_M2/GPIO1_D6_U)
- net I2C8_SDA_M2: now reaches U1.F25 (MIPI_CAMERA4_CLK_M0/PCIE30X2_CLKREQN_M3/HDMI_RX_SDA_M2/I2C8_SDA_M2/UART1_CTSN_M1/PWM15_IR_M3/GPIO1_D7_U)
- net DDR_CH1_CKB_C renamed DDR_CH1_CK_C_N
- net DDR_CH1_CKB_D renamed DDR_CH1_CK_D_N
- net DDR_CH1_CK_C renamed DDR_CH1_CK_C_P
- net DDR_CH1_CK_D renamed DDR_CH1_CK_D_P
- net DDR_CH1_DQS0N_C renamed DDR_CH1_DQS0_C_N
- net DDR_CH1_DQS0N_D renamed DDR_CH1_DQS0_D_N
- net DDR_CH1_DQS0P_C renamed DDR_CH1_DQS0_C_P
- net DDR_CH1_DQS0P_D renamed DDR_CH1_DQS0_D_P
- net DDR_CH1_DQS1N_C renamed DDR_CH1_DQS1_C_N
- net DDR_CH1_DQS1N_D renamed DDR_CH1_DQS1_D_N
- net DDR_CH1_DQS1P_C renamed DDR_CH1_DQS1_C_P
- net DDR_CH1_DQS1P_D renamed DDR_CH1_DQS1_D_P
- net I2C3_SCL_M0: no longer names the net of U1.G27 (I2C3_SCL_M0/UART3_TX_M0/SPI4_MOSI_M0/GPIO1_C1_Z)
- net I2C3_SDA_M0: no longer names the net of U1.G29 (I2C3_SDA_M0/UART3_RX_M0/SPI4_MISO_M0/GPIO1_C0_Z)
- net USB_1_OTG_DM renamed USB_1_OTG_DN
- net USB_2_OTG_DM renamed USB_2_OTG_DN
- new net: J1.S1 (SHIELD), J1.S2 (SHIELD), J1.S3 (SHIELD), J1.S4 (SHIELD)
- new net: C75.2, U23.C2 (VDDI)
- new net: R59.2, U23.H5 (DataStrobe)
- new net Net-(U23-VDDI): U23.C1 (NC)
- no-connect marks 61 -> 228
Other:
- moved on the sheet: C15, C17, C32, C36, C37, C38, C40, C41, C42, C43, C49, C50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
