File: hardware/motherboard/barebones_io.kicad_sch (KiCad schematic)
At the start: 266 parts, among them IC1 W25Q80DVSSIG, IC2 FUSB302BMPX, IC3 W25Q80DVSSIG, IC4 FUSB302BMPX, J1 12401610E4_2A, J10 54-00007, J11 54-00007, J12 10067847-001RLF, J13 SM02B-GHS-TB_LF__SN_, J14 SM05B-SRSS-TB_LF__SN_, J15 20455-040E-76, J16 524352671, J17 522070485, J18 G45AA1912100B1EU, J19 SM06B-SRSS-TB_LF__SN_, J2 1-2199119-5, J20 20682-040E-02, J3 1-2199119-5, J4 21992304, J5 12401610E4_2A, J6 SJ2-35894B-SMT-TR, J7 1-84953-4, J8 SM02B-GHS-TB_LF__SN_, J9 1040310811, SW1 EC05E1220401, SW2 EC05E1220401, SW3 EC05E1220401, U39 TPS65987DDHRSHR, U40 TXS0104EYZTR, U41 TPD4E004DRYR, U42 PCA9306DCTR, U43 9FGV0641AKILFT, U44 TPD4E05U06DQAR, U45 GL3523-ONY30, U46 TXS0104EYZTR, U47 TPS2553DBVR, U48 PI3DPX1207Q3ZHEX, U49 TPS65987DDHRSHR, U50 TXS0104EYZTR, U51 PCA9306DCTR, U52 OV9734-H16A, U53 TPS2553DBVR, U54 TPD4E004DRYR, U55 PI6C557-05BLEX, U56 PI6C557-05LEX, U57 PI6C557-03ALEX, U58 TPS2553DBVR, U59 TPD4E004DRYR, U60 TPD4E004DRYR, U61 PCA9306DCTR, U62 2N7002KW, U63 2N7002KW, U64 2N7002KW, U65 2N7002KW, U66 2N7002KW, U67 2N7002KW, U68 2N7002KW, U69 2N7002KW, U70 2N7002KW, Y3 C2E-25.000-10-1530-X-R, Y4 C2E-25.000-10-1530-X-R

Commit message: pushed many changes and added dedicated bms module
Parts:
- removed R203: 1.5k, Resistor_SMD:R_0402_1005Metric, symbol Device:R
- removed R228, R229, R230, R231, R232, R233, R234, R235, R249: 4.7k, Resistor_SMD:R_0402_1005Metric, symbol Device:R
- removed SW1, SW2, SW3: EC05E1220401, barebones:SW-SMD_EC05E1220401, symbol EC05E1220401:EC05E1220401
- added C563, C564: 0.1uF, Capacitor_SMD:C_0201_0603Metric, symbol Device:C
- added J25: F33X-1AAJ1-E8951, barebones:AMPHENOL_F33X-1AAJ1-E8951, symbol F33X-1AAJ1-E8951:F33X-1AAJ1-E8951
- added R226: 1.5k, Resistor_SMD:R_0402_1005Metric, symbol Device:R
Connections:
- net BACKLIGHT_DN: now also J25.29, J25.31; no longer J17.3, J17.4
- net BACKLIGHT_DP: now also J25.30, J25.32; no longer J17.1, J17.2
- net CAPS_P: now also R226.2
- net GND: now also C563.1, C564.1, J25.1, J25.26, J25.28, J25.33, J25.37, J25.43; no longer J16.26, J16.P1, J16.P2, J17.P1, J17.P2
- net KSI0: now also J25.2; no longer J16.1
- net KSI1: now also J25.3; no longer J16.2
- net KSI2: now also J25.4; no longer J16.3
- net KSI3: now also J25.5; no longer J16.4
- net KSI4: now also J25.6; no longer J16.5
- net KSI5: now also J25.7; no longer J16.6
- net KSI6: now also J25.8; no longer J16.7
- net KSI7: now also J25.9; no longer J16.8
- net KSO0: now also J25.10; no longer J16.9
- net KSO1: now also J25.11; no longer J16.10
- net KSO10: now also J25.20; no longer J16.19
- net KSO11: now also J25.21; no longer J16.20
- net KSO12: now also J25.22; no longer J16.21
- net KSO13: now also J25.23; no longer J16.22
- net KSO14: now also J25.24; no longer J16.23
- net KSO15: now also J25.25; no longer J16.24
- net KSO2: now also J25.12; no longer J16.11
- net KSO3: now also J25.13; no longer J16.12
- net KSO4: now also J25.14; no longer J16.13
- net KSO5: now also J25.15; no longer J16.14
- net KSO6: now also J25.16; no longer J16.15
- net KSO7: now also J25.17; no longer J16.16
- net KSO8: now also J25.18; no longer J16.17
- net KSO9: now also J25.19; no longer J16.18
- new net: J25.27, R226.1
- new net BOARD_ID: J25.38
- new net EC_CONTROL: J25.45
- new net TP_INT: J25.35
- new net TP_SCL: J25.34
- new net TP_SDA: J25.36
- new net VCC_4V0_SYS: C563.2, J25.40
- new net VCC_5V0_ALW: C564.2, J25.41
- no-connect marks 163 -> 172
Other:
- note removed: "BACKLIGHT"
- note removed: "MATRIX"
- note removed: "ROTARY ENCODERS"

Commit message: arranged the schematics in every sheet
Parts:
- removed C430: 4.7uF, Capacitor_SMD:C_0201_0603Metric, symbol Device:C
- removed C434, C435, C465, C466, C473, C475, C477, C478, C480, C481, C483, C485, C487, C490, C493, C494, C496, C498, C506, C515, C517: 0.1uF, Capacitor_SMD:C_0201_0603Metric, symbol Device:C
- removed C467, C468: 12pF, Capacitor_SMD:C_0201_0603Metric, symbol Device:C
- removed C484, C526, C527: 1uF, Capacitor_SMD:C_0201_0603Metric, symbol Device:C
- removed C505, C514: 100uF, Capacitor_SMD:C_0201_0603Metric, symbol Device:C
- removed C519, C520: 220pF, Capacitor_SMD:C_0201_0603Metric, symbol Device:C
- removed C530: 100pF, Capacitor_SMD:C_0201_0603Metric, symbol Device:C
- removed C539: 100nF, Capacitor_SMD:C_0603_1608Metric, symbol Device:C
- removed IC2: FUSB302BMPX, barebones:QFN50P250X250X80-15N, symbol FUSB302BMPX:FUSB302BMPX
- removed IC3: W25Q80DVSSIG, barebones:SOIC8-FLASH, symbol W25Q80DVSSIG:W25Q80DVSSIG
- removed J13, J8: SM02B-GHS-TB_LF__SN_, barebones:JST_SM02B-GHS-TB_LF__SN_, symbol SM02B-GHS-TB_LF__SN_:SM02B-GHS-TB_LF__SN_
- removed J19: SM06B-SRSS-TB_LF__SN_, SM06B-SRSS-TB_LF__SN_:JST_SM06B-SRSS-TB_LF__SN_, symbol SM06B-SRSS-TB_LF__SN_:SM06B-SRSS-TB_LF__SN_
- removed J6: SJ2-35894B-SMT-TR, barebones:CUI_SJ2-35894B-SMT-TR, symbol SJ2-35894B-SMT-TR:SJ2-35894B-SMT-TR
- removed L17: XAL7030-472MEB, XAL7030-472MEB:IND_XAL7030-472MEB, symbol XAL7030-472MEB:XAL7030-472MEB
- removed R148: 4.7k, Resistor_SMD:R_0402_1005Metric, symbol Device:R
- removed R155, R164, R165, R166, R167, R168, R169, R183: 10k, Resistor_SMD:R_0402_1005Metric, symbol Device:R
- removed R172: 6.81k, Resistor_SMD:R_0402_1005Metric, symbol Device:R
- removed R186: 68k, Resistor_SMD:R_0402_1005Metric, symbol Device:R
- removed R189, R190, R191: 2.2k, Resistor_SMD:R_0402_1005Metric, symbol Device:R
- removed TP10: MISO, TestPoint:TestPoint_Pad_D1.5mm, symbol Connector:TestPoint
- removed TP7: CHIP SELECT, TestPoint:TestPoint_Pad_D1.5mm, symbol Connector:TestPoint
- removed TP8: CLOCK, TestPoint:TestPoint_Pad_D1.5mm, symbol Connector:TestPoint
- removed TP9: MOSI, TestPoint:TestPoint_Pad_D1.5mm, symbol Connector:TestPoint
- removed U39, U49: TPS65987DDHRSHR, barebones:IC_TPS65987DDHRSHR, symbol TPS65987DDHRSHR:TPS65987DDHRSHR
- removed U45: GL3523-ONY30, barebones:QFN-48_L6.0-W6.0-P0.40-BL-EP3.8, symbol GL3523-ONY30:GL3523-ONY30
- removed U50: TXS0104EYZTR, barebones:BGA12N50P4X3_186X136X62N, symbol TXS0104EYZTR:TXS0104EYZTR
- removed U53: TPS2553DBVR, barebones:SOT95P280X145-6N, symbol TPS2553DBVR:TPS2553DBVR
- removed U61: PCA9306DCTR, barebones:SOP65P400X130-8N, symbol PCA9306DCTR:PCA9306DCTR
- removed U62, U63, U64, U66: 2N7002KW, 2N7002KW:SOT323, symbol 2N7002KW:2N7002KW
- removed Y4: C2E-25.000-10-1530-X-R, barebones:XTAL_C2E-25.000-10-1530-X-R, symbol C2E-25.000-10-1530-X-R:C2E-25.000-10-1530-X-R
- added C561, C562, C565, C566: 220pF, Capacitor_SMD:C_0201_0603Metric, symbol Device:C
- added C567, C568, C583, C587, C599: 1uF, Capacitor_SMD:C_0201_0603Metric, symbol Device:C
- added C569, C570, C571, C572, C573, C574, C575, C576: 10nF, Capacitor_SMD:C_0201_0603Metric, symbol Device:C
- added C577, C578, C585, C597, C608, C610: 10uF, Capacitor_SMD:C_0201_0603Metric, symbol Device:C
- added C579, C580, C581, C582: 22uF, Capacitor_SMD:C_0201_0603Metric, symbol Device:C
- added C584, C586, C588, C590, C591, C592, C593, C594, C598, C600, C607, C611: 0.1uF, Capacitor_SMD:C_0201_0603Metric, symbol Device:C
- added C595, C596: 12pF, Capacitor_SMD:C_0201_0603Metric, symbol Device:C
- added C609, C612: 120uF, Capacitor_SMD:C_0201_0603Metric, symbol Device:C
- added D1, D17: SMAJ15CA, Diode_SMD:D_SMA, symbol Diode:SMAJ15CA
- added Q1, Q3, Q5, Q6: BSS138, Package_TO_SOT_SMD:SOT-23, symbol Transistor_FET:BSS138
- added Q9: CSD18504Q5A, barebones:MOSFET_CSD19531Q5A, symbol CSD18504Q5A:CSD18504Q5A
- added R243, R244: 4.7k, Resistor_SMD:R_0402_1005Metric, symbol Device:R
- added R245, R246: 100k, Resistor_SMD:R_0402_1005Metric, symbol Device:R
- added R247, R248, R255, R257: 10k, Resistor_SMD:R_0402_1005Metric, symbol Device:R
- added R256, R258: 20.2k, Resistor_SMD:R_0402_1005Metric, symbol Device:R
- added U38: TPS65988DHRSHR, barebones:IC_TPS65987DDHRSHR, symbol TPS65988DHRSHR:TPS65988DHRSHR
- added U39, U49, U50, U61: CSD25402Q3A, barebones:TRANS_CSD25402Q3A, symbol Transistor_FET:CSD25402Q3A
- added U74, U77: 2N7002KW, 2N7002KW:SOT323, symbol 2N7002KW:2N7002KW
- added U79: USB5744_2G, barebones:QFN40P700X700X100-57N, symbol USB5744_2G:USB5744_2G
- added U82, U83: TPS2557DRBR, TPS2557DRBR:SON65P300X300X100-9N, symbol TPS2557DRBR:TPS2557DRBR
- added Y7: C2E-25.000-10-1530-X-R, barebones:XTAL_C2E-25.000-10-1530-X-R, symbol C2E-25.000-10-1530-X-R:C2E-25.000-10-1530-X-R
- C460: value 220pF -> 10uF
- C461: value 220pF -> 0.1uF
- C489: value 4.7uF -> 0.1uF
- R144: value 100k -> 43k
- R146: value 10k -> 56k
- R147, R176, R178: value 4.7k -> 10k
- R158, R159, R160, R187, R188: value 2.2k -> 10k
- R173: value 100k -> 12k
- R175: value 10k -> 15k
- R177: value 4.7k -> 200k
- R179: value 4.7k -> 100k
- R181: value 68k -> 10k
- R196, R197: value 1k -> 10k
Connections:
- net GL_USB30_FAULT_0 is gone; now on net VCC_3V3_S3: R180.1
- net I2C2_SCL_M4 is gone; now on net VCC_3V3_S3: R177.1
- net I2C2_SDA_M4 is gone; now on net VCC_3V3_S3: R176.1
- net TPS2_LDO_3V3 is gone; now on net GND: C492.1
- net VCC3V3_PCIE30_1 is gone; now on net VCC3V3_PCIE30: C452.2, C453.2, C454.2, J2.12 (P12), J2.14 (P14), J2.16 (P16), J2.18 (P18), J2.2 (P2), J2.4 (P4), J2.70 (P70), J2.72 (P72), J2.74 (P74)
- net VCC5V0_HDMI_TX0 is gone; now on net HDMI2_1_5V0: D12.1, R193.2, R202.2
- net VDD33 is gone; now on net VCC_3V3_S3: U48.12 (VDD33), U48.13 (VDD33), U48.26 (VDD33), U48.27 (VDD33), U48.31 (VDD33), U48.34 (VDD33), U48.35 (VDD33), U48.4 (VDD33), U48.5 (VDD33), U48.8 (VDD33)
- net FU_INT_L: now also R158.2
- net FU_INT_L2: no longer IC4.5 (INT_N)
- net FU_SCL_1: no longer U42.6 (SCL2)
- net FU_SCL_2: no longer IC4.6 (SCL)
- net FU_SDA_1: no longer U42.5 (SDA2)
- net FU_SDA_2: no longer IC4.7 (SDA)
- net GND: now also C500.2, R173.2, R175.1, R179.1, C561.2, C562.2, C565.2, C566.2, C567.2, C568.2, C569.2, C570.2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; no longer C461.2, IC4.15 (EP_GND), IC4.8 (GND_1), IC4.9 (GND_2), R173.1, R181.2, U40.D2 (GND), U42.1 (GND), U58.2 (GND)
- net GPIO3_B3_U: now also R179.2, U38.30 (GPIO3(HPD1)); no longer U40.D3 (A4)
- net GPIO3_B4_U: now also R174.2, U38.31 (GPIO4(HPD2)); no longer U40.C3 (A3)
- net HDMITX1_HPDIN_M1: now also Q3.3 (D)
- net HDMITX1_SCL_M1: now also Q5.2 (S)
- net HDMITX1_SDA_M1: now also Q6.2 (S)
- net HDMI_1_SDA_1: now also Q6.3 (D)
- net I2C4_SCL_M3: now also R149.1, U38.27 (I2C1_SCL); no longer U40.A3 (A1)
- net I2C4_SDA_M3: now also R150.1, U38.28 (I2C1_SDA); no longer R147.1, U40.B3 (A2)
- net TPS1_CLK: now also U38.38 (SPI_CLK)
- net TPS1_CS: now also U38.39 (~{SPI_CS})
- net TPS1_LDO_3V3: now also R146.2, R147.2, C578.1, U38.9 (LDO_3V3)
- net TPS1_MISO: now also U38.37 (SPI_PICO)
- net TPS1_MOSI: now also U38.36 (SPI_POCI)
- net USB1_CC1: now also C562.1, U38.24 (C1_CC1); no longer C460.1
- net USB1_CC2: now also C561.1, U38.26 (C1_CC2); no longer C461.1
- net USB20_HOST1_DM: now also U79.46 (USB2UP_DM)
- net USB20_HOST1_DP: now also U79.45 (USB2UP_DP)
- net USB2_CC1: now also C566.1, U38.45 (C2_CC1); no longer IC4.10 (CC1_1), IC4.11 (CC1_2)
- net USB2_CC2: now also C565.1, U38.47 (C2_CC2); no longer IC4.1 (CC2_1), IC4.14 (CC2_2)
- net USB30_2_SSRXN: now also C499.1
- net USB30_2_SSRXP: now also C590.1
- net USB30_2_SSTXN: now also U79.51 (USB3UP_RXDM)
- net USB30_2_SSTXP: now also U79.50 (USB3UP_RXDP)
- net USB3_0_DN: now also U79.9 (USB2DN_DM2/PRT_DIS_M2)
- net USB3_0_DP: now also U79.8 (USB2DN_DP2/PRT_DIS_P2)
- net USB3_0_RX_N: now also C593.1
- net USB3_0_RX_P: now also C594.1
- net USB3_0_TX_N: now also U79.14 (USB3DN_RXDM2)
- net USB3_0_TX_P: now also U79.13 (USB3DN_RXDP2)
- net USB3_0_VBUS: now also C609.2, U82.6 (OUT), U82.7 (OUT)
- net USB3_1_DN: now also U79.18 (USB2DN_DM3/PRT_DIS_M3)
- net USB3_1_DP: now also U79.17 (USB2DN_DP3/PRT_DIS_P3)
- net USB3_1_RX_N: now also C591.1
- net USB3_1_RX_P: now also C592.1
- net USB3_1_TX_N: now also U79.23 (USB3DN_RXDM3)
- net USB3_1_TX_P: now also U79.22 (USB3DN_RXDP3)
- net USB3_1_VBUS: now also C612.2, U83.6 (OUT), U83.7 (OUT); no longer U58.6 (OUT)
- net USB_1_OTG_DM: now also U38.53 (C1_USB_N(GPIO19))
- net USB_1_OTG_DP: now also U38.50 (C1_USB_P(GPIO18))
- net USB_2_OTG_DM: now also U38.55 (C2_USB_N(GPIO21))
- net USB_2_OTG_DP: now also U38.54 (C2_USB_P(GPIO20))
- net VBUS_A: now also C567.1, C568.1, C569.1, C570.1, C571.1, C572.1, C573.1, C574.1, C575.1, C576.1, C584.1, C588.1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; no longer IC4.2 (VBUS)
- net VCC_1V2_HUB: now also C599.2, C600.2, U79.12 (VDD12), U79.15 (VDD12), U79.21 (VDD12), U79.28 (VDD12), U79.33 (VDD12), U79.43 (VDD12), U79.49 (VDD12), U79.5 (VDD12)
- net VCC_1V8_SYS: now also R149.2, R150.2, R156.1, R157.1, R158.1, R187.1, R188.1; no longer C499.2, R146.1, R147.2, R159.1, R160.1, R175.1, R176.2, R177.2, U42.2 (VREF1)
- net VCC_3V3_ALW: now also R243.2, R244.2, U38.5 (VIN_3V3)
- net VCC_3V3_S0: now also Q5.1 (G)
- net VCC_3V3_S3: now also R178.1, R181.1, C597.2, C598.2, U79.16 (VDD33), U79.31 (VDD33), U79.44 (VDD33), U79.55 (VDD33)
- net VCC_3V3_SYS: now also R255.2, R257.2; no longer C449.2, C500.2, C511.2, IC4.3 (VDD_1), IC4.4 (VDD_2), R149.1, R150.1, R156.1, R157.1, R158.1, R178.1, R179.1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
- net VCC_4V0_SYS: now also C458.1, C459.1
- net VCC_5V0_PERIPH: now also C607.2, C608.2, C610.2, C611.2, U82.2 (IN), U82.3 (IN), U83.2 (IN), U83.3 (IN); no longer U58.1 (IN)
- net VCC_5V0_SYS: now also C500.1, C579.1, C580.1, C581.1, C582.1, U38.1 (PP_HV2), U38.11 (PP_HV1), U38.25 (PP1_CABLE), U38.46 (PP2_CABLE); no longer C458.1, C459.1, IC4.12 (VCONN_1), IC4.13 (VCONN_2)
- net at R197.1: now also Q6.1 (G)
- net at R144.2: now also R146.1, U38.6 (ADCIN1)
- net at U40.A1 (B1): no longer R150.2
- net at U40.B1 (B2): no longer R149.2
- net at R143.2: now also R147.1, U38.10 (ADCIN2)
- net at R195.1: now also Q1.3 (D), Q3.1 (G)
- net CFG_BC_EN: now reaches R178.2
- net CFG_BC_EN: now also U79.40 (SPI_DI/CFG_BC_EN/GPIO9)
- net at R198.2, R199.2: now also Q1.1 (G)
- net at C489.2: now also U60.6 (VCC)
- net at C492.2: now also U59.6 (VCC)
- net VBUS_DET: now reaches R175.2
- net VBUS_DET: now also R176.2, U79.37 (VBUS_DET/GPIO16)
- net at U40.C2 (OE): no longer R146.2
- net GL_USB30_EN_1: no longer names the net of U58.3 (EN)
- net GL_USB30_FAULT_1: no longer names the net of U58.4 (~{FAULT})
- net HDMI1_TX_SBDN renamed HDMI1_HP_DETECT
- net HDMI1_TX_SBDP renamed HDMI_1_SCL_1
- net HDMI_1_SCL_1: now also Q5.3 (D)
- net I2C1_IRQ_1: no longer names the net of U40.C1 (B3)
- net I2C5_SCL_M4: no longer names the net of R159.2
- net I2C5_SCL_M4: now also C461.2, R160.1, C583.2, C584.2, U39.4 (G), U49.4 (G); no longer U42.3 (SCL1)
- net I2C5_SDA_M4: no longer names the net of R160.2
- net I2C5_SDA_M4: now also U74.1; no longer U42.4 (SDA1)
- new net: C586.2, C587.2, C588.2, R247.2, R248.1, U50.4 (G), U61.4 (G)
- new net: R248.2, U77.1
- new net: U38.15 (DRAIN1), U38.19 (DRAIN1), U38.58 (DRAIN1), U38.8 (DRAIN1)
- new net: U38.52 (DRAIN2), U38.56 (DRAIN2), U38.57 (DRAIN2), U38.7 (DRAIN2)
- new net: R256.1, U82.5 (ILIM)
- new net: C594.2, U79.10 (USB3DN_TXDP2)
- new net: C587.1, R247.1, U50.5 (S), U61.5 (S)
- new net: C593.2, U79.11 (USB3DN_TXDM2)
- new net: C592.2, U79.19 (USB3DN_TXDP3)
- new net: C583.1, R159.1, U39.5 (S), U49.5 (S)
- new net: C499.2, U79.48 (USB3UP_TXDM)
- new net: R258.1, U83.5 (ILIM)
- new net: C511.2, U54.6 (VCC)
- new net: C449.2, U41.6 (VCC)
- new net: C591.2, U79.20 (USB3DN_TXDM3)
- new net: C590.2, U79.47 (USB3UP_TXDP)
- new net 12C1_EXTI_EC: U38.34 (~{I2C2_IRQ})
- new net CFG_NON_REM: R177.2, U79.41 (SPI_CE_N/CFG_NON_REM/GPIO7)
- new net GPIO3_B5_U: U38.29 (~{I2C1_IRQ})
- new net I2C1_SCL_EC: R243.1, U38.32 (I2C2_SCL)
- new net I2C1_SDA_EC: R244.1, U38.33 (I2C2_SDA)
- new net PP_EXT1: D17.1 (A1), R245.1, U38.48 (GPIO16(PP_EXT1)), U74.2
- new net PP_EXT2: D1.1 (A1), R246.1, U38.49 (GPIO17(PP_EXT2)), U77.2
- new net PRT_CTL2: R255.1, U79.35 (PRT_CTL2), U82.4 (EN), U82.8 (~{FAULT})
- new net PRT_CTL3: R257.1, U79.34 (PRT_CTL3), U83.4 (EN), U83.8 (~{FAULT})
- new net RBIAS: R173.1, U79.56 (RBIAS)
- new net SMCLK: R181.2, U79.38 (SPI_CLK/SMCLK/GPIO4)
- new net SMDAT: R180.2, U79.39 (SPI_DO/SMDAT/GPIO5)
- new net SYS_PWR: C460.1, C461.1, C585.1, C586.1, U39.1 (D), U39.2 (D), U39.3 (D), U50.1 (D), U50.2 (D), U50.3 (D)
- new net TPS1_LDO_1V8: C577.1, U38.35 (LDO_1V8)
- new net USB30_HUB_RST: U79.42 (RESET_N)
- new net USB_CTRL_RESET: U38.44 (HRESET)
- new net USB_MACRO_DN: U79.2 (USB2DN_DM1/PRT_DIS_M1)
- new net USB_MACRO_DP: U79.1 (USB2DN_DP1/PRT_DIS_P1)
- new net XTALI/CLK_IN: C595.2, U79.54 (XTALI/CLK_IN), Y7.3
- new net XTALO: C596.2, U79.53 (XTALO), Y7.1
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Other:
- note added: "40-PIN eDP CONNECTOR AUO B160ZAN01.U DISPLAY"
- note added: "CAPS FOR A4, A9, B4, B9 PINS"
- note added: "CLOCK GENERATOR"
- note added: "CONNECT TO 3V3 GPIO LINE"
- note added: "DISPLAY CONNECTOR"
- note added: "DISPLAYPORT + PD OVER USB-C"
- note added: "HDMI OUTPUT"
- note added: "KEYBOARD CONNECTOR"
- note added: "LEAVE THEM UNCONNECTED"
- note added: "M.2 SLOTS"
- note added: "USB 3.1 GEN 1 TYPE-A PORT"
- note added: "use the W25Q80JVNIQ"
- note removed: "1%"
- note removed: "40-PIN eDP CONNECTOR"
- note removed: "AUO B160ZAN01.U DISPLAY"
- note removed: "EC PROGRAMMING PINS"
- note removed: "HDMI PORTS"
- note removed: "HEADPHONE JACK"
- note removed: "LEFT SPEAKER"
- note removed: "RIGHT SPEAKER"
- note removed: "USB TYPE-A PORT"
- note removed: "USB TYPE-C PORTS"
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
Commit message: removed unused components and connections
Parts:
- removed C431: 0.1uF, Capacitor_SMD:C_0201_0603Metric, symbol Device:C
- removed IC4: FUSB302BMPX, barebones:QFN50P250X250X80-15N, symbol FUSB302BMPX:FUSB302BMPX
- removed J14: SM05B-SRSS-TB_LF__SN_, SM05B-SRSS-TB_LF__SN_:JST_SM05B-SRSS-TB_LF__SN_, symbol SM05B-SRSS-TB_LF__SN_:SM05B-SRSS-TB_LF__SN_
- removed J15: 20455-040E-76, 20455-040E-76:IPEX_20455-040E-76, symbol 20455-040E-76:20455-040E-76
- removed J16: 524352671, barebones:CON_524352671_MOL, symbol 524352671:524352671
- removed J17: 522070485, barebones:CON_522070485_MOL, symbol 522070485:522070485
- removed J7: 1-84953-4, 1-84953-4:TE_1-84953-4, symbol 1-84953-4:1-84953-4
- removed J9: 1040310811, barebones:104031-0811_MOL, symbol 1040310811:1040310811
- removed Q9: CSD18504Q5A, barebones:MOSFET_CSD19531Q5A, symbol CSD18504Q5A:CSD18504Q5A
- removed U40, U46: TXS0104EYZTR, barebones:BGA12N50P4X3_186X136X62N, symbol TXS0104EYZTR:TXS0104EYZTR
- removed U42, U51: PCA9306DCTR, barebones:SOP65P400X130-8N, symbol PCA9306DCTR:PCA9306DCTR
- removed U44: TPD4E05U06DQAR, barebones:IC_TPD4E05U06DQAR, symbol TPD4E05U06DQAR:TPD4E05U06DQAR
- removed U47, U58: TPS2553DBVR, barebones:SOT95P280X145-6N, symbol TPS2553DBVR:TPS2553DBVR
- removed U48: PI3DPX1207Q3ZHEX, barebones:QFN50P900X350X84-43N, symbol PI3DPX1207Q3ZHEX:PI3DPX1207Q3ZHEX
- removed U52: OV9734-H16A, OV9734-H16A:BGA16N27X30P8X4_253X172X80N, symbol OV9734-H16A:OV9734-H16A
- removed U55: PI6C557-05BLEX, barebones:TSSOP-20_L6.5-W4.4-P0.65-LS6.4-BL, symbol PI6C557-05BLEX:PI6C557-05BLEX
- removed U56: PI6C557-05LEX, easyeda2kicad:TSSOP-20_L6.5-W4.4-P0.65-LS6.4-BL, symbol PI6C557-05LEX:PI6C557-05LEX
- removed U57: PI6C557-03ALEX, easyeda2kicad:TSSOP-16_L5.0-W4.4-P0.65-LS6.4-BL, symbol PI6C557-03ALEX:PI6C557-03ALEX
- added C468: 10uF, Capacitor_SMD:C_0201_0603Metric, symbol Device:C
- added C605: 0.1uF, Capacitor_SMD:C_0201_0603Metric, symbol Device:C
Connections:
- net VCC_4V0_SYS is gone; now on net VCC_5V0_SYS: C458.1, C459.1, C563.2, J25.40
- net GND: now also C468.2, C605.2
- net TPS1_LDO_3V3: now also IC1.8 (VCC), C605.1
- net VCC_3V3_ALW: now also C468.1

Commit message: updated last changes
Parts:
- removed C458, C516, C544, C591: 0.1uF, Capacitor_SMD:C_0201_0603Metric, symbol Device:C
- removed C545: 10uF, Capacitor_SMD:C_0201_0603Metric, symbol Device:C
- removed C573, C574, C575, C576: 10nF, Capacitor_SMD:C_0201_0603Metric, symbol Device:C
- removed C581: 22uF, Capacitor_SMD:C_0201_0603Metric, symbol Device:C
- removed D12: SD103AWS-E3-08, SD103AWS-E3-08:SOD2713X115N, symbol SD103AWS-E3-08:SD103AWS-E3-08
- removed FPC1: FH12-6S-0.5SH, barebones:FPC-SMD_FH12-6S-0.5SH-55, symbol FH12-6S-0.5SH(55):FH12-6S-0.5SH
- removed IC1: W25Q80DVSSIG, barebones:SOIC8-FLASH, symbol W25Q80DVSSIG:W25Q80DVSSIG
- removed J20: 20682-040E-02, 20682-040E-02:IPEX_20682-040E-02, symbol 20682-040E-02:20682-040E-02
- removed J4: 21992304, barebones:TE_21992304, symbol 21992304:21992304
- removed Q5, Q6: BSS138, Package_TO_SOT_SMD:SOT-23, symbol Transistor_FET:BSS138
- removed R149, R150, R243, R244: 4.7k, Resistor_SMD:R_0402_1005Metric, symbol Device:R
- removed R151, R158, R187, R188, R192, R193, R196, R197: 10k, Resistor_SMD:R_0402_1005Metric, symbol Device:R
- removed R156, R157: 2.2k, Resistor_SMD:R_0402_1005Metric, symbol Device:R
- removed R202: 1.8k, Resistor_SMD:R_0402_1005Metric, symbol Device:R
- removed U39, U49, U50, U61: CSD25402Q3A, barebones:TRANS_CSD25402Q3A, symbol Transistor_FET:CSD25402Q3A
- removed U59, U60: TPD4E004DRYR, barebones:PSON50P145X100X60-6N, symbol TPD4E004DRYR:TPD4E004DRYR
- removed U82, U83: TPS2557DRBR, TPS2557DRBR:SON65P300X300X100-9N, symbol TPS2557DRBR:TPS2557DRBR
- added C547, C554: 10uF, Capacitor_SMD:C_0603_1608Metric, symbol Device:C
- added C553, C613, C624, C625, C626, C627, C628, C629, C630, C631, C632, C633, C634, C635, C636, C637, C697, C705, C706, C716, C724: 0.1uF, Capacitor_SMD:C_0201_0603Metric, symbol Device:C
- added C601: 22uF, Capacitor_SMD:C_0603_1608Metric, symbol Device:C
- added C606, C616: 100nF, Capacitor_SMD:C_0402_1005Metric, symbol Device:C
- added C614: 4.7uF, Capacitor_SMD:C_0402_1005Metric, symbol Device:C
- added C617, C618: 10uF, Capacitor_SMD:C_0402_1005Metric, symbol Device:C
- added C689: 1uF, Capacitor_SMD:C_0201_0603Metric, symbol Device:C
- added D19: TPD6E05U06RVZR, barebones:SON50P135X350X55-14N, symbol TPD6E05U06RVZR:TPD6E05U06RVZR
- added D20: SD103AWS-E3-08, barebones:SOD2713X115N, symbol SD103AWS-E3-08:SD103AWS-E3-08
- added J6: 2199119-4, barebones:TE_2199119-4, symbol 2199119-4:2199119-4
- added J7: 5034801200, barebones:CON_5034801200_MOL, symbol 5034801200:5034801200
- added J9: 20455-040E-76, barebones:IPEX_20455-040E-76, symbol 20455-040E-76:20455-040E-76
- added Q2, Q7, Q8, Q9: CSD25402Q3A, barebones:TRANS_CSD25402Q3A, symbol CSD25402Q3A:CSD25402Q3A
- added R155: 10k, Resistor_SMD:R_0402_1005Metric, symbol Device:R
- added R183: 100k, Resistor_SMD:R_0201_0603Metric, symbol Device:R
- added R186, R253, R259, R260, R261, R271, R272: 10k, Resistor_SMD:R_0201_0603Metric, symbol Device:R
- added R262, R263: 1.8k, Resistor_SMD:R_0201_0603Metric, symbol Device:R
- added R264: 200k, Resistor_SMD:R_0201_0603Metric, symbol Device:R
- added R269: 200R, Resistor_SMD:R_0201_0603Metric, symbol Device:R
- added U11, U20: PCA9306DCTR, barebones:SOP65P400X130-8N, symbol PCA9306DCTR:PCA9306DCTR
- added U15: TPS22919DCK, Package_TO_SOT_SMD:SOT-363_SC-70-6, symbol Power_Management:TPS22919DCK
- added U2: W25Q16JVUXIQ_TR, barebones:IC_W25Q16JVUXIQ_TR, symbol W25Q16JVUXIQ_TR:W25Q16JVUXIQ_TR
- added U85, U86: TPS2557DRBR, barebones:SON65P300X300X100-9N, symbol TPS2557DRBR:TPS2557DRBR
- C432, C433, C436, C437, C438, C439, C440, C441, C442, C443, C444, C445, C446, C447, C448, C449, C450, C451, C452, C453, C455, C456, C461, C463, C464, C469, C470, C471, C472, C474, C476, C479, C482, C486, C488, C491, C495, C497, C501, C502, C503, C504, C511, C528, C541, C561, C562, C563, C564, C565, C566, C567, C568, C583, C584, C586, C587, C588, C595, C596, C607, C608, C609, C610, C611, C612: footprint Capacitor_SMD:C_0201_0603Metric -> Capacitor_SMD:C_0402_1005Metric; KiLib_Generator (none) -> SMD_2terminal_chip_molded
- C454: value 100nF -> 10uF; footprint Capacitor_SMD:C_0201_0603Metric -> Capacitor_SMD:C_0402_1005Metric; KiLib_Generator (none) -> SMD_2terminal_chip_molded
- C457: value 100nF -> 100uF; footprint Capacitor_SMD:C_0201_0603Metric -> Capacitor_SMD:C_0402_1005Metric; KiLib_Generator (none) -> SMD_2terminal_chip_molded
- C459, C492, C592, C594, C600: value 0.1uF -> 100nF; footprint Capacitor_SMD:C_0201_0603Metric -> Capacitor_SMD:C_0402_1005Metric; KiLib_Generator (none) -> SMD_2terminal_chip_molded
- C460, C468, C577, C578, C579, C580, C582, C585: footprint Capacitor_SMD:C_0201_0603Metric -> Capacitor_SMD:C_0603_1608Metric; KiLib_Generator (none) -> SMD_2terminal_chip_molded
- C462, C593, C598: value 0.1uF -> 10uF; footprint Capacitor_SMD:C_0201_0603Metric -> Capacitor_SMD:C_0402_1005Metric; KiLib_Generator (none) -> SMD_2terminal_chip_molded
- C489: value 0.1uF -> 22uF; footprint Capacitor_SMD:C_0201_0603Metric -> Capacitor_SMD:C_0402_1005Metric; KiLib_Generator (none) -> SMD_2terminal_chip_molded
- C499, C500, C507, C508, C509, C510, C521, C531, C532, C533, C534, C535, C536, C537, C538, C543, C605: KiLib_Generator (none) -> SMD_2terminal_chip_molded
- C512, C513: footprint Capacitor_SMD:C_0201_0603Metric -> Capacitor_SMD:C_0805_2012Metric; KiLib_Generator (none) -> SMD_2terminal_chip_molded
- C529: value 100uF -> 0.1uF; KiLib_Generator (none) -> SMD_2terminal_chip_molded
- C569, C570, C571, C572: value 10nF -> 0.1uF; KiLib_Generator (none) -> SMD_2terminal_chip_molded
- C590: value 0.1uF -> 1uF; KiLib_Generator (none) -> SMD_2terminal_chip_molded
- C597: value 10uF -> 100nF; footprint Capacitor_SMD:C_0201_0603Metric -> Capacitor_SMD:C_0402_1005Metric; KiLib_Generator (none) -> SMD_2terminal_chip_molded
- C599: value 1uF -> 100nF; footprint Capacitor_SMD:C_0201_0603Metric -> Capacitor_SMD:C_0402_1005Metric; KiLib_Generator (none) -> SMD_2terminal_chip_molded
- D13: footprint SD103AWS-E3-08:SOD2713X115N -> barebones:SOD2713X115N
- J12: footprint 10067847-001RLF:AMPHENOL_10067847-001RLF -> barebones:AMPHENOL_10067847-001RLF
- R143, R144, R146, R147, R173, R174, R175, R176, R179, R180, R181, R194, R195, R199, R200, R201, R204, R205, R206, R207, R208, R209, R210, R211: footprint Resistor_SMD:R_0402_1005Metric -> Resistor_SMD:R_0201_0603Metric
- R177: value 200k -> 10k; footprint Resistor_SMD:R_0402_1005Metric -> Resistor_SMD:R_0201_0603Metric
- R178: value 10k -> 10R; footprint Resistor_SMD:R_0402_1005Metric -> Resistor_SMD:R_0201_0603Metric
- R182: value 10k -> 100k; footprint Resistor_SMD:R_0402_1005Metric -> Resistor_SMD:R_0201_0603Metric
- R184, R185: footprint Resistor_SMD:R_0402_1005Metric -> Resistor_SMD:R_0805_2012Metric
- U65, U67, U68, U69, U70, U74, U77: footprint 2N7002KW:SOT323 -> barebones:SOT323
Connections:
- net FU_INT_L2 is gone; now on net 12C1_EXTI_EC: R182.2
- net VCC5V0_SYS is gone; now on net VCC_5V0_SYS: U65.2
- net VCC5V_HDMI_TX1 is gone; now on net HDMI2_1_5V0: C528.2, C529.2
- net VCC_5V0_ALW is gone; now on net VCC_5V0_SYS: C564.2, J25.41
- net VCC_5V0_PERIPH is gone; now on net VCC_5V0_SYS: C607.2, C608.2, C610.2, C611.2
- net CFG_BC_EN: now also R178.1; no longer R178.2
- net CFG_NON_REM: now also R177.1; no longer R177.2
- net EDP_TX0_AUX_N: now also J9.16
- net EDP_TX0_AUX_P: now also J9.15
- net EDP_TX0_BL_EN: now also J9.32
- net EDP_TX0_BL_PWM: now also J9.33
- net EDP_TX0_HDP: now also J9.27
- net GND: now also C459.1, C462.1, C570.1, C592.1, C593.1, C594.1, R177.2, R178.2, R182.1, C547.2, C553.1, C554.2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; no longer C459.2, C462.2, C500.2, C521.2, C569.2, C570.2, C571.2, C572.2
- net GPIO3_B5_U: now also R183.2
- net HDMI0_TX0N_PORT/eDP0_TX_D0N: now also J9.12
- net HDMI0_TX0P_PORT/eDP0_TX_D0P: now also J9.13
- net HDMI0_TX1N_PORT/eDP0_TX_D1N: now also J9.9
- net HDMI0_TX1P_PORT/eDP0_TX_D1P: now also J9.10
- net HDMI0_TX2N_PORT/eDP0_TX_D2N: now also J9.6
- net HDMI0_TX2P_PORT/eDP0_TX_D2P: now also J9.7
- net HDMI0_TX3N_PORT/eDP0_TX_D3N: now also J9.3
- net HDMI0_TX3P_PORT/eDP0_TX_D3P: now also J9.4
- net HDMI1_TX_SBDN/eDP1_TX_AUXN: now also C689.2
- net HDMI1_TX_SBDP/eDP1_TX_AUXP: now also C590.2
- net HDMI2_1_5V0: now also D20.1, R262.2, R263.2, R264.2
- net HDMITX1_SCL_M1: now also R253.1, U11.3 (SCL1)
- net HDMITX1_SDA_M1: now also R261.1, U11.4 (SDA1)
- net HDMI_1_SCL_1: now also C590.1, R262.1, U11.6 (SCL2)
- net HDMI_1_SDA_1: now also R263.1, U11.5 (SDA2)
- net PCIE20_0_REFCLKN_SLOT: now also J6.49
- net PCIE20_0_REFCLKP_SLOT: now also J6.47
- net PCIE20_0_RXN: now also J6.43
- net PCIE20_0_RXP: now also J6.41
- net PCIE30X1_0_CLKREQn_M1_L: now also J6.53
- net PCIE30X1_0_PERSTn_M1_L: now also J6.52
- net PCIE30X1_0_WAKEn_M1_L: now also J6.55
- net PRT_CTL3: now also R255.1, U86.4 (EN), U86.8 (~{FAULT}); no longer R257.1
- net SDMMC_CLK: now also D19.11 (D2N)
- net SDMMC_CMD: now also D19.12 (D2P)
- net SDMMC_DAT0: now also D19.9 (D3P)
- net SDMMC_DAT1: now also D19.8 (D3N)
- net SDMMC_DAT2: now also D19.14 (D1P)
- net SDMMC_DAT3: now also D19.13 (D1N)
- net SYS_PWR: now also C547.1, C554.1, Q7.1, Q7.2, Q7.3, Q8.1, Q8.2, Q8.3
- net TMDS_CLOCK_1_DM: now also D15.5 (IO4); no longer D15.2 (IO2)
- net TMDS_CLOCK_1_DP: now also D15.4 (IO3); no longer D15.1 (IO1)
- net TMDS_DATA0_1_DM: now also D15.2 (IO2); no longer D15.5 (IO4)
- net TMDS_DATA0_1_DP: now also D15.1 (IO1); no longer D15.4 (IO3)
- net TPS1_CLK: now also U2.6 (CLK)
- net TPS1_CS: now also U2.1 (~{CS})
- net TPS1_LDO_3V3: now also C624.1, C637.1, U2.3 (~{WP}/IO2), U2.7 (~{HOLD}/~{RESET}/IO3), U2.8 (VCC)
- net TPS1_MISO: now also U2.2 (DO/IO1)
- net TPS1_MOSI: now also U2.5 (DI/IO0)
- net USB20_HOST0_DM: now also J6.5
- net USB20_HOST0_DP: now also J6.3
- net USB30_2_SSRXP: now also C500.1; no longer C590.1
- net USB3_0_DN: now also D10.12 (D2P), U79.18 (USB2DN_DM3/PRT_DIS_M3); no longer D10.14 (D1P), U79.9 (USB2DN_DM2/PRT_DIS_M2)
- net USB3_0_DP: now also D10.11 (D2N), U79.17 (USB2DN_DP3/PRT_DIS_P3); no longer D10.13 (D1N), U79.8 (USB2DN_DP2/PRT_DIS_P2)
- net USB3_0_RX_N: now also C521.1, D10.14 (D1P); no longer C593.1, D10.11 (D2N)
- net USB3_0_RX_P: now also C571.1, D10.13 (D1N); no longer C594.1, D10.12 (D2P)
- net USB3_0_TX_N: now also U79.23 (USB3DN_RXDM3); no longer U79.14 (USB3DN_RXDM2)
- net USB3_0_TX_P: now also U79.22 (USB3DN_RXDP3); no longer U79.13 (USB3DN_RXDP2)
- net USB3_0_VBUS: now also U86.6 (OUT), U86.7 (OUT)
- net USB3_1_DN: now also D11.11 (D2N), U79.25 (USB2DN_DM4/PRT_DIS_M4); no longer D11.13 (D1N), U79.18 (USB2DN_DM3/PRT_DIS_M3)
- net USB3_1_DP: now also D11.12 (D2P), U79.24 (USB2DN_DP4/PRT_DIS_P4); no longer D11.14 (D1P), U79.17 (USB2DN_DP3/PRT_DIS_P3)
- net USB3_1_RX_N: now also C569.1, D11.14 (D1P); no longer D11.11 (D2N)
- net USB3_1_RX_P: now also C572.1, D11.13 (D1N); no longer C592.1, D11.12 (D2P)
- net USB3_1_TX_N: now also U79.30 (USB3DN_RXDM4); no longer U79.23 (USB3DN_RXDM3)
- net USB3_1_TX_P: now also U79.29 (USB3DN_RXDP4); no longer U79.22 (USB3DN_RXDP3)
- net USB3_1_VBUS: now also U85.6 (OUT), U85.7 (OUT)
- net VBUS_A: now also Q2.1, Q2.2, Q2.3, Q9.1, Q9.2, Q9.3; no longer C569.1, C570.1, C571.1, C572.1
- net VCC3V3_PCIE30: now also C492.2, C592.2, C593.2, C594.2, C597.2, C598.2; no longer C455.2, C456.2, C457.2, J3.12 (P12), J3.14 (P14), J3.16 (P16), J3.18 (P18), J3.2 (P2), J3.4 (P4), J3.70 (P70), J3.72 (P72), J3.74 (P74)
- net VCC_12V_EDP: now also C570.2, C613.2, C614.2, J9.36, J9.37, J9.38, J9.39
- net VCC_1V2_HUB: now also C629.2, C630.2, C631.2, C632.2, C633.2, C634.2, C635.2, C636.2; no longer C599.2, C600.2
- net VCC_3V3_S0: now also R253.2, R259.2, R261.2, R269.2, R271.2, U11.2 (VREF1)
- net VCC_3V3_S3: now also C541.2, C543.2, R255.2, R257.2, C553.2, C625.2, C626.2, C627.2, C628.2, J9.18, J9.19, J9.20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; no longer C597.2, C598.2, R177.1, R178.1
- net VCC_3V3_SYS: now also C459.2, C462.2, C489.2, J6.2, J6.4, J6.72, J6.74, R155.1; no longer C462.1, C521.1, C541.2, C543.2, R255.2, R257.2
- net VCC_5V0_SYS: now also C601.1, D20.2, U85.2 (IN), U85.3 (IN), U86.2 (IN), U86.3 (IN); no longer C459.1, C500.1
- net at C586.2, C587.2, C588.2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: now also Q8.4, Q9.4
- net at R256.1: now also U86.5 (ILIM)
- net at U79.10 (USB3DN_TXDP2): no longer C594.2
- net at C587.1, R247.1: now also Q8.9, Q9.9
- net at U79.11 (USB3DN_TXDM2): no longer C593.2
- net HDMI1_HP_DETECT renamed HDMI_1_TX_SBDN
- net VCC_1V8_SYS renamed VCC_1V8_S3
- new net: C716.1, J7.4, U15.5 (QOD), U15.6 (OUT)
- new net: C724.2, R269.1, U20.7 (VREF2), U20.8 (EN)
- new net: C697.2, R264.1, U11.7 (VREF2), U11.8 (EN)
- new net CAM_DN: J7.3, U79.9 (USB2DN_DM2/PRT_DIS_M2)
- new net CAM_DP: J7.2, U79.8 (USB2DN_DP2/PRT_DIS_P2)
- new net CAM_SW: J7.5
- new net I2C3_SCL_M0: R260.1, U20.3 (SCL1)
- new net I2C3_SDA_M0: R272.1, U20.4 (SDA1)
- new net INT_ALS: J7.9
- new net MIC_CLK: J7.6
- new net MIC_DAT: J7.7
- new net MIC_SW: J7.8
- new net PCIE30X1_W_EN: J6.56, R155.2
- new net SCL_ALS: J7.10, R259.1, U20.6 (SCL2)
- new net SDA_ALS: J7.11, R271.1, U20.5 (SDA2)
- new net VCC3V3_PCIE30_1: C455.2, C456.2, C457.2, C599.2, C600.2, C606.2, C616.2, C617.2, C618.2, J3.12 (P12), J3.14 (P14), J3.16 (P16)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
- new net WEBCAM_EN: R186.2, U15.3 (ON)
- new net WEBCAM_PWR: C705.1, C706.1, U15.1 (IN)
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Other:
- note added: "40-PIN eDP CONNECTOR AUO B160QAN02.0 DISPLAY"
- note added: "KEYBOARD + TRACKPAD"
- note added: "WEBCAM CONNECTOR"
- note removed: "40-PIN eDP CONNECTOR AUO B160ZAN01.U DISPLAY"
- note removed: "6-PIN BACKLIGHT CONNECTOR"
- note removed: "CAPS FOR A4, A9, B4, B9 PINS"
- note removed: "LEAVE THEM UNCONNECTED"
- note removed: "use the W25Q80JVNIQ"
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
Commit message: started routing on LPDDR4x RAM
Parts:
- removed C437, C459: 100nF, Capacitor_SMD:C_0402_1005Metric, symbol Device:C
- removed C438, C462, C617: 10uF, Capacitor_SMD:C_0402_1005Metric, symbol Device:C
- removed C439, C489: 22uF, Capacitor_SMD:C_0402_1005Metric, symbol Device:C
- removed C457: 100uF, Capacitor_SMD:C_0402_1005Metric, symbol Device:C
- removed C507: 0.1uF, Capacitor_SMD:C_0201_0603Metric, symbol Device:C
- removed C568: 1uF, Capacitor_SMD:C_0402_1005Metric, symbol Device:C
- removed J1, J5: 12401610E4_2A, barebones:AMPHENOL_12401610E4_2A, symbol 12401610E4_2A:12401610E4_2A
- removed R183: 100k, Resistor_SMD:R_0201_0603Metric, symbol Device:R
- added C514, C723, C726, C741, C745, C746: 0.1uF, Capacitor_SMD:C_0402_1005Metric, symbol Device:C
- added C619, C620: 1uF, Capacitor_SMD:C_0603_1608Metric, symbol Device:C
- added C682, C683, C742, C747: 10uF, Capacitor_SMD:C_0603_1608Metric, symbol Device:C
- added C725: 10uF, Capacitor_SMD:C_0805_2012Metric, symbol Device:C
- added C733, C734, C735, C736, C737, C738, C739, C740, C743, C744: 22uF, Capacitor_SMD:C_0805_2012Metric, symbol Device:C
- added C752: 150uF, Capacitor_Tantalum_SMD:CP_EIA-7343-20_Kemet-V, symbol Device:C
- added D12, D2: SMAJ22A, Diode_SMD:D_SMA, symbol Diode:SMAJ22A
- added J23, J26: 10137062-00021LF, barebones:AMPHENOL_10137062-00021LF, symbol Connector:USB_C_Receptacle
- C452, C453, C455, C456, C492, C495, C497, C501, C502, C592, C594, C597, C599, C600, C606, C616: value 100nF -> 0.1uF
- C454, C588, C593, C598, C607, C610, C618: footprint Capacitor_SMD:C_0402_1005Metric -> Capacitor_SMD:C_0603_1608Metric
- C468, C577, C578, C579, C580, C582, C601: footprint Capacitor_SMD:C_0603_1608Metric -> Capacitor_SMD:C_0805_2012Metric
- C503, C608: footprint Capacitor_SMD:C_0402_1005Metric -> Capacitor_SMD:C_0805_2012Metric
- C504: value 100nF -> 0.1uF; footprint Capacitor_SMD:C_0402_1005Metric -> Capacitor_SMD:C_0603_1608Metric
- C509, C605, C624, C637: footprint Capacitor_SMD:C_0201_0603Metric -> Capacitor_SMD:C_0402_1005Metric
- C567: value 1uF -> 0.1uF
- C609, C612: value 120uF -> 0.1uF; footprint Capacitor_SMD:C_0402_1005Metric -> Capacitor_SMD:C_0805_2012Metric
- R143, R144, R146, R147, R174, R179: footprint Resistor_SMD:R_0201_0603Metric -> Resistor_SMD:R_0402_1005Metric
- R182: value 100k -> 10k; footprint Resistor_SMD:R_0201_0603Metric -> Resistor_SMD:R_0402_1005Metric
- R256, R258: value 20.2k -> 20k
Connections:
- net 12C1_EXTI_EC: no longer R182.2
- net GND: now also C503.1, C504.1, C619.2, C620.2, C682.1, C683.1, C723.2, C725.1, C726.1, C733.1, C734.1, C735.1, C736.1, C737.1, C738.1, C739.1, C740.1, C741.1, C742.1, C743.1, C744.1, C745.1, C746.1, C747.1, C752.2, D12.2 (A2), D2.2 (A2), J23.A1 (GND), J23.A12 (GND), J23.B1 (GND), J23.B12 (GND), J23.SH (SHIELD), J26.A1 (GND), J26.A12 (GND), J26.B1 (GND), J26.B12 (GND), J26.SH (SHIELD); no longer R182.1
- net GPIO3_B5_U: now also R182.1
- net PRT_CTL4: no longer U85.4 (EN)
- net SDMMC_CLK: now also D19.4 (D2N_1)
- net SDMMC_CMD: now also D19.3 (D2P_1)
- net SDMMC_DAT0: now also D19.6 (D3P_1)
- net SDMMC_DAT1: now also D19.7 (D3N_1)
- net SDMMC_DAT2: now also D19.1 (D1P_1)
- net SDMMC_DAT3: now also D19.2 (D1N_1)
- net TMDS_CLOCK_1_DM: now also D15.6 (104_1)
- net TMDS_CLOCK_1_DP: now also D15.7 (IO3_1)
- net TMDS_DATA0_1_DM: now also D15.9 (IO2_1)
- net TMDS_DATA0_1_DP: now also D15.10 (IO1_1)
- net TMDS_DATA1_1_DM: now also D14.6 (104_1)
- net TMDS_DATA1_1_DP: now also D14.7 (IO3_1)
- net TMDS_DATA2_1_DM: now also D14.9 (IO2_1)
- net TMDS_DATA2_1_DP: now also D14.10 (IO1_1)
- net USB1_CC1: now also U38.45 (C2_CC1), J26.A5 (CC1); no longer U38.24 (C1_CC1)
- net USB1_CC2: now also U38.47 (C2_CC2), J26.B5 (CC2); no longer U38.26 (C1_CC2)
- net USB1_TX1N: now also D7.10 (IO1_1), J26.A3 (TX1-)
- net USB1_TX1P: now also D7.9 (IO2_1), J26.A2 (TX1+)
- net USB1_TX2N: now also D6.1 (IO1), D6.10 (IO1_1), J26.B3 (TX2-); no longer D7.4 (IO3)
- net USB1_TX2P: now also D6.2 (IO2), D6.9 (IO2_1), J26.B2 (TX2+); no longer D7.5 (IO4)
- net USB2_CC1: now also U38.24 (C1_CC1), J23.A5 (CC1); no longer U38.45 (C2_CC1)
- net USB2_CC2: now also U38.26 (C1_CC2), J23.B5 (CC2); no longer U38.47 (C2_CC2)
- net USB2_TX1N: now also D8.1 (IO1), D8.10 (IO1_1), J23.A3 (TX1-); no longer D9.1 (IO1)
- net USB2_TX1P: now also D8.2 (IO2), D8.9 (IO2_1), J23.A2 (TX1+); no longer D9.2 (IO2)
- net USB2_TX2N: now also D9.1 (IO1), D9.10 (IO1_1), J23.B3 (TX2-); no longer D9.4 (IO3)
- net USB2_TX2P: now also D9.2 (IO2), D9.9 (IO2_1), J23.B2 (TX2+); no longer D9.5 (IO4)
- net USB3_0_DN: now also D10.11 (D2N), D10.4 (D2N_1); no longer D10.12 (D2P)
- net USB3_0_DP: now also D10.12 (D2P), D10.3 (D2P_1); no longer D10.11 (D2N)
- net USB3_0_RX_N: now also D10.1 (D1P_1)
- net USB3_0_RX_P: now also D10.2 (D1N_1)
- net USB3_0_TX_N: now also D10.6 (D3P_1), D10.9 (D3P), C514.1; no longer D10.8 (D3N)
- net USB3_0_TX_P: now also D10.7 (D3N_1), D10.8 (D3N); no longer D10.9 (D3P)
- net USB3_0_VBUS: now also C725.2, C733.2, C734.2, C735.2, C736.2, C737.2, C738.2, C739.2, C740.2, C743.2, C744.2
- net USB3_1_DN: now also D11.4 (D2N_1)
- net USB3_1_DP: now also D11.3 (D2P_1)
- net USB3_1_RX_N: now also D11.1 (D1P_1)
- net USB3_1_RX_P: now also D11.2 (D1N_1)
- net USB3_1_TX_N: now also D11.6 (D3P_1), D11.9 (D3P); no longer D11.8 (D3N)
- net USB3_1_TX_P: now also D11.7 (D3N_1), D11.8 (D3N); no longer D11.9 (D3P)
- net USB3_1_VBUS: now also C752.1
- net USB_1_OTG_DP: now also U38.54 (C2_USB_P(GPIO20)), U41.4, J26.A6 (D+), J26.B6 (D+); no longer U38.50 (C1_USB_P(GPIO18)), U41.1
- net USB_1_RX1N: now also D7.5 (IO4), D7.6 (104_1), J26.B10 (RX1-); no longer D6.4 (IO3)
- net USB_1_RX1P: now also D7.4 (IO3), D7.7 (IO3_1), J26.B11 (RX1+); no longer D6.5 (IO4)
- net USB_1_RX2N: now also D6.5 (IO4), D6.6 (104_1), J26.A10 (RX2-); no longer D6.1 (IO1)
- net USB_1_RX2P: now also D6.4 (IO3), D6.7 (IO3_1), J26.A11 (RX2+); no longer D6.2 (IO2)
- net USB_1_SBU1: now also U41.1, J26.A8 (SBU1); no longer U41.4
- net USB_1_SBU2: now also U41.2, J26.B8 (SBU2); no longer U41.5
- net USB_2_OTG_DP: now also U38.50 (C1_USB_P(GPIO18)), U54.4, J23.A6 (D+), J23.B6 (D+); no longer U38.54 (C2_USB_P(GPIO20)), U54.1
- net USB_2_RX1N: now also D8.5 (IO4), D8.6 (104_1), J23.B10 (RX1-); no longer D8.4 (IO3)
- net USB_2_RX1P: now also D8.4 (IO3), D8.7 (IO3_1), J23.B11 (RX1+); no longer D8.5 (IO4)
- net USB_2_RX2N: now also D9.5 (IO4), D9.6 (104_1), J23.A10 (RX2-); no longer D8.1 (IO1)
- net USB_2_RX2P: now also D9.4 (IO3), D9.7 (IO3_1), J23.A11 (RX2+); no longer D8.2 (IO2)
- net USB_2_SBU1: now also U54.1, J23.A8 (SBU1); no longer U54.4
- net USB_2_SBU2: now also U54.2, J23.B8 (SBU2); no longer U54.5
- net VCC3V3_PCIE30_1: now also C682.2, C683.2
- net VCC_3V3_S0: now also R182.2
- net VCC_3V3_S3: now also J12.4 (VDD), U85.4 (EN)
- net VCC_3V3_SYS: now also C726.2, C741.2, C742.2, C745.2, C746.2, C747.2
- net unconnected-(U38-DRAIN1-Pad15)_2: now reaches U38.15 (DRAIN1), U38.19 (DRAIN1), U38.58 (DRAIN1), U38.8 (DRAIN1)
- net unconnected-(U38-DRAIN2-Pad52)_1: now reaches U38.52 (DRAIN2), U38.56 (DRAIN2), U38.57 (DRAIN2), U38.7 (DRAIN2)
- net USB3_0_SSTX_N: now reaches J10.8 (SSTX-)
- net USB3_0_SSTX_N: now also C514.2
- net USB3_0_SSTX_P: now reaches C509.2, J10.9 (SSTX+)
- net I2C3_SCL_M0 renamed I2C8_SCL_M2
- net I2C3_SDA_M0 renamed I2C8_SDA_M2
- net USB_1_OTG_DM renamed USB_2_OTG_DN
- net USB_2_OTG_DN: now also U54.5, J23.A7 (D-), J23.B7 (D-); no longer U41.2
- net USB_2_OTG_DM renamed USB_1_OTG_DN
- net USB_1_OTG_DN: now also U41.5, J26.A7 (D-), J26.B7 (D-); no longer U54.2
- net VBUS_A renamed USB1_VBUS
- net USB1_VBUS: now also C619.1, D2.1 (A1), J26.A4 (VBUS), J26.A9 (VBUS), J26.B4 (VBUS), J26.B9 (VBUS); no longer C584.1, Q2.1, Q2.2, Q2.3, U38.13 (VBUS1)
- new net USB2_VBUS: C584.1, C620.1, C723.1, D12.1 (A1), J23.A4 (VBUS), J23.A9 (VBUS), J23.B4 (VBUS), J23.B9 (VBUS), Q2.1, Q2.2, Q2.3, U38.13 (VBUS1)
Other:
- moved on the sheet: C449, C499, C500, C503, C504, C508, C509, C510, C511, C512, C513, C521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
