File: hardware/motherboard/barebones_mems.kicad_sch (KiCad schematic)
At the start: 26 parts, among them U32 K4UCE3Q4AA-MGCL, U33 K4UCE3Q4AA-MGCL

Commit message: arranged the schematics in every sheet
Other:
- note added: "LPDDR4x MEMORY"
- moved on the sheet: C374, C375, C376, C377, C378, C379, C380, C381, C382, C383, C384, C385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

Commit message: updated last changes
Parts:
- removed C374, C378: 4.7uF, Capacitor_SMD:C_0201_0603Metric, symbol Device:C
- removed C375, C376, C377, C379, C380, C381, C386, C387, C392, C393: 100nF, Capacitor_SMD:C_0201_0603Metric, symbol Device:C
- removed C382, C388: 22uF, Capacitor_SMD:C_0201_0603Metric, symbol Device:C
- removed C383, C384, C389, C390: 10uF, Capacitor_SMD:C_0201_0603Metric, symbol Device:C
- removed C385, C391: 1uF, Capacitor_SMD:C_0201_0603Metric, symbol Device:C
- removed R122, R123, R124, R125: 200R, Resistor_SMD:R_0402_1005Metric, symbol Device:R
- added C417, C645, C660, C661: 22uF, Capacitor_SMD:C_0603_1608Metric, symbol Device:C
- added C421, C540, C646, C647, C663, C664, C666, C667: 10uF, Capacitor_SMD:C_0402_1005Metric, symbol Device:C
- added C581, C638, C639, C640, C641, C642, C643, C644, C648, C649, C650, C651, C652, C653, C654, C655, C657, C658, C662, C665, C668, C669, C670, C671, C672, C673, C674, C675, C676, C677, C678, C679, C680, C681, C682, C683: 0.1uF, Capacitor_SMD:C_0201_0603Metric, symbol Device:C
- added C656, C659: 4.7uF, Capacitor_SMD:C_0402_1005Metric, symbol Device:C
- added R133, R135, R138, R140: 240R, Resistor_SMD:R_0201_0603Metric, symbol Device:R
Connections:
- net GND: now also C417.2, C421.2, C540.2, C581.2, C638.2, C639.2, C640.2, C641.2, C642.2, C643.2, C644.2, C645.2, C646.2, C647.2, C648.2, C649.2, C650.2, C651.2, C652.2, C653.2, C654.2, C655.2, C656.2, C657.2, C658.2, C659.2, C660.2, C661.2, C662.2, C663.2, C664.2, C665.2, C666.2, C667.2, C668.2, C669.2, C670.2, C671.2, C672.2, C673.2, C674.2, C675.2, C676.2, C677.2, C678.2, C679.2, C680.2, C681.2, C682.2, C683.2
- net VCC_1V8_S3: now also C656.1, C657.1, C658.1, C659.1, C662.1, C665.1
- net VDDQ_DDR_S0: now also C645.1, C646.1, C647.1, C648.1, C649.1, C650.1, C651.1, C652.1, C653.1, C654.1, C655.1, C661.1, C664.1, C667.1, C669.1, C671.1, C673.1, C675.1, C677.1, C679.1, C681.1, C683.1, R133.2, R135.1, R138.2, R140.1
- net at U32.A8 (ZQ1): now also R140.2
- net at U32.A5 (ZQ0): now also R138.1
- net at U33.A8 (ZQ1): now also R135.2
- net at U33.A5 (ZQ0): now also R133.1
- net VDD_DDR_S0 renamed VDD2_DDR_S3
- net VDD2_DDR_S3: now also C417.1, C421.1, C540.1, C581.1, C638.1, C639.1, C640.1, C641.1, C642.1, C643.1, C644.1, C660.1, C663.1, C666.1, C668.1, C670.1, C672.1, C674.1, C676.1, C678.1, C680.1, C682.1
Other:
- moved on the sheet: U32, U33

Commit message: started routing on LPDDR4x RAM
Parts:
- removed C540: 10uF, Capacitor_SMD:C_0402_1005Metric, symbol Device:C
- removed C672, C674, C676, C678, C679, C680, C681, C682, C683: 0.1uF, Capacitor_SMD:C_0201_0603Metric, symbol Device:C
- added C480, C483, C484, C487, C490, C494, C496: 10uF, Capacitor_SMD:C_0603_1608Metric, symbol Device:C
- added C481, C485, C493: 22uF, Capacitor_SMD:C_0805_2012Metric, symbol Device:C
- added C727, C728, C729, C730: 0.1uF, Capacitor_SMD:C_0201_0603Metric, symbol Device:C
- C417: footprint Capacitor_SMD:C_0603_1608Metric -> Capacitor_SMD:C_0805_2012Metric
- C421: footprint Capacitor_SMD:C_0402_1005Metric -> Capacitor_SMD:C_0603_1608Metric
- C645, C660, C661: value 22uF -> 0.1uF; footprint Capacitor_SMD:C_0603_1608Metric -> Capacitor_SMD:C_0201_0603Metric
- C646, C647, C663, C664, C666, C667: value 10uF -> 0.1uF; footprint Capacitor_SMD:C_0402_1005Metric -> Capacitor_SMD:C_0201_0603Metric
Connections:
- net GND: now also C480.2, C481.2, C483.2, C484.2, C485.2, C487.2, C490.2, C493.2, C494.2, C496.2, C727.2, C728.2, C729.2, C730.2
- net VCC_1V8_S3: now also C727.1, C728.1, C729.1, C730.1
- net VDD2_DDR_S3: now also C645.1, C646.1, C647.1, C480.1, C493.1, C494.1, C496.1
- net VDDQ_DDR_S0: now also C481.1, C483.1, C484.1, C485.1, C487.1, C490.1; no longer C645.1, C646.1, C647.1
- net DDR_CH1_CKB_C renamed DDR_CH1_CK_C_N
- net DDR_CH1_CKB_D renamed DDR_CH1_CK_D_N
- net DDR_CH1_CK_C renamed DDR_CH1_CK_C_P
- net DDR_CH1_CK_D renamed DDR_CH1_CK_D_P
- net DDR_CH1_DQS0N_C renamed DDR_CH1_DQS0_C_N
- net DDR_CH1_DQS0N_D renamed DDR_CH1_DQS0_D_N
- net DDR_CH1_DQS0P_C renamed DDR_CH1_DQS0_C_P
- net DDR_CH1_DQS0P_D renamed DDR_CH1_DQS0_D_P
- net DDR_CH1_DQS1N_C renamed DDR_CH1_DQS1_C_N
- net DDR_CH1_DQS1N_D renamed DDR_CH1_DQS1_D_N
- net DDR_CH1_DQS1P_C renamed DDR_CH1_DQS1_C_P
- net DDR_CH1_DQS1P_D renamed DDR_CH1_DQS1_D_P
Other:
- moved on the sheet: R133, R135, U33
