File: hardware/motherboard/barebones_power.kicad_sch (KiCad schematic)
At the start: 370 parts, among them J21 SM02B-GHS-TB_LF__SN_, J23 874381343, Q1 STL40DN3LLH5, Q2 STL40DN3LLH5, Q3 AO3401A, Q5 CSD18504Q5A, Q6 CSD18504Q5A, U10 TPS259474ARPWR, U11 IHLP1616ABERR47M01, U12 RK806-1_C5156483, U13 IHLP1616ABERR47M01, U14 BQ25731RSNR, U15 BQ78350DBTR-R1, U16 BQ7692000PW, U17 BQ28Z610DRZR, U18 RK860-2, U19 RK860-2, U2 IHLP1616ABERR47M01, U20 TPS54628DDAR, U21 TPS62933DRLR, U22 RK860-3, U23 TPS62933DRLR, U24 TPS54628DDAR, U25 TPS54628DDAR, U26 TPS61170DRVR, U27 LM3940IMPX-3.3_NOPB, U28 TPS61160ADRVT, U29 TPS54628DDAR, U3 IHLP1616ABERR47M01, U4 TPS259474ARPWR, U5 IHLP1616ABERR47M01, U6 IHLP1616ABERR47M01, U7 LP5912-1.8DRVT, U73 BQ40Z50RSMR-R2, U74 TPD4E004DRYR, U77 NXFT15XH103FA2B025, U78 NXFT15XH103FA2B025, U79 NXFT15XH103FA2B025, U8 TPS2121RUXR, U80 NXFT15XH103FA2B025, U9 1N5819WT

Commit message: pushed many changes and added dedicated bms module
Parts:
- removed C561, C562, C563, C564, C565, C567, C568: 0.1uF, Capacitor_SMD:C_0402_1005Metric, symbol Device:C
- removed C566: 2.2uF, Capacitor_SMD:C_0402_1005Metric, symbol Device:C
- removed D21: 1N4148W, Diode_SMD:D_SOD-123, symbol Diode:1N4148W
- removed PAD0: NEUTRAL, barebones:7x10-PAD, symbol Connector:TestPoint
- removed PAD1: BATT_1P, barebones:7x10-PAD, symbol Connector:TestPoint
- removed PAD2: BATT_2P, barebones:7x10-PAD, symbol Connector:TestPoint
- removed PAD3: BATT_3P, barebones:7x10-PAD, symbol Connector:TestPoint
- removed PAD4: BATT_4P, barebones:7x10-PAD, symbol Connector:TestPoint
- removed PAD5: BATT_4N, barebones:7x10-PAD, symbol Connector:TestPoint
- removed PAD6: BATT_3N, barebones:7x10-PAD, symbol Connector:TestPoint
- removed PAD7: BATT_2N, barebones:7x10-PAD, symbol Connector:TestPoint
- removed Q3: AO3401A, Package_TO_SOT_SMD:SOT-23, symbol Transistor_FET:AO3401A
- removed R225, R93, R94: 5.1k, Resistor_SMD:R_0402_1005Metric, symbol Device:R
- removed R226: 100R, Resistor_SMD:R_0402_1005Metric, symbol Device:R
- removed R236, R237, R238, R239, R241, R243, R245, R246, R247: 100, Resistor_SMD:R_0402_1005Metric, symbol Device:R
- removed R240: 300, Resistor_SMD:R_0402_1005Metric, symbol Device:R
- removed R242, R244, R248: 10M, Resistor_SMD:R_0402_1005Metric, symbol Device:R
- removed R78, R79: 4.7k, Resistor_SMD:R_0402_1005Metric, symbol Device:R
- removed TP11: SMBD, TestPoint:TestPoint_Pad_D1.0mm, symbol Connector:TestPoint
- removed TP12: SMBC, TestPoint:TestPoint_Pad_D1.0mm, symbol Connector:TestPoint
- removed TP13: GND, TestPoint:TestPoint_Pad_D1.0mm, symbol Connector:TestPoint
- removed U74: TPD4E004DRYR, barebones:PSON50P145X100X60-6N, symbol TPD4E004DRYR:TPD4E004DRYR
- removed U77, U79, U80: NXFT15XH103FA2B025, barebones:NXFT15XH103FA2B025, symbol NXFT15XH103FA2B025:NXFT15XH103FA2B025
Connections:
- net GUAGE is gone; now on net PACK_P: C273.1, C275.2, C276.2, R68.2, R74.1
- net GND: no longer R59.1, U73.14 (NC), U73.17 (~{DISP}), U73.23 (PTC), U73.24 (PTCEN), U73.29 (NC), U73.33 (EXP), U73.33_1 (EXP), U73.7 (NC), U73.9 (VSS), U78.P$1
- net PACK_N: no longer R59.2
- net PACK_P: no longer Q6.1, Q6.2, Q6.3, U73.27 (PACK)
- net BAT: no longer names the net of U73.32 (BAT)
- removed net BATT_4P: Q5.1, Q5.2, Q5.3
- net CHG: no longer names the net of U73.31 (CHG)
- net DSG: no longer names the net of U73.28 (DSG)
- net PCHG: no longer names the net of U73.30 (PCHG)
- net SRN_BATT: no longer names the net of U73.6 (SRN)
- net SRP_BATT: no longer names the net of U73.8 (SRP)
- net TS1: no longer names the net of U73.10 (TS1)
- net TS1: no longer U78.P$2
- net TS2: no longer names the net of U73.11 (TS2)
- net TS3: no longer names the net of U73.12 (TS3)
- net TS4: no longer names the net of U73.13 (TS4)
- net VC1: no longer names the net of U73.5 (VC1)
- net VC2: no longer names the net of U73.4 (VC2)
- net VC3: no longer names the net of U73.3 (VC3)
- net VC4: no longer names the net of U73.2 (VC4)
- net VCC: no longer names the net of U73.26 (VCC)
- new net: U73.14 (NC), U73.29 (NC), U73.7 (NC)
- new net: U73.33 (EXP), U73.33_1 (EXP)
- now unconnected: Q5.5, Q5.6, Q5.7, Q5.8, Q6.5, Q6.6, Q6.7, Q6.8
- no-connect marks 19 -> 13
Other:
- note added: "BMS CONNECTOR"
- note added: "LOOK FOR FEMALE VERSION OF THIS"
- moved on the sheet: J23

Commit message: arranged the schematics in every sheet
Parts:
- removed C165, C166, C184, C189, C190, C339, C349, C368: 1uF, Capacitor_SMD:C_0402_1005Metric, symbol Device:C
- removed C180, C196: 4.7nF, Capacitor_SMD:C_0402_1005Metric, symbol Device:C
- removed C181, C198, C331, C345, C364: 10nF, Capacitor_SMD:C_0402_1005Metric, symbol Device:C
- removed C185, C195, C302, C328, C334, C343, C344, C348, C352, C363, C367, C371: 0.1uF, Capacitor_SMD:C_0402_1005Metric, symbol Device:C
- removed C303, C309, C330, C338: 100nF, Capacitor_SMD:C_0402_1005Metric, symbol Device:C
- removed C308, C329, C335, C336, C337: 10uF, Capacitor_SMD:C_0402_1005Metric, symbol Device:C
- removed C332, C333, C341, C342, C346, C347, C350, C351, C365, C366, C369, C370: 47uF, Capacitor_SMD:C_0402_1005Metric, symbol Device:C
- removed C340: 33nF, Capacitor_SMD:C_0402_1005Metric, symbol Device:C
- removed L11, L12, L13, L16, L9: XAL7030-472MEB, XAL7030-472MEB:IND_XAL7030-472MEB, symbol XAL7030-472MEB:XAL7030-472MEB
- removed Q1: STL40DN3LLH5, barebones:TRANS_STL40DN3LLH5, symbol STL40DN3LLH5:STL40DN3LLH5
- removed unit 1 of Q2
- removed Q5, Q6: CSD18504Q5A, barebones:MOSFET_CSD19531Q5A, symbol CSD18504Q5A:CSD18504Q5A
- removed R100, R104, R107, R109, R111, R117, R36, R39, R40, R43, R45, R47, R48: 10k, Resistor_SMD:R_0402_1005Metric, symbol Device:R
- removed R101, R108: 31.3k, Resistor_SMD:R_0402_1005Metric, symbol Device:R
- removed R106, R110, R99: 56k, Resistor_SMD:R_0402_1005Metric, symbol Device:R
- removed R116: 33.2k, Resistor_SMD:R_0402_1005Metric, symbol Device:R
- removed R35, R42: 27.4k, Resistor_SMD:R_0402_1005Metric, symbol Device:R
- removed R38, R46: 174k, Resistor_SMD:R_0402_1005Metric, symbol Device:R
- removed U23: TPS62933DRLR, barebones:SOTFL50P160X60-8N, symbol TPS62933DRLR:TPS62933DRLR
- removed U24, U25, U29: TPS54628DDAR, barebones:VREG_LM5017MR_NOPB, symbol TPS54628DDAR:TPS54628DDAR
- added C242, C251, C264, C280, C473, C478, C485, C487, C498, C505, C526, C527: 10uF, Capacitor_SMD:C_0402_1005Metric, symbol Device:C
- added C281: 22pF, Capacitor_SMD:C_0402_1005Metric, symbol Device:C
- added C282, C283, C290, C291: 10pF, Capacitor_SMD:C_0402_1005Metric, symbol Device:C
- added C475, C477, C483, C484, C494, C496, C515, C517, C603, C604: 22uF, Capacitor_SMD:C_0402_1005Metric, symbol Device:C
- added C480, C490, C506, C530: 0.1uF, Capacitor_SMD:C_0402_1005Metric, symbol Device:C
- added C481, C493, C514, C589: 1uF, Capacitor_SMD:C_0402_1005Metric, symbol Device:C
- added L17, L18, L19, L20: XAL7030-472MEB, XAL7030-472MEB:IND_XAL7030-472MEB, symbol XAL7030-472MEB:XAL7030-472MEB
- added Q11, Q12, Q13, Q14: CSD18543Q3A, barebones:TRANS_CSD18543Q3A, symbol Transistor_FET:CSD18543Q3A
- added R126, R128, R130, R135, R140, R148, R165, R168: 10k, Resistor_SMD:R_0402_1005Metric, symbol Device:R
- added R127, R129, R138: 56k, Resistor_SMD:R_0402_1005Metric, symbol Device:R
- added R155, R166: 100k, Resistor_SMD:R_0402_1005Metric, symbol Device:R
- added R164, R167: 30k, Resistor_SMD:R_0402_1005Metric, symbol Device:R
- added U45, U53, U62, U63: TPS54628DDAR, barebones:VREG_LM5017MR_NOPB, symbol TPS54628DDAR:TPS54628DDAR
- C304: value 10nF -> 8200pF
- C305: value 47uF -> 8200pF
- C306: value 47uF -> 0.1uF
- C310, C312: value 10uF -> 8200pF
- C311: value 10uF -> 0.1uF
- C313, C327: value 100nF -> 0.1uF
- C321: value 33nF -> 8200pF
- C322, C323: value 47uF -> 10uF
Connections:
- net BUCK_PWRON: now also R126.1; no longer U20.1 (EN)
- net GND: now also C305.2, C310.2, C312.2, C321.2, C242.1, C251.1, C264.1, C280.1, C473.1, C475.1, C477.1, C478.1, C480.1, C481.1, C483.1, C484.1, C485.1, C487.1, C490.1, C493.1, C494.1, C496.1, C498.1, C505.1, C506.1, C514.1, C515.1, C517.1, C526.1, C527.1, C530.1, C589.1, C603.1, C604.1, Q12.1 (S), Q12.2 (S), Q12.3 (S), Q14.5 (D), R128.1, R130.1, R140.1, R164.1, R167.1, U45.5 (GND), U53.5 (GND), U62.5 (GND), U63.5 (GND); no longer C305.1, C306.1, C307.1, C310.1, C311.1, C312.1, C313.1, C321.1, U10.8 (GND), U21.4 (GND), U4.8 (GND), U8.12 (GND), U8.3 (CP2), U8.4 (OV2), U8.5 (OV1), U8.6 (PR1)
- net HIDRV1: now also Q11.4 (G)
- net HIDRV2: now also Q13.4 (G); no longer Q2.2
- net LODRV1: now also Q12.4 (G)
- net LODRV2: now also Q14.4 (G)
- net PCIE30X4_PWREN_H: now also R165.1, R168.1; no longer U21.2 (EN)
- net PMIC_EXT_EN: now also R135.1, R148.1
- net VCC3V3_PCIE30: now also C290.1, C515.2, C517.2, L19.2, R155.1; no longer C310.2, C311.2, C312.2, C313.2
- net VCC_3V3_SYS: now also C291.1, C603.2, C604.2, L20.2, R166.1
- net VCC_4V0_SYS: now also C281.1, C475.2, C477.2, R127.1; no longer C305.2, C306.2, C307.2
- net VCC_5V0_ALW: now also C283.1, C494.2, C496.2, L18.2, R138.1
- net VCC_5V0_PERIPH: now also C282.1, C483.2, C484.2, L17.2, R129.1; no longer U21.3 (VIN)
- net VIN_CHRG_1: now also Q11.5 (D)
- net VIN_CHRG_2: now also Q11.1 (S), Q11.2 (S), Q11.3 (S), Q12.5 (D)
- net VIN_CHRG_3: now also Q13.1 (S), Q13.2 (S), Q13.3 (S), Q14.1 (S), Q14.2 (S), Q14.3 (S); no longer Q2.1
- net at U8.2 (IN2), U8.2_1 (IN2): no longer U10.6 (OUT)
- net at U21.7 (SS): no longer C321.2
- net at U20.2 (VFB): now also C281.2, R127.2, R128.2
- net at C327.2: now also L20.1, U63.6 (SW)
- net at L8.1, U20.6 (SW): now also C307.2
- net at U20.7 (VBST): now also C307.1
- net at C327.1: now also U63.7 (VBST)
- net at U8.7 (IN1), U8.7_1 (IN1): no longer U4.6 (OUT)
- net PP_HV1_1: no longer names the net of U4.5 (IN)
- net PP_HV1_2: no longer names the net of U10.5 (IN)
- net PP_HV_MAIN renamed SYS_PWR
- net SYS_PWR: now also C242.2, C251.2, C264.2, C280.2; no longer U8.1 (OUT), U8.1_1 (OUT), U8.8 (OUT), U8.8_1 (OUT)
- net PWM_VIN renamed VIN_CHRG_4
- net VIN_CHRG_4: now also C254.1, C255.1, C256.1, C257.1, C258.1, C259.1, C260.1, C261.1, C262.1, C268.1, C269.1, C273.2, C274.1, C322.2, C323.2, C324.2, C356.2, C357.2, R68.1, R73.1, U14.22 (VSYS), U20.8 (VIN), U26.6 (VIN), C473.2, C478.2, C480.2, C485.2, C487.2, C490.2, C498.2, C505.2, C506.2, C526.2, C527.2, C530.2, Q13.5 (D), U45.8 (VIN), U53.8 (VIN), U62.8 (VIN), U63.8 (VIN)
- net USB_SIG_STAT: no longer names the net of U8.9 (ST)
- removed net VSYS_MAIN: C254.1, C255.1, C256.1, C257.1, C258.1, C259.1, C260.1, C261.1, C262.1, C268.1, C269.1, C273.2, C274.1, C322.2, C323.2, C324.2, C356.2, C357.2, Q2.7-8, R68.1, R73.1, U14.22 (VSYS), U20.8 (VIN), U26.5 (CTRL), U26.6 (VIN)
- new net: R168.2, U63.1 (EN)
- new net: C291.2, R166.2, R167.2, U63.2 (VFB)
- new net: C589.2, U63.3 (VREG5)
- new net: C321.1, U63.4 (SS)
- new net: C283.2, R138.2, R140.2, U53.2 (VFB)
- new net: C282.2, R129.2, R130.2, U45.2 (VFB)
- new net: R135.2, U45.1 (EN)
- new net: C481.2, U45.3 (VREG5)
- new net: C305.1, U45.4 (SS)
- new net: C306.2, L17.1, U45.6 (SW)
- new net: C306.1, U45.7 (VBST)
- new net: C311.1, U53.7 (VBST)
- new net: C311.2, L18.1, U53.6 (SW)
- new net: R126.2, U20.1 (EN)
- new net: R165.2, U62.1 (EN)
- new net: C290.2, R155.2, R164.2, U62.2 (VFB)
- new net: C514.2, U62.3 (VREG5)
- new net: C312.1, U62.4 (SS)
- new net: C313.2, L19.1, U62.6 (SW)
- new net: C313.1, U62.7 (VBST)
- new net: R148.2, U53.1 (EN)
- new net: C493.2, U53.3 (VREG5)
- new net: C310.1, U53.4 (SS)
- new net: U8.1 (OUT), U8.1_1 (OUT), U8.8 (OUT), U8.8_1 (OUT)
- new net EDP_PWM11_M1: U26.5 (CTRL)
- no-connect marks 13 -> 7
Other:
- note added: "25V X5R capacitors"
- note added: "BUCK/BOOST CONVERTERS & LDOs"
- note added: "CONFIRM THIS MOSFET CONNECTIONS"
- note added: "DEDICATED PMICs"
- note added: "USE 10uH INDUCTOR"
- note added: "USE 22uH INDUCTOR"
- note added: "USE 4.7uH INDUCTOR"
- note removed: "3V3 BUCK CONVERTER"
- note removed: "3V3 LDO FOR EC"
- note removed: "4V BUCK CONVERTER"
- note removed: "5V BUCK CONVERTER"
- note removed: "5V BUCK CONVERTER FOR EC"
- note removed: "CPU_BIG0_VSEL"
- note removed: "CURRENT LIMITER"
- note removed: "POWER MUX"
- moved on the sheet: C167, C168, C169, C170, C171, C172, C173, C174, C175, C176, C177, C178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

Commit message: removed unused components and connections
Parts:
- removed C319, C320, C325, C326: 22uF, Capacitor_SMD:C_0402_1005Metric, symbol Device:C
- removed D2: MMSZ5V6T1G, barebones:MMSZ5V6T1G, symbol MMSZ5V6T1G:MMSZ5V6T1G
- removed Q2: STL40DN3LLH5, barebones:TRANS_STL40DN3LLH5, symbol STL40DN3LLH5:STL40DN3LLH5
- removed R105, R98: 100R, Resistor_SMD:R_0402_1005Metric, symbol Device:R
- removed R59: WSL25122L000FEA, barebones:RES_WSL25122L000FEA, symbol WSL25122L000FEA:WSL25122L000FEA
- removed U10, U4: TPS259474ARPWR, barebones:IC_TPS259474ARPWR, symbol TPS259474ARPWR:TPS259474ARPWR
- removed U15: BQ78350DBTR-R1, barebones:SOP50P640X120-30N, symbol BQ78350DBTR-R1:BQ78350DBTR-R1
- removed U16: BQ7692000PW, barebones:SOP65P640X120-20N, symbol BQ7692000PW:BQ7692000PW
- removed U17: BQ28Z610DRZR, barebones:IC_BQ27441DRZR-G1A, symbol BQ28Z610DRZR:BQ28Z610DRZR
- removed U21: TPS62933DRLR, barebones:SOTFL50P160X60-8N, symbol TPS62933DRLR:TPS62933DRLR
- removed U7: LP5912-1.8DRVT, barebones:SON65P200X200X80-7N, symbol LP5912-1.8DRVT:LP5912-1.8DRVT
- removed U73: BQ40Z50RSMR-R2, barebones:QFN40P400X400X100-33N, symbol BQ40Z50RSMR-R2:BQ40Z50RSMR-R2
- removed U78: NXFT15XH103FA2B025, barebones:NXFT15XH103FA2B025, symbol NXFT15XH103FA2B025:NXFT15XH103FA2B025
- removed U8: TPS2121RUXR, barebones:IC_TPS2121RUXR, symbol TPS2121RUXR:TPS2121RUXR
- added C302: 1uF, Capacitor_SMD:C_0402_1005Metric, symbol Device:C
- added C303, C308, C309: 22uF, Capacitor_SMD:C_0402_1005Metric, symbol Device:C
- added R93, R94: 100R, Resistor_SMD:R_0402_1005Metric, symbol Device:R
- C315: value 1uF -> 22uF
Connections:
- net GND: now also C315.2, C303.2, C308.2, C309.2
- net VCC_4V0_SYS: now also C317.1, C318.1
- net VDD_CPU_BIG0_S0: now also R93.1, R93.2
- net VDD_CPU_BIG1_S0: now also C302.1, C302.2, C303.1, C308.1, C309.1, R94.1, R94.2; no longer C315.2, C317.1, C318.1
Other:
- moved on the sheet: C220, C221, C222, C223, C224, C225, C226, C227, C228, C231, C232, C235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

Commit message: updated last changes
Parts:
- removed C220, C481, C493, C514: 1uF, Capacitor_SMD:C_0402_1005Metric, symbol Device:C
- removed C221, C222, C223, C224, C225, C226, C306, C307, C311, C313, C324, C327, C480, C490, C506, C540: 0.1uF, Capacitor_SMD:C_0402_1005Metric, symbol Device:C
- removed C259, C260, C261, C262, C264, C280, C473, C478, C485, C487, C498, C505: 10uF, Capacitor_SMD:C_0402_1005Metric, symbol Device:C
- removed C268, C269: 33uF, Capacitor_SMD:C_0402_1005Metric, symbol Device:C
- removed C281: 22pF, Capacitor_SMD:C_0402_1005Metric, symbol Device:C
- removed C282, C283, C290, C291: 10pF, Capacitor_SMD:C_0402_1005Metric, symbol Device:C
- removed C295, C475, C477, C483, C484, C494, C496, C515, C517: 22uF, Capacitor_SMD:C_0402_1005Metric, symbol Device:C
- removed C304, C305, C310, C312: 8200pF, Capacitor_SMD:C_0402_1005Metric, symbol Device:C
- removed J21: SM02B-GHS-TB_LF__SN_, barebones:JST_SM02B-GHS-TB_LF__SN_, symbol SM02B-GHS-TB_LF__SN_:SM02B-GHS-TB_LF__SN_
- removed J23: 874381343, barebones:MOLEX_874381343, symbol 874381343:874381343
- removed L1, L10, L2, L3, L5, L6, L7: 0.22uH, Inductor_SMD:L_0805_2012Metric, symbol Device:L
- removed L18, L19, L20, L4, L8: XAL7030-472MEB, XAL7030-472MEB:IND_XAL7030-472MEB, symbol XAL7030-472MEB:XAL7030-472MEB
- removed R102, R103, R88, R89, R96, R97: 2.2k, Resistor_SMD:R_0402_1005Metric, symbol Device:R
- removed R126, R128, R130, R135, R140, R148, R63: 10k, Resistor_SMD:R_0402_1005Metric, symbol Device:R
- removed R127, R129, R138: 56k, Resistor_SMD:R_0402_1005Metric, symbol Device:R
- removed R155: 100k, Resistor_SMD:R_0402_1005Metric, symbol Device:R
- removed R164: 30k, Resistor_SMD:R_0402_1005Metric, symbol Device:R
- removed R80, R81: 4.7k, Resistor_SMD:R_0402_1005Metric, symbol Device:R
- removed U11, U13, U2, U3, U5, U6: IHLP1616ABERR47M01, IHLP1616ABERR47M01:IHLP-ER2, symbol IHLP1616ABERR47M01:IHLP1616ABERR47M01
- removed U20, U45, U62, U63: TPS54628DDAR, barebones:VREG_LM5017MR_NOPB, symbol TPS54628DDAR:TPS54628DDAR
- removed U27: LM3940IMPX-3.3_NOPB, LM3940IMPX-3.3_NOPB:SOT230P700X180-4N, symbol LM3940IMPX-3.3_NOPB:LM3940IMPX-3.3_NOPB
- added BT1: BK-912-G, barebones:BAT_BK-912-G, symbol BK-912-G:BK-912-G
- added C189, C195, C319, C320, C576, C687, C688, C695, C696: 22uF, Capacitor_SMD:C_0402_1005Metric, symbol Device:C
- added C325, C326, C328, C329, C330, C331, C332: 10uF, Capacitor_SMD:C_0603_1608Metric, symbol Device:C
- added C334, C335: 33uF, Capacitor_SMD:C_0603_1608Metric, symbol Device:C
- added C341, C342, C350, C351, C684, C691, C692, C699, C700: 10uF, Capacitor_SMD:C_0402_1005Metric, symbol Device:C
- added C343, C345, C352, C575, C685, C690, C693, C701: 0.1uF, Capacitor_SMD:C_0402_1005Metric, symbol Device:C
- added C344: 47nF, Capacitor_SMD:C_0201_0603Metric, symbol Device:C
- added C346: 150pF, Capacitor_SMD:C_0402_1005Metric, symbol Device:C
- added C347, C348, C349, C366, C367, C368: 22uF, Capacitor_SMD:C_0603_1608Metric, symbol Device:C
- added C365: 150pF, Capacitor_SMD:C_0201_0603Metric, symbol Device:C
- added C591, C686, C694, C702: 33nF, Capacitor_SMD:C_0201_0603Metric, symbol Device:C
- added C703, C704: 47uF, Capacitor_SMD:C_0402_1005Metric, symbol Device:C
- added J17: 2200981671, barebones:CONN_2200980000-SD_16_MOL, symbol 2200981671:2200981671
- added L1, L2, L4, L6: FDSD0420-H-2R2M=P3, barebones:IND_FDSD0420-H-2R2M=P3, symbol FDSD0420-H-2R2M_P3:FDSD0420-H-2R2M=P3
- added L10, L12, L13, L16, L18, L19, L9: DFE252010F-R22M=P2, barebones:IND-SMD_L2.5-W2.0_MHCD252012B-2R2M-A8L, symbol DFE252010F-R22M=P2:DFE252010F-R22M=P2
- added L11, L21, L22, L23, L24, L25: DFE201610E-R47M=P2, barebones:INDC2016X100N, symbol DFE201610E-R47M_P2:DFE201610E-R47M=P2
- added L20, L3: DFEG7030D-4R7M=P3, barebones:IND_DFEG7030D-4R7M=P3, symbol DFEG7030D-4R7M_P3:DFEG7030D-4R7M=P3
- added L26, L7: XAL6030-332MEC, barebones:IND_XAL6030-332MEC, symbol XAL6030-332MEC:XAL6030-332MEC
- added R169, R188, R216, R239, R251: 10k, Resistor_SMD:R_0402_1005Metric, symbol Device:R
- added R172, R252: 31.3k, Resistor_SMD:R_0402_1005Metric, symbol Device:R
- added R187, R242, R64: 100k, Resistor_SMD:R_0402_1005Metric, symbol Device:R
- added R189, R217, R225, R228: 10k, Resistor_SMD:R_0201_0603Metric, symbol Device:R
- added R190: 30.1k, Resistor_SMD:R_0201_0603Metric, symbol Device:R
- added R191, R240: 49.9k, Resistor_SMD:R_0402_1005Metric, symbol Device:R
- added R203: 57.6k, Resistor_SMD:R_0402_1005Metric, symbol Device:R
- added R218: 3.74k, Resistor_SMD:R_0402_1005Metric, symbol Device:R
- added R227: 30.1k, Resistor_SMD:R_0402_1005Metric, symbol Device:R
- added R241: 73.2k, Resistor_SMD:R_0402_1005Metric, symbol Device:R
- added R45: 0R, Capacitor_SMD:C_0201_0603Metric, symbol Device:R
- added U10, U6, U7, U8: TPS62933DRLR, barebones:SOTFL50P160X60-8N, symbol TPS62933DRLR:TPS62933DRLR
- added U3: TLV75533PDBVR, barebones:SOT95P280X145-5N, symbol TLV75533PDBVR:TLV75533PDBVR
- added U4, U5: TPS56837RPAR, barebones:CONV_TPS56837RPAR, symbol TPS56837RPAR:TPS56837RPAR
- added VR1: TPS7A7002DDAR, barebones:VREG_TPS7A7002DDAR, symbol TPS7A7002DDAR:TPS7A7002DDAR
- C176, C204, C240, C241, C354, C355, C357, C362, C556, C557, C558, C559: footprint Capacitor_SMD:C_0402_1005Metric -> Capacitor_SMD:C_0201_0603Metric
- C227, C228, C237, C238: footprint Capacitor_SMD:C_0402_1005Metric -> Capacitor_SMD:C_0603_1608Metric
- C242: value 10uF -> 1uF; footprint Capacitor_SMD:C_0402_1005Metric -> Capacitor_SMD:C_0603_1608Metric
- C251, C254, C255, C256, C257, C258: value 10uF -> 0.1uF; footprint Capacitor_SMD:C_0402_1005Metric -> Capacitor_SMD:C_0603_1608Metric
- C285, C289: value 22uF -> 47uF
- C314: value 1uF -> 0.1uF
- C321: value 8200pF -> 0.1uF
- C322, C323, C526: value 10uF -> 0.1uF
- C358: value 33uF -> 0.1uF
- C359: value 0.47uF -> 47nF; footprint Capacitor_SMD:C_0402_1005Metric -> Capacitor_SMD:C_0201_0603Metric
- C530: value 0.1uF -> 10uF
- C589: value 1uF -> 22uF
- C603: value 22uF -> 0.1uF
- C604: value 22uF -> 10uF
- D3, D4: footprint B0530W-7-F:SOD3715X145N -> barebones:SOD3715X145N
- L14: footprint LQH5BPN100MT0L:IND_LQH5BPN100MT0L -> barebones:IND_LQH5BPN100MT0L
- L15: footprint LQH32PH220MNCL:IND_LQH32PH220MNCL -> barebones:IND_LQH32PH220MNCL
- L17: footprint XAL7030-472MEB:IND_XAL7030-472MEB -> barebones:IND_XAL7030-472MEB
- R114, R115, R55, R57, R66, R67, R72, R75, R76, R82: footprint Resistor_SMD:R_0402_1005Metric -> Resistor_SMD:R_0201_0603Metric
- R165, R168, R58: value 10k -> 100k
- R166: value 100k -> 10k
- R167: value 30k -> 31.3k
- R65: value 10 -> 10R; footprint Resistor_SMD:R_0402_1005Metric -> Resistor_SMD:R_0201_0603Metric
- R73, R74: value 10 -> 10R
- U12: value RK806-1_C5156483 -> RK806-1
- U22: footprint easyeda2kicad:WLCSP-20_L2.0-W1.6-R5-C4-P0.40-TL -> barebones:WLCSP-20_L2.0-W1.6-R5-C4-P0.40-TL
- U26: footprint TPS61170DRVR:SON65P200X200X80-7N -> barebones:SON65P200X200X80-7N
- U28: footprint TPS61160ADRVT:SON65P200X200X80-7N -> barebones:SON65P200X200X80-7N
- U9: footprint easyeda2kicad:SOD-523_L1.2-W0.8-LS1.6-RD -> barebones:SOD-523_L1.2-W0.8-LS1.6-RD
Connections:
- net INT_PMIC is gone; now on net PMIC_INT_L: R61.2
- net SPI_CS_PMIC is gone; now on net SPI2_CS0_M2: R58.1
- net BATT_PRES: now also J17.7
- net BUCK_PWRON: now also R189.2, R225.2, U4.1 (EN), U5.1 (EN)
- net GND: now also C242.2, C251.2, Q14.1 (S), Q14.2 (S), Q14.3 (S), R166.1, BT1.1, C189.2, C195.2, C319.2, C320.2, C325.1, C326.1, C328.1, C329.1, C330.1, C331.1, C332.1, C334.1, C335.1, C341.1, C342.1, C343.1, C344.1, C347.1, C348.1, C349.1, C350.1, C351.1, C352.1, C366.1, C367.1, C368.1, C575.1, C576.1, C591.1, C684.1, C685.1, C686.1, C687.1, C688.1, C690.1, C691.1, C692.1, C693.1, C694.1, C695.1, C696.1, C699.1, C700.1, C701.1, C702.1, C703.1, C704.1, J17.12, J17.13, J17.14, J17.15, J17.16, R169.1, R188.1, R189.1, R190.1, R216.1, R225.1, R227.1, R239.1, R251.1, R64.2, U10.1 (RT), U10.4 (GND), U4.3 (AGND), U4.9 (PGND), U5.3 (AGND), U5.9 (PGND), U6.1 (RT), U6.4 (GND), U7.1 (RT), U7.4 (GND), U8.1 (RT), U8.4 (GND); no longer C242.1, C251.1, C314.1, C321.2, C322.1, C323.1, C358.1, Q14.5 (D), R167.1, U22.A1 (VSEL), U53.5 (GND)
- net PACK_P: now also J17.1, J17.2, J17.3, J17.4, J17.5
- net PMIC_EXT_EN: now also R187.1
- net SMBC_BATT: now also J17.9
- net SMBD_BATT: now also J17.8
- net SPI2_MOSI_M2: now also R64.1
- net SW0_LX: now also L18.1
- net SW1: now also L13.2
- net SW10: now also L24.2
- net SW1_LX: now also L19.1
- net SW2: now also L12.1
- net SW2_LX: now also L10.1
- net SW3: now also L9.1
- net SW4: now also L16.1
- net SW5: now also L11.1
- net SW6: now also L25.2
- net SW7: now also L21.1
- net SW8: now also L22.2
- net SW9: now also L23.2
- net SYS_PWR: now also C242.1, C251.1, C254.1, C255.1, C256.1, C257.1, C258.1; no longer C242.2, C251.2
- net VCC1V8_PMU_DDR_S3: now also C195.1, L24.1
- net VCC3V3_PCIE30: now also C589.2, R167.1, C576.2, L2.2
- net VCC_1V1_NLDO_S3: now also C695.2, C696.2, L4.2, R218.1
- net VCC_2V0_PLDO_S3: now also C189.1, L21.2
- net VCC_3V3_ALW: now also C703.2, C704.2, L6.2, R252.1; no longer C358.2
- net VCC_3V3_S3: now also R55.1, R82.1, C319.1, L22.1
- net VCC_4V0_SYS: now also C366.2, C367.2, C368.2, L7.2, R240.2; no longer C292.1, C293.1, C300.1, C301.1, C317.1, C318.1, U18.D1 (VIN), U18.D2 (VIN), U18.E1 (VIN), U18.E2 (VIN), U19.D1 (VIN), U19.D2 (VIN), U19.E1 (VIN), U19.E2 (VIN), U22.D1 (VIN), U22.D2 (VIN), U22.E1 (VIN), U22.E2 (VIN)
- net VDDQ_DDR_S0: now also L23.1, R45.1; no longer C204.2, U12.66 (FB9)
- net VDD_CPU_BIG0_S0: no longer C294.1, C296.1, C297.1, C298.1, C299.1, R93.2
- net VDD_CPU_BIG1_S0: no longer C302.1, C303.1, C308.1, C309.1, C315.1, C316.1, R94.2
- net VDD_CPU_LIT_S0: now also L12.2
- net VDD_DDR_S0: now also L11.2
- net VDD_GPU_S0: now also L13.1
- net VDD_LOG_S0: now also L9.2
- net VDD_NPU_S0: no longer C284.1, C285.1, C286.1, C287.1, C288.1, C289.1, R92.2
- net VDD_VDENC_S0: now also L16.2
- net VIN_CHRG_2: now also L20.1
- net VIN_CHRG_3: now also Q14.5 (D), L20.2; no longer Q14.1 (S), Q14.2 (S), Q14.3 (S)
- net V_BAT_CMOS: now also BT1.S1, BT1.S2
- net PCIE30X4_PWREN_H_EN_1: now reaches R168.2
- net PCIE30X4_PWREN_H_EN_1: now also C603.2, U7.2 (EN)
- net at R166.2, R167.2: now also U6.8 (FB)
- net at C321.1: now also U7.6 (BST)
- net PCIE30X4_PWREN_H_EN_2: now reaches R165.2
- net PCIE30X4_PWREN_H_EN_2: now also C526.2, U6.2 (EN)
- net at C314.2: now also L2.1, U6.5 (SW)
- net FB5: no longer names the net of U12.47 (FB5)
- net VCC2_DDR_S3 renamed VDD2_DDR_S3
- net VDD2_DDR_S3: now also L25.1
- removed net VCC_3V3_SYS: C603.2, C604.2, R166.1, R55.1, R82.1
- net VCC_5V0_ALW: no longer names the net of C359.2
- net VCC_5V0_ALW: now also U5.5 (SS)
- net VCC_5V0_PERIPH: no longer names the net of L17.2
- removed net VIN_CHRG_4: C254.1, C255.1, C256.1, C257.1, C258.1, C273.2, C274.1, C322.2, C323.2, C356.2, C357.2, C360.2, C526.2, C527.2, C530.2, L15.1, Q13.5 (D), R68.1, R73.1, U14.22 (VSYS), U26.6 (VIN), U28.6 (VIN), U53.8 (VIN)
- new net: R169.2, R172.2, U7.8 (FB)
- new net: C284.1, C285.1, C286.1, C287.1, C288.1, C289.1, L18.2, R92.2
- new net: C314.1, U6.6 (BST)
- new net: C591.2, U6.7 (SS)
- new net: R228.2, U5.4 (PG)
- new net: C345.1, U4.7 (BOOT)
- new net: C702.2, U10.7 (SS)
- new net: R190.2, U4.10 (MODE)
- new net: C344.2, U4.5 (SS)
- new net: C322.2, L4.1, U8.5 (SW)
- new net: C294.1, C296.1, C297.1, C298.1, C299.1, C316.1, L19.2, R93.2
- new net: C694.2, U8.7 (SS)
- new net: C302.1, C303.1, C308.1, C309.1, C315.1, C320.1, L10.2, R94.2
- new net: R188.2, R218.2, U8.8 (FB)
- new net: C321.2, L1.1, U7.5 (SW)
- new net: R227.2, U5.10 (MODE)
- new net: C690.2, R187.2, U8.2 (EN)
- new net: C346.1, R203.1, R216.2, U4.2 (FB)
- new net: C346.2, R191.1, R203.2
- new net: R251.2, R252.2, U10.8 (FB)
- new net: C323.1, U10.6 (BST)
- new net: C323.2, L6.1, U10.5 (SW)
- new net: R242.2, U10.2 (EN)
- new net: C686.2, U7.7 (SS)
- new net: C322.1, U8.6 (BST)
- new net: C365.1, R239.2, R241.1, U5.2 (FB)
- new net: C365.2, R240.1, R241.2
- new net: C358.1, U5.7 (BOOT)
- new net: R217.2, U4.4 (PG)
- new net BK_0_PG: R217.1
- new net BK_1_PG: R228.1
- new net B_SW_0: C345.2, L26.1, U4.6 (SW)
- new net B_SW_1: C358.2, L7.1, U5.6 (SW)
- new net CPU_BIG1_VSEL: U22.A1 (VSEL)
- new net FB9: C204.2, R45.2, U12.66 (FB9)
- new net VCC3V3_PCIE30_1: C687.2, C688.2, L1.2, R172.1
- new net VCC_5V0_SYS: C292.1, C293.1, C300.1, C301.1, C317.1, C318.1, C347.2, C348.2, C349.2, C350.2, C351.2, C352.2, C356.2, C357.2, C360.2, C527.2, C530.2, C575.2, C604.2, C684.2, C685.2, C691.2, C692.2, C693.2, L15.1, L26.2, R191.2, U18.D1 (VIN), U18.D2 (VIN), U18.E1 (VIN), U18.E2 (VIN), U19.D1 (VIN), U19.D2 (VIN), U19.E1 (VIN), U19.E2 (VIN), U22.D1 (VIN), U22.D2 (VIN), U22.E1 (VIN), U22.E2 (VIN), U26.6 (VIN), U28.6 (VIN), U5.8 (VIN), U6.3 (VIN), U7.3 (VIN), U8.3 (VIN)
- new net VSYS_MAIN: C273.2, C274.1, C325.2, C326.2, C328.2, C329.2, C330.2, C331.2, C332.2, C334.2, C335.2, C341.2, C342.2, C343.2, C699.2, C700.2, C701.2, Q13.5 (D), R242.1, R68.1, R73.1, U10.3 (VIN), U14.22 (VSYS), U4.8 (VIN)
- no-connect marks 7 -> 9
Other:
- note added: "0.22uH"
- note added: "0.47uH"
- note added: "USE 2.2uH INDUCTOR"
- note added: "USE 3.3uH INDUCTOR"
- note added: "USE THE 2045321601 MALE COUNTERPART"
- note removed: "25V X5R capacitors"
- note removed: "LOOK FOR FEMALE VERSION OF THIS"
- note removed: "REMOVE ALL USES OF VCC_1V8_SYS"
- moved on the sheet: C167, C168, C169, C170, C171, C172, C173, C174, C175, C176, C177, C178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
