File: hardware/motherboard/barebones_power.kicad_sch (KiCad schematic)
At the start: 297 parts, among them J17 2200981671, Q11 CSD18543Q3A, Q12 CSD18543Q3A, Q13 CSD18543Q3A, Q14 CSD18543Q3A, U10 TPS62933DRLR, U12 RK806-1, U14 BQ25731RSNR, U18 RK860-2, U19 RK860-2, U22 RK860-3, U26 TPS61170DRVR, U28 TPS61160ADRVT, U3 TLV75533PDBVR, U4 TPS56837RPAR, U5 TPS56837RPAR, U53 TPS54628DDAR, U6 TPS62933DRLR, U7 TPS62933DRLR, U8 TPS62933DRLR, U9 1N5819WT

Commit message: started routing on LPDDR4x RAM
Parts:
- removed C167, C168, C169, C170, C171, C172, C173, C317, C318, C576, C589: 22uF, Capacitor_SMD:C_0402_1005Metric, symbol Device:C
- removed C255, C256, C257, C258: 0.1uF, Capacitor_SMD:C_0603_1608Metric, symbol Device:C
- removed C354, C357: 0.1uF, Capacitor_SMD:C_0201_0603Metric, symbol Device:C
- removed C355: 680pF, Capacitor_SMD:C_0201_0603Metric, symbol Device:C
- removed C356: 4.7uF, Capacitor_SMD:C_0402_1005Metric, symbol Device:C
- removed C358, C575: 0.1uF, Capacitor_SMD:C_0402_1005Metric, symbol Device:C
- removed C359: 47nF, Capacitor_SMD:C_0201_0603Metric, symbol Device:C
- removed C360, C361: 1uF, Capacitor_SMD:C_0402_1005Metric, symbol Device:C
- removed C362: 220nF, Capacitor_SMD:C_0201_0603Metric, symbol Device:C
- removed C365: 150pF, Capacitor_SMD:C_0201_0603Metric, symbol Device:C
- removed C367, C368: 22uF, Capacitor_SMD:C_0603_1608Metric, symbol Device:C
- removed C527, C530: 10uF, Capacitor_SMD:C_0402_1005Metric, symbol Device:C
- removed D4: B0530W-7-F, barebones:SOD3715X145N, symbol B0530W-7-F:B0530W-7-F
- removed L7: XAL6030-332MEC, barebones:IND_XAL6030-332MEC, symbol XAL6030-332MEC:XAL6030-332MEC
- removed R112: 87.6k, Resistor_SMD:R_0402_1005Metric, symbol Device:R
- removed R113, R239: 10k, Resistor_SMD:R_0402_1005Metric, symbol Device:R
- removed R114, R228: 10k, Resistor_SMD:R_0201_0603Metric, symbol Device:R
- removed R115: 10R, Resistor_SMD:R_0201_0603Metric, symbol Device:R
- removed R227: 30.1k, Resistor_SMD:R_0402_1005Metric, symbol Device:R
- removed R240: 49.9k, Resistor_SMD:R_0402_1005Metric, symbol Device:R
- removed R241: 73.2k, Resistor_SMD:R_0402_1005Metric, symbol Device:R
- removed R45: 0R, Capacitor_SMD:C_0201_0603Metric, symbol Device:R
- removed U10, U6, U7, U8: TPS62933DRLR, barebones:SOTFL50P160X60-8N, symbol TPS62933DRLR:TPS62933DRLR
- removed U5: TPS56837RPAR, barebones:CONV_TPS56837RPAR, symbol TPS56837RPAR:TPS56837RPAR
- added C311, C312, C313: 22uF, Capacitor_SMD:C_0603_1608Metric, symbol Device:C
- added C324, C337: 10uF, Capacitor_SMD:C_0805_2012Metric, symbol Device:C
- added C333, C336, C338, C339, C340, C731, C732: 22uF, Capacitor_SMD:C_0805_2012Metric, symbol Device:C
- added C363: 56pF, Capacitor_SMD:C_0402_1005Metric, symbol Device:C
- added C369, C371, C374, C375, C381, C384, C385: 47uF, Capacitor_SMD:C_1210_3225Metric, symbol Device:C
- added C382, C383, C540, C672: 0.1uF, Capacitor_SMD:C_0402_1005Metric, symbol Device:C
- added C386: 0.047uF, Capacitor_SMD:C_0402_1005Metric, symbol Device:C
- added C387: 4.7uF, Capacitor_SMD:C_0402_1005Metric, symbol Device:C
- added C552, C568: 10uF, Capacitor_SMD:C_0402_1005Metric, symbol Device:C
- added C617, C679: 10uF, Capacitor_SMD:C_1206_3216Metric, symbol Device:C
- added C674: 33nF, Capacitor_SMD:C_0201_0603Metric, symbol Device:C
- added C676, C678: 22uF, Capacitor_SMD:C_1210_3225Metric, symbol Device:C
- added C680, C681: 22uF, Capacitor_SMD:C_1206_3216Metric, symbol Device:C
- added C753: 0.1uF, Capacitor_SMD:C_0201_0603Metric, symbol Device:C
- added J20: 5055671571, barebones:CONN_505567_15_MOL, symbol 5055671571:5055671571
- added L5: XFL4015-471MEC, barebones:IND-SMD_L4.0-W4.0_XFL4020-102MEB, symbol XFL4015-471MEC:XFL4015-471MEC
- added L7: FDSD0420-H-2R2M=P3, barebones:IND_XAL6030-332MEC, symbol FDSD0420-H-2R2M_P3:FDSD0420-H-2R2M=P3
- added L8: XAL7030-152MEC, barebones:INDDFN750X750X310-2N, symbol XAL7030-152MEC:XAL7030-152MEC
- added Q5: BSS138, Package_TO_SOT_SMD:SOT-23, symbol Transistor_FET:BSS138
- added R183: 100k, Resistor_SMD:R_0402_1005Metric, symbol Device:R
- added R196: 10k, Resistor_SMD:R_0201_0603Metric, symbol Device:R
- added R197: 49.9k, Resistor_SMD:R_0201_0603Metric, symbol Device:R
- added R202, R220, R234: 10k, Resistor_SMD:R_0402_1005Metric, symbol Device:R
- added R213: 57.6k, Resistor_SMD:R_0402_1005Metric, symbol Device:R
- added R235: 52.3k, Resistor_SMD:R_0402_1005Metric, symbol Device:R
- added U24: TPS56C215RNNR, barebones:QFN50P350X350X100-18N, symbol TPS56C215RNNR:TPS56C215RNNR
- added U29, U39, U40, U42, U44: TPS62933DRLR, barebones:SOTFL50P160X60-8N, symbol TPS62933DRLR:TPS62933DRLR
- C176, C204, C591, C686: footprint Capacitor_SMD:C_0201_0603Metric -> Capacitor_SMD:C_0402_1005Metric
- C177, C178, C179, C187, C188, C189, C192, C193, C195, C199, C200, C201, C207, C208, C213, C214, C215, C216, C218, C219, C246, C247, C249, C275, C276, C319, C320, C343, C691, C692, C695, C696: footprint Capacitor_SMD:C_0402_1005Metric -> Capacitor_SMD:C_0805_2012Metric
- C182, C191, C197, C205, C206, C210, C211, C217, C229, C230, C233, C234, C236, C239, C244, C245, C252, C263, C265, C267, C270, C271, C277, C278, C279, C285, C286, C287, C288, C289, C292, C293, C296, C297, C298, C299, C300, C301, C303, C308, C309, C315, C316, C685, C690: footprint Capacitor_SMD:C_0402_1005Metric -> Capacitor_SMD:C_0603_1608Metric
- C202: value 22uF -> 10uF; footprint Capacitor_SMD:C_0402_1005Metric -> Capacitor_SMD:C_0805_2012Metric
- C209: value 10uF -> 22uF; footprint Capacitor_SMD:C_0402_1005Metric -> Capacitor_SMD:C_0805_2012Metric
- C242, C251, C254: footprint Capacitor_SMD:C_0603_1608Metric -> Capacitor_SMD:C_0805_2012Metric
- C248: value 47uF -> 22uF; footprint Capacitor_SMD:C_0402_1005Metric -> Capacitor_SMD:C_0805_2012Metric
- C325, C326, C328, C329, C348, C349: footprint Capacitor_SMD:C_0603_1608Metric -> Capacitor_SMD:C_1210_3225Metric
- C330, C331, C332: value 10uF -> 22uF; footprint Capacitor_SMD:C_0603_1608Metric -> Capacitor_SMD:C_0805_2012Metric
- C334: value 33uF -> 22uF; footprint Capacitor_SMD:C_0603_1608Metric -> Capacitor_SMD:C_0805_2012Metric
- C335: value 33uF -> 47uF; footprint Capacitor_SMD:C_0603_1608Metric -> Capacitor_SMD:C_0805_2012Metric
- C341, C342, C703, C704: footprint Capacitor_SMD:C_0402_1005Metric -> Capacitor_SMD:C_1210_3225Metric
- C347: value 22uF -> 0.1uF; footprint Capacitor_SMD:C_0603_1608Metric -> Capacitor_SMD:C_0402_1005Metric
- C350, C351: value 10uF -> 22uF; footprint Capacitor_SMD:C_0402_1005Metric -> Capacitor_SMD:C_0603_1608Metric
- C353: value 4.7uF -> 22uF; footprint Capacitor_SMD:C_0402_1005Metric -> Capacitor_SMD:C_0603_1608Metric
- C366: value 22uF -> 47uF; footprint Capacitor_SMD:C_0603_1608Metric -> Capacitor_SMD:C_1210_3225Metric
- C604, C687: footprint Capacitor_SMD:C_0402_1005Metric -> Capacitor_SMD:C_1206_3216Metric
- C684: value 10uF -> 22uF; footprint Capacitor_SMD:C_0402_1005Metric -> Capacitor_SMD:C_1206_3216Metric
- C688: value 22uF -> 10uF; footprint Capacitor_SMD:C_0402_1005Metric -> Capacitor_SMD:C_1206_3216Metric
- C693: footprint Capacitor_SMD:C_0402_1005Metric -> Capacitor_SMD:C_0201_0603Metric
- Q11, Q12, Q13, Q14: footprint barebones:TRANS_CSD18543Q3A -> Package_SON:VSON-8_3.3x3.3mm_P0.65mm_NexFET
- R187: footprint Resistor_SMD:R_0402_1005Metric -> Resistor_SMD:R_0201_0603Metric
- R225: value 10k -> 140k; footprint Resistor_SMD:R_0201_0603Metric -> Resistor_SMD:R_0402_1005Metric
Connections:
- net BACKLIGHT_PWM: now also Q5.1 (G); no longer U28.5 (CTRL)
- net BATT_PRES: now also J20.7; no longer J17.7
- net BUCK_PWRON: now also R196.2, U24.15 (EN); no longer R225.2
- net GND: now also C330.2, C331.2, C332.2, C334.2, C335.2, C350.2, C351.2, C353.2, C311.2, C312.2, C313.2, C324.2, C333.2, C336.2, C337.2, C338.2, C339.2, C340.2, C369.1, C371.1, C374.1, C375.1, C381.1, C382.1, C383.1, C384.1, C385.1, C386.1, C387.1, C540.1, C552.1, C568.1, C617.1, C672.1, C674.1, C676.1, C678.1, C679.1, C680.1, C681.1, C731.1, C732.1, C753.1, J20.10, J20.11, J20.12, J20.13, J20.14, J20.15, Q5.2 (S), R196.1, R197.1, R202.1, R220.1, U24.10 (PGND), U24.12 (AGND), U24.3 (PGND), U24.4 (PGND), U24.5 (PGND), U24.8 (PGND), U24.9 (PGND), U29.1 (RT), U29.4 (GND), U39.1 (RT), U39.4 (GND), U40.1 (RT), U40.4 (GND), U42.1 (RT), U42.4 (GND), U44.1 (RT), U44.4 (GND); no longer C330.1, C331.1, C332.1, C334.1, C335.1, C347.1, C350.1, C351.1, C352.1, C353.1, J17.12, J17.13, J17.14, J17.15, J17.16, R225.1, U26.3 (GND), U26.7 (THERMALPAD), U28.3 (GND), U28.7 (THERMALPAD)
- net PACK_P: now also J20.1, J20.2, J20.3, J20.4, J20.5, J20.6; no longer J17.1, J17.2, J17.3, J17.4, J17.5
- net PCIE30X4_PWREN_H: now also R183.1
- net PCIE30X4_PWREN_H_EN_1: now also U42.2 (EN)
- net PCIE30X4_PWREN_H_EN_2: now also U40.2 (EN)
- net SMBC_BATT: now also J20.9; no longer J17.9
- net SMBD_BATT: now also J20.8; no longer J17.8
- net VCC1V8_PMU_DDR_S3: now also C248.1
- net VCC3V3_PCIE30: now also C684.2, C687.2
- net VCC3V3_PCIE30_1: now also C680.2, C681.2; no longer C687.2, C688.2
- net VCC_12V_EDP: now also R225.1, C676.2, C678.2, L7.2; no longer C353.2, D3.C
- net VCC_1V1_NLDO_S3: now also C731.2, C732.2
- net VCC_2V0_PLDO_S3: now also C330.1
- net VCC_3V3_S3: now also C209.1, C338.1; no longer C319.1
- net VCC_4V0_SYS: now also C292.1, C293.1, C300.1, C301.1, C315.1, C316.1, U18.D1 (VIN), U18.D2 (VIN), U18.E1 (VIN), U18.E2 (VIN), U19.D1 (VIN), U19.D2 (VIN), U19.E1 (VIN), U19.E2 (VIN), U22.D1 (VIN), U22.D2 (VIN), U22.E1 (VIN), U22.E2 (VIN), C363.1, C369.2, C371.2, C374.2, L8.2, R213.1
- net VCC_5V0_SYS: now also Q5.3 (D); no longer C292.1, C293.1, C300.1, C301.1, C347.2, C350.2, C351.2, C352.2, C604.2, C684.2, C685.2, C691.2, C692.2, C693.2, L15.1, U18.D1 (VIN), U18.D2 (VIN), U18.E1 (VIN), U18.E2 (VIN), U19.D1 (VIN), U19.D2 (VIN), U19.E1 (VIN), U19.E2 (VIN), U22.D1 (VIN), U22.D2 (VIN), U22.E1 (VIN), U22.E2 (VIN), U26.6 (VIN), U28.6 (VIN)
- net VDD2_DDR_S3: now also C324.1
- net VDDQ_DDR_S0: now also C202.1, C337.1; no longer C209.1
- net VDD_CPU_BIG0_S0: now also C294.1, C296.1, C297.1, C298.1, C299.1, C350.1, L19.2, R93.2, C311.1
- net VDD_CPU_BIG1_S0: now also C302.1, C303.1, C308.1, C309.1, C353.1, L10.2, R94.2, C312.1, C313.1
- net VDD_DDR_S0: now also C331.1, C332.1, C334.1, C333.1
- net VDD_GPU_S0: now also C335.1; no longer C248.1
- net VDD_LOG_S0: now also C336.1; no longer C202.1
- net VDD_NPU_S0: now also C284.1, C285.1, C286.1, C287.1, C288.1, C289.1, C351.1, L18.2, R92.2
- net VDD_VDENC_S0: now also C319.1, C320.1, C339.1, C340.1
- net at R169.2, R172.2: now also U42.8 (FB)
- net at C314.2, L2.1: now also U40.5 (SW)
- net at C314.1: now also U40.6 (BST)
- net at C591.2: now also U40.7 (SS)
- net at R166.2, R167.2: now also U40.8 (FB)
- net at C702.2: now also U29.7 (SS)
- net at U26.1 (FB): no longer L14.1
- net at C322.2, L4.1: now also U39.5 (SW)
- net at C694.2: now also U39.7 (SS)
- net at R188.2, R218.2: now also U39.8 (FB)
- net at C321.2, L1.1: now also U42.5 (SW)
- net at R187.2: now also C753.2, U39.2 (EN); no longer C690.2
- net at R251.2, R252.2: now also U29.8 (FB)
- net at C323.1: now also U29.6 (BST)
- net at C323.2, L6.1: now also U29.5 (SW)
- net at R242.2: now also U29.2 (EN)
- net at C321.1: now also U42.6 (BST)
- net at C686.2: now also U42.7 (SS)
- net at C322.1: now also U39.6 (BST)
- net BACKLIGHT_DN: no longer names the net of U28.1 (FB)
- net EDP_PWM11_M1: no longer names the net of U26.5 (CTRL)
- removed net EDP_SW: D3.A, L14.2, U26.4 (SW)
- net PWM_SW: no longer names the net of U28.4 (SW)
- net PWM_SW: no longer L15.2
- net VSYS_MAIN renamed VIN
- net VIN: now also C604.2, C685.2, C688.2, C690.2, C691.2, C692.2, C693.2, C375.2, C381.2, C382.2, C383.2, C384.2, C385.2, C552.2, C568.2, C617.2, C672.2, C679.2, U24.11 (VIN), U24.2 (VIN), U29.3 (VIN), U39.3 (VIN), U40.3 (VIN), U42.3 (VIN), U44.3 (VIN); no longer C330.2, C331.2, C332.2, C334.2, C335.2
- new net: C347.1, U44.6 (BST)
- new net: C347.2, L7.1, U44.5 (SW)
- new net: C363.2, R213.2, R220.2, U24.13 (FB)
- new net: R202.2, R225.2, U44.8 (FB)
- new net: C352.1, U24.1 (BOOT)
- new net: C386.2, U24.14 (SS)
- new net: R234.1, U24.16 (PGOOD)
- new net: C387.2, R234.2, R235.1, U24.17 (VREG5)
- new net: R197.2, R235.2, U24.18 (MODE)
- new net: C540.2, R183.2, U44.2 (EN)
- new net: C674.2, U44.7 (SS)
- new net MAIN_SW: C352.2, L8.1, U24.6 (SW), U24.7 (SW)
- no-connect marks 9 -> 6
Other:
- note removed: "USE 10uH INDUCTOR"
- note removed: "USE 22uH INDUCTOR"
- moved on the sheet: BT1, C177, C178, C204, C227, C228, C237, C238, C273, C274, C275, C276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
